Commit message: Use ur5 prefix for ur5 links
This is necessary to rename "base_link" to "ur5_base_link"

File: mobipick_description/urdf/mobipick/mobipick_model.urdf.xacro (robot description, xacro)
@@ -19,7 +19,7 @@
   <xacro:structure prefix="" height="0.1" />
   <!-- arm -->
-  <xacro:ur5_robot prefix="" joint_limited="true"/>
+  <xacro:ur5_robot prefix="ur5_" joint_limited="true"/>
   <!-- sensor -->
-  <xacro:robotiq_ft_300 parent="tool0" prefix="" >
+  <xacro:robotiq_ft_300 parent="ur5_tool0" prefix="" >
       <pose xyz="0 0 0" rpy="0 0 0" />
       <!-- <pose xyz="0 0 0.009" rpy="0 0 0" /> -->
@@ -39,5 +39,5 @@
   <joint name="${prefix}struct_ur5_joint" type="fixed">
     <parent link="StructBaseSupport" />
-    <child link = "base_link" />
+    <child link = "ur5_base_link" />
     <origin xyz="0.0 0.0 0.0025" rpy="0.0 0.0 0.0" />
   </joint>
