Commit message: introduced prefix parameters to urdf, srdf and config files
This allows us to compile a new robot description for every instance
of a robot we want to deploy using xacro, which will include a prefix
for every joint and link. Therefore many config files need to be
parameterized, too. All in all this makes it possible to set a tf_prefix
for our robot without using the inconsistently used and therefore not
correctly working rosparam 'tf_prefix'.

File: mobipick_description/urdf/mobipick/mobipick.gazebo.xacro (robot description, xacro)
@@ -1,15 +1,16 @@
 <?xml version="1.0"?>
 <robot xmlns:xacro="http://ros.org/wiki/xacro">
-  <xacro:arg name="robot_namespace" default="" />
-  <!-- Common -->
-  <xacro:include filename="$(find mobipick_description)/urdf/common.gazebo.xacro" />
-  <xacro:controller_plugin_gazebo robot_namespace="$(arg robot_namespace)"/>
-  <!-- MiR100 mobile base -->
-  <!-- UR5 arm -->
-  <!-- TODO -->
-  <!-- force torque sensor-->
-  <!-- TODO -->
-  <!-- Robotiq gripper -->
-  <xacro:include filename="$(find mobipick_description)/urdf/robotiq_2f_140/robotiq_2f_140.gazebo.xacro" />
-  <xacro:mimic_joint_plugins_gazebo prefix="gripper_" robot_namespace=""/>
+  <xacro:macro name="mobipick_gazebo" params="robot_namespace prefix">
+    <!-- Common -->
+    <xacro:include filename="$(find mobipick_description)/urdf/common.gazebo.xacro" />
+    <xacro:controller_plugin_gazebo robot_namespace="${robot_namespace}"/>
+    <!-- MiR100 mobile base -->
+    <!-- UR5 arm -->
+    <!-- TODO -->
+    <!-- force torque sensor-->
+    <!-- TODO -->
+    <!-- Robotiq gripper -->
+    <xacro:include filename="$(find mobipick_description)/urdf/robotiq_2f_140/robotiq_2f_140.gazebo.xacro" />
+    <xacro:mimic_joint_plugins_gazebo prefix="${prefix}gripper_" robot_namespace="${robot_namespace}"/>
+  </xacro:macro>
 </robot>

File: mobipick_description/urdf/mobipick/mobipick_v1_model.urdf.xacro (robot description, xacro)
@@ -4,31 +4,39 @@
   <xacro:arg name="robot" default="mobipick-hb" />      <!-- can be "mobipick-hb" or "mobipick-os" -->
   <xacro:property name="robot" value="$(arg robot)" />  <!-- necessary because args cannot be accessed inside ${} expressions -->
+  <xacro:arg name="tf_prefix" default="" />
+  <xacro:property name="tf_prefix_" value="$(arg tf_prefix)" />
+  <xacro:if value="${tf_prefix_ == ''}">
+    <xacro:property name="prefix" value="" />
+  </xacro:if>
+  <xacro:unless value="${tf_prefix_ == ''}">
+    <xacro:property name="prefix" value="${tf_prefix_}/" />
+  </xacro:unless>
   <!-- ############# MIR100 BASE ############## -->
   <xacro:include filename="$(find mir_description)/urdf/include/mir_100_v1.urdf.xacro" />
-  <xacro:mir_100 prefix=""/>
+  <xacro:mir_100 prefix="${prefix}"/>
   <!-- ############## STRUCTURE ############### -->
   <xacro:include filename="$(find mobipick_description)/urdf/structure/mobipick_structure.urdf.xacro" />
-  <joint name="mir_struct_joint" type="fixed">
-    <parent link="surface" />
-    <child link = "structure_part_down" />
+  <joint name="${prefix}mir_struct_joint" type="fixed">
+    <parent link="${prefix}surface" />
+    <child link="${prefix}structure_part_down" />
     <origin xyz="0.0 0.0 0.0" rpy="0.0 0.0 0.0" />
   </joint>
   <xacro:if value="${robot == 'mobipick-hb'}">
-    <xacro:structure prefix="structure_" height="0.058" variant="v1" />
+    <xacro:structure prefix="${prefix}structure_" height="0.058" variant="v1" />
   </xacro:if>
   <xacro:if value="${robot == 'mobipick-os'}">
-    <xacro:structure prefix="structure_" height="0.058" variant="v2" />
+    <xacro:structure prefix="${prefix}structure_" height="0.058" variant="v2" />
   </xacro:if>
   <!-- ############### UR5 ARM ################ -->
   <xacro:include filename="$(find mobipick_description)/urdf/ur5/ur5.urdf.xacro" />
-  <joint name="struct_ur5_joint" type="fixed">
-    <parent link="structure_pedestal_surface" />
-    <child link = "ur5_base_link" />
+  <joint name="${prefix}struct_ur5_joint" type="fixed">
+      <parent link="${prefix}structure_pedestal_surface" />
+      <child link="${prefix}ur5_base_link" />
     <origin xyz="0.0 0.0 0.0025" rpy="0.0 0.0 0.0" />
   </joint>
-  <xacro:ur5_robot prefix="ur5_" joint_limited="true"/>
+  <xacro:ur5_robot prefix="${prefix}ur5_" joint_limited="true"/>
   <!-- ############## FT SENSOR ############### -->
   <xacro:include filename="$(find mobipick_description)/urdf/robotiq_ft_300/robotiq_ft_300.urdf.xacro" />
-  <xacro:robotiq_ft_300 parent="ur5_tool0" prefix="" >
+  <xacro:robotiq_ft_300 parent="${prefix}ur5_tool0" prefix="${prefix}" >
       <pose xyz="0 0 0" rpy="0 0 0" />
       <!-- <pose xyz="0 0 0.009" rpy="0 0 0" /> -->
@@ -41,10 +49,10 @@
   <xacro:property name="coupling_inner_length" value="0.008" />
   <xacro:property name="coupling_mass" value="0.100" />
-  <joint name="ft300_coupling_joint" type="fixed">
+  <joint name="${prefix}ft300_coupling_joint" type="fixed">
     <origin xyz="0 0 ${coupling_inner_length / 2}" rpy="0 0 ${-pi/2}" />
-    <parent link="fts_toolside" />
-    <child link="gripper_coupling_link" />
+    <parent link="${prefix}fts_toolside" />
+    <child link="${prefix}gripper_coupling_link" />
   </joint>
-  <link name="gripper_coupling_link">
+  <link name="${prefix}gripper_coupling_link">
     <origin xyz="0 0 0" rpy="0 0 0" />
     <visual>
@@ -65,30 +73,31 @@
     </xacro:cylinder_inertial>
   </link>
-  <gazebo reference="gripper_coupling_link">
+  <gazebo reference="${prefix}gripper_coupling_link">
     <material>Gazebo/FlatBlack</material>
   </gazebo>
-  <joint name="coupling_2f140_joint" type="fixed">
+  <joint name="${prefix}coupling_2f140_joint" type="fixed">
     <origin xyz="0 0 ${coupling_inner_length / 2}" rpy="0 0 0" />
-    <parent link="gripper_coupling_link" />
-    <child link="gripper_robotiq_arg2f_base_link" />
+    <parent link="${prefix}gripper_coupling_link" />
+    <child link="${prefix}gripper_robotiq_arg2f_base_link" />
   </joint>
-  <xacro:robotiq_arg2f_140 prefix="gripper_"/>
+  <xacro:robotiq_arg2f_140 prefix="${prefix}gripper_"/>
   <!-- ############### SENSOR MOUNT + 3D CAM  ################ -->
   <xacro:include filename="$(find mobipick_description)/urdf/sensors/gripper_cam.urdf.xacro" />
-  <joint name="sensor_mount_joint" type="fixed">
+  <joint name="${prefix}sensor_mount_joint" type="fixed">
     <origin xyz="0.0 0.0 -0.005" rpy="0.0 ${-pi/2} 0.0" />
-    <parent link="fts_toolside" />
-    <child link="sensor_mount_link" />
+    <parent link="${prefix}fts_toolside" />
+    <child link="${prefix}sensor_mount_link" />
   </joint>
-  <gripper_cam />
+  <gripper_cam prefix="${prefix}" />
   <!-- ############### DUAL XTION MOUNT + XTIONS ################ -->
   <xacro:include filename="$(find mobipick_description)/urdf/sensors/dual_xtions.urdf.xacro" />
-  <joint name="dual_xtion_mount_joint" type="fixed">
+  <joint name="${prefix}dual_xtion_mount_joint" type="fixed">
     <origin xyz="0.37 0.0 -0.02" rpy="0 0 0" />
-    <parent link="structure_pedestal" />
-    <child link="dual_xtion_mount_link" />
+    <parent link="${prefix}structure_pedestal" />
+    <child link="${prefix}dual_xtion_mount_link" />
   </joint>
-  <dual_xtions />
+  <dual_xtions prefix="${prefix}" />
   <!-- ################ GAZEBO ################ -->
   <xacro:include filename="$(find mobipick_description)/urdf/mobipick/mobipick.gazebo.xacro" />
+  <xacro:mobipick_gazebo prefix="${prefix}" robot_namespace="" />
 </robot>

File: mobipick_description/urdf/sensors/dual_xtions.urdf.xacro (robot description, xacro)
@@ -5,33 +5,33 @@
   <!-- distance between center of camera and camera_link -->
   <xacro:property name="xtion_cam_py" value="0.069"/>
-  <xacro:macro name="dual_xtions" params="">
-    <link name="dual_xtion_mount_link" />
-    <joint name="dual_xtion_left_mount" type="fixed">
-      <parent link="dual_xtion_mount_link" />
-      <child link="dual_xtion_left_mount_link" />
+  <xacro:macro name="dual_xtions" params="prefix">
+    <link name="${prefix}dual_xtion_mount_link" />
+    <joint name="${prefix}dual_xtion_left_mount" type="fixed">
+      <parent link="${prefix}dual_xtion_mount_link" />
+      <child link="${prefix}dual_xtion_left_mount_link" />
       <origin xyz="0 0.06 0" rpy="0.0 1.571 0.0" />
     </joint>
-    <dual_xtion_mount side="left" />
-    <joint name="dual_xtion_right_mount" type="fixed">
-      <parent link="dual_xtion_mount_link" />
-      <child link="dual_xtion_right_mount_link" />
+    <dual_xtion_mount side="left" prefix="${prefix}" />
+    <joint name="${prefix}dual_xtion_right_mount" type="fixed">
+      <parent link="${prefix}dual_xtion_mount_link" />
+      <child link="${prefix}dual_xtion_right_mount_link" />
       <origin xyz="0 -0.06 0" rpy="0.0 -1.571 3.142" />
     </joint>
-    <dual_xtion_mount side="right" />
-    <joint name="dual_xtion_bottom_joint" type="fixed">
-      <parent link="dual_xtion_mount_link" />
-      <child link="dual_xtion_bottom_link" />
+    <dual_xtion_mount side="right" prefix="${prefix}" />
+    <joint name="${prefix}dual_xtion_bottom_joint" type="fixed">
+      <parent link="${prefix}dual_xtion_mount_link" />
+      <child link="${prefix}dual_xtion_bottom_link" />
       <origin xyz="0.045 ${xtion_cam_py} -0.032" rpy="0 0.262 0" />
     </joint>
-    <sensor_xtion camera_name="dual_xtion_bottom" />
-    <joint name="dual_xtion_top_joint" type="fixed">
-      <parent link="dual_xtion_mount_link" />
-      <child link="dual_xtion_top_link" />
+    <sensor_xtion camera_name="dual_xtion_bottom" prefix="${prefix}" />
+    <joint name="${prefix}dual_xtion_top_joint" type="fixed">
+      <parent link="${prefix}dual_xtion_mount_link" />
+      <child link="${prefix}dual_xtion_top_link" />
       <origin xyz="0.045 ${xtion_cam_py} 0.032" rpy="0 -0.262 0" />
     </joint>
-    <sensor_xtion camera_name="dual_xtion_top" />
+    <sensor_xtion camera_name="dual_xtion_top" prefix="${prefix}" />
   </xacro:macro>
-  <xacro:macro name="dual_xtion_mount" params="side">
-    <link name="dual_xtion_${side}_mount_link">
+  <xacro:macro name="dual_xtion_mount" params="side prefix">
+    <link name="${prefix}dual_xtion_${side}_mount_link">
       <origin xyz="0 0 0" rpy="0 0 0" />
       <visual>
@@ -59,5 +59,5 @@
       </inertial>
     </link>
-    <gazebo reference="dual_xtion_${side}_mount_link">
+    <gazebo reference="${prefix}dual_xtion_${side}_mount_link">
       <material>Gazebo/FlatBlack</material>
     </gazebo>
@@ -66,6 +66,6 @@
   <!-- ######################## ASUS Xtion Pro Live ######################## -->
   <!-- ##################################################################### -->
-  <xacro:macro name="sensor_xtion" params="camera_name">
-    <link name="${camera_name}_link">
+  <xacro:macro name="sensor_xtion" params="camera_name prefix">
+    <link name="${prefix}${camera_name}_link">
       <visual>
         <origin xyz="0 0 0" />
@@ -85,32 +85,32 @@
       </xacro:box_inertial>
     </link>
-    <gazebo reference="${camera_name}_link">
+    <gazebo reference="${prefix}${camera_name}_link">
       <material>Gazebo/FlatBlack</material>
     </gazebo>
-    <joint name="${camera_name}_rgb_joint" type="fixed">
+    <joint name="${prefix}${camera_name}_rgb_joint" type="fixed">
       <origin xyz="0 -0.045 0" rpy="0 0 0" />
-      <parent link="${camera_name}_link"/>
-      <child link="${camera_name}_rgb_frame" />
+      <parent link="${prefix}${camera_name}_link"/>
+      <child link="${prefix}${camera_name}_rgb_frame" />
     </joint>
-    <link name="${camera_name}_rgb_frame"/>
-    <joint name="${camera_name}_rgb_optical_joint" type="fixed">
+    <link name="${prefix}${camera_name}_rgb_frame"/>
+    <joint name="${prefix}${camera_name}_rgb_optical_joint" type="fixed">
       <origin xyz="0 0 0" rpy="${-pi/2} 0 ${-pi/2}" />
-      <parent link="${camera_name}_rgb_frame" />
-      <child link="${camera_name}_rgb_optical_frame" />
+      <parent link="${prefix}${camera_name}_rgb_frame" />
+      <child link="${prefix}${camera_name}_rgb_optical_frame" />
     </joint>
-    <link name="${camera_name}_rgb_optical_frame"/>
-    <joint name="${camera_name}_depth_joint" type="fixed">
+    <link name="${prefix}${camera_name}_rgb_optical_frame"/>
+    <joint name="${prefix}${camera_name}_depth_joint" type="fixed">
       <origin xyz="0 -0.02 0" rpy="0 0 0" />
-      <parent link="${camera_name}_link"/>
-      <child link="${camera_name}_depth_frame" />
+      <parent link="${prefix}${camera_name}_link"/>
+      <child link="${prefix}${camera_name}_depth_frame" />
     </joint>
-    <link name="${camera_name}_depth_frame"/>
-    <joint name="${camera_name}_depth_optical_joint" type="fixed">
+    <link name="${prefix}${camera_name}_depth_frame"/>
+    <joint name="${prefix}${camera_name}_depth_optical_joint" type="fixed">
       <origin xyz="0 0 0" rpy="${-pi/2} 0 ${-pi/2}" />
-      <parent link="${camera_name}_depth_frame" />
-      <child link="${camera_name}_depth_optical_frame" />
+      <parent link="${prefix}${camera_name}_depth_frame" />
+      <child link="${prefix}${camera_name}_depth_optical_frame" />
     </joint>
-    <link name="${camera_name}_depth_optical_frame"/>
-    <sim_3dsensor/>  <!-- NOTE: sim_3dsensor macro from gripper_cam is used here -->
+    <link name="${prefix}${camera_name}_depth_optical_frame"/>
+    <sim_3dsensor prefix="${prefix}" />  <!-- NOTE: sim_3dsensor macro from gripper_cam is used here -->
   </xacro:macro>
 </robot>
