Commit message: introduced prefix parameters to urdf, srdf and config files
This allows us to compile a new robot description for every instance
of a robot we want to deploy using xacro, which will include a prefix
for every joint and link. Therefore many config files need to be
parameterized, too. All in all this makes it possible to set a tf_prefix
for our robot without using the inconsistently used and therefore not
correctly working rosparam 'tf_prefix'.

File: mobipick_description/urdf/sensors/gripper_cam.urdf.xacro (robot description, xacro)
@@ -8,21 +8,21 @@
   <!-- distance between center of camera and camera_link -->
   <xacro:property name="astra_cam_py" value="0.0485"/>
-  <xacro:macro name="gripper_cam" params="">
-    <sensor_mount />
-    <joint name="gripper_astra_joint" type="fixed">
+  <xacro:macro name="gripper_cam" params="prefix">
+    <sensor_mount prefix="${prefix}" />
+    <joint name="${prefix}gripper_astra_joint" type="fixed">
       <origin xyz="-0.032 0.033 -0.065" rpy="${pi/2} ${pi/2} ${-pi/2}" />
-      <parent link="sensor_mount_link"/>
-      <child link="gripper_astra_link"/>
-    </joint>
-    <sensor_astra_mini_s camera_name="gripper_astra" />
-    <joint name="gripper_pico_flexx_joint" type="fixed">
+      <parent link="${prefix}sensor_mount_link"/>
+      <child link="${prefix}gripper_astra_link"/>
+    </joint>
+    <sensor_astra_mini_s camera_name="gripper_astra" prefix="${prefix}" />
+    <joint name="${prefix}gripper_pico_flexx_joint" type="fixed">
       <origin xyz="0.01545 0.0001 0.008" rpy="${-pi/2} 0.0 -0.03650298564336946" />
-      <parent link="sensor_mount_pico_holder_link"/>
-      <child link="gripper_pico_flexx_link"/>
-    </joint>
-    <sensor_pico_flexx camera_name="gripper_pico_flexx" />
-  </xacro:macro>
-  <xacro:macro name="sensor_mount">
-    <link name="sensor_mount_link">
+      <parent link="${prefix}sensor_mount_pico_holder_link"/>
+      <child link="${prefix}gripper_pico_flexx_link"/>
+    </joint>
+    <sensor_pico_flexx camera_name="gripper_pico_flexx" prefix="${prefix}" />
+  </xacro:macro>
+  <xacro:macro name="sensor_mount" params="prefix">
+    <link name="${prefix}sensor_mount_link">
       <visual>
         <geometry>
@@ -47,13 +47,13 @@
       </inertial>
     </link>
-    <gazebo reference="sensor_mount_link">
+    <gazebo reference="${prefix}sensor_mount_link">
       <material>Gazebo/Grey</material>
     </gazebo>
-    <joint name="sensor_mount_bracket_joint" type="fixed">
+    <joint name="${prefix}sensor_mount_bracket_joint" type="fixed">
       <origin xyz="0 0 0" rpy="0 0 0" />
-      <parent link="sensor_mount_link"/>
-      <child link="sensor_mount_bracket_link" />
-    </joint>
-    <link name="sensor_mount_bracket_link">
+      <parent link="${prefix}sensor_mount_link"/>
+      <child link="${prefix}sensor_mount_bracket_link" />
+    </joint>
+    <link name="${prefix}sensor_mount_bracket_link">
       <visual>
         <geometry>
@@ -78,13 +78,13 @@
       </inertial>
     </link>
-    <gazebo reference="sensor_mount_bracket_link">
+    <gazebo reference="${prefix}sensor_mount_bracket_link">
       <material>Gazebo/Grey</material>
     </gazebo>
-    <joint name="sensor_mount_pico_holder_joint" type="fixed">
+    <joint name="${prefix}sensor_mount_pico_holder_joint" type="fixed">
       <origin xyz="-0.00325 0.11187 0" rpy="0 0 ${-33.5 / 180.0 * pi}" /> <!-- angle can be adjusted from -15 to -50 degrees (corresponds to downward angle of the pico flexx) -->
-      <parent link="sensor_mount_link"/>
-      <child link="sensor_mount_pico_holder_link" />
-    </joint>
-    <link name="sensor_mount_pico_holder_link">
+      <parent link="${prefix}sensor_mount_link"/>
+      <child link="${prefix}sensor_mount_pico_holder_link" />
+    </joint>
+    <link name="${prefix}sensor_mount_pico_holder_link">
       <visual>
         <geometry>
@@ -109,5 +109,5 @@
       </inertial>
     </link>
-    <gazebo reference="sensor_mount_pico_holder_link">
+    <gazebo reference="${prefix}sensor_mount_pico_holder_link">
       <material>Gazebo/Grey</material>
     </gazebo>
@@ -116,6 +116,6 @@
   <!-- ######################## Orbbec Astra Mini S ######################## -->
   <!-- ##################################################################### -->
-  <xacro:macro name="sensor_astra_mini_s" params="camera_name">
-    <link name="${camera_name}_link">
+  <xacro:macro name="sensor_astra_mini_s" params="camera_name prefix">
+    <link name="${prefix}${camera_name}_link">
       <visual>
         <origin xyz="0 0 0" />
@@ -135,35 +135,35 @@
       </xacro:box_inertial>
     </link>
-    <gazebo reference="${camera_name}_link">
+    <gazebo reference="${prefix}${camera_name}_link">
       <material>Gazebo/FlatBlack</material>
     </gazebo>
-    <joint name="${camera_name}_rgb_joint" type="fixed">
+    <joint name="${prefix}${camera_name}_rgb_joint" type="fixed">
       <origin xyz="0 -0.045 0" rpy="0 0 0" />
-      <parent link="${camera_name}_link"/>
-      <child link="${camera_name}_rgb_frame" />
-    </joint>
-    <link name="${camera_name}_rgb_frame"/>
-    <joint name="${camera_name}_rgb_optical_joint" type="fixed">
+      <parent link="${prefix}${camera_name}_link"/>
+      <child link="${prefix}${camera_name}_rgb_frame" />
+    </joint>
+    <link name="${prefix}${camera_name}_rgb_frame"/>
+    <joint name="${prefix}${camera_name}_rgb_optical_joint" type="fixed">
       <origin xyz="0 0 0" rpy="${-pi/2} 0 ${-pi/2}" />
-      <parent link="${camera_name}_rgb_frame" />
-      <child link="${camera_name}_rgb_optical_frame" />
-    </joint>
-    <link name="${camera_name}_rgb_optical_frame"/>
-    <joint name="${camera_name}_depth_joint" type="fixed">
+      <parent link="${prefix}${camera_name}_rgb_frame" />
+      <child link="${prefix}${camera_name}_rgb_optical_frame" />
+    </joint>
+    <link name="${prefix}${camera_name}_rgb_optical_frame"/>
+    <joint name="${prefix}${camera_name}_depth_joint" type="fixed">
       <origin xyz="0 -0.02 0" rpy="0 0 0" />
-      <parent link="${camera_name}_link"/>
-      <child link="${camera_name}_depth_frame" />
-    </joint>
-    <link name="${camera_name}_depth_frame"/>
-    <joint name="${camera_name}_depth_optical_joint" type="fixed">
+      <parent link="${prefix}${camera_name}_link"/>
+      <child link="${prefix}${camera_name}_depth_frame" />
+    </joint>
+    <link name="${prefix}${camera_name}_depth_frame"/>
+    <joint name="${prefix}${camera_name}_depth_optical_joint" type="fixed">
       <origin xyz="-0.025 0 0" rpy="0 0 0" />   <!-- calibration not necessary, depth_ir_offset used instead -->
-      <parent link="${camera_name}_rgb_optical_frame" />
-      <child link="${camera_name}_depth_optical_frame" />
-    </joint>
-    <link name="${camera_name}_depth_optical_frame"/>
-    <sim_3dsensor/>
-  </xacro:macro>
-  <xacro:macro name="sim_3dsensor">
-    <gazebo reference="${camera_name}_depth_frame">
+      <parent link="${prefix}${camera_name}_rgb_optical_frame" />
+      <child link="${prefix}${camera_name}_depth_optical_frame" />
+    </joint>
+    <link name="${prefix}${camera_name}_depth_optical_frame"/>
+    <sim_3dsensor prefix="${prefix}"/>
+  </xacro:macro>
+  <xacro:macro name="sim_3dsensor" params="prefix">
+    <gazebo reference="${prefix}${camera_name}_depth_frame">
       <sensor type="depth" name="${camera_name}">
         <always_on>true</always_on>
@@ -190,5 +190,5 @@
           <cameraInfoTopicName>rgb/camera_info</cameraInfoTopicName>
           <depthImageCameraInfoTopicName>depth_registered/camera_info</depthImageCameraInfoTopicName>
-          <frameName>${camera_name}_depth_optical_frame</frameName>
+          <frameName>${prefix}${camera_name}_depth_optical_frame</frameName>
           <distortion_k1>0.0</distortion_k1>
           <distortion_k2>0.0</distortion_k2>
@@ -205,6 +205,6 @@
   <!-- ######################## PMD CamBoard pico flexx ######################## -->
   <!-- ######################################################################### -->
-  <xacro:macro name="sensor_pico_flexx" params="camera_name">
-    <link name="${camera_name}_link">
+  <xacro:macro name="sensor_pico_flexx" params="camera_name prefix">
+    <link name="${prefix}${camera_name}_link">
       <visual>
         <origin xyz="0 0 0" />
@@ -224,23 +224,23 @@
       </xacro:box_inertial>
     </link>
-    <gazebo reference="${camera_name}_link">
+    <gazebo reference="${prefix}${camera_name}_link">
       <material>Gazebo/FlatBlack</material>
     </gazebo>
-    <joint name="${camera_name}_depth_joint" type="fixed">
+    <joint name="${prefix}${camera_name}_depth_joint" type="fixed">
       <origin xyz="0.0072 0.0081 0.0" rpy="0 0 0" />
-      <parent link="${camera_name}_link"/>
-      <child link="${camera_name}_frame" />
-    </joint>
-    <link name="${camera_name}_frame"/>
-    <joint name="${camera_name}_optical_joint" type="fixed">
+      <parent link="${prefix}${camera_name}_link"/>
+      <child link="${prefix}${camera_name}_frame" />
+    </joint>
+    <link name="${prefix}${camera_name}_frame"/>
+    <joint name="${prefix}${camera_name}_optical_joint" type="fixed">
       <origin xyz="0 0 0" rpy="${-pi/2} 0 ${-pi/2}" />
-      <parent link="${camera_name}_frame" />
-      <child link="${camera_name}_optical_frame" />
-    </joint>
-    <link name="${camera_name}_optical_frame"/>
-    <sim_pico_flexx/>
-  </xacro:macro>
-  <xacro:macro name="sim_pico_flexx">
-    <gazebo reference="${camera_name}_frame">
+      <parent link="${prefix}${camera_name}_frame" />
+      <child link="${prefix}${camera_name}_optical_frame" />
+    </joint>
+    <link name="${prefix}${camera_name}_optical_frame"/>
+    <sim_pico_flexx prefix="${prefix}"/>
+  </xacro:macro>
+  <xacro:macro name="sim_pico_flexx" params="prefix">
+    <gazebo reference="${prefix}${camera_name}_frame">
       <sensor type="depth" name="${camera_name}">
         <always_on>true</always_on>
@@ -268,5 +268,5 @@
           <cameraInfoTopicName>camera_info</cameraInfoTopicName>
           <depthImageCameraInfoTopicName>depth/camera_info</depthImageCameraInfoTopicName>
-          <frameName>${camera_name}_optical_frame</frameName>
+          <frameName>${prefix}${camera_name}_optical_frame</frameName>
           <distortion_k1>0.0</distortion_k1>
           <distortion_k2>0.0</distortion_k2>
