Commit message: Fix UR5 mounting position

File: mobipick_description/urdf/mobipick/mobipick_v1_model.urdf.xacro (robot description, xacro)
@@ -31,5 +31,5 @@
   </joint>
   <joint name="struct_ur5_joint" type="fixed">
-    <parent link="structure_pedestal" />
+    <parent link="structure_pedestal_surface" />
     <child link = "ur5_base_link" />
     <origin xyz="0.0 0.0 0.0025" rpy="0.0 0.0 0.0" />

Commit message: mobipick: Reorder mobipick xacro

File: mobipick_description/urdf/mobipick/mobipick_v1_model.urdf.xacro (robot description, xacro)
@@ -2,27 +2,16 @@
 <robot xmlns:xacro="http://ros.org/wiki/xacro"
        name="mobipick">
-  <!-- mir_100 -->
+  <!-- ############## BASE_LINK  ############## -->
+  <link name="base_link" />
+  <joint name="base_joint" type="fixed">
+    <parent link="base_link" />
+    <child link="mir_base" />
+    <origin xyz="0.0 0.0 0.0" rpy="0.0 0.0 0.0" />
+  </joint>
+  <!-- ############# MIR100 BASE ############## -->
   <xacro:include filename="$(find mobipick_description)/urdf/mir_100/mir_100_v1.urdf.xacro" />
-  <!-- structure -->
+  <xacro:mir_100 prefix="mir_"/>
+  <!-- ############## STRUCTURE ############### -->
   <xacro:include filename="$(find mobipick_description)/urdf/structure/mobipick_structure.urdf.xacro" />
-  <!-- ur5 -->
-  <xacro:include filename="$(find mobipick_description)/urdf/ur5/ur5.urdf.xacro" />
-  <!-- ft_300 -->
-  <xacro:include filename="$(find mobipick_description)/urdf/robotiq_ft_300/robotiq_ft_300.urdf.xacro" />
-  <!-- 2f_140 -->
-  <xacro:include filename="$(find mobipick_description)/urdf/robotiq_2f_140/robotiq_arg2f_140_model_macro.xacro" />
-  <!-- mobile robot -->
-  <xacro:mir_100 prefix="mir_"/>
-  <!-- structure -->
-  <xacro:structure prefix="structure_" height="0.1" />
-  <!-- arm -->
-  <xacro:ur5_robot prefix="ur5_" joint_limited="true"/>
-  <!-- sensor -->
-  <xacro:robotiq_ft_300 parent="ur5_tool0" prefix="" >
-      <pose xyz="0 0 0" rpy="0 0 0" />
-      <!-- <pose xyz="0 0 0.009" rpy="0 0 0" /> -->
-  </xacro:robotiq_ft_300>
-  <!-- gripper -->
-  <xacro:robotiq_arg2f_140 prefix="gripper_"/>
   <joint name="mir_struct_joint" type="fixed">
     <parent link="mir_surface" />
@@ -30,4 +19,7 @@
     <origin xyz="0.0 0.0 0.0" rpy="0.0 0.0 0.0" />
   </joint>
+  <xacro:structure prefix="structure_" height="0.1" />
+  <!-- ############### UR5 ARM ################ -->
+  <xacro:include filename="$(find mobipick_description)/urdf/ur5/ur5.urdf.xacro" />
   <joint name="struct_ur5_joint" type="fixed">
     <parent link="structure_pedestal_surface" />
@@ -35,4 +27,13 @@
     <origin xyz="0.0 0.0 0.0025" rpy="0.0 0.0 0.0" />
   </joint>
+  <xacro:ur5_robot prefix="ur5_" joint_limited="true"/>
+  <!-- ############## FT SENSOR ############### -->
+  <xacro:include filename="$(find mobipick_description)/urdf/robotiq_ft_300/robotiq_ft_300.urdf.xacro" />
+  <xacro:robotiq_ft_300 parent="ur5_tool0" prefix="" >
+      <pose xyz="0 0 0" rpy="0 0 0" />
+      <!-- <pose xyz="0 0 0.009" rpy="0 0 0" /> -->
+  </xacro:robotiq_ft_300>
+  <!-- ############### GRIPPER ################ -->
+  <xacro:include filename="$(find mobipick_description)/urdf/robotiq_2f_140/robotiq_arg2f_140_model_macro.xacro" />
   <joint name="ft300_2f140_joint" type="fixed">
     <origin xyz="0 0 0" rpy="0 0 0" />
@@ -41,11 +42,6 @@
     <axis xyz="0 0 1" />
   </joint>
-  <link name="base_link" />
-  <joint name="base_joint" type="fixed">
-    <parent link="base_link" />
-    <child link="mir_base" />
-    <origin xyz="0.0 0.0 0.0" rpy="0.0 0.0 0.0" />
-  </joint>
-  <!-- gazebo -->
+  <xacro:robotiq_arg2f_140 prefix="gripper_"/>
+  <!-- ################ GAZEBO ################ -->
   <xacro:include filename="$(find mobipick_description)/urdf/mobipick/mobipick.gazebo.xacro" />
 </robot>

Commit message: mobipick: Remove mir_prefix
... to make it compatible with standalone MiR ros_control config

File: mobipick_description/urdf/mobipick/mobipick_v1_model.urdf.xacro (robot description, xacro)
@@ -6,14 +6,14 @@
   <joint name="base_joint" type="fixed">
     <parent link="base_link" />
-    <child link="mir_base" />
+    <child link="base" />
     <origin xyz="0.0 0.0 0.0" rpy="0.0 0.0 0.0" />
   </joint>
   <!-- ############# MIR100 BASE ############## -->
   <xacro:include filename="$(find mobipick_description)/urdf/mir_100/mir_100_v1.urdf.xacro" />
-  <xacro:mir_100 prefix="mir_"/>
+  <xacro:mir_100 prefix=""/>
   <!-- ############## STRUCTURE ############### -->
   <xacro:include filename="$(find mobipick_description)/urdf/structure/mobipick_structure.urdf.xacro" />
   <joint name="mir_struct_joint" type="fixed">
-    <parent link="mir_surface" />
+    <parent link="surface" />
     <child link = "structure_part_down" />
     <origin xyz="0.0 0.0 0.0" rpy="0.0 0.0 0.0" />

Commit message: Add gripper camera

File: mobipick_description/urdf/mobipick/mobipick_v1_model.urdf.xacro (robot description, xacro)
@@ -33,7 +33,14 @@
     <parent link="fts_toolside" />
     <child link="gripper_robotiq_arg2f_base_link" />
-    <axis xyz="0 0 1" />
   </joint>
   <xacro:robotiq_arg2f_140 prefix="gripper_"/>
+  <!-- ############### SENSOR MOUNT + 3D CAM  ################ -->
+  <xacro:include filename="$(find mobipick_description)/urdf/sensors/gripper_cam.urdf.xacro" />
+  <joint name="sensor_mount_joint" type="fixed">
+    <origin xyz="0.0 0.0 0.01" rpy="0.0 ${-pi/2} ${pi/2}" />
+    <parent link="gripper_robotiq_arg2f_base_link" />
+    <child link="sensor_mount_link" />
+  </joint>
+  <gripper_cam />
   <!-- ################ GAZEBO ################ -->
   <xacro:include filename="$(find mobipick_description)/urdf/mobipick/mobipick.gazebo.xacro" />

Commit message: urdf: Add Mobipick v2 structure

File: mobipick_description/urdf/mobipick/mobipick_v1_model.urdf.xacro (robot description, xacro)
@@ -12,5 +12,5 @@
     <origin xyz="0.0 0.0 0.0" rpy="0.0 0.0 0.0" />
   </joint>
-  <xacro:structure prefix="structure_" height="0.1" />
+  <xacro:structure prefix="structure_" height="0.1" variant="v1" />
   <!-- ############### UR5 ARM ################ -->
   <xacro:include filename="$(find mobipick_description)/urdf/ur5/ur5.urdf.xacro" />

File: mobipick_description/urdf/structure/mobipick_structure.urdf.xacro (robot description, xacro)
@@ -2,5 +2,9 @@
 <robot xmlns:xacro="http://ros.org/wiki/xacro">
   <xacro:include filename="$(find mobipick_description)/urdf/common_properties.urdf.xacro" />
-  <xacro:macro name="structure" params="prefix height">
+  <!-- variant can be one of:
+       - v1: The original Mobipick in Bremen, built for the Hybr-iT project
+       - v2: The newer Mobipicks: one in Osnabrueck, two in Bremen for the UPLINX project
+  -->
+  <xacro:macro name="structure" params="prefix height variant='v1'">
     <link name="${prefix}part_down">
       <inertial>
@@ -18,5 +22,5 @@
         <origin xyz="0 0 0" rpy="0 0 0" />
         <geometry>
-          <mesh filename="package://mobipick_description/meshes/structure/visual/v1/part_down.stl" />
+          <mesh filename="package://mobipick_description/meshes/structure/visual/${variant}/part_down.stl" />
         </geometry>
         <xacro:insert_block name="material_aluminum" />
@@ -25,5 +29,5 @@
         <origin xyz="0 0 0" rpy="0 0 0" />
         <geometry>
-          <mesh filename="package://mobipick_description/meshes/structure/collision/v1/part_down.stl" />
+          <mesh filename="package://mobipick_description/meshes/structure/collision/${variant}/part_down.stl" />
         </geometry>
       </collision>
@@ -47,5 +51,5 @@
         <origin xyz="0 0 0" rpy="0 0 0" />
         <geometry>
-          <mesh filename="package://mobipick_description/meshes/structure/visual/v1/part_up.stl" />
+          <mesh filename="package://mobipick_description/meshes/structure/visual/${variant}/part_up.stl" />
         </geometry>
         <xacro:insert_block name="material_aluminum" />
@@ -54,5 +58,5 @@
         <origin xyz="0 0 0" rpy="0 0 0" />
         <geometry>
-          <mesh filename="package://mobipick_description/meshes/structure/collision/v1/part_up.stl" />
+          <mesh filename="package://mobipick_description/meshes/structure/collision/${variant}/part_up.stl" />
         </geometry>
       </collision>
@@ -76,5 +80,5 @@
         <origin xyz="0 0 0" rpy="0 0 0" />
         <geometry>
-          <mesh filename="package://mobipick_description/meshes/structure/visual/v1/pedestal.stl" />
+          <mesh filename="package://mobipick_description/meshes/structure/visual/${variant}/pedestal.stl" />
         </geometry>
         <xacro:insert_block name="material_aluminum" />
@@ -83,5 +87,5 @@
         <origin xyz="0 0 0" rpy="0 0 0" />
         <geometry>
-          <mesh filename="package://mobipick_description/meshes/structure/collision/v1/pedestal.stl" />
+          <mesh filename="package://mobipick_description/meshes/structure/collision/${variant}/pedestal.stl" />
         </geometry>
       </collision>
@@ -110,6 +114,12 @@
       <axis xyz="0 0 1" />
     </joint>
+    <xacro:if value="${variant == 'v1'}">
+      <xacro:property name="pedestal_height" value="0.2492" />
+    </xacro:if>
+    <xacro:if value="${variant == 'v2'}">
+      <xacro:property name="pedestal_height" value="0.2291" />
+    </xacro:if>
     <joint name="${prefix}Tischaufbau_base_joint" type="fixed">
-      <origin xyz="0 0 0.25" rpy="0 0 0" />
+      <origin xyz="0 0 ${pedestal_height}" rpy="0 0 0" />
       <parent link="${prefix}pedestal" />
       <child link="${prefix}pedestal_surface" />

Commit message: Fix gripper rotation

File: mobipick_description/urdf/mobipick/mobipick_v1_model.urdf.xacro (robot description, xacro)
@@ -30,5 +30,5 @@
   <xacro:include filename="$(find mobipick_description)/urdf/robotiq_2f_140/robotiq_arg2f_140_model_macro.xacro" />
   <joint name="ft300_2f140_joint" type="fixed">
-    <origin xyz="0 0 0" rpy="0 0 0" />
+    <origin xyz="0 0 0" rpy="0 0 ${-pi/2}" />
     <parent link="fts_toolside" />
     <child link="gripper_robotiq_arg2f_base_link" />

Commit message: Fix structure height + sensor mount placement
... based on the astra_and_pico_2018-05-07-15-27-52-filtered.bag rosbag.

File: mobipick_description/urdf/mobipick/mobipick_v1_model.urdf.xacro (robot description, xacro)
@@ -12,5 +12,5 @@
     <origin xyz="0.0 0.0 0.0" rpy="0.0 0.0 0.0" />
   </joint>
-  <xacro:structure prefix="structure_" height="0.1" variant="v1" />
+  <xacro:structure prefix="structure_" height="0.065" variant="v1" />
   <!-- ############### UR5 ARM ################ -->
   <xacro:include filename="$(find mobipick_description)/urdf/ur5/ur5.urdf.xacro" />
@@ -38,5 +38,5 @@
   <xacro:include filename="$(find mobipick_description)/urdf/sensors/gripper_cam.urdf.xacro" />
   <joint name="sensor_mount_joint" type="fixed">
-    <origin xyz="0.0 0.0 0.01" rpy="0.0 ${-pi/2} ${pi/2}" />
+    <origin xyz="0.0 0.0 -0.02" rpy="0.0 ${-pi/2} ${pi/2}" />
     <parent link="gripper_robotiq_arg2f_base_link" />
     <child link="sensor_mount_link" />

Commit message: URDF: Fix orientation of FT sensor (closes #1)

File: mobipick_description/urdf/mobipick/mobipick_v1_model.urdf.xacro (robot description, xacro)
@@ -38,5 +38,5 @@
   <xacro:include filename="$(find mobipick_description)/urdf/sensors/gripper_cam.urdf.xacro" />
   <joint name="sensor_mount_joint" type="fixed">
-    <origin xyz="0.0 0.0 -0.02" rpy="0.0 ${-pi/2} ${pi/2}" />
+    <origin xyz="0.0 0.0 -0.005" rpy="0.0 ${-pi/2} ${pi/2}" />
     <parent link="gripper_robotiq_arg2f_base_link" />
     <child link="sensor_mount_link" />

Commit message: URDF: Change parent of sensor_mount_link

File: mobipick_description/urdf/mobipick/mobipick_v1_model.urdf.xacro (robot description, xacro)
@@ -38,6 +38,6 @@
   <xacro:include filename="$(find mobipick_description)/urdf/sensors/gripper_cam.urdf.xacro" />
   <joint name="sensor_mount_joint" type="fixed">
-    <origin xyz="0.0 0.0 -0.005" rpy="0.0 ${-pi/2} ${pi/2}" />
-    <parent link="gripper_robotiq_arg2f_base_link" />
+    <origin xyz="0.0 0.0 -0.005" rpy="0.0 ${-pi/2} 0.0" />
+    <parent link="fts_toolside" />
     <child link="sensor_mount_link" />
   </joint>

Commit message: URDF: Add gripper coupling

File: mobipick_description/urdf/mobipick/mobipick_v1_model.urdf.xacro (robot description, xacro)
@@ -29,7 +29,39 @@
   <!-- ############### GRIPPER ################ -->
   <xacro:include filename="$(find mobipick_description)/urdf/robotiq_2f_140/robotiq_arg2f_140_model_macro.xacro" />
-  <joint name="ft300_2f140_joint" type="fixed">
-    <origin xyz="0 0 0" rpy="0 0 ${-pi/2}" />
+  <!-- gripper coupling (ISO 9409-1-50-4-M / Robotiq AGC-CPL-062-002_20171219) -->
+  <xacro:property name="coupling_radius" value="0.0375" />
+  <xacro:property name="coupling_outer_length" value="0.014" />
+  <xacro:property name="coupling_inner_length" value="0.008" />
+  <xacro:property name="coupling_mass" value="0.100" />
+  <joint name="ft300_coupling_joint" type="fixed">
+    <origin xyz="0 0 ${coupling_inner_length / 2}" rpy="0 0 ${-pi/2}" />
     <parent link="fts_toolside" />
+    <child link="gripper_coupling_link" />
+  </joint>
+  <link name="gripper_coupling_link">
+    <origin xyz="0 0 0" rpy="0 0 0" />
+    <visual>
+      <origin xyz="0 0 0" rpy="0 0 0" />
+      <geometry>
+        <cylinder radius="${coupling_radius}" length="${coupling_outer_length}" />
+      </geometry>
+      <xacro:insert_block name="material_black" />
+    </visual>
+    <collision>
+      <origin xyz="0 0 0" rpy="0 0 0" />
+      <geometry>
+        <cylinder radius="${coupling_radius}" length="${coupling_outer_length}" />
+      </geometry>
+    </collision>
+    <xacro:cylinder_inertial radius="${coupling_radius}" length="${coupling_outer_length}" mass="${coupling_mass}">
+      <origin xyz="0.0 0.0 0.0" rpy="0 0 0" />
+    </xacro:cylinder_inertial>
+  </link>
+  <gazebo reference="gripper_coupling_link">
+    <material>Gazebo/FlatBlack</material>
+  </gazebo>
+  <joint name="coupling_2f140_joint" type="fixed">
+    <origin xyz="0 0 ${coupling_inner_length / 2}" rpy="0 0 0" />
+    <parent link="gripper_coupling_link" />
     <child link="gripper_robotiq_arg2f_base_link" />
   </joint>

Commit message: URDF: Add xacro argument 'robot'

File: mobipick_description/urdf/mobipick/mobipick_v1_model.urdf.xacro (robot description, xacro)
@@ -2,4 +2,6 @@
 <robot xmlns:xacro="http://ros.org/wiki/xacro"
        name="mobipick">
+  <xacro:arg name="robot" default="mobipick-hb" />      <!-- can be "mobipick-hb" or "mobipick-os" -->
+  <xacro:property name="robot" value="$(arg robot)" />  <!-- necessary because args cannot be accessed inside ${} expressions -->
   <!-- ############# MIR100 BASE ############## -->
   <xacro:include filename="$(find mobipick_description)/urdf/mir_100/mir_100_v1.urdf.xacro" />
@@ -12,5 +14,10 @@
     <origin xyz="0.0 0.0 0.0" rpy="0.0 0.0 0.0" />
   </joint>
-  <xacro:structure prefix="structure_" height="0.058" variant="v1" />
+  <xacro:if value="${robot == 'mobipick-hb'}">
+    <xacro:structure prefix="structure_" height="0.058" variant="v1" />
+  </xacro:if>
+  <xacro:if value="${robot == 'mobipick-os'}">
+    <xacro:structure prefix="structure_" height="0.058" variant="v2" />
+  </xacro:if>
   <!-- ############### UR5 ARM ################ -->
   <xacro:include filename="$(find mobipick_description)/urdf/ur5/ur5.urdf.xacro" />

Commit message: URDF: Add dual xtions

File: mobipick_description/urdf/mobipick/mobipick_v1_model.urdf.xacro (robot description, xacro)
@@ -82,4 +82,12 @@
   </joint>
   <gripper_cam />
+  <!-- ############### DUAL XTION MOUNT + XTIONS ################ -->
+  <xacro:include filename="$(find mobipick_description)/urdf/sensors/dual_xtions.urdf.xacro" />
+  <joint name="dual_xtion_mount_joint" type="fixed">
+    <origin xyz="0.35 -0.18 0.0" rpy="0.0 0.0 ${-45.0 / 180.0 * pi}" />   <!-- TODO HENDRIK -->
+    <parent link="structure_pedestal" />
+    <child link="dual_xtion_mount_link" />
+  </joint>
+  <dual_xtions />
   <!-- ################ GAZEBO ################ -->
   <xacro:include filename="$(find mobipick_description)/urdf/mobipick/mobipick.gazebo.xacro" />

Commit message: Add dual xtion mount for people tracking

File: mobipick_description/urdf/mobipick/mobipick_v1_model.urdf.xacro (robot description, xacro)
@@ -85,5 +85,5 @@
   <xacro:include filename="$(find mobipick_description)/urdf/sensors/dual_xtions.urdf.xacro" />
   <joint name="dual_xtion_mount_joint" type="fixed">
-    <origin xyz="0.35 -0.18 0.0" rpy="0.0 0.0 ${-45.0 / 180.0 * pi}" />   <!-- TODO HENDRIK -->
+    <origin xyz="0.37 0.0 -0.02" rpy="0 0 0" />
     <parent link="structure_pedestal" />
     <child link="dual_xtion_mount_link" />

File: mobipick_description/urdf/sensors/dual_xtions.urdf.xacro (robot description, xacro)
@@ -9,36 +9,39 @@
   <xacro:property name="xtion_cam_py" value="0.069"/>
   <xacro:macro name="dual_xtions" params="">
-    <dual_xtion_mount />
+    <link name="dual_xtion_mount_link" />
+    <joint name="dual_xtion_left_mount" type="fixed">
+      <parent link="dual_xtion_mount_link" />
+      <child link="dual_xtion_left_mount_link" />
+      <origin xyz="0 0.06 0" rpy="0.0 1.571 0.0" />
+    </joint>
+    <dual_xtion_mount side="left" />
+    <joint name="dual_xtion_right_mount" type="fixed">
+      <parent link="dual_xtion_mount_link" />
+      <child link="dual_xtion_right_mount_link" />
+      <origin xyz="0 -0.06 0" rpy="0.0 -1.571 3.142" />
+    </joint>
+    <dual_xtion_mount side="right" />
     <joint name="dual_xtion_bottom_joint" type="fixed">
-      <origin xyz="0.04 ${xtion_cam_py} ${dual_xtion_mount_z - 0.04}" rpy="0 ${22.0 / 180.0 * pi} 0" />   <!-- TODO HENDRIK -->
-      <parent link="dual_xtion_mount_link"/>
-      <child link="dual_xtion_bottom_link"/>
+      <parent link="dual_xtion_mount_link" />
+      <child link="dual_xtion_bottom_link" />
+      <origin xyz="0.045 0.069 0.032" rpy="0 -0.262 0" />
     </joint>
     <sensor_xtion camera_name="dual_xtion_bottom" />
     <joint name="dual_xtion_top_joint" type="fixed">
-      <origin xyz="0.04 ${xtion_cam_py} ${dual_xtion_mount_z + 0.02}" rpy="0 ${-22.0 / 180.0 * pi} 0" />   <!-- TODO HENDRIK -->
-      <parent link="dual_xtion_mount_link"/>
-      <child link="dual_xtion_top_link"/>
+      <parent link="dual_xtion_mount_link" />
+      <child link="dual_xtion_top_link" />
+      <origin xyz="0.045 0.069 -0.032" rpy="0 0.262 0" />
     </joint>
     <sensor_xtion camera_name="dual_xtion_top" />
   </xacro:macro>
-  <xacro:macro name="dual_xtion_mount">
-    <link name="dual_xtion_mount_link">
+  <xacro:macro name="dual_xtion_mount" params="side">
+    <link name="dual_xtion_${side}_mount_link">
+      <origin xyz="0 0 0" rpy="0 0 0" />
       <visual>
-        <origin xyz="0 0 ${dual_xtion_mount_z / 2}" />
+        <origin xyz="0 0 0" rpy="0 0 0" />
         <geometry>
-          <box size="${dual_xtion_mount_x} ${dual_xtion_mount_y} ${dual_xtion_mount_z}" />
+          <mesh scale="0.001 0.001 0.001" filename="package://mobipick_description/meshes/sensors/peotrac_mount.stl" />
         </geometry>
-        <xacro:insert_block name="material_black" />
       </visual>
-      <collision>
-        <origin xyz="0 0 ${dual_xtion_mount_z / 2}" />
-        <geometry>
-          <box size="${dual_xtion_mount_x} ${dual_xtion_mount_y} ${dual_xtion_mount_z}" />
-        </geometry>
-      </collision>
-      <xacro:box_inertial mass="${dual_xtion_mount_mass}" x="${dual_xtion_mount_x}" y="${dual_xtion_mount_y}" z="${dual_xtion_mount_z}">
-        <origin xyz="0 0 ${dual_xtion_mount_z / 2}" />
-      </xacro:box_inertial>
     </link>
     <gazebo reference="dual_xtion_mount_link">
