Commit message: urdf: Remove dual xtions

File: mobipick_description/urdf/mobipick/mobipick_v1_model.urdf.xacro (robot description, xacro)
@@ -91,11 +91,13 @@
   <gripper_cam prefix="${prefix}" />
   <!-- ############### DUAL XTION MOUNT + XTIONS ################ -->
-  <xacro:include filename="$(find mobipick_description)/urdf/sensors/dual_xtions.urdf.xacro" />
-  <joint name="${prefix}dual_xtion_mount_joint" type="fixed">
-    <origin xyz="0.37 0.0 -0.02" rpy="0 0 0" />
-    <parent link="${prefix}structure_pedestal" />
-    <child link="${prefix}dual_xtion_mount_link" />
-  </joint>
-  <dual_xtions prefix="${prefix}" />
+  <xacro:if value="${robot == 'mobipick-hb'}">
+    <xacro:include filename="$(find mobipick_description)/urdf/sensors/dual_xtions.urdf.xacro" />
+    <joint name="${prefix}dual_xtion_mount_joint" type="fixed">
+      <origin xyz="0.37 0.0 -0.02" rpy="0 0 0" />
+      <parent link="${prefix}structure_pedestal" />
+      <child link="${prefix}dual_xtion_mount_link" />
+    </joint>
+    <dual_xtions prefix="${prefix}" />
+  </xacro:if>
   <!-- ################ GAZEBO ################ -->
   <xacro:include filename="$(find mobipick_description)/urdf/mobipick/mobipick.gazebo.xacro" />

File: mobipick_moveit_config/config/mobipick.srdf.xacro (robot description, xacro)
@@ -145,8 +145,4 @@
     <disable_collisions link1="${tf_prefix}back_laser_link" link2="${tf_prefix}br_caster_rotation_link" reason="Never" />
     <disable_collisions link1="${tf_prefix}back_laser_link" link2="${tf_prefix}br_caster_wheel_link" reason="Never" />
-    <disable_collisions link1="${tf_prefix}back_laser_link" link2="${tf_prefix}dual_xtion_bottom_link" reason="Never" />
-    <disable_collisions link1="${tf_prefix}back_laser_link" link2="${tf_prefix}dual_xtion_left_mount_link" reason="Never" />
-    <disable_collisions link1="${tf_prefix}back_laser_link" link2="${tf_prefix}dual_xtion_right_mount_link" reason="Never" />
-    <disable_collisions link1="${tf_prefix}back_laser_link" link2="${tf_prefix}dual_xtion_top_link" reason="Never" />
     <disable_collisions link1="${tf_prefix}back_laser_link" link2="${tf_prefix}fl_caster_rotation_link" reason="Never" />
     <disable_collisions link1="${tf_prefix}back_laser_link" link2="${tf_prefix}fl_caster_wheel_link" reason="Never" />
@@ -189,8 +185,4 @@
     <disable_collisions link1="${tf_prefix}base_link" link2="${tf_prefix}br_caster_rotation_link" reason="Adjacent" />
     <disable_collisions link1="${tf_prefix}base_link" link2="${tf_prefix}br_caster_wheel_link" reason="Never" />
-    <disable_collisions link1="${tf_prefix}base_link" link2="${tf_prefix}dual_xtion_bottom_link" reason="Never" />
-    <disable_collisions link1="${tf_prefix}base_link" link2="${tf_prefix}dual_xtion_left_mount_link" reason="Never" />
-    <disable_collisions link1="${tf_prefix}base_link" link2="${tf_prefix}dual_xtion_right_mount_link" reason="Never" />
-    <disable_collisions link1="${tf_prefix}base_link" link2="${tf_prefix}dual_xtion_top_link" reason="Never" />
     <disable_collisions link1="${tf_prefix}base_link" link2="${tf_prefix}fl_caster_rotation_link" reason="Adjacent" />
     <disable_collisions link1="${tf_prefix}base_link" link2="${tf_prefix}fl_caster_wheel_link" reason="Never" />
@@ -217,8 +209,4 @@
     <disable_collisions link1="${tf_prefix}bl_caster_rotation_link" link2="${tf_prefix}br_caster_rotation_link" reason="Never" />
     <disable_collisions link1="${tf_prefix}bl_caster_rotation_link" link2="${tf_prefix}br_caster_wheel_link" reason="Never" />
-    <disable_collisions link1="${tf_prefix}bl_caster_rotation_link" link2="${tf_prefix}dual_xtion_bottom_link" reason="Never" />
-    <disable_collisions link1="${tf_prefix}bl_caster_rotation_link" link2="${tf_prefix}dual_xtion_left_mount_link" reason="Never" />
-    <disable_collisions link1="${tf_prefix}bl_caster_rotation_link" link2="${tf_prefix}dual_xtion_right_mount_link" reason="Never" />
-    <disable_collisions link1="${tf_prefix}bl_caster_rotation_link" link2="${tf_prefix}dual_xtion_top_link" reason="Never" />
     <disable_collisions link1="${tf_prefix}bl_caster_rotation_link" link2="${tf_prefix}fl_caster_rotation_link" reason="Never" />
     <disable_collisions link1="${tf_prefix}bl_caster_rotation_link" link2="${tf_prefix}fl_caster_wheel_link" reason="Never" />
@@ -259,8 +247,4 @@
     <disable_collisions link1="${tf_prefix}bl_caster_wheel_link" link2="${tf_prefix}br_caster_rotation_link" reason="Never" />
     <disable_collisions link1="${tf_prefix}bl_caster_wheel_link" link2="${tf_prefix}br_caster_wheel_link" reason="Never" />
-    <disable_collisions link1="${tf_prefix}bl_caster_wheel_link" link2="${tf_prefix}dual_xtion_bottom_link" reason="Never" />
-    <disable_collisions link1="${tf_prefix}bl_caster_wheel_link" link2="${tf_prefix}dual_xtion_left_mount_link" reason="Never" />
-    <disable_collisions link1="${tf_prefix}bl_caster_wheel_link" link2="${tf_prefix}dual_xtion_right_mount_link" reason="Never" />
-    <disable_collisions link1="${tf_prefix}bl_caster_wheel_link" link2="${tf_prefix}dual_xtion_top_link" reason="Never" />
     <disable_collisions link1="${tf_prefix}bl_caster_wheel_link" link2="${tf_prefix}fl_caster_rotation_link" reason="Never" />
     <disable_collisions link1="${tf_prefix}bl_caster_wheel_link" link2="${tf_prefix}fl_caster_wheel_link" reason="Never" />
@@ -300,8 +284,4 @@
     <disable_collisions link1="${tf_prefix}bl_caster_wheel_link" link2="${tf_prefix}ur5_wrist_3_link" reason="Never" />
     <disable_collisions link1="${tf_prefix}br_caster_rotation_link" link2="${tf_prefix}br_caster_wheel_link" reason="Adjacent" />
-    <disable_collisions link1="${tf_prefix}br_caster_rotation_link" link2="${tf_prefix}dual_xtion_bottom_link" reason="Never" />
-    <disable_collisions link1="${tf_prefix}br_caster_rotation_link" link2="${tf_prefix}dual_xtion_left_mount_link" reason="Never" />
-    <disable_collisions link1="${tf_prefix}br_caster_rotation_link" link2="${tf_prefix}dual_xtion_right_mount_link" reason="Never" />
-    <disable_collisions link1="${tf_prefix}br_caster_rotation_link" link2="${tf_prefix}dual_xtion_top_link" reason="Never" />
     <disable_collisions link1="${tf_prefix}br_caster_rotation_link" link2="${tf_prefix}fl_caster_rotation_link" reason="Never" />
     <disable_collisions link1="${tf_prefix}br_caster_rotation_link" link2="${tf_prefix}fl_caster_wheel_link" reason="Never" />
@@ -340,8 +320,4 @@
     <disable_collisions link1="${tf_prefix}br_caster_rotation_link" link2="${tf_prefix}ur5_wrist_2_link" reason="Never" />
     <disable_collisions link1="${tf_prefix}br_caster_rotation_link" link2="${tf_prefix}ur5_wrist_3_link" reason="Never" />
-    <disable_collisions link1="${tf_prefix}br_caster_wheel_link" link2="${tf_prefix}dual_xtion_bottom_link" reason="Never" />
-    <disable_collisions link1="${tf_prefix}br_caster_wheel_link" link2="${tf_prefix}dual_xtion_left_mount_link" reason="Never" />
-    <disable_collisions link1="${tf_prefix}br_caster_wheel_link" link2="${tf_prefix}dual_xtion_right_mount_link" reason="Never" />
-    <disable_collisions link1="${tf_prefix}br_caster_wheel_link" link2="${tf_prefix}dual_xtion_top_link" reason="Never" />
     <disable_collisions link1="${tf_prefix}br_caster_wheel_link" link2="${tf_prefix}fl_caster_rotation_link" reason="Never" />
     <disable_collisions link1="${tf_prefix}br_caster_wheel_link" link2="${tf_prefix}fl_caster_wheel_link" reason="Never" />
@@ -380,59 +356,4 @@
     <disable_collisions link1="${tf_prefix}br_caster_wheel_link" link2="${tf_prefix}ur5_wrist_2_link" reason="Never" />
     <disable_collisions link1="${tf_prefix}br_caster_wheel_link" link2="${tf_prefix}ur5_wrist_3_link" reason="Never" />
-    <disable_collisions link1="${tf_prefix}dual_xtion_bottom_link" link2="${tf_prefix}dual_xtion_left_mount_link" reason="Adjacent" />
-    <disable_collisions link1="${tf_prefix}dual_xtion_bottom_link" link2="${tf_prefix}dual_xtion_right_mount_link" reason="Adjacent" />
-    <disable_collisions link1="${tf_prefix}dual_xtion_bottom_link" link2="${tf_prefix}dual_xtion_top_link" reason="Adjacent" />
-    <disable_collisions link1="${tf_prefix}dual_xtion_bottom_link" link2="${tf_prefix}fl_caster_rotation_link" reason="Never" />
-    <disable_collisions link1="${tf_prefix}dual_xtion_bottom_link" link2="${tf_prefix}fl_caster_wheel_link" reason="Never" />
-    <disable_collisions link1="${tf_prefix}dual_xtion_bottom_link" link2="${tf_prefix}fr_caster_rotation_link" reason="Never" />
-    <disable_collisions link1="${tf_prefix}dual_xtion_bottom_link" link2="${tf_prefix}fr_caster_wheel_link" reason="Never" />
-    <disable_collisions link1="${tf_prefix}dual_xtion_bottom_link" link2="${tf_prefix}front_laser_link" reason="Never" />
-    <disable_collisions link1="${tf_prefix}dual_xtion_bottom_link" link2="${tf_prefix}left_wheel_link" reason="Never" />
-    <disable_collisions link1="${tf_prefix}dual_xtion_bottom_link" link2="${tf_prefix}right_wheel_link" reason="Never" />
-    <disable_collisions link1="${tf_prefix}dual_xtion_bottom_link" link2="${tf_prefix}structure_part_down" reason="Never" />
-    <disable_collisions link1="${tf_prefix}dual_xtion_bottom_link" link2="${tf_prefix}structure_part_up" reason="Never" />
-    <disable_collisions link1="${tf_prefix}dual_xtion_bottom_link" link2="${tf_prefix}structure_pedestal" reason="Adjacent" />
-    <disable_collisions link1="${tf_prefix}dual_xtion_bottom_link" link2="${tf_prefix}ur5_base_link" reason="Never" />
-    <disable_collisions link1="${tf_prefix}dual_xtion_bottom_link" link2="${tf_prefix}ur5_shoulder_link" reason="Never" />
-    <disable_collisions link1="${tf_prefix}dual_xtion_bottom_link" link2="${tf_prefix}ur5_upper_arm_link" reason="Never" />
-    <disable_collisions link1="${tf_prefix}dual_xtion_left_mount_link" link2="${tf_prefix}dual_xtion_right_mount_link" reason="Adjacent" />
-    <disable_collisions link1="${tf_prefix}dual_xtion_left_mount_link" link2="${tf_prefix}dual_xtion_top_link" reason="Adjacent" />
-    <disable_collisions link1="${tf_prefix}dual_xtion_left_mount_link" link2="${tf_prefix}fl_caster_rotation_link" reason="Never" />
-    <disable_collisions link1="${tf_prefix}dual_xtion_left_mount_link" link2="${tf_prefix}fl_caster_wheel_link" reason="Never" />
-    <disable_collisions link1="${tf_prefix}dual_xtion_left_mount_link" link2="${tf_prefix}fr_caster_rotation_link" reason="Never" />
-    <disable_collisions link1="${tf_prefix}dual_xtion_left_mount_link" link2="${tf_prefix}fr_caster_wheel_link" reason="Never" />
-    <disable_collisions link1="${tf_prefix}dual_xtion_left_mount_link" link2="${tf_prefix}front_laser_link" reason="Never" />
-    <disable_collisions link1="${tf_prefix}dual_xtion_left_mount_link" link2="${tf_prefix}left_wheel_link" reason="Never" />
-    <disable_collisions link1="${tf_prefix}dual_xtion_left_mount_link" link2="${tf_prefix}right_wheel_link" reason="Never" />
-    <disable_collisions link1="${tf_prefix}dual_xtion_left_mount_link" link2="${tf_prefix}structure_part_down" reason="Never" />
-    <disable_collisions link1="${tf_prefix}dual_xtion_left_mount_link" link2="${tf_prefix}structure_part_up" reason="Default" />
-    <disable_collisions link1="${tf_prefix}dual_xtion_left_mount_link" link2="${tf_prefix}structure_pedestal" reason="Adjacent" />
-    <disable_collisions link1="${tf_prefix}dual_xtion_left_mount_link" link2="${tf_prefix}ur5_base_link" reason="Never" />
-    <disable_collisions link1="${tf_prefix}dual_xtion_left_mount_link" link2="${tf_prefix}ur5_shoulder_link" reason="Never" />
-    <disable_collisions link1="${tf_prefix}dual_xtion_right_mount_link" link2="${tf_prefix}dual_xtion_top_link" reason="Adjacent" />
-    <disable_collisions link1="${tf_prefix}dual_xtion_right_mount_link" link2="${tf_prefix}fl_caster_rotation_link" reason="Never" />
-    <disable_collisions link1="${tf_prefix}dual_xtion_right_mount_link" link2="${tf_prefix}fl_caster_wheel_link" reason="Never" />
-    <disable_collisions link1="${tf_prefix}dual_xtion_right_mount_link" link2="${tf_prefix}fr_caster_rotation_link" reason="Never" />
-    <disable_collisions link1="${tf_prefix}dual_xtion_right_mount_link" link2="${tf_prefix}fr_caster_wheel_link" reason="Never" />
-    <disable_collisions link1="${tf_prefix}dual_xtion_right_mount_link" link2="${tf_prefix}front_laser_link" reason="Never" />
-    <disable_collisions link1="${tf_prefix}dual_xtion_right_mount_link" link2="${tf_prefix}left_wheel_link" reason="Never" />
-    <disable_collisions link1="${tf_prefix}dual_xtion_right_mount_link" link2="${tf_prefix}right_wheel_link" reason="Never" />
-    <disable_collisions link1="${tf_prefix}dual_xtion_right_mount_link" link2="${tf_prefix}structure_part_down" reason="Never" />
-    <disable_collisions link1="${tf_prefix}dual_xtion_right_mount_link" link2="${tf_prefix}structure_part_up" reason="Default" />
-    <disable_collisions link1="${tf_prefix}dual_xtion_right_mount_link" link2="${tf_prefix}structure_pedestal" reason="Adjacent" />
-    <disable_collisions link1="${tf_prefix}dual_xtion_right_mount_link" link2="${tf_prefix}ur5_base_link" reason="Never" />
-    <disable_collisions link1="${tf_prefix}dual_xtion_right_mount_link" link2="${tf_prefix}ur5_shoulder_link" reason="Never" />
-    <disable_collisions link1="${tf_prefix}dual_xtion_top_link" link2="${tf_prefix}fl_caster_rotation_link" reason="Never" />
-    <disable_collisions link1="${tf_prefix}dual_xtion_top_link" link2="${tf_prefix}fl_caster_wheel_link" reason="Never" />
-    <disable_collisions link1="${tf_prefix}dual_xtion_top_link" link2="${tf_prefix}fr_caster_rotation_link" reason="Never" />
-    <disable_collisions link1="${tf_prefix}dual_xtion_top_link" link2="${tf_prefix}fr_caster_wheel_link" reason="Never" />
-    <disable_collisions link1="${tf_prefix}dual_xtion_top_link" link2="${tf_prefix}front_laser_link" reason="Never" />
-    <disable_collisions link1="${tf_prefix}dual_xtion_top_link" link2="${tf_prefix}left_wheel_link" reason="Never" />
-    <disable_collisions link1="${tf_prefix}dual_xtion_top_link" link2="${tf_prefix}right_wheel_link" reason="Never" />
-    <disable_collisions link1="${tf_prefix}dual_xtion_top_link" link2="${tf_prefix}structure_part_down" reason="Never" />
-    <disable_collisions link1="${tf_prefix}dual_xtion_top_link" link2="${tf_prefix}structure_part_up" reason="Never" />
-    <disable_collisions link1="${tf_prefix}dual_xtion_top_link" link2="${tf_prefix}structure_pedestal" reason="Adjacent" />
-    <disable_collisions link1="${tf_prefix}dual_xtion_top_link" link2="${tf_prefix}ur5_base_link" reason="Never" />
-    <disable_collisions link1="${tf_prefix}dual_xtion_top_link" link2="${tf_prefix}ur5_shoulder_link" reason="Never" />
     <disable_collisions link1="${tf_prefix}fl_caster_rotation_link" link2="${tf_prefix}fl_caster_wheel_link" reason="Adjacent" />
     <disable_collisions link1="${tf_prefix}fl_caster_rotation_link" link2="${tf_prefix}fr_caster_rotation_link" reason="Never" />

Commit message: joint_limits: Update wrist_3 limits again
Restrict the limits a bit because the cables would be stretched too much
otherwise.

File: mobipick_description/urdf/mobipick/mobipick_v1_model.urdf.xacro (robot description, xacro)
@@ -42,5 +42,5 @@
   <xacro:ur5_robot prefix="${prefix}ur5_" joint_limited="true"
     shoulder_lift_lower_limit="${-pi - 0.82}" shoulder_lift_upper_limit="${0.82}"
-    wrist_3_lower_limit="0.0001" wrist_3_upper_limit="${2 * pi}"
+    wrist_3_lower_limit="${0.25 * pi}" wrist_3_upper_limit="${1.75 * pi}"
     transmission_hw_interface="$(arg transmission_hw_interface)"
     kinematics_file="${load_yaml('$(arg kinematics_config)')}" />

File: mobipick_moveit_config/config/mobipick.srdf.xacro (robot description, xacro)
@@ -53,5 +53,5 @@
         <joint name="${tf_prefix}ur5_wrist_1_joint" value="-0.95" />
         <joint name="${tf_prefix}ur5_wrist_2_joint" value="1.57" />
-        <joint name="${tf_prefix}ur5_wrist_3_joint" value="-1.57" />
+        <joint name="${tf_prefix}ur5_wrist_3_joint" value="4.71" />
     </group_state>
     <group_state name="observe100cm_left" group="arm">
@@ -61,5 +61,5 @@
         <joint name="${tf_prefix}ur5_wrist_1_joint" value="-0.95" />
         <joint name="${tf_prefix}ur5_wrist_2_joint" value="1.57" />
-        <joint name="${tf_prefix}ur5_wrist_3_joint" value="-1.57" />
+        <joint name="${tf_prefix}ur5_wrist_3_joint" value="4.71" />
     </group_state>
     <group_state name="observe100cm_right" group="arm">
@@ -69,5 +69,5 @@
         <joint name="${tf_prefix}ur5_wrist_1_joint" value="-0.95" />
         <joint name="${tf_prefix}ur5_wrist_2_joint" value="1.57" />
-        <joint name="${tf_prefix}ur5_wrist_3_joint" value="-1.57" />
+        <joint name="${tf_prefix}ur5_wrist_3_joint" value="4.71" />
     </group_state>
     <group_state name="observe100cm_back" group="arm">
@@ -77,5 +77,5 @@
         <joint name="${tf_prefix}ur5_wrist_1_joint" value="-0.95" />
         <joint name="${tf_prefix}ur5_wrist_2_joint" value="1.57" />
-        <joint name="${tf_prefix}ur5_wrist_3_joint" value="-1.57" />
+        <joint name="${tf_prefix}ur5_wrist_3_joint" value="4.71" />
     </group_state>
     <group_state name="transport" group="arm">
@@ -109,5 +109,5 @@
         <joint name="${tf_prefix}ur5_wrist_1_joint" value="-1.15" />
         <joint name="${tf_prefix}ur5_wrist_2_joint" value="1.57" />
-        <joint name="${tf_prefix}ur5_wrist_3_joint" value="-1.57" />
+        <joint name="${tf_prefix}ur5_wrist_3_joint" value="4.71" />
     </group_state>
     <group_state name="pick" group="arm">

Commit message: SRDF: Remove group_state "pick"
This is not used anywhere AFAIK and is now outside the new joint limits
(see previous commit)

File: mobipick_description/urdf/mobipick/mobipick_v1_model.urdf.xacro (robot description, xacro)
@@ -47,5 +47,5 @@
          mess up the path simplification (planner produces a feasible plan, but path
          "simplification" introduces jumps from one configuration to the opposite one).
-       * shoulder_lift_upper_limit=0.72: all values > 0.72 are in self collision
+       * shoulder_lift_upper_limit=0.74: all values > 0.74 are in self collision
          (this limit is just an optimization)
        * elbow_joint_upper_limit=2.93: all values > 2.93 are in self collision
@@ -56,5 +56,5 @@
   <xacro:ur5_robot prefix="${prefix}ur5_" joint_limited="true"
     shoulder_pan_lower_limit="${-pi}"   shoulder_pan_upper_limit="${pi}"
-    shoulder_lift_lower_limit="${-pi}"  shoulder_lift_upper_limit="0.72"
+    shoulder_lift_lower_limit="${-pi}"  shoulder_lift_upper_limit="0.74"
     elbow_joint_lower_limit="0.0"       elbow_joint_upper_limit="2.93"
     wrist_1_lower_limit="${-pi}"        wrist_1_upper_limit="${pi}"

File: mobipick_moveit_config/config/mobipick.srdf.xacro (robot description, xacro)
@@ -110,12 +110,4 @@
         <joint name="${tf_prefix}ur5_wrist_2_joint" value="1.57" />
         <joint name="${tf_prefix}ur5_wrist_3_joint" value="4.71" />
-    </group_state>
-    <group_state name="pick" group="arm">
-        <joint name="${tf_prefix}ur5_shoulder_pan_joint" value="-1.4668672720538538" />
-        <joint name="${tf_prefix}ur5_shoulder_lift_joint" value="0.05980873107910156" />
-        <joint name="${tf_prefix}ur5_elbow_joint" value="-1.440704647694723" />
-        <joint name="${tf_prefix}ur5_wrist_1_joint" value="-0.3296421209918421" />
-        <joint name="${tf_prefix}ur5_wrist_2_joint" value="-1.6553095022784632" />
-        <joint name="${tf_prefix}ur5_wrist_3_joint" value="2.775566339492798" />
     </group_state>
     <group_state name="open" group="gripper">

Commit message: Change xacro comment to work around xacro bug
Since xacro 1.14.11, xacro now also evaluates expressions in comments
and throws an error if the substition argument is undefined. In xacro
1.14.12, this error was changed to a warning.

This commit removes that warning.

Workaround for https://github.com/ros/xacro/issues/309 .

File: mobipick_description/urdf/mobipick/mobipick_v1_model.urdf.xacro (robot description, xacro)
@@ -3,5 +3,5 @@
        name="mobipick">
   <xacro:arg name="robot" default="mobipick-os" />      <!-- can be "mobipick-hb" or "mobipick-os" -->
-  <xacro:property name="robot" value="$(arg robot)" />  <!-- necessary because args cannot be accessed inside ${} expressions -->
+  <xacro:property name="robot" value="$(arg robot)" />  <!-- necessary because args cannot be accessed inside $ {} expressions -->
   <xacro:arg name="tf_prefix" default="" />
   <xacro:property name="tf_prefix_" value="$(arg tf_prefix)" />

Commit message: Revert "Change xacro comment to work around xacro bug"
This reverts commit e00944028aae9d622c25492708834afc610c9e0f.

This is no longer necessary since xacro 1.14.13.

File: mobipick_description/urdf/mobipick/mobipick_v1_model.urdf.xacro (robot description, xacro)
@@ -3,5 +3,5 @@
        name="mobipick">
   <xacro:arg name="robot" default="mobipick-os" />      <!-- can be "mobipick-hb" or "mobipick-os" -->
-  <xacro:property name="robot" value="$(arg robot)" />  <!-- necessary because args cannot be accessed inside $ {} expressions -->
+  <xacro:property name="robot" value="$(arg robot)" />  <!-- necessary because args cannot be accessed inside ${} expressions -->
   <xacro:arg name="tf_prefix" default="" />
   <xacro:property name="tf_prefix_" value="$(arg tf_prefix)" />
