Commit message: Use FT-Sensor description from robotiq repository instead of own copy

File: mobipick_description/urdf/mobipick/mobipick_v1_model.urdf.xacro (robot description, xacro)
@@ -46,9 +46,15 @@
   <xacro:cable_guide prefix="${prefix}" />
   <!-- ############## FT SENSOR ############### -->
-  <xacro:include filename="$(find mobipick_description)/urdf/robotiq_ft_300/robotiq_ft_300.urdf.xacro" />
-  <xacro:robotiq_ft_300 parent="${prefix}ur5_tool0" prefix="${prefix}" >
-      <pose xyz="0 0 0" rpy="0 0 0" />
-      <!-- <pose xyz="0 0 0.009" rpy="0 0 0" /> -->
-  </xacro:robotiq_ft_300>
+  <xacro:include filename="$(find robotiq_ft_sensor)/urdf/robotiq_ft300.urdf.xacro"/>
+  <xacro:robotiq_ft300 parent="${prefix}ur5_tool0" prefix="${prefix}">
+		<origin xyz="0 0 -0.004" rpy="0 0 ${-pi/2}"/>
+	</xacro:robotiq_ft300>
+  <!-- Colorize the sensor black  -->
+  <gazebo reference="${prefix}ft300_mounting_plate">
+      <material>Gazebo/FlatBlack</material>
+  </gazebo>
+  <gazebo reference="${prefix}ft300_sensor">
+      <material>Gazebo/FlatBlack</material>
+  </gazebo>
   <!-- ############### GRIPPER ################ -->
   <xacro:include filename="$(find mobipick_description)/urdf/robotiq_2f_140/robotiq_arg2f_140_model_macro.xacro" />
@@ -60,5 +66,5 @@
   <joint name="${prefix}ft300_coupling_joint" type="fixed">
     <origin xyz="0 0 ${coupling_inner_length / 2}" rpy="0 0 ${-pi/2}" />
-    <parent link="${prefix}fts_toolside" />
+    <parent link="${prefix}robotiq_ft_frame_id" />
     <child link="${prefix}gripper_coupling_link" />
   </joint>
@@ -95,5 +101,5 @@
   <joint name="${prefix}sensor_mount_joint" type="fixed">
     <origin xyz="0.0 0.0 -0.005" rpy="0.0 ${-pi/2} 0.0" />
-    <parent link="${prefix}fts_toolside" />
+    <parent link="${prefix}robotiq_ft_frame_id" />
     <child link="${prefix}sensor_mount_link" />
   </joint>

Commit message: Use defined xacro property in Robotiq FT sensor

File: mobipick_description/urdf/mobipick/mobipick_v1_model.urdf.xacro (robot description, xacro)
@@ -46,7 +46,12 @@
   <xacro:cable_guide prefix="${prefix}" />
   <!-- ############## FT SENSOR ############### -->
+  <!-- gripper coupling (ISO 9409-1-50-4-M / Robotiq AGC-CPL-062-002_20171219) -->
+  <xacro:property name="coupling_radius" value="0.0375" />
+  <xacro:property name="coupling_outer_length" value="0.014" />
+  <xacro:property name="coupling_inner_length" value="0.008" />
+  <xacro:property name="coupling_mass" value="0.100" />
   <xacro:include filename="$(find robotiq_ft_sensor)/urdf/robotiq_ft300.urdf.xacro"/>
   <xacro:robotiq_ft300 parent="${prefix}ur5_tool0" prefix="${prefix}">
-		<origin xyz="0 0 -0.004" rpy="0 0 ${-pi/2}"/>
+		<origin xyz="0 0 ${-coupling_inner_length / 2}" rpy="0 0 ${-pi/2}"/>
 	</xacro:robotiq_ft300>
   <!-- Colorize the sensor black  -->
@@ -59,9 +64,4 @@
   <!-- ############### GRIPPER ################ -->
   <xacro:include filename="$(find mobipick_description)/urdf/robotiq_2f_140/robotiq_arg2f_140_model_macro.xacro" />
-  <!-- gripper coupling (ISO 9409-1-50-4-M / Robotiq AGC-CPL-062-002_20171219) -->
-  <xacro:property name="coupling_radius" value="0.0375" />
-  <xacro:property name="coupling_outer_length" value="0.014" />
-  <xacro:property name="coupling_inner_length" value="0.008" />
-  <xacro:property name="coupling_mass" value="0.100" />
   <joint name="${prefix}ft300_coupling_joint" type="fixed">
     <origin xyz="0 0 ${coupling_inner_length / 2}" rpy="0 0 ${-pi/2}" />

Commit message: add Intel RealSense 2 D435 and D455 camera options
The Mobipick in Bremen has a temporary Intel camera that might become
permanent, so its a config option.

File: mobipick_description/urdf/mobipick/mobipick_v1_model.urdf.xacro (robot description, xacro)
@@ -4,4 +4,11 @@
   <xacro:arg name="robot" default="mobipick-os" />      <!-- can be "mobipick-hb" or "mobipick-os" -->
   <xacro:property name="robot" value="$(arg robot)" />  <!-- necessary because args cannot be accessed inside ${} expressions -->
+  <!--
+    Main camera type, Can be "astra" for Orbbec Astra Mini S,
+    'intel_d455' for Intel RealSense D455 or 'intel_d435' for Intel RealSense D435,
+    changes the main 3D camera that is mounted on the endeffector." />
+  -->
+  <xacro:arg name="main_camera" default="astra" />
+  <xacro:property name="main_camera" value="$(arg main_camera)" />
   <xacro:arg name="tf_prefix" default="" />
   <xacro:property name="tf_prefix_" value="$(arg tf_prefix)" />
@@ -99,6 +106,16 @@
   </joint>
   <xacro:robotiq_arg2f_140 prefix="${prefix}gripper_"/>
-  <!-- ############### SENSOR MOUNT + 3D CAM  ################ -->
-  <xacro:include filename="$(find mobipick_description)/urdf/sensors/gripper_cam.urdf.xacro" />
+  <!-- ############### SENSOR MOUNT + 3D CAMS  ################ -->
+  <xacro:include filename="$(find mobipick_description)/urdf/sensors/sensor_mount.urdf.xacro" />
+  <xacro:if value="${main_camera == 'astra'}">
+    <xacro:include filename="$(find mobipick_description)/urdf/sensors/astra_cam.urdf.xacro" />
+  </xacro:if>
+  <xacro:if value="${main_camera == 'intel_d455'}">
+    <xacro:include filename="$(find mobipick_description)/urdf/sensors/d455_cam.urdf.xacro" />
+  </xacro:if>
+  <xacro:if value="${main_camera == 'intel_d435'}">
+    <xacro:include filename="$(find mobipick_description)/urdf/sensors/d435_cam.urdf.xacro" />
+  </xacro:if>
+  <xacro:include filename="$(find mobipick_description)/urdf/sensors/pico_cam.urdf.xacro" />
   <joint name="${prefix}sensor_mount_joint" type="fixed">
     <origin xyz="0.0 0.0 -0.005" rpy="0.0 ${-pi/2} 0.0" />
@@ -106,5 +123,15 @@
     <child link="${prefix}sensor_mount_link" />
   </joint>
-  <xacro:gripper_cam prefix="${prefix}" />
+  <xacro:sensor_mount prefix="${prefix}" />
+  <xacro:if value="${main_camera == 'astra'}">
+    <xacro:astra_cam prefix="${prefix}" />
+  </xacro:if>
+  <xacro:if value="${main_camera == 'intel_d455'}">
+    <xacro:intel_d455_cam prefix="${prefix}" />
+  </xacro:if>
+  <xacro:if value="${main_camera == 'intel_d435'}">
+    <xacro:intel_d435_cam prefix="${prefix}" />
+  </xacro:if>
+  <xacro:pico_cam prefix="${prefix}" />
   <!-- ############### DUAL XTION MOUNT + XTIONS ################ -->
   <xacro:if value="${robot == 'mobipick-hb'}">

File: mobipick_description/urdf/sensors/dual_xtions.urdf.xacro (robot description, xacro)
@@ -112,5 +112,5 @@
     </joint>
     <link name="${prefix}${camera_name}_depth_optical_frame"/>
-    <xacro:sim_3dsensor prefix="${prefix}" />  <!-- NOTE: sim_3dsensor macro from gripper_cam is used here -->
+    <xacro:sim_3dsensor prefix="${prefix}" />  <!-- NOTE: sim_3dsensor macro from astra/intel_xxx is used here -->
   </xacro:macro>
 </robot>
