Commit message: make gazebo grasp fix optional by improving physics settings

File: mobipick_description/urdf/mobipick/mobipick_v1_model.urdf.xacro (robot description, xacro)
@@ -20,4 +20,6 @@
   </xacro:unless>
   <xacro:arg name="transmission_hw_interface" default="hardware_interface/PositionJointInterface"/>
+  <xacro:arg name="grasp_fix" default="false" />  <!-- legacy gazebo_grasp_fix plugin on the gripper, see robotiq_arg2f_140_model_macro.xacro -->
+  <xacro:property name="grasp_fix_required" value="$(arg grasp_fix)" />
   <xacro:arg name="joint_limits_parameters_file" default="$(find mobipick_description)/config/joint_limits.yaml"/>  <!-- path the to the yaml with the ur5 joint limits. -->
   <xacro:arg name="kinematics_config" default="$(find mobipick_description)/config/ur5_calibration.yaml"/>  <!-- path the to the yaml with the arms calibration parameters. -->

File: mobipick_description/urdf/robotiq_2f_140/robotiq_arg2f_140_model_macro.xacro (robot description, xacro)
@@ -219,6 +219,8 @@
     <link name="${prefix}tcp" />
   </xacro:macro>
-  <!-- GRASP HACK -->
-  <xacro:property name="grasp_fix_required" default="true" />
+  <!-- Optional gazebo_grasp_fix plugin (legacy "grasp hack" that welds a grasped object to the gripper).
+       Off by default: objects are held by friction (see robotiq_fingertips_65mm.xacro). Enable with the
+       grasp_fix launch/xacro argument, or define grasp_fix_required before including this file. -->
+  <xacro:property name="grasp_fix_required" default="false" />
   <xacro:if value="${grasp_fix_required}">
     <xacro:include filename="$(find mobipick_description)/urdf/robotiq_2f_140/gzplugin_grasp_fix.urdf.xacro"/>

File: mobipick_description/urdf/robotiq_2f_140/robotiq_arg2f_140_model_sim_floating.urdf.xacro (robot description, xacro)
@@ -9,5 +9,4 @@
     <xacro:property name="prefix" value="${tf_prefix_}/" />
   </xacro:unless>
-  <xacro:property name="grasp_fix_required" value="false" /> <!-- do not use grasp fix plugin -->
   <xacro:include filename="$(find mobipick_description)/urdf/robotiq_2f_140/robotiq_arg2f_140_model_macro.xacro" />
   <xacro:include filename="$(find mobipick_description)/urdf/common.gazebo.xacro" />

File: mobipick_description/urdf/robotiq_2f_140/robotiq_fingertips_65mm.xacro (robot description, xacro)
@@ -2,4 +2,23 @@
 <robot xmlns:xacro="http://ros.org/wiki/xacro">
   <xacro:include filename="$(find mobipick_description)/urdf/common_properties.urdf.xacro" />
+  <!-- ODE contact parameters of the fingertip pads. Objects are held by friction alone (the gazebo_grasp_fix plugin is off by default, see grasp_fix arg),
+       which needs two things: a persistent contact and a real squeeze force.
+       * min_depth lets the pad sink 2 mm into the object before ODE pushes back. With the default 0 (and
+         contact_surface_layer 0 in our worlds) the contacts flicker while the object is carried and it slowly
+         creeps out of the gripper. Objects need the same setting on their side (see mobipick_gazebo/urdf).
+       * The squeeze force is set by the torque limit and position gain of mobipick_gripper_effort_controller.
+       Measured with test/grasp_rig (multimeter, 0.35 kg, carried and shaken at 1.6 m/s^2, fast physics profile):
+       without min_depth or with < 1 Nm finger torque the object tilts 40 deg during the lift and falls when the
+       gripper is moved, with these values it moves < 5 mm.
+       The properties can be overridden by defining them before including this file. -->
+  <xacro:property name="fingertip_mu" default="5.0" />
+  <!-- kp is the contact stiffness, see https://classic.gazebosim.org/tutorials?tut=physics_params&cat=physics
+       (5000 = soft pad, 1e6 = rigid). The pads used to be soft (5000) to gain contact area; with min_depth that
+       is not needed, and 1e5 halved the slip of the multimeter and was the difference between holding and
+       dropping the relay when the fingers barely touch it. -->
+  <xacro:property name="fingertip_kp" default="1e5" />
+  <xacro:property name="fingertip_kd" default="1.0" />
+  <xacro:property name="fingertip_min_depth" default="0.002" />
+  <xacro:property name="fingertip_max_vel" default="0.01" /> <!-- ODE default -->
   <xacro:macro name="robotiq_fingertip_65mm" params="prefix fingerprefix stroke">
     <link name="${prefix}${fingerprefix}_robotiq_fingertip_65mm">
@@ -34,12 +53,10 @@
       <material>Gazebo/Grey</material>
       <!-- high friction value to prevent objects from slipping the gripper fingers -->
-      <mu1>5.0</mu1>
-      <mu2>5.0</mu2>
-      <!-- a low kp (stiffness value) allows some penetration of the material making the gripper "soft".
-           The reason to prefer a soft gripper is to increase friction by increasing the contact area,
-           specially when the surface of the object to grasp is irregular, e.g. a mesh
-           see: https://classic.gazebosim.org/tutorials?tut=physics_params&cat=physics -->
-      <kp>5000.0</kp> <!-- 5000.0 - medium gripper finger "softness", 1000000.0 - hard/rigid gripper finger -->
-      <kd>1.0</kd>
+      <mu1>${fingertip_mu}</mu1>
+      <mu2>${fingertip_mu}</mu2>
+      <kp>${fingertip_kp}</kp>
+      <kd>${fingertip_kd}</kd>
+      <minDepth>${fingertip_min_depth}</minDepth>
+      <maxVel>${fingertip_max_vel}</maxVel>
     </gazebo>
   </xacro:macro>

File: mobipick_gazebo/urdf/bleach_cleanser.urdf.xacro (robot description, xacro)
@@ -35,4 +35,5 @@
     <kp>1e+06</kp> <!-- high stiffness -->
     <kd>1.0</kd> <!-- normal damping -->
+    <minDepth>0.002</minDepth> <!-- persistent contact with the gripper pads, see robotiq_fingertips_65mm.xacro -->
   </gazebo>
 </robot>

File: mobipick_gazebo/urdf/coke_can.urdf.xacro (robot description, xacro)
@@ -26,4 +26,5 @@
     <kp>1e+06</kp> <!-- high stiffness -->
     <kd>1.0</kd> <!-- normal damping -->
+    <minDepth>0.002</minDepth> <!-- persistent contact with the gripper pads, see robotiq_fingertips_65mm.xacro -->
   </gazebo>
 </robot>

File: mobipick_gazebo/urdf/cracker_box.urdf.xacro (robot description, xacro)
@@ -35,4 +35,5 @@
     <kp>1e+06</kp> <!-- high stiffness -->
     <kd>1.0</kd> <!-- normal damping -->
+    <minDepth>0.002</minDepth> <!-- persistent contact with the gripper pads, see robotiq_fingertips_65mm.xacro -->
   </gazebo>
 </robot>

File: mobipick_gazebo/urdf/gelatin_box.urdf.xacro (robot description, xacro)
@@ -35,4 +35,5 @@
     <kp>1e+06</kp> <!-- high stiffness -->
     <kd>1.0</kd> <!-- normal damping -->
+    <minDepth>0.002</minDepth> <!-- persistent contact with the gripper pads, see robotiq_fingertips_65mm.xacro -->
   </gazebo>
 </robot>

File: mobipick_gazebo/urdf/hot_glue_gun.urdf.xacro (robot description, xacro)
@@ -32,4 +32,5 @@
     <kp>1e+06</kp> <!-- high stiffness -->
     <kd>1.0</kd> <!-- normal damping -->
+    <minDepth>0.002</minDepth> <!-- persistent contact with the gripper pads, see robotiq_fingertips_65mm.xacro -->
   </gazebo>
 </robot>

File: mobipick_gazebo/urdf/klt.urdf.xacro (robot description, xacro)
@@ -68,4 +68,5 @@
     <kp>1e+06</kp> <!-- high stiffness -->
     <kd>1.0</kd> <!-- normal damping -->
+    <minDepth>0.002</minDepth> <!-- persistent contact with the gripper pads, see robotiq_fingertips_65mm.xacro -->
   </gazebo>
 </robot>

File: mobipick_gazebo/urdf/multimeter.urdf.xacro (robot description, xacro)
@@ -35,4 +35,5 @@
     <kp>1e+06</kp> <!-- high stiffness -->
     <kd>1.0</kd> <!-- normal damping -->
+    <minDepth>0.002</minDepth> <!-- persistent contact with the gripper pads, see robotiq_fingertips_65mm.xacro -->
   </gazebo>
 </robot>

File: mobipick_gazebo/urdf/mustard_bottle.urdf.xacro (robot description, xacro)
@@ -35,4 +35,5 @@
     <kp>1e+06</kp> <!-- high stiffness -->
     <kd>1.0</kd> <!-- normal damping -->
+    <minDepth>0.002</minDepth> <!-- persistent contact with the gripper pads, see robotiq_fingertips_65mm.xacro -->
   </gazebo>
 </robot>

File: mobipick_gazebo/urdf/potted_meat_can.urdf.xacro (robot description, xacro)
@@ -35,4 +35,5 @@
     <kp>1e+06</kp> <!-- high stiffness -->
     <kd>1.0</kd> <!-- normal damping -->
+    <minDepth>0.002</minDepth> <!-- persistent contact with the gripper pads, see robotiq_fingertips_65mm.xacro -->
   </gazebo>
 </robot>

File: mobipick_gazebo/urdf/power_drill.urdf.xacro (robot description, xacro)
@@ -35,4 +35,5 @@
     <kp>1e+06</kp> <!-- high stiffness -->
     <kd>1.0</kd> <!-- normal damping -->
+    <minDepth>0.002</minDepth> <!-- persistent contact with the gripper pads, see robotiq_fingertips_65mm.xacro -->
   </gazebo>
 </robot>

File: mobipick_gazebo/urdf/power_drill_with_grip.urdf.xacro (robot description, xacro)
@@ -32,4 +32,5 @@
     <kp>1e+06</kp> <!-- high stiffness -->
     <kd>1.0</kd> <!-- normal damping -->
+    <minDepth>0.002</minDepth> <!-- persistent contact with the gripper pads, see robotiq_fingertips_65mm.xacro -->
   </gazebo>
 </robot>

File: mobipick_gazebo/urdf/relay.urdf.xacro (robot description, xacro)
@@ -35,4 +35,5 @@
     <kp>1e+06</kp> <!-- high stiffness -->
     <kd>1.0</kd> <!-- normal damping -->
+    <minDepth>0.002</minDepth> <!-- persistent contact with the gripper pads, see robotiq_fingertips_65mm.xacro -->
   </gazebo>
 </robot>

File: mobipick_gazebo/urdf/screwdriver.urdf.xacro (robot description, xacro)
@@ -35,4 +35,5 @@
     <kp>1e+06</kp> <!-- high stiffness -->
     <kd>1.0</kd> <!-- normal damping -->
+    <minDepth>0.002</minDepth> <!-- persistent contact with the gripper pads, see robotiq_fingertips_65mm.xacro -->
   </gazebo>
 </robot>

File: mobipick_gazebo/urdf/sugar_box.urdf.xacro (robot description, xacro)
@@ -35,4 +35,5 @@
     <kp>1e+06</kp> <!-- high stiffness -->
     <kd>1.0</kd> <!-- normal damping -->
+    <minDepth>0.002</minDepth> <!-- persistent contact with the gripper pads, see robotiq_fingertips_65mm.xacro -->
   </gazebo>
 </robot>

File: mobipick_gazebo/urdf/tomato_soup_can.urdf.xacro (robot description, xacro)
@@ -35,4 +35,5 @@
     <kp>1e+06</kp> <!-- high stiffness -->
     <kd>1.0</kd> <!-- normal damping -->
+    <minDepth>0.002</minDepth> <!-- persistent contact with the gripper pads, see robotiq_fingertips_65mm.xacro -->
   </gazebo>
 </robot>
