Commit message: Remove "world" frames

File: mobipick_description/urdf/MiR_100/MiR_100_v1_model.urdf.xacro (robot description, xacro)
@@ -4,10 +4,4 @@
   <!-- structure -->
   <xacro:include filename="$(find mobipick_description)/urdf/MiR_100/MiR_100_v1.urdf.xacro" />
-  <link name="world" />
   <xacro:MiR_100 prefix=""/>
-  <joint name="world_joint" type="fixed">
-    <parent link="world" />
-    <child link="mir100_base" />
-    <origin xyz="0.0 0.0 0.0" rpy="0.0 0.0 0.0" />
-  </joint>
 </robot>

File: mobipick_description/urdf/mobipick/mobipick_model.urdf.xacro (robot description, xacro)
@@ -13,5 +13,4 @@
   <!-- 2f_140 -->
   <xacro:include filename="$(find mobipick_description)/urdf/robotiq_2f_140/robotiq_arg2f_140_model_macro.xacro" />
-  <link name="world" />
   <!-- mobile robot -->
   <xacro:MiR_100 prefix=""/>
@@ -27,9 +26,4 @@
   <!-- gripper -->
   <xacro:robotiq_arg2f_140 prefix=""/>
-  <joint name="world_joint" type="fixed">
-    <parent link="world" />
-    <child link = "mir100_base" />
-    <origin xyz="0.0 0.0 0.0" rpy="0.0 0.0 0.0" />
-  </joint>
   <joint name="mir100_struct_joint" type="fixed">
     <parent link="MiR100BaseSupport" />

File: mobipick_description/urdf/structure/mobipick_structure_model.urdf.xacro (robot description, xacro)
@@ -4,10 +4,4 @@
   <!-- structure -->
   <xacro:include filename="$(find mobipick_description)/urdf/structure/mobipick_structure.urdf.xacro" />
-  <link name="world" />
   <xacro:structure prefix="" height="0.1" />
-  <joint name="world_joint" type="fixed">
-    <parent link="world" />
-    <child link="StructPartDown" />
-    <origin xyz="0.0 0.0 0.0" rpy="0.0 0.0 0.0" />
-  </joint>
 </robot>

File: mobipick_description/urdf/ur5/ur5_joint_limited_robot.urdf.xacro (robot description, xacro)
@@ -8,9 +8,3 @@
   <!-- arm -->
   <xacro:ur5_robot prefix="" joint_limited="true"/>
-  <link name="world" />
-  <joint name="world_joint" type="fixed">
-    <parent link="world" />
-    <child link = "base_link" />
-    <origin xyz="0.0 0.0 0.0" rpy="0.0 0.0 0.0" />
-  </joint>
 </robot>

File: mobipick_description/urdf/ur5/ur5_robot.urdf.xacro (robot description, xacro)
@@ -8,9 +8,3 @@
   <!-- arm -->
   <xacro:ur5_robot prefix="" joint_limited="false"/>
-  <link name="world" />
-  <joint name="world_joint" type="fixed">
-    <parent link="world" />
-    <child link = "base_link" />
-    <origin xyz="0.0 0.0 0.0" rpy="0.0 0.0 0.0" />
-  </joint>
 </robot>
