Commit message: Rename mir100_base => base_link

File: mobipick_description/urdf/MiR_100/MiR_100_v1.urdf.xacro (robot description, xacro)
@@ -3,5 +3,5 @@
   <xacro:property name="pi" value="3.14159265" />
   <xacro:macro name="MiR_100" params="prefix">
-    <link name="${prefix}mir100_base">
+    <link name="${prefix}base_link">
       <inertial>
         <origin xyz="-7.8373351882E-004 0 0.2060599945" rpy="${1.5 * pi} ${0.5 * pi} ${0.5 * pi}" />
@@ -31,7 +31,7 @@
       </collision>
     </link>
-    <joint name="${prefix}mir100_base_joint" type="fixed">
+    <joint name="${prefix}base_link_joint" type="fixed">
       <origin xyz="0 0 0.352" rpy="0 0 0" />
-      <parent link="${prefix}mir100_base" />
+      <parent link="${prefix}base_link" />
       <child link="${prefix}MiR100BaseSupport" />
       <axis xyz="0 0 1" />
