Commit message: added a new link base_link for compatibility (leaving the previous base_link from the mir was generating errors while testing gazebo)

File: mobipick_description/urdf/mir_100/mir_100_v1_model.urdf.xacro (robot description, xacro)
@@ -4,4 +4,10 @@
   <!-- structure -->
   <xacro:include filename="$(find mobipick_description)/urdf/mir_100/mir_100_v1.urdf.xacro" />
+  <link name="base_link" />
+  <joint name="base_joint" type="fixed">
+    <parent link="base_link" />
+    <child link="base" />
+    <origin xyz="0.0 0.0 0.0" rpy="0.0 0.0 0.0" />
+  </joint>
   <xacro:mir_100 prefix=""/>
 </robot>

File: mobipick_description/urdf/mobipick/mobipick_v1_model.urdf.xacro (robot description, xacro)
@@ -41,3 +41,9 @@
     <axis xyz="0 0 1" />
   </joint>
+  <link name="base_link" />
+  <joint name="base_joint" type="fixed">
+    <parent link="base_link" />
+    <child link="mir_base" />
+    <origin xyz="0.0 0.0 0.0" rpy="0.0 0.0 0.0" />
+  </joint>
 </robot>
