Commit message: mir: Rename active wheel joints
Old names: base_link_left_act_wheel_joint,i base_link_right_act_wheel_joint
New name: left_wheel_joint, right_wheel_joint

File: mobipick_description/urdf/mir_100/mir_100.transmission.xacro (robot description, xacro)
@@ -4,5 +4,5 @@
     <transmission name="${prefix}${locationprefix}_act_wheel_trans">
       <type>transmission_interface/SimpleTransmission</type>
-      <joint name="${prefix}base_link_${locationprefix}_act_wheel_joint">
+      <joint name="${prefix}${locationprefix}_wheel_joint">
         <hardwareInterface>hardware_interface/VelocityJointInterface</hardwareInterface>
       </joint>

File: mobipick_description/urdf/mir_100/mir_100_v1.urdf.xacro (robot description, xacro)
@@ -120,5 +120,5 @@
   </xacro:macro>
   <xacro:macro name="actuated_wheel_joint" params="prefix locationprefix locationright">
-    <joint name="${prefix}base_link_${locationprefix}_act_wheel_joint" type="continuous">
+    <joint name="${prefix}${locationprefix}_wheel_joint" type="continuous">
       <origin xyz="${mir_100_act_wheel_dx} ${-mir_100_act_wheel_dy * locationright} ${mir_100_act_wheel_radius}" rpy="0 0 0" />
       <parent link="${prefix}base_link" />

File: mobipick_description/urdf/mir_100/mir_100_v1_model_diff_controller.urdf.xacro (robot description, xacro)
@@ -12,6 +12,6 @@
   <xacro:set_all_wheel_frictions prefix=""/>
   <xacro:diff_controller_plugin_gazebo prefix=""
-    left_wheel_joint="base_link_left_act_wheel_joint"
-    right_wheel_joint="base_link_right_act_wheel_joint"
+    left_wheel_joint="left_wheel_joint"
+    right_wheel_joint="right_wheel_joint"
     wheel_separation="${2*mir_100_act_wheel_dy}"
     wheel_radius="${mir_100_act_wheel_radius}"/>
