Commit message: mir: Rename base_link -> base_footprint, base -> base_link

File: mobipick_description/urdf/mir_100/mir_100.gazebo.xacro (robot description, xacro)
@@ -16,5 +16,5 @@
         <commandTopic>mobile_base_controller/cmd_vel</commandTopic>
         <odometryTopic>mobile_base_controller/odom</odometryTopic>
-        <robotBaseFrame>base_link</robotBaseFrame>
+        <robotBaseFrame>base_footprint</robotBaseFrame>
         <wheelAcceleration>2.8</wheelAcceleration>
         <publishWheelJointState>true</publishWheelJointState>

File: mobipick_description/urdf/mir_100/mir_100.transmission.xacro (robot description, xacro)
@@ -4,5 +4,5 @@
     <transmission name="${prefix}${locationprefix}_act_wheel_trans">
       <type>transmission_interface/SimpleTransmission</type>
-      <joint name="${prefix}base_${locationprefix}_act_wheel_joint">
+      <joint name="${prefix}base_link_${locationprefix}_act_wheel_joint">
         <hardwareInterface>hardware_interface/VelocityJointInterface</hardwareInterface>
       </joint>

File: mobipick_description/urdf/mir_100/mir_100_v1.urdf.xacro (robot description, xacro)
@@ -62,5 +62,5 @@
       <inertial>
         <!-- <origin xyz="0 0 -0.042500000044" rpy="${0.5 * pi} ${24 * deg_to_rad} ${1.5 * pi}" /> -->
-	<origin xyz="0 0 -0.042500000044" rpy="${24 * deg_to_rad} 0 ${0.5 * pi} " />
+        <origin xyz="0 0 -0.042500000044" rpy="${24 * deg_to_rad} 0 ${0.5 * pi} " />
         <mass value="0.3097539019" />
         <inertia
@@ -120,7 +120,7 @@
   </xacro:macro>
   <xacro:macro name="actuated_wheel_joint" params="prefix locationprefix locationright">
-    <joint name="${prefix}base_${locationprefix}_act_wheel_joint" type="continuous">
+    <joint name="${prefix}base_link_${locationprefix}_act_wheel_joint" type="continuous">
       <origin xyz="${mir_100_act_wheel_dx} ${-mir_100_act_wheel_dy * locationright} ${mir_100_act_wheel_radius}" rpy="0 0 0" />
-      <parent link="${prefix}base" />
+      <parent link="${prefix}base_link" />
       <child link="${prefix}${locationprefix}_act_wheel" />
       <axis xyz="0 1 0" />
@@ -129,12 +129,12 @@
   </xacro:macro>
   <xacro:macro name="front_caster_wheel_joints" params="prefix locationprefix locationright">
-    <joint name="${prefix}base_front_${locationprefix}_wheel_base_joint" type="continuous">
+    <joint name="${prefix}base_link_front_${locationprefix}_wheel_base_joint" type="continuous">
       <origin xyz="${mir_100_front_caster_wheel_base_dx} ${-mir_100_caster_wheel_base_dy * locationright} ${mir_100_caster_wheel_base_dz}" rpy="0 0 0" />
-      <parent link="${prefix}base" />
+      <parent link="${prefix}base_link" />
       <child link="${prefix}front_${locationprefix}_caster_wheel_base" />
       <axis xyz="0 0 1" />
       <joint_properties damping="0.0" friction="0.0"/>
     </joint>
-    <joint name="${prefix}base_front_${locationprefix}_wheel_joint" type="continuous">
+    <joint name="${prefix}base_link_front_${locationprefix}_wheel_joint" type="continuous">
       <origin xyz="${mir_100_caster_wheel_dx} ${-mir_100_caster_wheel_dy * locationright} ${mir_100_caster_wheel_dz}" rpy="0 0 0" />
       <parent link="${prefix}front_${locationprefix}_caster_wheel_base" />
@@ -144,12 +144,12 @@
   </xacro:macro>
   <xacro:macro name="back_caster_wheel_joints" params="prefix locationprefix locationright">
-    <joint name="${prefix}base_back_${locationprefix}_wheel_base_joint" type="continuous">
+    <joint name="${prefix}base_link_back_${locationprefix}_wheel_base_joint" type="continuous">
       <origin xyz="${mir_100_back_caster_wheel_base_dx} ${-mir_100_caster_wheel_base_dy * locationright} ${mir_100_caster_wheel_base_dz}" rpy="0 0 0" />
-      <parent link="${prefix}base" />
+      <parent link="${prefix}base_link" />
       <child link="${prefix}back_${locationprefix}_caster_wheel_base" />
       <axis xyz="0 0 1" />
       <joint_properties damping="0.0" friction="0.0"/>
     </joint>
-    <joint name="${prefix}base_back_${locationprefix}_wheel_joint" type="continuous">
+    <joint name="${prefix}base_link_back_${locationprefix}_wheel_joint" type="continuous">
       <origin xyz="${mir_100_caster_wheel_dx} ${-mir_100_caster_wheel_dy * locationright} ${mir_100_caster_wheel_dz}" rpy="0 0 0" />
       <parent link="${prefix}back_${locationprefix}_caster_wheel_base" />
@@ -159,7 +159,7 @@
   </xacro:macro>
   <xacro:macro name="mir_100" params="prefix">
-    <link name="${prefix}base">
-      <inertial>
-	 <origin xyz="0 0 0.1623852639" rpy="0 0 0" />
+    <link name="${prefix}base_link">
+      <inertial>
+        <origin xyz="0 0 0.1623852639" rpy="0 0 0" />
         <mass value="${mir_100_base_mass}" />
         <xacro:box_inertia m="${mir_100_base_mass}" x="0.9" y="0.58" z="0.3" />
@@ -193,7 +193,7 @@
     <xacro:back_caster_wheel_joints prefix="${prefix}" locationprefix="left" locationright="-1"/>
     <xacro:back_caster_wheel_joints prefix="${prefix}" locationprefix="right" locationright="1"/>
-    <joint name="${prefix}base_surface_joint" type="fixed">
+    <joint name="${prefix}base_link_surface_joint" type="fixed">
       <origin xyz="0 0 0.352" rpy="0 0 0" />
-      <parent link="${prefix}base" />
+      <parent link="${prefix}base_link" />
       <child link="${prefix}surface" />
       <axis xyz="0 0 1" />

File: mobipick_description/urdf/mir_100/mir_100_v1_model.urdf.xacro (robot description, xacro)
@@ -4,8 +4,8 @@
   <!-- structure -->
   <xacro:include filename="$(find mobipick_description)/urdf/mir_100/mir_100_v1.urdf.xacro" />
-  <link name="base_link" />
+  <link name="base_footprint" />
   <joint name="base_joint" type="fixed">
-    <parent link="base_link" />
-    <child link="base" />
+    <parent link="base_footprint" />
+    <child link="base_link" />
     <origin xyz="0.0 0.0 0.0" rpy="0.0 0.0 0.0" />
   </joint>

File: mobipick_description/urdf/mir_100/mir_100_v1_model_diff_controller.urdf.xacro (robot description, xacro)
@@ -3,8 +3,8 @@
   <xacro:include filename="$(find mobipick_description)/urdf/mir_100/mir_100_v1.urdf.xacro" />
   <xacro:include filename="$(find mobipick_description)/urdf/mir_100/mir_100.gazebo.xacro" />
-  <link name="base_link" />
+  <link name="base_footprint" />
   <joint name="base_joint" type="fixed">
-    <parent link="base_link" />
-    <child link="base" />
+    <parent link="base_footprint" />
+    <child link="base_link" />
     <origin xyz="0.0 0.0 0.0" rpy="0.0 0.0 0.0" />
   </joint>
@@ -12,6 +12,6 @@
   <xacro:set_all_wheel_frictions prefix=""/>
   <xacro:diff_controller_plugin_gazebo prefix=""
-    left_wheel_joint="base_left_act_wheel_joint"
-    right_wheel_joint="base_right_act_wheel_joint"
+    left_wheel_joint="base_link_left_act_wheel_joint"
+    right_wheel_joint="base_link_right_act_wheel_joint"
     wheel_separation="${2*mir_100_act_wheel_dy}"
     wheel_radius="${mir_100_act_wheel_radius}"/>

File: mobipick_description/urdf/mir_100/mir_100_v1_model_ros_control.urdf.xacro (robot description, xacro)
@@ -4,8 +4,8 @@
   <xacro:include filename="$(find mobipick_description)/urdf/mir_100/mir_100.gazebo.xacro" />
   <xacro:include filename="$(find mobipick_description)/urdf/common.gazebo.xacro" />
-  <link name="base_link" />
+  <link name="base_footprint" />
   <joint name="base_joint" type="fixed">
-    <parent link="base_link" />
-    <child link="base" />
+    <parent link="base_footprint" />
+    <child link="base_link" />
     <origin xyz="0.0 0.0 0.0" rpy="0.0 0.0 0.0" />
   </joint>

File: mobipick_description/urdf/mobipick/mobipick_v1_model.urdf.xacro (robot description, xacro)
@@ -3,8 +3,8 @@
        name="mobipick">
   <!-- ############## BASE_LINK  ############## -->
-  <link name="base_link" />
+  <link name="base_footprint" />
   <joint name="base_joint" type="fixed">
-    <parent link="base_link" />
-    <child link="base" />
+    <parent link="base_footprint" />
+    <child link="base_link" />
     <origin xyz="0.0 0.0 0.0" rpy="0.0 0.0 0.0" />
   </joint>

Commit message: urdf: Rename wheel links + joints

File: mobipick_description/urdf/mir_100/mir_100.gazebo.xacro (robot description, xacro)
@@ -34,10 +34,10 @@
   </xacro:macro>
   <xacro:macro name="set_all_wheel_frictions" params="prefix">
-    <xacro:set_wheel_friction link="${prefix}left_act_wheel" friction="200"/>
-    <xacro:set_wheel_friction link="${prefix}right_act_wheel" friction="200"/>
-    <xacro:set_wheel_friction link="${prefix}front_left_caster_wheel" friction="1"/>
-    <xacro:set_wheel_friction link="${prefix}front_right_caster_wheel" friction="1"/>
-    <xacro:set_wheel_friction link="${prefix}back_left_caster_wheel" friction="1"/>
-    <xacro:set_wheel_friction link="${prefix}back_right_caster_wheel" friction="1"/>
+    <xacro:set_wheel_friction link="${prefix}left_wheel_link" friction="200"/>
+    <xacro:set_wheel_friction link="${prefix}right_wheel_link" friction="200"/>
+    <xacro:set_wheel_friction link="${prefix}fl_caster_wheel_link" friction="1"/>
+    <xacro:set_wheel_friction link="${prefix}fr_caster_wheel_link" friction="1"/>
+    <xacro:set_wheel_friction link="${prefix}bl_caster_wheel_link" friction="1"/>
+    <xacro:set_wheel_friction link="${prefix}br_caster_wheel_link" friction="1"/>
   </xacro:macro>
 </robot>

File: mobipick_description/urdf/mir_100/mir_100.transmission.xacro (robot description, xacro)
@@ -2,10 +2,10 @@
 <robot xmlns:xacro="http://ros.org/wiki/xacro">
   <xacro:macro name="mir_100_wheel_transmission" params="prefix locationprefix">
-    <transmission name="${prefix}${locationprefix}_act_wheel_trans">
+    <transmission name="${prefix}${locationprefix}_wheel_trans">
       <type>transmission_interface/SimpleTransmission</type>
       <joint name="${prefix}${locationprefix}_wheel_joint">
         <hardwareInterface>hardware_interface/VelocityJointInterface</hardwareInterface>
       </joint>
-      <actuator name="${prefix}${locationprefix}_act_wheel_motor">
+      <actuator name="${prefix}${locationprefix}_wheel_motor">
         <hardwareInterface>hardware_interface/VelocityJointInterface</hardwareInterface>
         <mechanicalReduction>1</mechanicalReduction>

File: mobipick_description/urdf/mir_100/mir_100_v1.urdf.xacro (robot description, xacro)
@@ -25,5 +25,5 @@
   <xacro:property name="imu_stdev" value="0.00017" />
   <xacro:macro name="actuated_wheel_link" params="prefix locationprefix">
-    <link name="${prefix}${locationprefix}_act_wheel">
+    <link name="${prefix}${locationprefix}_wheel_link">
       <xacro:cylinder_inertial mass="${mir_100_act_wheel_mass}" radius="${mir_100_act_wheel_radius}" length="${mir_100_act_wheel_width}">
         <origin xyz="0 0 0" rpy="${0.5 * pi} 0 0" />
@@ -43,10 +43,10 @@
       </collision>
     </link>
-    <gazebo reference="${prefix}${locationprefix}_act_wheel">
+    <gazebo reference="${prefix}${locationprefix}_wheel_link">
       <material>Gazebo/DarkGrey</material>
     </gazebo>
   </xacro:macro>
   <xacro:macro name="caster_wheel_links" params="prefix locationprefix">
-    <link name="${prefix}${locationprefix}_caster_wheel_base">
+    <link name="${prefix}${locationprefix}_caster_rotation_link">
       <inertial>
         <!-- <origin xyz="0 0 -0.042500000044" rpy="${0.5 * pi} ${24 * deg_to_rad} ${1.5 * pi}" /> -->
@@ -75,8 +75,8 @@
       </collision>
     </link>
-    <gazebo reference="${prefix}${locationprefix}_caster_wheel_base">
+    <gazebo reference="${prefix}${locationprefix}_caster_rotation_link">
       <material>Gazebo/Grey</material>
     </gazebo>
-    <link name="${prefix}${locationprefix}_caster_wheel">
+    <link name="${prefix}${locationprefix}_caster_wheel_link">
       <xacro:cylinder_inertial mass="${mir_100_caster_wheel_mass}" radius="${mir_100_caster_wheel_radius}" length="${mir_100_caster_wheel_width}">
         <origin xyz="0 0 0" rpy="${0.5 * pi} 0 0" />
@@ -96,5 +96,5 @@
       </collision>
     </link>
-    <gazebo reference="${prefix}${locationprefix}_caster_wheel">
+    <gazebo reference="${prefix}${locationprefix}_caster_wheel_link">
       <material>Gazebo/DarkGrey</material>
     </gazebo>
@@ -104,5 +104,5 @@
       <origin xyz="0.0 ${-mir_100_act_wheel_dy * locationright} ${mir_100_act_wheel_radius}" rpy="0 0 0" />
       <parent link="${prefix}base_link" />
-      <child link="${prefix}${locationprefix}_act_wheel" />
+      <child link="${prefix}${locationprefix}_wheel_link" />
       <axis xyz="0 1 0" />
       <limit effort="100" velocity="20.0" />
@@ -110,30 +110,30 @@
   </xacro:macro>
   <xacro:macro name="front_caster_wheel_joints" params="prefix locationprefix locationright">
-    <joint name="${prefix}base_link_front_${locationprefix}_wheel_base_joint" type="continuous">
+    <joint name="${prefix}${locationprefix}_caster_rotation_joint" type="continuous">
       <origin xyz="${mir_100_front_caster_wheel_base_dx} ${-mir_100_caster_wheel_base_dy * locationright} ${mir_100_caster_wheel_base_dz}" rpy="0 0 0" />
       <parent link="${prefix}base_link" />
-      <child link="${prefix}front_${locationprefix}_caster_wheel_base" />
+      <child link="${prefix}${locationprefix}_caster_rotation_link" />
       <axis xyz="0 0 1" />
       <dynamics damping="0.01" friction="0.0"/>
     </joint>
-    <joint name="${prefix}base_link_front_${locationprefix}_wheel_joint" type="continuous">
+    <joint name="${prefix}${locationprefix}_caster_wheel_joint" type="continuous">
       <origin xyz="${mir_100_caster_wheel_dx} ${-mir_100_caster_wheel_dy * locationright} ${mir_100_caster_wheel_dz}" rpy="0 0 0" />
-      <parent link="${prefix}front_${locationprefix}_caster_wheel_base" />
-      <child link="${prefix}front_${locationprefix}_caster_wheel" />
+      <parent link="${prefix}${locationprefix}_caster_rotation_link" />
+      <child link="${prefix}${locationprefix}_caster_wheel_link" />
       <axis xyz="0 1 0" />
     </joint>
   </xacro:macro>
   <xacro:macro name="back_caster_wheel_joints" params="prefix locationprefix locationright">
-    <joint name="${prefix}base_link_back_${locationprefix}_wheel_base_joint" type="continuous">
+    <joint name="${prefix}${locationprefix}_caster_rotation_joint" type="continuous">
       <origin xyz="${mir_100_back_caster_wheel_base_dx} ${-mir_100_caster_wheel_base_dy * locationright} ${mir_100_caster_wheel_base_dz}" rpy="0 0 0" />
       <parent link="${prefix}base_link" />
-      <child link="${prefix}back_${locationprefix}_caster_wheel_base" />
+      <child link="${prefix}${locationprefix}_caster_rotation_link" />
       <axis xyz="0 0 1" />
       <dynamics damping="0.01" friction="0.0"/>
     </joint>
-    <joint name="${prefix}base_link_back_${locationprefix}_wheel_joint" type="continuous">
+    <joint name="${prefix}${locationprefix}_caster_wheel_joint" type="continuous">
       <origin xyz="${mir_100_caster_wheel_dx} ${-mir_100_caster_wheel_dy * locationright} ${mir_100_caster_wheel_dz}" rpy="0 0 0" />
-      <parent link="${prefix}back_${locationprefix}_caster_wheel_base" />
-      <child link="${prefix}back_${locationprefix}_caster_wheel" />
+      <parent link="${prefix}${locationprefix}_caster_rotation_link" />
+      <child link="${prefix}${locationprefix}_caster_wheel_link" />
       <axis xyz="0 1 0" />
     </joint>
@@ -202,14 +202,14 @@
     <xacro:actuated_wheel_link prefix="${prefix}" locationprefix="left"/>
     <xacro:actuated_wheel_link prefix="${prefix}" locationprefix="right"/>
-    <xacro:caster_wheel_links prefix="${prefix}" locationprefix="front_left"/>
-    <xacro:caster_wheel_links prefix="${prefix}" locationprefix="front_right"/>
-    <xacro:caster_wheel_links prefix="${prefix}" locationprefix="back_left"/>
-    <xacro:caster_wheel_links prefix="${prefix}" locationprefix="back_right"/>
+    <xacro:caster_wheel_links prefix="${prefix}" locationprefix="fl"/>
+    <xacro:caster_wheel_links prefix="${prefix}" locationprefix="fr"/>
+    <xacro:caster_wheel_links prefix="${prefix}" locationprefix="bl"/>
+    <xacro:caster_wheel_links prefix="${prefix}" locationprefix="br"/>
     <xacro:actuated_wheel_joint prefix="${prefix}" locationprefix="left" locationright="-1"/>
     <xacro:actuated_wheel_joint prefix="${prefix}" locationprefix="right" locationright="1"/>
-    <xacro:front_caster_wheel_joints prefix="${prefix}" locationprefix="left" locationright="-1"/>
-    <xacro:front_caster_wheel_joints prefix="${prefix}" locationprefix="right" locationright="1"/>
-    <xacro:back_caster_wheel_joints prefix="${prefix}" locationprefix="left" locationright="-1"/>
-    <xacro:back_caster_wheel_joints prefix="${prefix}" locationprefix="right" locationright="1"/>
+    <xacro:front_caster_wheel_joints prefix="${prefix}" locationprefix="fl" locationright="-1"/>
+    <xacro:front_caster_wheel_joints prefix="${prefix}" locationprefix="fr" locationright="1"/>
+    <xacro:back_caster_wheel_joints prefix="${prefix}" locationprefix="bl" locationright="-1"/>
+    <xacro:back_caster_wheel_joints prefix="${prefix}" locationprefix="br" locationright="1"/>
     <joint name="${prefix}base_link_surface_joint" type="fixed">
       <origin xyz="${mir_100_act_wheel_dx} 0 0.352" rpy="0 0 0" />
