Commit message: Add caster wheels to mir

File: mobipick_description/urdf/mir_100/mir_100_v1.urdf.xacro (robot description, xacro)
@@ -2,21 +2,145 @@
 <robot xmlns:xacro="http://ros.org/wiki/xacro">
   <xacro:property name="pi" value="3.14159265" />
-  <xacro:macro name="mir_100" params="prefix">
-    <link name="${prefix}base">
+  <xacro:macro name="actuated_wheel_link" params="prefix locationprefix">
+    <link name="${prefix}${locationprefix}_act_wheel">
       <inertial>
-        <origin xyz="-7.8373351882E-004 0 0.2060599945" rpy="${1.5 * pi} ${0.5 * pi} ${0.5 * pi}" />
-        <mass value="62.5" />
+        <origin xyz="0 0 0" rpy="${0.5 * pi} ${0.5 * pi} 0" />
+        <mass value="1.0" />
         <inertia
-            ixx="5.9"
+            ixx="0.0021285829616"
             ixy="0"
             ixz="0"
-            iyy="4.55"
+            iyy="0.0011566983393"
             iyz="0"
-            izz="2.2" />
+            izz="0.0011566983393" />
       </inertial>
       <visual>
         <origin xyz="0 0 0" rpy="0 0 0" />
         <geometry>
-          <mesh filename="package://mobipick_description/meshes/mir_100/visual/mir100_v_1_5.stl" />
+          <mesh filename="package://mobipick_description/meshes/mir_100/visual/actuated_wheel.stl" />
+        </geometry>
+        <material name="">
+          <color rgba="1.0 0.0 0.0 1" />
+        </material>
+      </visual>
+      <collision>
+        <origin xyz="0 0 0" rpy="0 0 0" />
+        <geometry>
+          <mesh filename="package://mobipick_description/meshes/mir_100/collision/actuated_wheel.stl" />
+        </geometry>
+      </collision>
+    </link>
+  </xacro:macro>
+  <xacro:macro name="caster_wheel_links" params="prefix locationprefix">
+    <link name="${prefix}${locationprefix}_caster_wheel_base">
+      <inertial>
+        <origin xyz="0 0 -0.042500000044" rpy="${0.5 * pi} ${24 / 180 * pi} ${1.5 * pi}" />
+        <mass value="0.3097539019" />
+        <inertia
+            ixx="0.0005844517978"
+            ixy="0"
+            ixz="0"
+            iyy="0.00052872551237"
+            iyz="0"
+            izz="0.00017923555074" />
+      </inertial>
+      <visual>
+        <origin xyz="0 0 0" rpy="0 0 0" />
+        <geometry>
+          <mesh filename="package://mobipick_description/meshes/mir_100/visual/caster_wheel_base.stl" />
+        </geometry>
+        <material name="">
+          <color rgba="0.4 0.4 0.4 1" />
+        </material>
+      </visual>
+      <collision>
+        <origin xyz="0 0 0" rpy="0 0 0" />
+        <geometry>
+          <mesh filename="package://mobipick_description/meshes/mir_100/collision/caster_wheel_base.stl" />
+        </geometry>
+      </collision>
+    </link>
+    <link name="${prefix}${locationprefix}_caster_wheel">
+      <inertial>
+        <origin xyz="0 0 0" rpy="${0.5 * pi} ${0.5 * pi} 0" />
+        <mass value="1.0" />
+        <inertia
+            ixx="0.0021285829616"
+            ixy="0"
+            ixz="0"
+            iyy="0.0011566983393"
+            iyz="0"
+            izz="0.0011566983393" />
+      </inertial>
+      <visual>
+        <origin xyz="0 0 0" rpy="0 0 0" />
+        <geometry>
+          <mesh filename="package://mobipick_description/meshes/mir_100/visual/caster_wheel.stl" />
+        </geometry>
+        <material name="">
+          <color rgba="0.4 0.4 0.4 1" />
+        </material>
+      </visual>
+      <collision>
+        <origin xyz="0 0 0" rpy="0 0 0" />
+        <geometry>
+          <mesh filename="package://mobipick_description/meshes/mir_100/collision/caster_wheel.stl" />
+        </geometry>
+      </collision>
+    </link>
+  </xacro:macro>
+  <xacro:macro name="actuated_wheel_joint" params="prefix locationprefix locationright">
+    <joint name="${prefix}base_${locationprefix}_act_wheel_joint" type="continuous">
+      <origin xyz="-0.037646 ${-0.222604 * locationright} 0.0625" rpy="0 0 0" />
+      <parent link="${prefix}base" />
+      <child link="${prefix}${locationprefix}_act_wheel" />
+      <axis xyz="0 1 0" />
+    </joint>
+  </xacro:macro>
+  <xacro:macro name="front_caster_wheel_joints" params="prefix locationprefix locationright">
+    <joint name="${prefix}base_front_${locationprefix}_wheel_base_joint" type="continuous">
+      <origin xyz="0.3037 ${-0.203 * locationright} 0.1565" rpy="0 0 0" />
+      <parent link="${prefix}base" />
+      <child link="${prefix}front_${locationprefix}_caster_wheel_base" />
+      <axis xyz="0 0 1" />
+    </joint>
+    <joint name="${prefix}base_front_${locationprefix}_wheel_joint" type="continuous">
+      <origin xyz="-0.0382 0 -0.094" rpy="0 0 0" />
+      <parent link="${prefix}front_${locationprefix}_caster_wheel_base" />
+      <child link="${prefix}front_${locationprefix}_caster_wheel" />
+      <axis xyz="0 1 0" />
+    </joint>
+  </xacro:macro>
+  <xacro:macro name="back_caster_wheel_joints" params="prefix locationprefix locationright">
+    <joint name="${prefix}base_back_${locationprefix}_wheel_base_joint" type="continuous">
+      <origin xyz="-0.3078 ${-0.203 * locationright} 0.1565" rpy="0 0 0" />
+      <parent link="${prefix}base" />
+      <child link="${prefix}back_${locationprefix}_caster_wheel_base" />
+      <axis xyz="0 0 1" />
+    </joint>
+    <joint name="${prefix}base_back_${locationprefix}_wheel_joint" type="continuous">
+      <origin xyz="-0.0382 0 -0.094" rpy="0 0 0" />
+      <parent link="${prefix}back_${locationprefix}_caster_wheel_base" />
+      <child link="${prefix}back_${locationprefix}_caster_wheel" />
+      <axis xyz="0 1 0" />
+    </joint>
+  </xacro:macro>
+  <xacro:macro name="mir_100" params="prefix">
+    <link name="${prefix}base">
+      <inertial>
+        <origin xyz="0 -0.2528237011 0.1623852639" rpy="${0.5 * pi} ${0.5 * pi} 0" />
+        <mass value="60.0" />
+        <inertia
+            ixx="2.104161731"
+            ixy="0"
+            ixz="0"
+            iyy="1.927704596"
+            iyz="0"
+            izz="0.194324673" />
+      </inertial>
+      <visual>
+        <origin xyz="0 0 0" rpy="0 0 0" />
+        <geometry>
+          <mesh filename="package://mobipick_description/meshes/mir_100/visual/mir_100_base.stl" />
         </geometry>
         <material name="">
@@ -27,8 +151,20 @@
         <origin xyz="0 0 0" rpy="0 0 0" />
         <geometry>
-          <mesh filename="package://mobipick_description/meshes/mir_100/collision/mir100_v_1_5.stl" />
+          <mesh filename="package://mobipick_description/meshes/mir_100/collision/mir_100_base.stl" />
         </geometry>
       </collision>
     </link>
+    <xacro:actuated_wheel_link prefix="${prefix}" locationprefix="left"/>
+    <xacro:actuated_wheel_link prefix="${prefix}" locationprefix="right"/>
+    <xacro:caster_wheel_links prefix="${prefix}" locationprefix="front_left"/>
+    <xacro:caster_wheel_links prefix="${prefix}" locationprefix="front_right"/>
+    <xacro:caster_wheel_links prefix="${prefix}" locationprefix="back_left"/>
+    <xacro:caster_wheel_links prefix="${prefix}" locationprefix="back_right"/>
+    <xacro:actuated_wheel_joint prefix="${prefix}" locationprefix="left" locationright="-1"/>
+    <xacro:actuated_wheel_joint prefix="${prefix}" locationprefix="right" locationright="1"/>
+    <xacro:front_caster_wheel_joints prefix="${prefix}" locationprefix="left" locationright="-1"/>
+    <xacro:front_caster_wheel_joints prefix="${prefix}" locationprefix="right" locationright="1"/>
+    <xacro:back_caster_wheel_joints prefix="${prefix}" locationprefix="left" locationright="-1"/>
+    <xacro:back_caster_wheel_joints prefix="${prefix}" locationprefix="right" locationright="1"/>
     <joint name="${prefix}base_surface_joint" type="fixed">
       <origin xyz="0 0 0.352" rpy="0 0 0" />

File: mobipick_description/urdf/mir_100/mir_100_v1_model.urdf.xacro (robot description, xacro)
@@ -1,7 +1,7 @@
 <?xml version="1.0"?>
 <robot xmlns:xacro="http://ros.org/wiki/xacro"
-       name="mir_100_v1" >
+       name="mir_100_v2" >
   <!-- structure -->
-  <xacro:include filename="$(find mobipick_description)/urdf/mir_100/mir_100_v1.urdf.xacro" />
+  <xacro:include filename="$(find mobipick_description)/urdf/mir_100/mir_100_v2.urdf.xacro" />
   <link name="world" />
   <xacro:mir_100 prefix=""/>

Commit message: MiR100: Rename ${prefix}base => base_link

File: mobipick_description/urdf/mir_100/mir_100_v1.urdf.xacro (robot description, xacro)
@@ -93,5 +93,5 @@
     <joint name="${prefix}base_${locationprefix}_act_wheel_joint" type="continuous">
       <origin xyz="-0.037646 ${-0.222604 * locationright} 0.0625" rpy="0 0 0" />
-      <parent link="${prefix}base" />
+      <parent link="base_link" />
       <child link="${prefix}${locationprefix}_act_wheel" />
       <axis xyz="0 1 0" />
@@ -101,5 +101,5 @@
     <joint name="${prefix}base_front_${locationprefix}_wheel_base_joint" type="continuous">
       <origin xyz="0.3037 ${-0.203 * locationright} 0.1565" rpy="0 0 0" />
-      <parent link="${prefix}base" />
+      <parent link="base_link" />
       <child link="${prefix}front_${locationprefix}_caster_wheel_base" />
       <axis xyz="0 0 1" />
@@ -115,5 +115,5 @@
     <joint name="${prefix}base_back_${locationprefix}_wheel_base_joint" type="continuous">
       <origin xyz="-0.3078 ${-0.203 * locationright} 0.1565" rpy="0 0 0" />
-      <parent link="${prefix}base" />
+      <parent link="base_link" />
       <child link="${prefix}back_${locationprefix}_caster_wheel_base" />
       <axis xyz="0 0 1" />
@@ -127,5 +127,5 @@
   </xacro:macro>
   <xacro:macro name="mir_100" params="prefix">
-    <link name="${prefix}base">
+    <link name="base_link">
       <inertial>
         <origin xyz="0 -0.2528237011 0.1623852639" rpy="${0.5 * pi} ${0.5 * pi} 0" />
@@ -169,5 +169,5 @@
     <joint name="${prefix}base_surface_joint" type="fixed">
       <origin xyz="0 0 0.352" rpy="0 0 0" />
-      <parent link="${prefix}base" />
+      <parent link="base_link" />
       <child link="${prefix}surface" />
       <axis xyz="0 0 1" />

Commit message: commented unnecessary pi definitions

File: mobipick_description/urdf/mir_100/mir_100_v1.urdf.xacro (robot description, xacro)
@@ -1,5 +1,5 @@
 <?xml version="1.0"?>
 <robot xmlns:xacro="http://ros.org/wiki/xacro">
-  <xacro:property name="pi" value="3.14159265" />
+  <!-- <xacro:property name="pi" value="3.14159265" /> -->
   <xacro:macro name="actuated_wheel_link" params="prefix locationprefix">
     <link name="${prefix}${locationprefix}_act_wheel">

File: mobipick_description/urdf/structure/mobipick_structure.urdf.xacro (robot description, xacro)
@@ -1,5 +1,5 @@
 <?xml version="1.0"?>
 <robot xmlns:xacro="http://ros.org/wiki/xacro">
-  <xacro:property name="pi" value="3.14159265" />
+  <!-- <xacro:property name="pi" value="3.14159265" /> -->
   <xacro:macro name="structure" params="prefix height">
     <link name="${prefix}part_down">

File: mobipick_description/urdf/ur5/ur5.urdf.xacro (robot description, xacro)
@@ -3,5 +3,5 @@
   <xacro:include filename="$(find mobipick_description)/urdf/ur5/ur.transmission.xacro" />
   <xacro:include filename="$(find mobipick_description)/urdf/ur5/ur.gazebo.xacro" />
-  <xacro:property name="pi" value="3.14159265" />
+  <!-- <xacro:property name="pi" value="3.14159265" /> -->
   <!-- Inertia parameters -->
   <xacro:property name="base_mass" value="4.0" />  <!-- This mass might be incorrect -->

Commit message: set the base_link to base again (for completeness), cleaned some of the parameters of the model, added links/calls to transmission and gazebo xacros

File: mobipick_description/urdf/mir_100/mir_100_v1.urdf.xacro (robot description, xacro)
@@ -1,5 +1,19 @@
 <?xml version="1.0"?>
 <robot xmlns:xacro="http://ros.org/wiki/xacro">
+  <xacro:include filename="$(find mobipick_description)/urdf/mir_100/mir_100.transmission.xacro" />
+  <xacro:include filename="$(find mobipick_description)/urdf/mir_100/mir_100.gazebo.xacro" />
   <!-- <xacro:property name="pi" value="3.14159265" /> -->
+  <xacro:property name="deg_to_rad" value="0.017453293" />
+  <xacro:property name="mir_100_act_wheel_dx" value="-0.037646" />
+  <xacro:property name="mir_100_act_wheel_dy" value="0.222604" />
+  <xacro:property name="mir_100_act_wheel_radius" value="0.0625" />
+  <xacro:property name="mir_100_caster_wheel_radius" value="${mir_100_act_wheel_radius}" />
+  <xacro:property name="mir_100_caster_wheel_dx" value="-0.0382" />
+  <xacro:property name="mir_100_caster_wheel_dy" value="0" />
+  <xacro:property name="mir_100_caster_wheel_dz" value="-0.094" />
+  <xacro:property name="mir_100_front_caster_wheel_base_dx" value="0.3037" />
+  <xacro:property name="mir_100_back_caster_wheel_base_dx" value="-0.3078" />
+  <xacro:property name="mir_100_caster_wheel_base_dy" value="0.203" />
+  <xacro:property name="mir_100_caster_wheel_base_dz" value="${mir_100_caster_wheel_radius-mir_100_caster_wheel_dz}" />
   <xacro:macro name="actuated_wheel_link" params="prefix locationprefix">
     <link name="${prefix}${locationprefix}_act_wheel">
@@ -35,5 +49,5 @@
     <link name="${prefix}${locationprefix}_caster_wheel_base">
       <inertial>
-        <origin xyz="0 0 -0.042500000044" rpy="${0.5 * pi} ${24 / 180 * pi} ${1.5 * pi}" />
+        <origin xyz="0 0 -0.042500000044" rpy="${0.5 * pi} ${24 * deg_to_rad} ${1.5 * pi}" />
         <mass value="0.3097539019" />
         <inertia
@@ -92,6 +106,6 @@
   <xacro:macro name="actuated_wheel_joint" params="prefix locationprefix locationright">
     <joint name="${prefix}base_${locationprefix}_act_wheel_joint" type="continuous">
-      <origin xyz="-0.037646 ${-0.222604 * locationright} 0.0625" rpy="0 0 0" />
-      <parent link="base_link" />
+      <origin xyz="${mir_100_act_wheel_dx} ${-mir_100_act_wheel_dy * locationright} ${mir_100_act_wheel_radius}" rpy="0 0 0" />
+      <parent link="${prefix}base" />
       <child link="${prefix}${locationprefix}_act_wheel" />
       <axis xyz="0 1 0" />
@@ -100,11 +114,11 @@
   <xacro:macro name="front_caster_wheel_joints" params="prefix locationprefix locationright">
     <joint name="${prefix}base_front_${locationprefix}_wheel_base_joint" type="continuous">
-      <origin xyz="0.3037 ${-0.203 * locationright} 0.1565" rpy="0 0 0" />
-      <parent link="base_link" />
+      <origin xyz="${mir_100_front_caster_wheel_base_dx} ${-mir_100_caster_wheel_base_dy * locationright} ${mir_100_caster_wheel_base_dz}" rpy="0 0 0" />
+      <parent link="${prefix}base" />
       <child link="${prefix}front_${locationprefix}_caster_wheel_base" />
       <axis xyz="0 0 1" />
     </joint>
     <joint name="${prefix}base_front_${locationprefix}_wheel_joint" type="continuous">
-      <origin xyz="-0.0382 0 -0.094" rpy="0 0 0" />
+      <origin xyz="${mir_100_caster_wheel_dx} ${-mir_100_caster_wheel_dy * locationright} ${mir_100_caster_wheel_dz}" rpy="0 0 0" />
       <parent link="${prefix}front_${locationprefix}_caster_wheel_base" />
       <child link="${prefix}front_${locationprefix}_caster_wheel" />
@@ -114,11 +128,11 @@
   <xacro:macro name="back_caster_wheel_joints" params="prefix locationprefix locationright">
     <joint name="${prefix}base_back_${locationprefix}_wheel_base_joint" type="continuous">
-      <origin xyz="-0.3078 ${-0.203 * locationright} 0.1565" rpy="0 0 0" />
-      <parent link="base_link" />
+      <origin xyz="${mir_100_back_caster_wheel_base_dx} ${-mir_100_caster_wheel_base_dy * locationright} ${mir_100_caster_wheel_base_dz}" rpy="0 0 0" />
+      <parent link="${prefix}base" />
       <child link="${prefix}back_${locationprefix}_caster_wheel_base" />
       <axis xyz="0 0 1" />
     </joint>
     <joint name="${prefix}base_back_${locationprefix}_wheel_joint" type="continuous">
-      <origin xyz="-0.0382 0 -0.094" rpy="0 0 0" />
+      <origin xyz="${mir_100_caster_wheel_dx} ${-mir_100_caster_wheel_dy * locationright} ${mir_100_caster_wheel_dz}" rpy="0 0 0" />
       <parent link="${prefix}back_${locationprefix}_caster_wheel_base" />
       <child link="${prefix}back_${locationprefix}_caster_wheel" />
@@ -127,5 +141,5 @@
   </xacro:macro>
   <xacro:macro name="mir_100" params="prefix">
-    <link name="base_link">
+    <link name="${prefix}base">
       <inertial>
         <origin xyz="0 -0.2528237011 0.1623852639" rpy="${0.5 * pi} ${0.5 * pi} 0" />
@@ -169,9 +183,11 @@
     <joint name="${prefix}base_surface_joint" type="fixed">
       <origin xyz="0 0 0.352" rpy="0 0 0" />
-      <parent link="base_link" />
+      <parent link="${prefix}base" />
       <child link="${prefix}surface" />
       <axis xyz="0 0 1" />
     </joint>
     <link name="${prefix}surface"/>
+    <xacro:mir_100_wheel_transmissions prefix="${prefix}"/>
+    <xacro:mir_100_gazebo prefix="${prefix}"/>
   </xacro:macro>
 </robot>

Commit message: Added properties, fixed some parameters (inc. inertial) and removed gazebo-related stuff

File: mobipick_description/urdf/mir_100/mir_100_v1.urdf.xacro (robot description, xacro)
@@ -2,11 +2,15 @@
 <robot xmlns:xacro="http://ros.org/wiki/xacro">
   <xacro:include filename="$(find mobipick_description)/urdf/mir_100/mir_100.transmission.xacro" />
-  <xacro:include filename="$(find mobipick_description)/urdf/mir_100/mir_100.gazebo.xacro" />
   <!-- <xacro:property name="pi" value="3.14159265" /> -->
   <xacro:property name="deg_to_rad" value="0.017453293" />
+  <xacro:property name="mir_100_base_mass" value="58.0" />
+  <xacro:property name="mir_100_act_wheel_radius" value="0.0625" />
+  <xacro:property name="mir_100_act_wheel_width" value="0.032" />
+  <xacro:property name="mir_100_act_wheel_mass" value="1.0" />
   <xacro:property name="mir_100_act_wheel_dx" value="-0.037646" />
   <xacro:property name="mir_100_act_wheel_dy" value="0.222604" />
-  <xacro:property name="mir_100_act_wheel_radius" value="0.0625" />
   <xacro:property name="mir_100_caster_wheel_radius" value="${mir_100_act_wheel_radius}" />
+  <xacro:property name="mir_100_caster_wheel_width" value="${mir_100_act_wheel_width}" />
+  <xacro:property name="mir_100_caster_wheel_mass" value="${mir_100_act_wheel_mass}" />
   <xacro:property name="mir_100_caster_wheel_dx" value="-0.0382" />
   <xacro:property name="mir_100_caster_wheel_dy" value="0" />
@@ -16,10 +20,17 @@
   <xacro:property name="mir_100_caster_wheel_base_dy" value="0.203" />
   <xacro:property name="mir_100_caster_wheel_base_dz" value="${mir_100_caster_wheel_radius-mir_100_caster_wheel_dz}" />
+  <xacro:macro name="cylinder_inertia" params="m r h">
+    <inertia ixx="${m*(3*r*r+h*h)/12}" ixy="0" ixz="0" iyy="${m*(3*r*r+h*h)/12}" iyz="0" izz="${m*r*r/2}"/>
+  </xacro:macro>
+  <xacro:macro name="box_inertia" params="m x y z">
+    <inertia ixx="${m*(y*y+z*z)/12}" ixy="0" ixz="0" iyy="${m*(x*x+z*z)/12}" iyz="0" izz="${m*(x*x+z*z)/12}"/>
+  </xacro:macro>
   <xacro:macro name="actuated_wheel_link" params="prefix locationprefix">
     <link name="${prefix}${locationprefix}_act_wheel">
       <inertial>
-        <origin xyz="0 0 0" rpy="${0.5 * pi} ${0.5 * pi} 0" />
-        <mass value="1.0" />
-        <inertia
+        <!-- <origin xyz="0 0 0" rpy="${0.5 * pi} ${0.5 * pi} 0" /> -->
+        <origin xyz="0 0 0" rpy="${0.5 * pi} 0 0" />
+        <mass value="${mir_100_act_wheel_mass}" />
+        <!-- <inertia
             ixx="0.0021285829616"
             ixy="0"
@@ -27,5 +38,6 @@
             iyy="0.0011566983393"
             iyz="0"
-            izz="0.0011566983393" />
+            izz="0.0011566983393" /> -->
+        <xacro:cylinder_inertia m="${mir_100_act_wheel_mass}" r="${mir_100_act_wheel_radius}" h="${mir_100_act_wheel_width}" />
       </inertial>
       <visual>
@@ -49,5 +61,6 @@
     <link name="${prefix}${locationprefix}_caster_wheel_base">
       <inertial>
-        <origin xyz="0 0 -0.042500000044" rpy="${0.5 * pi} ${24 * deg_to_rad} ${1.5 * pi}" />
+        <!-- <origin xyz="0 0 -0.042500000044" rpy="${0.5 * pi} ${24 * deg_to_rad} ${1.5 * pi}" /> -->
+	<origin xyz="0 0 -0.042500000044" rpy="${24 * deg_to_rad} 0 ${0.5 * pi} " />
         <mass value="0.3097539019" />
         <inertia
@@ -77,7 +90,8 @@
     <link name="${prefix}${locationprefix}_caster_wheel">
       <inertial>
-        <origin xyz="0 0 0" rpy="${0.5 * pi} ${0.5 * pi} 0" />
-        <mass value="1.0" />
-        <inertia
+        <!-- <origin xyz="0 0 0" rpy="${0.5 * pi} ${0.5 * pi} 0" /> -->
+        <origin xyz="0 0 0" rpy="${0.5 * pi} 0 0" />
+        <mass value="${mir_100_caster_wheel_mass}" />
+        <!-- <inertia
             ixx="0.0021285829616"
             ixy="0"
@@ -85,5 +99,6 @@
             iyy="0.0011566983393"
             iyz="0"
-            izz="0.0011566983393" />
+            izz="0.0011566983393" /> -->
+        <xacro:cylinder_inertia m="${mir_100_act_wheel_mass}" r="${mir_100_act_wheel_radius}" h="${mir_100_act_wheel_width}" />
       </inertial>
       <visual>
@@ -110,4 +125,5 @@
       <child link="${prefix}${locationprefix}_act_wheel" />
       <axis xyz="0 1 0" />
+      <limit effort="100" velocity="20.0" />
     </joint>
   </xacro:macro>
@@ -118,4 +134,5 @@
       <child link="${prefix}front_${locationprefix}_caster_wheel_base" />
       <axis xyz="0 0 1" />
+      <joint_properties damping="0.0" friction="0.0"/>
     </joint>
     <joint name="${prefix}base_front_${locationprefix}_wheel_joint" type="continuous">
@@ -132,4 +149,5 @@
       <child link="${prefix}back_${locationprefix}_caster_wheel_base" />
       <axis xyz="0 0 1" />
+      <joint_properties damping="0.0" friction="0.0"/>
     </joint>
     <joint name="${prefix}base_back_${locationprefix}_wheel_joint" type="continuous">
@@ -143,13 +161,7 @@
     <link name="${prefix}base">
       <inertial>
-        <origin xyz="0 -0.2528237011 0.1623852639" rpy="${0.5 * pi} ${0.5 * pi} 0" />
-        <mass value="60.0" />
-        <inertia
-            ixx="2.104161731"
-            ixy="0"
-            ixz="0"
-            iyy="1.927704596"
-            iyz="0"
-            izz="0.194324673" />
+	 <origin xyz="0 0 0.1623852639" rpy="0 0 0" />
+        <mass value="${mir_100_base_mass}" />
+        <xacro:box_inertia m="${mir_100_base_mass}" x="0.9" y="0.58" z="0.3" />
       </inertial>
       <visual>
@@ -189,5 +201,4 @@
     <link name="${prefix}surface"/>
     <xacro:mir_100_wheel_transmissions prefix="${prefix}"/>
-    <xacro:mir_100_gazebo prefix="${prefix}"/>
   </xacro:macro>
 </robot>

Commit message: Fix box_inertia macro

File: mobipick_description/urdf/mir_100/mir_100_v1.urdf.xacro (robot description, xacro)
@@ -24,5 +24,5 @@
   </xacro:macro>
   <xacro:macro name="box_inertia" params="m x y z">
-    <inertia ixx="${m*(y*y+z*z)/12}" ixy="0" ixz="0" iyy="${m*(x*x+z*z)/12}" iyz="0" izz="${m*(x*x+z*z)/12}"/>
+    <inertia ixx="${m*(y*y+z*z)/12}" ixy="0" ixz="0" iyy="${m*(x*x+z*z)/12}" iyz="0" izz="${m*(x*x+y*y)/12}"/>
   </xacro:macro>
   <xacro:macro name="actuated_wheel_link" params="prefix locationprefix">
