Commit message: Move base_footprint into MiR100 macro

File: mobipick_description/urdf/mir_100/mir_100_v1.urdf.xacro (robot description, xacro)
@@ -159,4 +159,10 @@
   </xacro:macro>
   <xacro:macro name="mir_100" params="prefix">
+  <link name="${prefix}base_footprint" />
+  <joint name="${prefix}base_joint" type="fixed">
+    <parent link="${prefix}base_footprint" />
+    <child link="${prefix}base_link" />
+    <origin xyz="0 0 0" rpy="0 0 0" />
+  </joint>
     <link name="${prefix}base_link">
       <inertial>

File: mobipick_description/urdf/mir_100/mir_100_v1_model.urdf.xacro (robot description, xacro)
@@ -2,12 +2,6 @@
 <robot xmlns:xacro="http://ros.org/wiki/xacro"
        name="mir_100" >
-  <!-- structure -->
+  <!-- MiR100 base -->
   <xacro:include filename="$(find mobipick_description)/urdf/mir_100/mir_100_v1.urdf.xacro" />
-  <link name="base_footprint" />
-  <joint name="base_joint" type="fixed">
-    <parent link="base_footprint" />
-    <child link="base_link" />
-    <origin xyz="0.0 0.0 0.0" rpy="0.0 0.0 0.0" />
-  </joint>
   <xacro:mir_100 prefix=""/>
 </robot>

File: mobipick_description/urdf/mir_100/mir_100_v1_model_diff_controller.urdf.xacro (robot description, xacro)
@@ -3,10 +3,4 @@
   <xacro:include filename="$(find mobipick_description)/urdf/mir_100/mir_100_v1.urdf.xacro" />
   <xacro:include filename="$(find mobipick_description)/urdf/mir_100/mir_100.gazebo.xacro" />
-  <link name="base_footprint" />
-  <joint name="base_joint" type="fixed">
-    <parent link="base_footprint" />
-    <child link="base_link" />
-    <origin xyz="0.0 0.0 0.0" rpy="0.0 0.0 0.0" />
-  </joint>
   <xacro:mir_100 prefix=""/>
   <xacro:set_all_wheel_frictions prefix=""/>

File: mobipick_description/urdf/mir_100/mir_100_v1_model_ros_control.urdf.xacro (robot description, xacro)
@@ -4,10 +4,4 @@
   <xacro:include filename="$(find mobipick_description)/urdf/mir_100/mir_100.gazebo.xacro" />
   <xacro:include filename="$(find mobipick_description)/urdf/common.gazebo.xacro" />
-  <link name="base_footprint" />
-  <joint name="base_joint" type="fixed">
-    <parent link="base_footprint" />
-    <child link="base_link" />
-    <origin xyz="0.0 0.0 0.0" rpy="0.0 0.0 0.0" />
-  </joint>
   <xacro:mir_100 prefix=""/>
   <xacro:set_all_wheel_frictions prefix=""/>

File: mobipick_description/urdf/mobipick/mobipick_v1_model.urdf.xacro (robot description, xacro)
@@ -2,11 +2,4 @@
 <robot xmlns:xacro="http://ros.org/wiki/xacro"
        name="mobipick">
-  <!-- ############## BASE_LINK  ############## -->
-  <link name="base_footprint" />
-  <joint name="base_joint" type="fixed">
-    <parent link="base_footprint" />
-    <child link="base_link" />
-    <origin xyz="0.0 0.0 0.0" rpy="0.0 0.0 0.0" />
-  </joint>
   <!-- ############# MIR100 BASE ############## -->
   <xacro:include filename="$(find mobipick_description)/urdf/mir_100/mir_100_v1.urdf.xacro" />

Commit message: Shift base_link to center of actuated wheels
This is important for twist + odom calculations; also, this fits with
the TF data from the real MiR robot.

File: mobipick_description/urdf/mir_100/mir_100_v1.urdf.xacro (robot description, xacro)
@@ -8,5 +8,5 @@
   <xacro:property name="mir_100_act_wheel_width" value="0.032" />
   <xacro:property name="mir_100_act_wheel_mass" value="1.0" />
-  <xacro:property name="mir_100_act_wheel_dx" value="-0.037646" />
+  <xacro:property name="mir_100_act_wheel_dx" value="0.037646" />
   <xacro:property name="mir_100_act_wheel_dy" value="0.222604" />
   <xacro:property name="mir_100_caster_wheel_radius" value="${mir_100_act_wheel_radius}" />
@@ -16,6 +16,6 @@
   <xacro:property name="mir_100_caster_wheel_dy" value="0" />
   <xacro:property name="mir_100_caster_wheel_dz" value="-0.094" />
-  <xacro:property name="mir_100_front_caster_wheel_base_dx" value="0.3037" />
-  <xacro:property name="mir_100_back_caster_wheel_base_dx" value="-0.3078" />
+  <xacro:property name="mir_100_front_caster_wheel_base_dx" value="0.341346" />
+  <xacro:property name="mir_100_back_caster_wheel_base_dx" value="-0.270154" />
   <xacro:property name="mir_100_caster_wheel_base_dy" value="0.203" />
   <xacro:property name="mir_100_caster_wheel_base_dz" value="${mir_100_caster_wheel_radius-mir_100_caster_wheel_dz}" />
@@ -121,5 +121,5 @@
   <xacro:macro name="actuated_wheel_joint" params="prefix locationprefix locationright">
     <joint name="${prefix}${locationprefix}_wheel_joint" type="continuous">
-      <origin xyz="${mir_100_act_wheel_dx} ${-mir_100_act_wheel_dy * locationright} ${mir_100_act_wheel_radius}" rpy="0 0 0" />
+      <origin xyz="0.0 ${-mir_100_act_wheel_dy * locationright} ${mir_100_act_wheel_radius}" rpy="0 0 0" />
       <parent link="${prefix}base_link" />
       <child link="${prefix}${locationprefix}_act_wheel" />
@@ -167,10 +167,10 @@
     <link name="${prefix}base_link">
       <inertial>
-        <origin xyz="0 0 0.1623852639" rpy="0 0 0" />
+        <origin xyz="${mir_100_act_wheel_dx} 0 0.20" rpy="0 0 0" />
         <mass value="${mir_100_base_mass}" />
         <xacro:box_inertia m="${mir_100_base_mass}" x="0.9" y="0.58" z="0.3" />
       </inertial>
       <visual>
-        <origin xyz="0 0 0" rpy="0 0 0" />
+        <origin xyz="${mir_100_act_wheel_dx} 0 0" rpy="0 0 0" />
         <geometry>
           <mesh filename="package://mobipick_description/meshes/mir_100/visual/mir_100_base.stl" />
@@ -181,5 +181,5 @@
       </visual>
       <collision>
-        <origin xyz="0 0 0" rpy="0 0 0" />
+        <origin xyz="${mir_100_act_wheel_dx} 0 0" rpy="0 0 0" />
         <geometry>
           <mesh filename="package://mobipick_description/meshes/mir_100/collision/mir_100_base.stl" />
@@ -200,5 +200,5 @@
     <xacro:back_caster_wheel_joints prefix="${prefix}" locationprefix="right" locationright="1"/>
     <joint name="${prefix}base_link_surface_joint" type="fixed">
-      <origin xyz="0 0 0.352" rpy="0 0 0" />
+      <origin xyz="${mir_100_act_wheel_dx} 0 0.352" rpy="0 0 0" />
       <parent link="${prefix}base_link" />
       <child link="${prefix}surface" />

Commit message: Add damping to caster wheels
This stops them from spinning around madly when the robot is dropped on
the side, and also makes them behave more realistically in general.

File: mobipick_description/urdf/mir_100/mir_100_v1.urdf.xacro (robot description, xacro)
@@ -135,5 +135,5 @@
       <child link="${prefix}front_${locationprefix}_caster_wheel_base" />
       <axis xyz="0 0 1" />
-      <joint_properties damping="0.0" friction="0.0"/>
+      <dynamics damping="0.01" friction="0.0"/>
     </joint>
     <joint name="${prefix}base_link_front_${locationprefix}_wheel_joint" type="continuous">
@@ -150,5 +150,5 @@
       <child link="${prefix}back_${locationprefix}_caster_wheel_base" />
       <axis xyz="0 0 1" />
-      <joint_properties damping="0.0" friction="0.0"/>
+      <dynamics damping="0.01" friction="0.0"/>
     </joint>
     <joint name="${prefix}base_link_back_${locationprefix}_wheel_joint" type="continuous">

Commit message: Add remaining Gazebo colors

File: mobipick_description/urdf/mir_100/mir_100_v1.urdf.xacro (robot description, xacro)
@@ -3,4 +3,5 @@
   <xacro:include filename="$(find mobipick_description)/urdf/mir_100/mir_100.transmission.xacro" />
   <xacro:include filename="$(find mobipick_description)/urdf/mir_100/mir_100.gazebo.xacro" />
+  <xacro:include filename="$(find mobipick_description)/urdf/mir_100/materials.xacro" />
   <!-- <xacro:property name="pi" value="3.14159265" /> -->
   <xacro:property name="deg_to_rad" value="0.017453293" />
@@ -47,7 +48,5 @@
           <mesh filename="package://mobipick_description/meshes/mir_100/visual/actuated_wheel.stl" />
         </geometry>
-        <material name="">
-          <color rgba="1.0 0.0 0.0 1" />
-        </material>
+        <material name="mir_dark_grey" />
       </visual>
       <collision>
@@ -58,4 +57,7 @@
       </collision>
     </link>
+    <gazebo reference="${prefix}${locationprefix}_act_wheel">
+      <material>Gazebo/DarkGrey</material>
+    </gazebo>
   </xacro:macro>
   <xacro:macro name="caster_wheel_links" params="prefix locationprefix">
@@ -78,7 +80,5 @@
           <mesh filename="package://mobipick_description/meshes/mir_100/visual/caster_wheel_base.stl" />
         </geometry>
-        <material name="">
-          <color rgba="0.4 0.4 0.4 1" />
-        </material>
+        <material name="mir_silver" />
       </visual>
       <collision>
@@ -89,4 +89,7 @@
       </collision>
     </link>
+    <gazebo reference="${prefix}${locationprefix}_caster_wheel_base">
+      <material>Gazebo/Grey</material>
+    </gazebo>
     <link name="${prefix}${locationprefix}_caster_wheel">
       <inertial>
@@ -108,7 +111,5 @@
           <mesh filename="package://mobipick_description/meshes/mir_100/visual/caster_wheel.stl" />
         </geometry>
-        <material name="">
-          <color rgba="0.4 0.4 0.4 1" />
-        </material>
+        <material name="mir_dark_grey" />
       </visual>
       <collision>
@@ -119,4 +120,7 @@
       </collision>
     </link>
+    <gazebo reference="${prefix}${locationprefix}_caster_wheel">
+      <material>Gazebo/DarkGrey</material>
+    </gazebo>
   </xacro:macro>
   <xacro:macro name="actuated_wheel_joint" params="prefix locationprefix locationright">
@@ -177,7 +181,5 @@
           <mesh filename="package://mobipick_description/meshes/mir_100/visual/mir_100_base.stl" />
         </geometry>
-        <material name="">
-          <color rgba="0.8 0.8 0.8 1" />
-        </material>
+        <material name="mir_white" />
       </visual>
       <collision>
@@ -188,4 +190,7 @@
       </collision>
     </link>
+    <gazebo reference="${prefix}base_link">
+      <material>Gazebo/White</material>
+    </gazebo>
     <xacro:actuated_wheel_link prefix="${prefix}" locationprefix="left"/>
     <xacro:actuated_wheel_link prefix="${prefix}" locationprefix="right"/>

File: mobipick_description/urdf/structure/mobipick_structure.urdf.xacro (robot description, xacro)
@@ -1,4 +1,5 @@
 <?xml version="1.0"?>
 <robot xmlns:xacro="http://ros.org/wiki/xacro">
+  <xacro:include filename="$(find mobipick_description)/urdf/structure/materials.xacro" />
   <!-- <xacro:property name="pi" value="3.14159265" /> -->
   <xacro:macro name="structure" params="prefix height">
@@ -20,7 +21,5 @@
           <mesh filename="package://mobipick_description/meshes/structure/visual/part_down.stl" />
         </geometry>
-        <material name="">
-          <color rgba="0.8 0.8 0.8 1" />
-        </material>
+        <material name="structure_aluminum" />
       </visual>
       <collision>
@@ -31,4 +30,7 @@
       </collision>
     </link>
+    <gazebo reference="${prefix}part_down">
+      <material>Gazebo/Grey</material>
+    </gazebo>
     <link name="${prefix}part_up">
       <inertial>
@@ -48,7 +50,5 @@
           <mesh filename="package://mobipick_description/meshes/structure/visual/part_up.stl" />
         </geometry>
-        <material name="">
-          <color rgba="0.8 0.8 0.8 1" />
-        </material>
+        <material name="structure_aluminum" />
       </visual>
       <collision>
@@ -59,4 +59,7 @@
       </collision>
     </link>
+    <gazebo reference="${prefix}part_up">
+      <material>Gazebo/Grey</material>
+    </gazebo>
     <link name="${prefix}pedestal">
       <inertial>
@@ -76,7 +79,5 @@
           <mesh filename="package://mobipick_description/meshes/structure/visual/pedestal.stl" />
         </geometry>
-        <material name="">
-          <color rgba="0.8 0.8 0.8 1" />
-        </material>
+        <material name="structure_aluminum" />
       </visual>
       <collision>
@@ -87,4 +88,7 @@
       </collision>
     </link>
+    <gazebo reference="${prefix}pedestal">
+      <material>Gazebo/Grey</material>
+    </gazebo>
     <link name="${prefix}pedestal_surface"/>
     <!-- <joint name="${prefix}structure_vertical_joint" type="prismatic">

Commit message: Fix whitespace

File: mobipick_description/urdf/mir_100/mir_100_v1.urdf.xacro (robot description, xacro)
@@ -68,10 +68,10 @@
         <mass value="0.3097539019" />
         <inertia
-            ixx="0.0005844517978"
-            ixy="0"
-            ixz="0"
-            iyy="0.00052872551237"
-            iyz="0"
-            izz="0.00017923555074" />
+          ixx="0.0005844517978"
+          ixy="0"
+          ixz="0"
+          iyy="0.00052872551237"
+          iyz="0"
+          izz="0.00017923555074" />
       </inertial>
       <visual>
@@ -164,10 +164,10 @@
   </xacro:macro>
   <xacro:macro name="mir_100" params="prefix">
-  <link name="${prefix}base_footprint" />
-  <joint name="${prefix}base_joint" type="fixed">
-    <parent link="${prefix}base_footprint" />
-    <child link="${prefix}base_link" />
-    <origin xyz="0 0 0" rpy="0 0 0" />
-  </joint>
+    <link name="${prefix}base_footprint" />
+    <joint name="${prefix}base_joint" type="fixed">
+      <parent link="${prefix}base_footprint" />
+      <child link="${prefix}base_link" />
+      <origin xyz="0 0 0" rpy="0 0 0" />
+    </joint>
     <link name="${prefix}base_link">
       <inertial>

File: mobipick_description/urdf/robotiq_2f_140/robotiq_fingertips_65mm.xacro (robot description, xacro)
@@ -8,9 +8,9 @@
         <mass value="3.3455E-2" />
         <inertia ixx="13.66E-6"
-		 ixy="0"
-		 ixz="0"
-		 iyy="11.784E-6"
-		 iyz="0"
-		 izz="2.15E-6" />
+          ixy="0"
+          ixz="0"
+          iyy="11.784E-6"
+          iyz="0"
+          izz="2.15E-6" />
       </inertial>
       <visual>

File: mobipick_description/urdf/structure/mobipick_structure.urdf.xacro (robot description, xacro)
@@ -9,10 +9,10 @@
         <mass value="3.349376" />
         <inertia
-            ixx="0.432077541"
-            ixy="0"
-            ixz="0"
-            iyy="0.369249471"
-            iyz="0"
-            izz="0.179676981" />
+          ixx="0.432077541"
+          ixy="0"
+          ixz="0"
+          iyy="0.369249471"
+          iyz="0"
+          izz="0.179676981" />
       </inertial>
       <visual>
@@ -38,10 +38,10 @@
         <mass value="4.64704" />
         <inertia
-            ixx="0.549473755"
-            ixy="0"
-            ixz="0"
-            iyy="0.436580833"
-            iyz="0"
-            izz="0.245971089" />
+          ixx="0.549473755"
+          ixy="0"
+          ixz="0"
+          iyy="0.436580833"
+          iyz="0"
+          izz="0.245971089" />
       </inertial>
       <visual>
@@ -67,10 +67,10 @@
         <mass value="2.354023413" />
         <inertia
-            ixx="0.049542988"
-            ixy="0"
-            ixz="0"
-            iyy="0.042530187"
-            iyz="0"
-            izz="0.020198776" />
+          ixx="0.049542988"
+          ixy="0"
+          ixz="0"
+          iyy="0.042530187"
+          iyz="0"
+          izz="0.020198776" />
       </inertial>
       <visual>

Commit message: Add IMU sensor

File: mobipick_description/urdf/mir_100/mir_100_v1.urdf.xacro (robot description, xacro)
@@ -2,4 +2,5 @@
 <robot xmlns:xacro="http://ros.org/wiki/xacro">
   <xacro:include filename="$(find mobipick_description)/urdf/common_properties.urdf.xacro" />
+  <xacro:include filename="$(find mobipick_description)/urdf/sensors/imu.gazebo.urdf.xacro" />
   <xacro:include filename="$(find mobipick_description)/urdf/mir_100/mir_100.transmission.xacro" />
   <xacro:include filename="$(find mobipick_description)/urdf/mir_100/mir_100.gazebo.xacro" />
@@ -21,4 +22,5 @@
   <xacro:property name="mir_100_caster_wheel_base_dy" value="0.203" />
   <xacro:property name="mir_100_caster_wheel_base_dz" value="${mir_100_caster_wheel_radius-mir_100_caster_wheel_dz}" />
+  <xacro:property name="imu_stdev" value="0.00017" />
   <xacro:macro name="actuated_wheel_link" params="prefix locationprefix">
     <link name="${prefix}${locationprefix}_act_wheel">
@@ -164,4 +166,13 @@
       <material>Gazebo/White</material>
     </gazebo>
+    <!-- IMU -->
+    <joint name="${prefix}base_link_to_imu_joint" type="fixed">
+      <parent link="${prefix}base_link" />
+      <child link="${prefix}imu_link" />
+      <origin xyz="0.0 0.0 0.25" rpy="0 0 0" />  <!-- same as real MiR -->
+    </joint>
+    <link name="${prefix}imu_link" />
+    <xacro:imu_gazebo link="${prefix}imu_link" imu_topic="imu_data" update_rate="50.0" stdev="${imu_stdev}" />
+    <!-- wheels -->
     <xacro:actuated_wheel_link prefix="${prefix}" locationprefix="left"/>
     <xacro:actuated_wheel_link prefix="${prefix}" locationprefix="right"/>

Commit message: gazebo: Use EKF instead of direct TF from plugin

File: mobipick_description/urdf/mir_100/mir_100_v1.urdf.xacro (robot description, xacro)
@@ -175,4 +175,13 @@
     <link name="${prefix}imu_link" />
     <xacro:imu_gazebo link="${prefix}imu_link" imu_topic="imu_data" update_rate="50.0" stdev="${imu_stdev}" />
+    <!-- Create an alias for imu_link. This is necessary because the real MiR's
+         TF has imu_link, but the imu_data topic is published in the imu_frame
+         frame. -->
+    <joint name="${prefix}imu_link_to_imu_frame_joint" type="fixed">
+      <parent link="${prefix}imu_link" />
+      <child link="${prefix}imu_frame" />
+      <origin xyz="0 0 0" rpy="0 0 0" />
+    </joint>
+    <link name="${prefix}imu_frame" />
     <!-- Laser scanners -->
     <joint name="${prefix}base_link_to_front_laser_joint" type="fixed">
