Commit message: urdf: Simplify caster wheel macros

File: mobipick_description/urdf/mir_100/mir_100_v1.urdf.xacro (robot description, xacro)
@@ -24,5 +24,12 @@
   <xacro:property name="mir_100_caster_wheel_base_dz" value="${mir_100_caster_wheel_radius-mir_100_caster_wheel_dz}" />
   <xacro:property name="imu_stdev" value="0.00017" />
-  <xacro:macro name="actuated_wheel_link" params="prefix locationprefix">
+  <xacro:macro name="actuated_wheel" params="prefix locationprefix locationright">
+    <joint name="${prefix}${locationprefix}_wheel_joint" type="continuous">
+      <origin xyz="0.0 ${-mir_100_act_wheel_dy * locationright} ${mir_100_act_wheel_radius}" rpy="0 0 0" />
+      <parent link="${prefix}base_link" />
+      <child link="${prefix}${locationprefix}_wheel_link" />
+      <axis xyz="0 1 0" />
+      <limit effort="100" velocity="20.0" />
+    </joint>
     <link name="${prefix}${locationprefix}_wheel_link">
       <xacro:cylinder_inertial mass="${mir_100_act_wheel_mass}" radius="${mir_100_act_wheel_radius}" length="${mir_100_act_wheel_width}">
@@ -47,5 +54,13 @@
     </gazebo>
   </xacro:macro>
-  <xacro:macro name="caster_wheel_links" params="prefix locationprefix">
+  <xacro:macro name="caster_wheel" params="prefix locationprefix locationright wheel_base_dx">
+    <!-- caster hub -->
+    <joint name="${prefix}${locationprefix}_caster_rotation_joint" type="continuous">
+      <origin xyz="${wheel_base_dx} ${-mir_100_caster_wheel_base_dy * locationright} ${mir_100_caster_wheel_base_dz}" rpy="0 0 0" />
+      <parent link="${prefix}base_link" />
+      <child link="${prefix}${locationprefix}_caster_rotation_link" />
+      <axis xyz="0 0 1" />
+      <dynamics damping="0.01" friction="0.0"/>
+    </joint>
     <link name="${prefix}${locationprefix}_caster_rotation_link">
       <inertial>
@@ -78,43 +93,5 @@
       <material>Gazebo/Grey</material>
     </gazebo>
-    <link name="${prefix}${locationprefix}_caster_wheel_link">
-      <xacro:cylinder_inertial mass="${mir_100_caster_wheel_mass}" radius="${mir_100_caster_wheel_radius}" length="${mir_100_caster_wheel_width}">
-        <origin xyz="0 0 0" rpy="${0.5 * pi} 0 0" />
-      </xacro:cylinder_inertial>
-      <visual>
-        <origin xyz="0 0 0" rpy="0 0 0" />
-        <geometry>
-          <mesh filename="package://mobipick_description/meshes/mir_100/visual/caster_wheel.stl" />
-        </geometry>
-        <xacro:insert_block name="material_dark_grey" />
-      </visual>
-      <collision>
-        <origin xyz="0 0 0" rpy="0 0 0" />
-        <geometry>
-          <mesh filename="package://mobipick_description/meshes/mir_100/collision/caster_wheel.stl" />
-        </geometry>
-      </collision>
-    </link>
-    <gazebo reference="${prefix}${locationprefix}_caster_wheel_link">
-      <material>Gazebo/DarkGrey</material>
-    </gazebo>
-  </xacro:macro>
-  <xacro:macro name="actuated_wheel_joint" params="prefix locationprefix locationright">
-    <joint name="${prefix}${locationprefix}_wheel_joint" type="continuous">
-      <origin xyz="0.0 ${-mir_100_act_wheel_dy * locationright} ${mir_100_act_wheel_radius}" rpy="0 0 0" />
-      <parent link="${prefix}base_link" />
-      <child link="${prefix}${locationprefix}_wheel_link" />
-      <axis xyz="0 1 0" />
-      <limit effort="100" velocity="20.0" />
-    </joint>
-  </xacro:macro>
-  <xacro:macro name="front_caster_wheel_joints" params="prefix locationprefix locationright">
-    <joint name="${prefix}${locationprefix}_caster_rotation_joint" type="continuous">
-      <origin xyz="${mir_100_front_caster_wheel_base_dx} ${-mir_100_caster_wheel_base_dy * locationright} ${mir_100_caster_wheel_base_dz}" rpy="0 0 0" />
-      <parent link="${prefix}base_link" />
-      <child link="${prefix}${locationprefix}_caster_rotation_link" />
-      <axis xyz="0 0 1" />
-      <dynamics damping="0.01" friction="0.0"/>
-    </joint>
+    <!-- caster wheel -->
     <joint name="${prefix}${locationprefix}_caster_wheel_joint" type="continuous">
       <origin xyz="${mir_100_caster_wheel_dx} ${-mir_100_caster_wheel_dy * locationright} ${mir_100_caster_wheel_dz}" rpy="0 0 0" />
@@ -123,19 +100,25 @@
       <axis xyz="0 1 0" />
     </joint>
-  </xacro:macro>
-  <xacro:macro name="back_caster_wheel_joints" params="prefix locationprefix locationright">
-    <joint name="${prefix}${locationprefix}_caster_rotation_joint" type="continuous">
-      <origin xyz="${mir_100_back_caster_wheel_base_dx} ${-mir_100_caster_wheel_base_dy * locationright} ${mir_100_caster_wheel_base_dz}" rpy="0 0 0" />
-      <parent link="${prefix}base_link" />
-      <child link="${prefix}${locationprefix}_caster_rotation_link" />
-      <axis xyz="0 0 1" />
-      <dynamics damping="0.01" friction="0.0"/>
-    </joint>
-    <joint name="${prefix}${locationprefix}_caster_wheel_joint" type="continuous">
-      <origin xyz="${mir_100_caster_wheel_dx} ${-mir_100_caster_wheel_dy * locationright} ${mir_100_caster_wheel_dz}" rpy="0 0 0" />
-      <parent link="${prefix}${locationprefix}_caster_rotation_link" />
-      <child link="${prefix}${locationprefix}_caster_wheel_link" />
-      <axis xyz="0 1 0" />
-    </joint>
+    <link name="${prefix}${locationprefix}_caster_wheel_link">
+      <xacro:cylinder_inertial mass="${mir_100_caster_wheel_mass}" radius="${mir_100_caster_wheel_radius}" length="${mir_100_caster_wheel_width}">
+        <origin xyz="0 0 0" rpy="${0.5 * pi} 0 0" />
+      </xacro:cylinder_inertial>
+      <visual>
+        <origin xyz="0 0 0" rpy="0 0 0" />
+        <geometry>
+          <mesh filename="package://mobipick_description/meshes/mir_100/visual/caster_wheel.stl" />
+        </geometry>
+        <xacro:insert_block name="material_dark_grey" />
+      </visual>
+      <collision>
+        <origin xyz="0 0 0" rpy="0 0 0" />
+        <geometry>
+          <mesh filename="package://mobipick_description/meshes/mir_100/collision/caster_wheel.stl" />
+        </geometry>
+      </collision>
+    </link>
+    <gazebo reference="${prefix}${locationprefix}_caster_wheel_link">
+      <material>Gazebo/DarkGrey</material>
+    </gazebo>
   </xacro:macro>
   <xacro:macro name="mir_100" params="prefix">
@@ -200,16 +183,10 @@
     <xacro:sick_s300 link="${prefix}back_laser_link" topic="b_scan" />
     <!-- wheels -->
-    <xacro:actuated_wheel_link prefix="${prefix}" locationprefix="left"/>
-    <xacro:actuated_wheel_link prefix="${prefix}" locationprefix="right"/>
-    <xacro:caster_wheel_links prefix="${prefix}" locationprefix="fl"/>
-    <xacro:caster_wheel_links prefix="${prefix}" locationprefix="fr"/>
-    <xacro:caster_wheel_links prefix="${prefix}" locationprefix="bl"/>
-    <xacro:caster_wheel_links prefix="${prefix}" locationprefix="br"/>
-    <xacro:actuated_wheel_joint prefix="${prefix}" locationprefix="left" locationright="-1"/>
-    <xacro:actuated_wheel_joint prefix="${prefix}" locationprefix="right" locationright="1"/>
-    <xacro:front_caster_wheel_joints prefix="${prefix}" locationprefix="fl" locationright="-1"/>
-    <xacro:front_caster_wheel_joints prefix="${prefix}" locationprefix="fr" locationright="1"/>
-    <xacro:back_caster_wheel_joints prefix="${prefix}" locationprefix="bl" locationright="-1"/>
-    <xacro:back_caster_wheel_joints prefix="${prefix}" locationprefix="br" locationright="1"/>
+    <xacro:actuated_wheel prefix="${prefix}" locationprefix="left" locationright="-1"/>
+    <xacro:actuated_wheel prefix="${prefix}" locationprefix="right" locationright="1"/>
+    <xacro:caster_wheel prefix="${prefix}" locationprefix="fl" locationright="-1" wheel_base_dx="${mir_100_front_caster_wheel_base_dx}"/>
+    <xacro:caster_wheel prefix="${prefix}" locationprefix="fr" locationright="1" wheel_base_dx="${mir_100_front_caster_wheel_base_dx}"/>
+    <xacro:caster_wheel prefix="${prefix}" locationprefix="bl" locationright="-1" wheel_base_dx="${mir_100_back_caster_wheel_base_dx}"/>
+    <xacro:caster_wheel prefix="${prefix}" locationprefix="br" locationright="1" wheel_base_dx="${mir_100_back_caster_wheel_base_dx}"/>
     <joint name="${prefix}base_link_surface_joint" type="fixed">
       <origin xyz="${mir_100_act_wheel_dx} 0 0.352" rpy="0 0 0" />

Commit message: urdf: Adjust laser scanner tfs to mobipick-hb

File: mobipick_description/urdf/mir_100/mir_100_v1.urdf.xacro (robot description, xacro)
@@ -172,5 +172,6 @@
       <child link="${prefix}front_laser_link" />
       <!-- on real MiR (depends on calibration): <origin xyz="0.416 0.243 0.200" rpy="0.0 0.0 0.795" /> -->
-      <origin xyz="0.4288 0.2358 0.1914" rpy="${-pi} 0.0 ${pi/4}" />  <!-- from visually matching up the meshes of the MiR and the laser scanner -->
+      <!-- <origin xyz="0.4288 0.2358 0.1914" rpy="${-pi} 0.0 ${pi/4}" />  from visually matching up the meshes of the MiR and the laser scanner -->
+      <origin xyz="0.420 0.240 0.200" rpy="0.0 0.0 0.804" />  <!-- from the TFs published by the real mobipick-hb -->
     </joint>
     <xacro:sick_s300 link="${prefix}front_laser_link" topic="f_scan" />
@@ -179,5 +180,6 @@
       <child link="${prefix}back_laser_link" />
       <!-- on real MiR: <origin xyz="-0.360 -0.252 0.200" rpy="0.0 0.0 -2.348" /> -->
-      <origin xyz="-0.3548 -0.2352 0.1914" rpy="${-pi} 0.0 ${-0.75 * pi}" />  <!-- from visually matching up the meshes of the MiR and the laser scanner -->
+      <!-- <origin xyz="-0.3548 -0.2352 0.1914" rpy="${-pi} 0.0 ${-0.75 * pi}" />  from visually matching up the meshes of the MiR and the laser scanner -->
+      <origin xyz="-0.364 -0.239 0.200" rpy="0.0 0.0 -2.349" />  <!-- from the TFs published by the real mobipick-hb -->
     </joint>
     <xacro:sick_s300 link="${prefix}back_laser_link" topic="b_scan" />

File: mobipick_description/urdf/sensors/sick_s300.urdf.xacro (robot description, xacro)
@@ -9,4 +9,5 @@
     <link name="${link}">
       <visual>
+        <origin xyz="0.0 0.0 0.0" rpy="${pi} 0 0" />
         <geometry>
           <mesh filename="package://mobipick_description/meshes/sensors/sick_lms-100.stl" />
@@ -16,4 +17,5 @@
       </visual>
       <collision>
+        <origin xyz="0.0 0.0 0.0" rpy="${pi} 0 0" />
         <geometry>
           <mesh filename="package://mobipick_description/meshes/sensors/sick_lms-100.stl" />
