Commit message: gripper: Use PID in mimic, tune gains, add damping
Using the PID controller solves the last "parachute" problem (that the
wheels intermittently lose contact with the ground due to the use of the
Gazebo joint->SetAngle() function.

Also in this commit:

* lower max joint velocity to 0.7
* increase max_effort of the controller to 10 (in reality it should stay
  below 1 Nm)
* lowered the gains
* added damping

File: mobipick_description/urdf/robotiq_2f_140/robotiq_2f_140.gazebo.xacro (robot description, xacro)
@@ -1,11 +1,14 @@
 <?xml version="1.0"?>
 <robot xmlns:xacro="http://ros.org/wiki/xacro">
-  <xacro:macro name="mimic_joint_plugin_gazebo" params="name_prefix parent_joint mimic_joint multiplier offset robot_namespace">
+  <xacro:macro name="mimic_joint_plugin_gazebo" params="name_prefix parent_joint mimic_joint has_pid:=false multiplier:=1.0 offset:=0 sensitiveness:=0.0 max_effort:=1.0 robot_namespace">
     <gazebo>
       <plugin name="${name_prefix}mimic_joint_plugin" filename="libroboticsgroup_gazebo_mimic_joint_plugin.so">
         <joint>${parent_joint}</joint>
         <mimicJoint>${mimic_joint}</mimicJoint>
+        <hasPID>${has_pid}</hasPID>                       <!-- if set to true, PID parameters from "/gazebo_ros_control/pid_gains/${mimic_joint}" are loaded -->
         <multiplier>${multiplier}</multiplier>
         <offset>${offset}</offset>
+        <sensitiveness>${sensitiveness}</sensitiveness>   <!-- if absolute difference between setpoint and process value is below this threshold, do nothing; 0.0 = disable [rad] -->
+        <maxEffort>${max_effort}</maxEffort>              <!-- only taken into account if has_pid:=true [Nm] -->
         <xacro:unless value="${robot_namespace == ''}">
           <robotNamespace>($robot_namespace)</robotNamespace>
@@ -16,9 +19,9 @@
   <!-- plugin from https://github.com/roboticsgroup/roboticsgroup_gazebo_plugins used to simulate the mimic joints -->
   <xacro:macro name="mimic_joint_plugins_gazebo" params="prefix robot_namespace">
-    <xacro:mimic_joint_plugin_gazebo name_prefix="${prefix}right_outer_knuckle" parent_joint="${prefix}finger_joint" mimic_joint="${prefix}right_outer_knuckle_joint" multiplier="-1.0" offset="0" robot_namespace="${robot_namespace}"/>
-    <xacro:mimic_joint_plugin_gazebo name_prefix="${prefix}left_inner_knuckle" parent_joint="${prefix}finger_joint" mimic_joint="${prefix}left_inner_knuckle_joint" multiplier="-1.0" offset="0" robot_namespace="${robot_namespace}"/>
-    <xacro:mimic_joint_plugin_gazebo name_prefix="${prefix}right_inner_knuckle" parent_joint="${prefix}finger_joint" mimic_joint="${prefix}right_inner_knuckle_joint" multiplier="-1.0" offset="0" robot_namespace="${robot_namespace}"/>
-    <xacro:mimic_joint_plugin_gazebo name_prefix="${prefix}left_inner_finger" parent_joint="${prefix}finger_joint" mimic_joint="${prefix}left_inner_finger_joint" multiplier="1" offset="0" robot_namespace="${robot_namespace}"/>
-    <xacro:mimic_joint_plugin_gazebo name_prefix="${prefix}right_inner_finger" parent_joint="${prefix}finger_joint" mimic_joint="${prefix}right_inner_finger_joint" multiplier="1" offset="0" robot_namespace="${robot_namespace}"/>
+    <xacro:mimic_joint_plugin_gazebo name_prefix="${prefix}right_outer_knuckle" parent_joint="${prefix}finger_joint" mimic_joint="${prefix}right_outer_knuckle_joint" has_pid="true" multiplier="-1.0" max_effort="10.0" robot_namespace="${robot_namespace}"/>
+    <xacro:mimic_joint_plugin_gazebo name_prefix="${prefix}left_inner_knuckle"  parent_joint="${prefix}finger_joint" mimic_joint="${prefix}left_inner_knuckle_joint"  has_pid="true" multiplier="-1.0" max_effort="10.0" robot_namespace="${robot_namespace}"/>
+    <xacro:mimic_joint_plugin_gazebo name_prefix="${prefix}right_inner_knuckle" parent_joint="${prefix}finger_joint" mimic_joint="${prefix}right_inner_knuckle_joint" has_pid="true" multiplier="-1.0" max_effort="10.0" robot_namespace="${robot_namespace}"/>
+    <xacro:mimic_joint_plugin_gazebo name_prefix="${prefix}left_inner_finger"   parent_joint="${prefix}finger_joint" mimic_joint="${prefix}left_inner_finger_joint"   has_pid="true" multiplier="1"    max_effort="10.0" robot_namespace="${robot_namespace}"/>
+    <xacro:mimic_joint_plugin_gazebo name_prefix="${prefix}right_inner_finger"  parent_joint="${prefix}finger_joint" mimic_joint="${prefix}right_inner_finger_joint"  has_pid="true" multiplier="1"    max_effort="10.0" robot_namespace="${robot_namespace}"/>
   </xacro:macro>
 </robot>

File: mobipick_description/urdf/robotiq_2f_140/robotiq_arg2f_140_model_macro.xacro (robot description, xacro)
@@ -130,4 +130,5 @@
     </joint>
   </xacro:macro>
+  <!-- === 2x inner knuckle joint ================================================================================== -->
   <xacro:macro name="inner_knuckle_joint" params="prefix fingerprefix reflect">
     <joint name="${prefix}${fingerprefix}_inner_knuckle_joint" type="revolute">
@@ -136,8 +137,10 @@
       <child link="${prefix}${fingerprefix}_inner_knuckle" />
       <axis xyz="1 0 0" />
-      <limit lower="-0.8757" upper="0" velocity="2.0" effort="1000" />
+      <limit lower="-0.8757" upper="0" velocity="0.7" effort="1000" />
       <mimic joint="${prefix}finger_joint" multiplier="-1" offset="0" />
+      <dynamics damping="0.02" friction="0.0" />
     </joint>
   </xacro:macro>
+  <!-- === 2x finger tip joint (second movable joint in series) ===================================================== -->
   <xacro:macro name="inner_finger_joint" params="prefix fingerprefix">
     <joint name="${prefix}${fingerprefix}_inner_finger_joint" type="revolute">
@@ -146,10 +149,12 @@
       <child link="${prefix}${fingerprefix}_inner_finger" />
       <axis xyz="1 0 0" />
-      <limit lower="0" upper="0.8757" velocity="2.0" effort="1000" />
+      <limit lower="0" upper="0.8757" velocity="0.7" effort="1000" />
       <mimic joint="${prefix}finger_joint" multiplier="1" offset="0" />
+      <dynamics damping="0.001" friction="0.0" />
     </joint>
   </xacro:macro>
   <xacro:include filename="$(find mobipick_description)/urdf/robotiq_2f_140/robotiq_arg2f.xacro" />
-  <xacro:macro name="finger_joint" params="prefix">
+  <!-- === outer knuckle joint (first movable joint in series) ===================================================== -->
+  <xacro:macro name="finger_joint" params="prefix">   <!-- = "left_outer_knuckle_joint" -->
     <joint name="${prefix}finger_joint" type="revolute">
       <origin xyz="0 -0.030601 0.054905" rpy="${pi / 2 + .725} 0 0" />
@@ -157,5 +162,6 @@
       <child link="${prefix}left_outer_knuckle" />
       <axis xyz="-1 0 0" />
-      <limit lower="0" upper="0.755" velocity="2.0" effort="1000" />
+      <limit lower="0" upper="0.755" velocity="0.7" effort="1000" />
+      <dynamics damping="0.02" friction="0.0" />
     </joint>
     <xacro:finger_joints prefix="${prefix}" fingerprefix="left" reflect="1.0"/>
@@ -167,9 +173,11 @@
       <child link="${prefix}right_outer_knuckle" />
       <axis xyz="1 0 0" />
-      <limit lower="-0.755" upper="0" velocity="2.0" effort="1000" />
-    <mimic joint="${prefix}finger_joint" multiplier="-1" offset="0" />
+      <limit lower="-0.755" upper="0" velocity="0.7" effort="1000" />
+      <mimic joint="${prefix}finger_joint" multiplier="-1" offset="0" />
+      <dynamics damping="0.02" friction="0.0" />
     </joint>
     <xacro:finger_joints prefix="${prefix}" fingerprefix="right" reflect="-1.0"/>
   </xacro:macro>
+  <!-- =========================================================================================================== -->
   <xacro:include filename="$(find mobipick_description)/urdf/robotiq_2f_140/robotiq_fingertips_65mm.xacro" />
   <xacro:macro name="robotiq_arg2f_140" params="prefix">

Commit message: URDF: robotiq gripper: close kinematic loop
This finally turns our gripper into a true parallel gripper and fixes grasping the power drill!

File: mobipick_description/urdf/robotiq_2f_140/robotiq_2f_140.gazebo.xacro (robot description, xacro)
@@ -22,8 +22,4 @@
   <xacro:macro name="mimic_joint_plugins_gazebo" params="prefix robot_namespace">
     <xacro:mimic_joint_plugin_gazebo name_prefix="${prefix}right_outer_knuckle" parent_joint="${prefix}finger_joint" mimic_joint="${prefix}right_outer_knuckle_joint" has_pid="true" multiplier="-1.0" max_effort="10.0" robot_namespace="${robot_namespace}"/>
-    <xacro:mimic_joint_plugin_gazebo name_prefix="${prefix}left_inner_knuckle"  parent_joint="${prefix}finger_joint" mimic_joint="${prefix}left_inner_knuckle_joint"  has_pid="true" multiplier="-1.0" max_effort="10.0" robot_namespace="${robot_namespace}"/>
-    <xacro:mimic_joint_plugin_gazebo name_prefix="${prefix}right_inner_knuckle" parent_joint="${prefix}finger_joint" mimic_joint="${prefix}right_inner_knuckle_joint" has_pid="true" multiplier="-1.0" max_effort="10.0" robot_namespace="${robot_namespace}"/>
-    <xacro:mimic_joint_plugin_gazebo name_prefix="${prefix}left_inner_finger"   parent_joint="${prefix}finger_joint" mimic_joint="${prefix}left_inner_finger_joint"   has_pid="true" multiplier="1"    max_effort="10.0" robot_namespace="${robot_namespace}"/>
-    <xacro:mimic_joint_plugin_gazebo name_prefix="${prefix}right_inner_finger"  parent_joint="${prefix}finger_joint" mimic_joint="${prefix}right_inner_finger_joint"  has_pid="true" multiplier="1"    max_effort="10.0" robot_namespace="${robot_namespace}"/>
   </xacro:macro>
 </robot>

File: mobipick_description/urdf/robotiq_2f_140/robotiq_arg2f.xacro (robot description, xacro)
@@ -32,4 +32,5 @@
     <xacro:inner_knuckle_joint prefix="${prefix}" fingerprefix="${fingerprefix}" reflect="${reflect}"/>
     <xacro:inner_finger_joint prefix="${prefix}" fingerprefix="${fingerprefix}"/>
+    <xacro:inner_knuckle_to_finger_joint prefix="${prefix}" fingerprefix="${fingerprefix}"/>
   </xacro:macro>
   <xacro:macro name="finger_links" params="prefix fingerprefix stroke">

File: mobipick_description/urdf/robotiq_2f_140/robotiq_arg2f_140_model_macro.xacro (robot description, xacro)
@@ -158,4 +158,19 @@
       <dynamics damping="0.001" friction="0.0" />
     </joint>
+  </xacro:macro>
+  <xacro:include filename="$(find mobipick_description)/urdf/robotiq_2f_140/robotiq_arg2f.xacro" />
+  <!-- === 2x inner knuckle to inner finger joint ===================================================== -->
+  <xacro:macro name="inner_knuckle_to_finger_joint" params="prefix fingerprefix">
+    <!-- This joint closes the kinematic loop. Since loops are not allowed in URDF, but they are allowed in SDF, this is an SDF fragment. -->
+    <gazebo>
+      <joint name="${prefix}${fingerprefix}_inner_knuckle_to_finger_joint" type="revolute">
+        <pose relative_to="${prefix}${fingerprefix}_inner_knuckle">0 0.1 -0.0022 0 0 0</pose>
+        <axis>
+          <xyz>1 0 0</xyz>
+        </axis>
+        <parent>${prefix}${fingerprefix}_inner_knuckle</parent>
+        <child>${prefix}${fingerprefix}_inner_finger</child>
+      </joint>
+    </gazebo>
   </xacro:macro>
   <xacro:include filename="$(find mobipick_description)/urdf/robotiq_2f_140/robotiq_arg2f.xacro" />
