Commit message: gripper: Add Gazebo colors

File: mobipick_description/urdf/robotiq_2f_140/robotiq_arg2f.xacro (robot description, xacro)
@@ -24,4 +24,7 @@
       </collision>
     </link>
+    <gazebo reference="${prefix}robotiq_arg2f_base_link">
+      <material>Gazebo/FlatBlack</material>
+    </gazebo>
   </xacro:macro>
   <xacro:macro name="finger_joints" params="prefix fingerprefix reflect">

File: mobipick_description/urdf/robotiq_2f_140/robotiq_arg2f_140_model_macro.xacro (robot description, xacro)
@@ -10,10 +10,10 @@
         <mass value="0.00853198276973456" />
         <inertia
-            ixx="2.89328108496468E-06"
-            ixy="-1.57935047237397E-19"
-            ixz="-1.93980378593255E-19"
-            iyy="1.86719750325683E-06"
-            iyz="-1.21858577871576E-06"
-            izz="1.21905238907251E-06" />
+          ixx="2.89328108496468E-06"
+          ixy="-1.57935047237397E-19"
+          ixz="-1.93980378593255E-19"
+          iyy="1.86719750325683E-06"
+          iyz="-1.21858577871576E-06"
+          izz="1.21905238907251E-06" />
       </inertial>
       <visual>
@@ -31,4 +31,7 @@
       </collision>
     </link>
+    <gazebo reference="${prefix}${fingerprefix}_outer_knuckle">
+      <material>Gazebo/Grey</material>
+    </gazebo>
   </xacro:macro>
   <xacro:macro name="outer_finger" params="prefix fingerprefix stroke">
@@ -59,4 +62,7 @@
       </collision>
     </link>
+    <gazebo reference="${prefix}${fingerprefix}_outer_finger">
+      <material>Gazebo/FlatBlack</material>
+    </gazebo>
   </xacro:macro>
   <xacro:macro name="inner_knuckle" params="prefix fingerprefix stroke">
@@ -87,4 +93,7 @@
       </collision>
     </link>
+    <gazebo reference="${prefix}${fingerprefix}_inner_knuckle">
+      <material>Gazebo/FlatBlack</material>
+    </gazebo>
   </xacro:macro>
   <xacro:macro name="inner_finger" params="prefix fingerprefix stroke">
@@ -115,4 +124,7 @@
       </collision>
     </link>
+    <gazebo reference="${prefix}${fingerprefix}_inner_finger">
+      <material>Gazebo/FlatBlack</material>
+    </gazebo>
   </xacro:macro>
   <xacro:macro name="outer_finger_joint" params="prefix fingerprefix">

File: mobipick_description/urdf/robotiq_2f_140/robotiq_fingertips_65mm.xacro (robot description, xacro)
@@ -30,4 +30,7 @@
       </collision>
     </link>
+    <gazebo reference="${prefix}${fingerprefix}_robotiq_fingertip_65mm">
+      <material>Gazebo/Grey</material>
+    </gazebo>
   </xacro:macro>
   <xacro:macro name="fingertip_joint" params="prefix fingerprefix">

Commit message: URDF: Fix robotiq_arg2f_base_link_coarse
* Reduce length by 0.0078875 m to fit fine mesh.

* Rotate to match robotiq_arg2f_base_link_fine. The mesh and the URDF were
rotated in opposing directions, so that the net result is the same (but
the URDF can now use a yaw angle of 0).

File: mobipick_description/urdf/robotiq_2f_140/robotiq_arg2f.xacro (robot description, xacro)
@@ -18,5 +18,5 @@
       </visual>
       <collision>
-        <origin xyz="0 0 0" rpy="0 0 ${pi / 2}" />
+        <origin xyz="0 0 0" rpy="0 0 0" />
         <geometry>
           <mesh filename="package://mobipick_description/meshes/robotiq_2f_140/robotiq_arg2f_base_link_coarse.stl" />

Commit message: URDF: Extract remaining robotiq materials, fix typo
This also fixes the material name "robotiq_light_grey /", which caused
problems during Unity export.

File: mobipick_description/urdf/robotiq_2f_140/robotiq_arg2f.xacro (robot description, xacro)
@@ -1,4 +1,5 @@
 <?xml version="1.0"?>
 <robot xmlns:xacro="http://ros.org/wiki/xacro">
+  <xacro:include filename="$(find mobipick_description)/urdf/common_properties.urdf.xacro" />
   <xacro:macro name="robotiq_arg2f_base_link" params="prefix">
     <link name="${prefix}robotiq_arg2f_base_link">
@@ -13,7 +14,5 @@
           <mesh filename="package://mobipick_description/meshes/robotiq_2f_140/robotiq_arg2f_base_link_fine.stl" />
         </geometry>
-        <material name="">
-          <color rgba="0.1 0.1 0.1 1" />
-        </material>
+        <xacro:insert_block name="material_black" />
       </visual>
       <collision>

File: mobipick_description/urdf/robotiq_2f_140/robotiq_fingertips_65mm.xacro (robot description, xacro)
@@ -1,4 +1,5 @@
 <?xml version="1.0"?>
 <robot xmlns:xacro="http://ros.org/wiki/xacro">
+  <xacro:include filename="$(find mobipick_description)/urdf/common_properties.urdf.xacro" />
   <xacro:macro name="robotiq_fingertip_65mm" params="prefix fingerprefix stroke">
     <link name="${prefix}${fingerprefix}_robotiq_fingertip_65mm">
@@ -19,7 +20,5 @@
           <mesh filename="package://mobipick_description/meshes/robotiq_2f_140/robotiq_arg2f_${stroke}_fingertip_65mm.stl" />
         </geometry>
-        <material name="robotiq_light_grey /">
-          <color rgba="0.5 0.5 0.5 1" />
-        </material>
+        <xacro:insert_block name="material_grey" />
       </visual>
       <collision>

File: mobipick_description/urdf/robotiq_ft_300/robotiq_ft_300.urdf.xacro (robot description, xacro)
@@ -1,4 +1,5 @@
 <?xml version="1.0"?>
 <robot xmlns:xacro="http://ros.org/wiki/xacro" name="robotiq_ft_300">
+  <xacro:include filename="$(find mobipick_description)/urdf/common_properties.urdf.xacro" />
   <xacro:macro name="robotiq_ft_300" params="parent prefix *origin">
     <!-- mount the fts to the robot -->
@@ -21,7 +22,5 @@
           <mesh filename="package://mobipick_description/meshes/robotiq_ft_300/visual/robotiq_ft_300.stl"/>
         </geometry>
-        <material name="">
-          <color rgba="0.25 0.25 0.25 1" />
-        </material>
+        <xacro:insert_block name="material_black" />
       </visual>
       <collision>

File: mobipick_description/urdf/robotiq_ft_300/robotiq_fts150.urdf.xacro (robot description, xacro)
@@ -1,4 +1,5 @@
 <?xml version="1.0"?>
 <robot xmlns:xacro="http://ros.org/wiki/xacro" name="robotiq_fts150">
+  <xacro:include filename="$(find mobipick_description)/urdf/common_properties.urdf.xacro" />
     <xacro:macro name="robotiq_fts150" params="parent prefix *origin">
         <!-- mount the fts to the robot -->
@@ -20,5 +21,5 @@
                     <mesh filename="package://robotiq_force_torque_sensor/meshes/visual/robotiq_fts150.stl"/>
                 </geometry>
-                <material name="black"/>
+                <xacro:insert_block name="material_black" />
             </visual>
             <collision>
