Commit message: adjusted link names in gazebo grasp fix plugin with prefix

File: mobipick_description/urdf/robotiq_2f_140/gzplugin_grasp_fix.urdf.xacro (robot description, xacro)
@@ -1,21 +1,21 @@
 <?xml version="1.0" encoding="UTF-8"?>
 <root xmlns:xacro="http://ros.org/wiki/xacro">
-  <xacro:macro name="gzplugin_grasp_fix">
+  <xacro:macro name="gzplugin_grasp_fix" params="prefix">
     <gazebo>
       <plugin name="gazebo_grasp_fix" filename="libgazebo_grasp_fix.so">
         <arm>
           <arm_name>arm</arm_name>
-          <palm_link>ur5_wrist_3_link</palm_link>
+          <palm_link>${prefix}ur5_wrist_3_link</palm_link>
           <!-- NOTE: the commented-out links have fixed joints with other
                links, so they are not present in the SDF any more. -->
-          <gripper_link>gripper_left_outer_knuckle          </gripper_link>
+          <gripper_link>${prefix}gripper_left_outer_knuckle          </gripper_link>
           <!-- <gripper_link>gripper_left_outer_finger           </gripper_link> -->
-          <gripper_link>gripper_left_inner_finger           </gripper_link>
+          <gripper_link>${prefix}gripper_left_inner_finger           </gripper_link>
           <!-- <gripper_link>gripper_left_robotiq_fingertip_65mm </gripper_link> -->
-          <gripper_link>gripper_left_inner_knuckle          </gripper_link>
-          <gripper_link>gripper_right_inner_knuckle         </gripper_link>
-          <gripper_link>gripper_right_outer_knuckle         </gripper_link>
+          <gripper_link>${prefix}gripper_left_inner_knuckle          </gripper_link>
+          <gripper_link>${prefix}gripper_right_inner_knuckle         </gripper_link>
+          <gripper_link>${prefix}gripper_right_outer_knuckle         </gripper_link>
           <!-- <gripper_link>gripper_right_outer_finger          </gripper_link> -->
-          <gripper_link>gripper_right_inner_finger          </gripper_link>
+          <gripper_link>${prefix}gripper_right_inner_finger          </gripper_link>
           <!-- <gripper_link>gripper_right_robotiq_fingertip_65mm</gripper_link> -->
         </arm>

File: mobipick_description/urdf/robotiq_2f_140/robotiq_arg2f_140_model_macro.xacro (robot description, xacro)
@@ -207,4 +207,4 @@
   <!-- GRASP HACK -->
   <xacro:include filename="$(find mobipick_description)/urdf/robotiq_2f_140/gzplugin_grasp_fix.urdf.xacro"/>
-  <gzplugin_grasp_fix/>
+  <gzplugin_grasp_fix prefix="${prefix}"/>
 </robot>

Commit message: fixes issue 29: Objects slipping mobipick gripper in simulation, now it should be ok

File: mobipick_description/urdf/robotiq_2f_140/gzplugin_grasp_fix.urdf.xacro (robot description, xacro)
@@ -20,8 +20,27 @@
           <!-- <gripper_link>gripper_right_robotiq_fingertip_65mm</gripper_link> -->
         </arm>
-        <forces_angle_tolerance>120</forces_angle_tolerance>
-        <update_rate>8</update_rate>
+        <!-- Is the tolerance angle (in degrees) between two force vectors to be considered "opposing forces".
+             If the angle is smaller than this, they are not opposing. -->
+        <forces_angle_tolerance>90</forces_angle_tolerance> <!-- NOTE: min value: 90 degree-->
+        <!-- Is the rate at which all contact points are checked against the "gripping criterion".
+             Note that in-between such updates, existing contact points may be collected at a higher rate
+             (the Gazebo world update rate). The update_rate is only the rate at which they are processed,
+              which takes a bit of computation time, and therefore should be lower than the gazebo world update rate. -->
+        <update_rate>50</update_rate>
+        <!-- Is the number of times in the update loop (running at update_rate) that an object has to be detected as "gripped"
+             in order to attach the object. Adjust this with the update rate.-->
         <grip_count_threshold>4</grip_count_threshold>
+        <!-- Is the maximum number of a counter: At each update iteration (running at update_rate), if the "gripping criterion"
+             is met for an object, a counter for this object is increased. max_grip_count is the maximum number recorded for an object.
+             As soon as the counter goes beyond this number, the counter is stopped. As soon as the "gripping criterion" does not hold any more,
+             the number will start to decrease again, (by 1 each time the object is detected as "not grasped" in an update iteration).
+             So this counter is like a "buffer" which, when it is full, maintains the state, and when it is empty, again, the object is released.
+             This should be at least double of grip_count_threshold. -->
         <max_grip_count>16</max_grip_count>
+        <!-- Is the distance which the gripper links are allowed to move away from the object during* a grasp without the object being detached,
+             even if there are currently no actual contacts on the object. This condition can happen if the fingers "wobble"
+             or move ever so slightly away from the object, and therefore the "gripping criterion" fails in a few subsequent update iterations.
+             This setting is to make the behaviour more stable. Setting this number too high will also lead to the object not being detached
+             even if the grippers have opened up to release it, so use this with care. -->
         <release_tolerance>0.01</release_tolerance>
         <disable_collisions_on_attach>false</disable_collisions_on_attach>

File: mobipick_gazebo/urdf/klt.urdf.xacro (robot description, xacro)
@@ -20,9 +20,45 @@
       </geometry>
     </visual>
-    <collision>
+    <!--<collision>
       <origin xyz="0 0 0" rpy="0 0 0" />
       <geometry>
         <mesh filename="package://mobipick_gazebo/meshes/collision/klt.stl" />
       </geometry>
+    </collision>-->
+    <!--klt collision model made up from boxes, klt bounding box as reported from dope : 0.297 0.197 0.1469-->
+    <!-- klt base -->
+    <collision>
+      <origin xyz="0 0 -0.06345" rpy="0 0 0" /> <!--klt thickness = 0.02 ; (0.1469 - 0.02 = 0.1269) / 2-->
+      <geometry>
+            <box size="0.297 0.197 0.02" />
+      </geometry>
+    </collision>
+    <!-- right klt wall -->
+    <collision>
+      <origin xyz="0 0.0885 0" rpy="0 0 0" /> <!--(0.197 - 0.02 = 0.177) / 2-->
+      <geometry>
+        <box size="0.297 0.02 0.1469" />
+      </geometry>
+    </collision>
+    <!-- left klt wall -->
+    <collision>
+      <origin xyz="0 -0.0885 0" rpy="0 0 0" /> <!--(0.197 - 0.02 = 0.177) / 2-->
+      <geometry>
+        <box size="0.297 0.02 0.1469" />
+      </geometry>
+    </collision>
+    <!-- front klt wall -->
+    <collision>
+      <origin xyz="0.1385 0 0" rpy="0 0 0" /> <!--(0.297 - 0.02 = 0.277 ) / 2-->
+      <geometry>
+        <box size="0.02 0.197 0.1469" />
+      </geometry>
+    </collision>
+    <!-- back klt wall -->
+    <collision>
+      <origin xyz="-0.1385 0 0" rpy="0 0 0" /> <!--(0.297 - 0.02 = 0.277 ) / 2-->
+      <geometry>
+        <box size="0.02 0.197 0.1469" />
+      </geometry>
     </collision>
   </link>

File: mobipick_gazebo/urdf/multimeter.urdf.xacro (robot description, xacro)
@@ -25,6 +25,6 @@
       <origin xyz="0 0 0" rpy="0 0 0" />
       <geometry>
-        <!-- <box size="${bb_size_x} ${bb_size_y} ${bb_size_z}" /> -->
-        <mesh filename="package://mobipick_gazebo/meshes/collision//multimeter.stl" />
+         <box size="${bb_size_x} ${bb_size_y} ${bb_size_z}" />
+        <!--<mesh filename="package://mobipick_gazebo/meshes/collision//multimeter.stl" />-->
       </geometry>
     </collision>

File: mobipick_gazebo/urdf/relay.urdf.xacro (robot description, xacro)
@@ -25,6 +25,6 @@
       <origin xyz="0 0 0" rpy="0 0 0" />
       <geometry>
-        <!-- <box size="${bb_size_x} ${bb_size_y} ${bb_size_z}" /> -->
-        <mesh filename="package://mobipick_gazebo/meshes/collision/relay.stl" />
+         <box size="${bb_size_x} ${bb_size_y} ${bb_size_z}" />
+        <!--<mesh filename="package://mobipick_gazebo/meshes/collision/relay.stl" />-->
       </geometry>
     </collision>
