Commit message: Adjust robotiq fingertip position

File: mobipick_description/urdf/robotiq_2f_140/robotiq_arg2f_140_model_macro.xacro (robot description, xacro)
@@ -168,5 +168,5 @@
       <axis xyz="1 0 0" />
       <limit lower="0" upper="0.725" velocity="2.0" effort="1000" />
-    <mimic joint="finger_joint" multiplier="-1" offset="0" />
+    <mimic joint="${prefix}finger_joint" multiplier="-1" offset="0" />
     </joint>
     <xacro:finger_joints prefix="${prefix}" fingerprefix="right" reflect="-1.0"/>

File: mobipick_description/urdf/robotiq_2f_140/robotiq_fingertips_65mm.xacro (robot description, xacro)
@@ -5,5 +5,5 @@
       <inertial>
         <!-- <origin xyz="0 32.3E-03 -3.4587E-03" rpy="0 0 0" /> -->
-        <origin xyz="0 0 0" rpy="0 0 0" />
+        <origin xyz="0 0.0323 -0.003459" rpy="${pi} ${0.5 * pi} ${0.5 * pi}" />
         <mass value="3.3455E-2" />
         <inertia ixx="13.66E-6"
@@ -33,5 +33,5 @@
   <xacro:macro name="fingertip_joint" params="prefix fingerprefix">
     <joint name="${prefix}${fingerprefix}_fingertip_joint" type="fixed">
-      <origin xyz="0 0 0" rpy="0 0 0" />
+      <origin xyz="0 0.013513 -0.018469" rpy="0 0 0" />
       <parent link="${prefix}${fingerprefix}_inner_finger" />
       <child link="${prefix}${fingerprefix}_robotiq_fingertip_65mm" />

Commit message: Robotiq gripper: add missing prefix

File: mobipick_description/urdf/robotiq_2f_140/robotiq_arg2f_140_model_macro.xacro (robot description, xacro)
@@ -162,5 +162,5 @@
   </xacro:macro>
   <xacro:macro name="right_outer_knuckle_joint" params="prefix">
-    <joint name="right_outer_knuckle_joint" type="revolute">
+    <joint name="${prefix}right_outer_knuckle_joint" type="revolute">
       <origin xyz="0 0.030601 0.054905" rpy="${pi / 2 + .725} 0 ${pi}" />
       <parent link="${prefix}robotiq_arg2f_base_link" />

Commit message: fixed bugs related to the limits of the passive joints of the gripper

File: mobipick_description/urdf/robotiq_2f_140/robotiq_arg2f_140_model_macro.xacro (robot description, xacro)
@@ -136,5 +136,5 @@
       <child link="${prefix}${fingerprefix}_inner_knuckle" />
       <axis xyz="1 0 0" />
-      <limit lower="0" upper="0.8757" velocity="2.0" effort="1000" />
+      <limit lower="-0.8757" upper="0" velocity="2.0" effort="1000" />
       <mimic joint="${prefix}finger_joint" multiplier="-1" offset="0" />
     </joint>
@@ -167,5 +167,5 @@
       <child link="${prefix}right_outer_knuckle" />
       <axis xyz="1 0 0" />
-      <limit lower="0" upper="0.725" velocity="2.0" effort="1000" />
+      <limit lower="-0.725" upper="0" velocity="2.0" effort="1000" />
     <mimic joint="${prefix}finger_joint" multiplier="-1" offset="0" />
     </joint>

Commit message: fixed limits of gripper joints taking into account the fingertips

File: mobipick_description/urdf/robotiq_2f_140/robotiq_arg2f_140_model_macro.xacro (robot description, xacro)
@@ -157,5 +157,5 @@
       <child link="${prefix}left_outer_knuckle" />
       <axis xyz="-1 0 0" />
-      <limit lower="0" upper="0.775" velocity="2.0" effort="1000" />
+      <limit lower="0" upper="0.755" velocity="2.0" effort="1000" />
     </joint>
     <xacro:finger_joints prefix="${prefix}" fingerprefix="left" reflect="1.0"/>
@@ -167,5 +167,5 @@
       <child link="${prefix}right_outer_knuckle" />
       <axis xyz="1 0 0" />
-      <limit lower="-0.725" upper="0" velocity="2.0" effort="1000" />
+      <limit lower="-0.755" upper="0" velocity="2.0" effort="1000" />
     <mimic joint="${prefix}finger_joint" multiplier="-1" offset="0" />
     </joint>

Commit message: robotiq: Remove backup files

File: mobipick_description/urdf/robotiq_2f_140/robotiq_arg2f_140_model_macro.xacro (robot description, xacro)
@@ -108,5 +108,5 @@
         <origin xyz="0 0 0" rpy="0 0 0" />
         <geometry>
-          <mesh filename="package://mobipick_description/meshes/robotiq_2f_140/robotiq_arg2f_${stroke}_inner_finger_ed.stl" />
+          <mesh filename="package://mobipick_description/meshes/robotiq_2f_140/robotiq_arg2f_${stroke}_inner_finger.stl" />
         </geometry>
         <material name="">
@@ -117,5 +117,5 @@
         <origin xyz="0 0 0" rpy="0 0 0" />
         <geometry>
-          <mesh filename="package://mobipick_description/meshes/robotiq_2f_140/robotiq_arg2f_${stroke}_inner_finger_ed.stl" />
+          <mesh filename="package://mobipick_description/meshes/robotiq_2f_140/robotiq_arg2f_${stroke}_inner_finger.stl" />
         </geometry>
       </collision>

Commit message: gripper: extract materials.xacro

File: mobipick_description/urdf/robotiq_2f_140/robotiq_arg2f_140_model_macro.xacro (robot description, xacro)
@@ -2,4 +2,6 @@
 <robot xmlns:xacro="http://ros.org/wiki/xacro">
   <xacro:include filename="$(find mobipick_description)/urdf/robotiq_2f_140/robotiq_arg2f_transmission.xacro" />
+  <!-- Import Rviz colors -->
+  <xacro:include filename="$(find mobipick_description)/urdf/robotiq_2f_140/materials.xacro" />
   <xacro:macro name="outer_knuckle" params="prefix fingerprefix stroke">
     <link name="${prefix}${fingerprefix}_outer_knuckle">
@@ -20,7 +22,5 @@
           <mesh filename="package://mobipick_description/meshes/robotiq_2f_140/robotiq_arg2f_${stroke}_outer_knuckle.stl" />
         </geometry>
-        <material name="">
-          <color rgba="0.792156862745098 0.819607843137255 0.933333333333333 1" />
-        </material>
+        <material name="robotiq_silver" />
       </visual>
       <collision>
@@ -50,7 +50,5 @@
           <mesh filename="package://mobipick_description/meshes/robotiq_2f_140/robotiq_arg2f_${stroke}_outer_finger.stl" />
         </geometry>
-        <material name="">
-          <color rgba="0.1 0.1 0.1 1" />
-        </material>
+        <material name="robotiq_almost_black" />
       </visual>
       <collision>
@@ -80,7 +78,5 @@
           <mesh filename="package://mobipick_description/meshes/robotiq_2f_140/robotiq_arg2f_${stroke}_inner_knuckle.stl" />
         </geometry>
-        <material name="">
-          <color rgba="0.1 0.1 0.1 1" />
-        </material>
+        <material name="robotiq_almost_black" />
       </visual>
       <collision>
@@ -110,7 +106,5 @@
           <mesh filename="package://mobipick_description/meshes/robotiq_2f_140/robotiq_arg2f_${stroke}_inner_finger.stl" />
         </geometry>
-        <material name="">
-          <color rgba="0.1 0.1 0.1 1" />
-        </material>
+        <material name="robotiq_almost_black" />
       </visual>
       <collision>

File: mobipick_description/urdf/robotiq_2f_140/robotiq_fingertips_65mm.xacro (robot description, xacro)
@@ -19,5 +19,5 @@
           <mesh filename="package://mobipick_description/meshes/robotiq_2f_140/robotiq_arg2f_${stroke}_fingertip_65mm.stl" />
         </geometry>
-        <material name="">
+        <material name="robotiq_light_grey /">
           <color rgba="0.5 0.5 0.5 1" />
         </material>

Commit message: urdf: Add gripper tool center point

File: mobipick_description/urdf/robotiq_2f_140/robotiq_arg2f_140_model_macro.xacro (robot description, xacro)
@@ -197,4 +197,11 @@
     <xacro:fingertip_joint prefix="${prefix}" fingerprefix="left"/>
     <xacro:fingertip_joint prefix="${prefix}" fingerprefix="right"/>
+    <!-- Tool Center Point: Center of the fingertips when gripper is closed -->
+    <joint name="${prefix}tcp_joint" type="fixed">
+      <origin xyz="0 0 0.1975" rpy="0 ${-pi/2} 0" />
+      <parent link="${prefix}robotiq_arg2f_base_link" />
+      <child link="${prefix}tcp" />
+    </joint>
+    <link name="${prefix}tcp" />
   </xacro:macro>
   <!-- GRASP HACK -->

Commit message: add grasp_fix_required xacro property to optionally disable gazebo grasp fix

File: mobipick_description/urdf/robotiq_2f_140/robotiq_arg2f_140_model_macro.xacro (robot description, xacro)
@@ -220,5 +220,8 @@
   </xacro:macro>
   <!-- GRASP HACK -->
-  <xacro:include filename="$(find mobipick_description)/urdf/robotiq_2f_140/gzplugin_grasp_fix.urdf.xacro"/>
-  <xacro:gzplugin_grasp_fix prefix="${prefix}"/>
+  <xacro:property name="grasp_fix_required" default="true" />
+  <xacro:if value="${grasp_fix_required}">
+    <xacro:include filename="$(find mobipick_description)/urdf/robotiq_2f_140/gzplugin_grasp_fix.urdf.xacro"/>
+    <xacro:gzplugin_grasp_fix prefix="${prefix}"/>
+  </xacro:if>
 </robot>
