Commit message: gripper fingers urdf: use box instead of mesh for collision as it produces less vibration of the fingers when grasping objects

File: mobipick_description/urdf/robotiq_2f_140/robotiq_fingertips_65mm.xacro (robot description, xacro)
@@ -23,7 +23,9 @@
       </visual>
       <collision>
-        <origin xyz="0 0 0" rpy="0 0 0" />
+        <origin xyz="0.00005 0.0325 -0.0035" rpy="0 0 0"/>
         <geometry>
-          <mesh filename="package://mobipick_description/meshes/robotiq_2f_140/robotiq_arg2f_${stroke}_fingertip_65mm.stl" />
+          <!-- <mesh filename="package://mobipick_description/meshes/robotiq_2f_140/robotiq_arg2f_${stroke}_fingertip_65mm.stl" /> -->
+          <!-- using box instead of mesh for collision produces less vibration of the fingers when grasping objects -->
+          <box size="0.0271 0.065 0.007"/> <!-- values ok for stroke of 140, only? -->
         </geometry>
       </collision>
