Commit message: Move materials to common_properties.urdf.xacro

File: mobipick_description/urdf/common_properties.urdf.xacro (robot description, xacro)
@@ -8,4 +8,9 @@
     <material name="white">
       <color rgba="1 1 1 1"/>
+    </material>
+  </xacro:property>
+  <xacro:property name="material_almost_white">
+    <material name="almost_white">
+      <color rgba="0.9 0.9 0.9 1" />
     </material>
   </xacro:property>
@@ -30,3 +35,13 @@
     </material>
   </xacro:property>
+  <xacro:property name="material_aluminum">
+    <material name="aluminum">
+      <color rgba="0.8 0.8 0.8 1" />
+    </material>
+  </xacro:property>
+  <xacro:property name="material_silver">
+    <material name="silver">
+      <color rgba="0.79 0.82 0.93 1" />
+    </material>
+  </xacro:property>
 </robot>

File: mobipick_description/urdf/mir_100/mir_100_v1.urdf.xacro (robot description, xacro)
@@ -1,7 +1,7 @@
 <?xml version="1.0"?>
 <robot xmlns:xacro="http://ros.org/wiki/xacro">
+  <xacro:include filename="$(find mobipick_description)/urdf/common_properties.urdf.xacro" />
   <xacro:include filename="$(find mobipick_description)/urdf/mir_100/mir_100.transmission.xacro" />
   <xacro:include filename="$(find mobipick_description)/urdf/mir_100/mir_100.gazebo.xacro" />
-  <xacro:include filename="$(find mobipick_description)/urdf/mir_100/materials.xacro" />
   <!-- <xacro:property name="pi" value="3.14159265" /> -->
   <xacro:property name="deg_to_rad" value="0.017453293" />
@@ -48,5 +48,5 @@
           <mesh filename="package://mobipick_description/meshes/mir_100/visual/actuated_wheel.stl" />
         </geometry>
-        <material name="mir_dark_grey" />
+        <xacro:insert_block name="material_dark_grey" />
       </visual>
       <collision>
@@ -80,5 +80,5 @@
           <mesh filename="package://mobipick_description/meshes/mir_100/visual/caster_wheel_base.stl" />
         </geometry>
-        <material name="mir_silver" />
+        <xacro:insert_block name="material_silver" />
       </visual>
       <collision>
@@ -111,5 +111,5 @@
           <mesh filename="package://mobipick_description/meshes/mir_100/visual/caster_wheel.stl" />
         </geometry>
-        <material name="mir_dark_grey" />
+        <xacro:insert_block name="material_dark_grey" />
       </visual>
       <collision>
@@ -181,5 +181,5 @@
           <mesh filename="package://mobipick_description/meshes/mir_100/visual/mir_100_base.stl" />
         </geometry>
-        <material name="mir_white" />
+        <xacro:insert_block name="material_white" />
       </visual>
       <collision>

File: mobipick_description/urdf/robotiq_2f_140/robotiq_arg2f_140_model_macro.xacro (robot description, xacro)
@@ -1,7 +1,6 @@
 <?xml version="1.0"?>
 <robot xmlns:xacro="http://ros.org/wiki/xacro">
+  <xacro:include filename="$(find mobipick_description)/urdf/common_properties.urdf.xacro" />
   <xacro:include filename="$(find mobipick_description)/urdf/robotiq_2f_140/robotiq_arg2f_transmission.xacro" />
-  <!-- Import Rviz colors -->
-  <xacro:include filename="$(find mobipick_description)/urdf/robotiq_2f_140/materials.xacro" />
   <xacro:macro name="outer_knuckle" params="prefix fingerprefix stroke">
     <link name="${prefix}${fingerprefix}_outer_knuckle">
@@ -22,5 +21,5 @@
           <mesh filename="package://mobipick_description/meshes/robotiq_2f_140/robotiq_arg2f_${stroke}_outer_knuckle.stl" />
         </geometry>
-        <material name="robotiq_silver" />
+        <xacro:insert_block name="material_silver" />
       </visual>
       <collision>
@@ -53,5 +52,5 @@
           <mesh filename="package://mobipick_description/meshes/robotiq_2f_140/robotiq_arg2f_${stroke}_outer_finger.stl" />
         </geometry>
-        <material name="robotiq_almost_black" />
+        <xacro:insert_block name="material_black" />
       </visual>
       <collision>
@@ -84,5 +83,5 @@
           <mesh filename="package://mobipick_description/meshes/robotiq_2f_140/robotiq_arg2f_${stroke}_inner_knuckle.stl" />
         </geometry>
-        <material name="robotiq_almost_black" />
+        <xacro:insert_block name="material_black" />
       </visual>
       <collision>
@@ -115,5 +114,5 @@
           <mesh filename="package://mobipick_description/meshes/robotiq_2f_140/robotiq_arg2f_${stroke}_inner_finger.stl" />
         </geometry>
-        <material name="robotiq_almost_black" />
+        <xacro:insert_block name="material_black" />
       </visual>
       <collision>

File: mobipick_description/urdf/sensors/gripper_cam.urdf.xacro (robot description, xacro)
@@ -20,7 +20,5 @@
           <mesh filename="package://mobipick_description/meshes/sensors/sensor_mount.stl" scale="0.001 0.001 0.001" />
         </geometry>
-        <material name="almost_white">
-          <color rgba="0.9 0.9 0.9 1" />
-        </material>
+        <xacro:insert_block name="material_almost_white" />
       </visual>
       <collision>

File: mobipick_description/urdf/structure/mobipick_structure.urdf.xacro (robot description, xacro)
@@ -1,5 +1,5 @@
 <?xml version="1.0"?>
 <robot xmlns:xacro="http://ros.org/wiki/xacro">
-  <xacro:include filename="$(find mobipick_description)/urdf/structure/materials.xacro" />
+  <xacro:include filename="$(find mobipick_description)/urdf/common_properties.urdf.xacro" />
   <!-- <xacro:property name="pi" value="3.14159265" /> -->
   <xacro:macro name="structure" params="prefix height">
@@ -21,5 +21,5 @@
           <mesh filename="package://mobipick_description/meshes/structure/visual/part_down.stl" />
         </geometry>
-        <material name="structure_aluminum" />
+        <xacro:insert_block name="material_aluminum" />
       </visual>
       <collision>
@@ -50,5 +50,5 @@
           <mesh filename="package://mobipick_description/meshes/structure/visual/part_up.stl" />
         </geometry>
-        <material name="structure_aluminum" />
+        <xacro:insert_block name="material_aluminum" />
       </visual>
       <collision>
@@ -79,5 +79,5 @@
           <mesh filename="package://mobipick_description/meshes/structure/visual/pedestal.stl" />
         </geometry>
-        <material name="structure_aluminum" />
+        <xacro:insert_block name="material_aluminum" />
       </visual>
       <collision>

Commit message: Remove "pi" definition from xacro
Seems to be available by default...

File: mobipick_description/urdf/common_properties.urdf.xacro (robot description, xacro)
@@ -4,5 +4,4 @@
  -->
 <robot name="xacro_properties" xmlns:xacro="http://ros.org/wiki/xacro">
-  <xacro:property name="M_PI" value="3.1415926535897931" /> <!-- TODO: pi -->
   <xacro:property name="material_white">
     <material name="white">

File: mobipick_description/urdf/mir_100/mir_100_v1.urdf.xacro (robot description, xacro)
@@ -4,5 +4,4 @@
   <xacro:include filename="$(find mobipick_description)/urdf/mir_100/mir_100.transmission.xacro" />
   <xacro:include filename="$(find mobipick_description)/urdf/mir_100/mir_100.gazebo.xacro" />
-  <!-- <xacro:property name="pi" value="3.14159265" /> -->
   <xacro:property name="deg_to_rad" value="0.017453293" />
   <xacro:property name="mir_100_base_mass" value="58.0" />

File: mobipick_description/urdf/structure/mobipick_structure.urdf.xacro (robot description, xacro)
@@ -2,5 +2,4 @@
 <robot xmlns:xacro="http://ros.org/wiki/xacro">
   <xacro:include filename="$(find mobipick_description)/urdf/common_properties.urdf.xacro" />
-  <!-- <xacro:property name="pi" value="3.14159265" /> -->
   <xacro:macro name="structure" params="prefix height">
     <link name="${prefix}part_down">

File: mobipick_description/urdf/ur5/ur5.urdf.xacro (robot description, xacro)
@@ -3,5 +3,4 @@
   <xacro:include filename="$(find mobipick_description)/urdf/ur5/ur.transmission.xacro" />
   <xacro:include filename="$(find mobipick_description)/urdf/ur5/ur.gazebo.xacro" />
-  <!-- <xacro:property name="pi" value="3.14159265" /> -->
   <!-- Inertia parameters -->
   <xacro:property name="base_mass" value="0.300" />  <!-- This mass might be incorrect, the others are from the UR5 FAQ -->

Commit message: Unify inertial xacro macros

File: mobipick_description/urdf/common_properties.urdf.xacro (robot description, xacro)
@@ -4,4 +4,5 @@
  -->
 <robot name="xacro_properties" xmlns:xacro="http://ros.org/wiki/xacro">
+  <!-- #################### RViz materials #################### -->
   <xacro:property name="material_white">
     <material name="white">
@@ -44,3 +45,32 @@
     </material>
   </xacro:property>
+  <!-- #################### inertials with origin #################### -->
+  <!-- see https://secure.wikimedia.org/wikipedia/en/wiki/List_of_moment_of_inertia_tensors -->
+  <xacro:macro name="sphere_inertial" params="radius mass *origin">
+    <inertial>
+      <mass value="${mass}" />
+      <xacro:insert_block name="origin" />
+      <inertia ixx="${0.4 * mass * radius * radius}" ixy="0.0" ixz="0.0"
+        iyy="${0.4 * mass * radius * radius}" iyz="0.0"
+        izz="${0.4 * mass * radius * radius}" />
+    </inertial>
+  </xacro:macro>
+  <xacro:macro name="cylinder_inertial" params="radius length mass *origin">
+    <inertial>
+      <mass value="${mass}" />
+      <xacro:insert_block name="origin" />
+      <inertia ixx="${0.0833333 * mass * (3 * radius * radius + length * length)}" ixy="0.0" ixz="0.0"
+        iyy="${0.0833333 * mass * (3 * radius * radius + length * length)}" iyz="0.0"
+        izz="${0.5 * mass * radius * radius}" />
+    </inertial>
+  </xacro:macro>
+  <xacro:macro name="box_inertial" params="x y z mass *origin">
+    <inertial>
+      <mass value="${mass}" />
+      <xacro:insert_block name="origin" />
+      <inertia ixx="${0.0833333 * mass * (y*y + z*z)}" ixy="0.0" ixz="0.0"
+        iyy="${0.0833333 * mass * (x*x + z*z)}" iyz="0.0"
+        izz="${0.0833333 * mass * (x*x + y*y)}" />
+    </inertial>
+  </xacro:macro>
 </robot>

File: mobipick_description/urdf/mir_100/mir_100_v1.urdf.xacro (robot description, xacro)
@@ -21,25 +21,9 @@
   <xacro:property name="mir_100_caster_wheel_base_dy" value="0.203" />
   <xacro:property name="mir_100_caster_wheel_base_dz" value="${mir_100_caster_wheel_radius-mir_100_caster_wheel_dz}" />
-  <xacro:macro name="cylinder_inertia" params="m r h">
-    <inertia ixx="${m*(3*r*r+h*h)/12}" ixy="0" ixz="0" iyy="${m*(3*r*r+h*h)/12}" iyz="0" izz="${m*r*r/2}"/>
-  </xacro:macro>
-  <xacro:macro name="box_inertia" params="m x y z">
-    <inertia ixx="${m*(y*y+z*z)/12}" ixy="0" ixz="0" iyy="${m*(x*x+z*z)/12}" iyz="0" izz="${m*(x*x+y*y)/12}"/>
-  </xacro:macro>
   <xacro:macro name="actuated_wheel_link" params="prefix locationprefix">
     <link name="${prefix}${locationprefix}_act_wheel">
-      <inertial>
-        <!-- <origin xyz="0 0 0" rpy="${0.5 * pi} ${0.5 * pi} 0" /> -->
+      <xacro:cylinder_inertial mass="${mir_100_act_wheel_mass}" radius="${mir_100_act_wheel_radius}" length="${mir_100_act_wheel_width}">
         <origin xyz="0 0 0" rpy="${0.5 * pi} 0 0" />
-        <mass value="${mir_100_act_wheel_mass}" />
-        <!-- <inertia
-            ixx="0.0021285829616"
-            ixy="0"
-            ixz="0"
-            iyy="0.0011566983393"
-            iyz="0"
-            izz="0.0011566983393" /> -->
-        <xacro:cylinder_inertia m="${mir_100_act_wheel_mass}" r="${mir_100_act_wheel_radius}" h="${mir_100_act_wheel_width}" />
-      </inertial>
+      </xacro:cylinder_inertial>
       <visual>
         <origin xyz="0 0 0" rpy="0 0 0" />
@@ -92,17 +76,7 @@
     </gazebo>
     <link name="${prefix}${locationprefix}_caster_wheel">
-      <inertial>
-        <!-- <origin xyz="0 0 0" rpy="${0.5 * pi} ${0.5 * pi} 0" /> -->
+      <xacro:cylinder_inertial mass="${mir_100_caster_wheel_mass}" radius="${mir_100_caster_wheel_radius}" length="${mir_100_caster_wheel_width}">
         <origin xyz="0 0 0" rpy="${0.5 * pi} 0 0" />
-        <mass value="${mir_100_caster_wheel_mass}" />
-        <!-- <inertia
-            ixx="0.0021285829616"
-            ixy="0"
-            ixz="0"
-            iyy="0.0011566983393"
-            iyz="0"
-            izz="0.0011566983393" /> -->
-        <xacro:cylinder_inertia m="${mir_100_caster_wheel_mass}" r="${mir_100_caster_wheel_radius}" h="${mir_100_caster_wheel_width}" />
-      </inertial>
+      </xacro:cylinder_inertial>
       <visual>
         <origin xyz="0 0 0" rpy="0 0 0" />
@@ -170,9 +144,7 @@
     </joint>
     <link name="${prefix}base_link">
-      <inertial>
+      <xacro:box_inertial mass="${mir_100_base_mass}" x="0.9" y="0.58" z="0.3">
         <origin xyz="${mir_100_act_wheel_dx} 0 0.20" rpy="0 0 0" />
-        <mass value="${mir_100_base_mass}" />
-        <xacro:box_inertia m="${mir_100_base_mass}" x="0.9" y="0.58" z="0.3" />
-      </inertial>
+      </xacro:box_inertial>
       <visual>
         <origin xyz="${mir_100_act_wheel_dx} 0 0" rpy="0 0 0" />

File: mobipick_description/urdf/sensors/gripper_cam.urdf.xacro (robot description, xacro)
@@ -64,9 +64,7 @@
         </geometry>
       </collision>
-      <inertial>
-        <mass value="${astra_s_mass}" />
+      <xacro:box_inertial mass="${astra_s_mass}" x="0.0325" y="0.12" z="0.0375">
         <origin xyz="${-0.0325 / 2} ${-astra_cam_py} 0.0" />
-        <xacro:box_inertia m="${astra_s_mass}" x="0.0325" y="0.12" z="0.0375" />
-      </inertial>
+      </xacro:box_inertial>
     </link>
     <gazebo reference="${camera_name}_link">

File: mobipick_description/urdf/ur5/ur5.urdf.xacro (robot description, xacro)
@@ -1,4 +1,5 @@
 <?xml version="1.0"?>
 <robot xmlns:xacro="http://ros.org/wiki/xacro">
+  <xacro:include filename="$(find mobipick_description)/urdf/common_properties.urdf.xacro" />
   <xacro:include filename="$(find mobipick_description)/urdf/ur5/ur.transmission.xacro" />
   <xacro:include filename="$(find mobipick_description)/urdf/ur5/ur.gazebo.xacro" />
@@ -58,13 +59,4 @@
   <xacro:property name="forearm_radius" value="0.040" />    <!-- manually measured -->
   <xacro:property name="wrist_radius" value="0.045" />      <!-- manually measured -->
-  <xacro:macro name="cylinder_inertial" params="radius length mass *origin">
-    <inertial>
-      <mass value="${mass}" />
-      <xacro:insert_block name="origin" />
-      <inertia ixx="${0.0833333 * mass * (3 * radius * radius + length * length)}" ixy="0.0" ixz="0.0"
-        iyy="${0.0833333 * mass * (3 * radius * radius + length * length)}" iyz="0.0"
-        izz="${0.5 * mass * radius * radius}" />
-    </inertial>
-  </xacro:macro>
   <xacro:macro name="ur5_robot" params="prefix joint_limited">
     <link name="${prefix}base_link" >

Commit message: Add laser scanners

File: mobipick_description/urdf/common_properties.urdf.xacro (robot description, xacro)
@@ -8,4 +8,9 @@
     <material name="white">
       <color rgba="1 1 1 1"/>
+    </material>
+  </xacro:property>
+  <xacro:property name="material_yellow">
+    <material name="yellow">
+      <color rgba="${255/255} ${226/255} ${0/255} 1"/>
     </material>
   </xacro:property>

File: mobipick_description/urdf/mir_100/mir_100_v1.urdf.xacro (robot description, xacro)
@@ -3,4 +3,5 @@
   <xacro:include filename="$(find mobipick_description)/urdf/common_properties.urdf.xacro" />
   <xacro:include filename="$(find mobipick_description)/urdf/sensors/imu.gazebo.urdf.xacro" />
+  <xacro:include filename="$(find mobipick_description)/urdf/sensors/sick_s300.urdf.xacro" />
   <xacro:include filename="$(find mobipick_description)/urdf/mir_100/mir_100.transmission.xacro" />
   <xacro:include filename="$(find mobipick_description)/urdf/mir_100/mir_100.gazebo.xacro" />
@@ -174,4 +175,19 @@
     <link name="${prefix}imu_link" />
     <xacro:imu_gazebo link="${prefix}imu_link" imu_topic="imu_data" update_rate="50.0" stdev="${imu_stdev}" />
+    <!-- Laser scanners -->
+    <joint name="${prefix}base_link_to_front_laser_joint" type="fixed">
+      <parent link="${prefix}base_link" />
+      <child link="${prefix}front_laser_link" />
+      <!-- on real MiR (depends on calibration): <origin xyz="0.416 0.243 0.200" rpy="0.0 0.0 0.795" /> -->
+      <origin xyz="0.4288 0.2358 0.1914" rpy="${-pi} 0.0 ${pi/4}" />  <!-- from visually matching up the meshes of the MiR and the laser scanner -->
+    </joint>
+    <xacro:sick_s300 link="${prefix}front_laser_link" topic="f_scan" />
+    <joint name="${prefix}base_link_to_back_laser_joint" type="fixed">
+      <parent link="${prefix}base_link" />
+      <child link="${prefix}back_laser_link" />
+      <!-- on real MiR: <origin xyz="-0.360 -0.252 0.200" rpy="0.0 0.0 -2.348" /> -->
+      <origin xyz="-0.3548 -0.2352 0.1914" rpy="${-pi} 0.0 ${-0.75 * pi}" />  <!-- from visually matching up the meshes of the MiR and the laser scanner -->
+    </joint>
+    <xacro:sick_s300 link="${prefix}back_laser_link" topic="b_scan" />
     <!-- wheels -->
     <xacro:actuated_wheel_link prefix="${prefix}" locationprefix="left"/>
