Commit message: Fix UR5 inertias

File: mobipick_description/urdf/ur5/ur5.urdf.xacro (robot description, xacro)
@@ -5,11 +5,11 @@
   <!-- <xacro:property name="pi" value="3.14159265" /> -->
   <!-- Inertia parameters -->
-  <xacro:property name="base_mass" value="4.0" />  <!-- This mass might be incorrect -->
+  <xacro:property name="base_mass" value="0.300" />  <!-- This mass might be incorrect, the others are from the UR5 FAQ -->
   <xacro:property name="shoulder_mass" value="3.7000" />
   <xacro:property name="upper_arm_mass" value="8.3930" />
-  <xacro:property name="forearm_mass" value="2.2750" />
+  <xacro:property name="forearm_mass" value="2.33" />
   <xacro:property name="wrist_1_mass" value="1.2190" />
   <xacro:property name="wrist_2_mass" value="1.2190" />
-  <xacro:property name="wrist_3_mass" value="0.1879" />
+  <xacro:property name="wrist_3_mass" value="0.1897" />
   <xacro:property name="shoulder_cog" value="0.0 0.00193 -0.02561" />
   <xacro:property name="upper_arm_cog" value="0.0 -0.024201 0.2125" />
@@ -83,5 +83,5 @@
         </geometry>
       </collision>
-      <xacro:cylinder_inertial radius="0.06" length="0.05" mass="${base_mass}">
+      <xacro:cylinder_inertial radius="0.075" length="0.024" mass="${base_mass}">
         <origin xyz="0.0 0.0 0.0" rpy="0 0 0" />
       </xacro:cylinder_inertial>
@@ -114,5 +114,5 @@
         </geometry>
       </collision>
-      <xacro:cylinder_inertial radius="0.06" length="0.15" mass="${shoulder_mass}">
+      <xacro:cylinder_inertial radius="0.06" length="0.14" mass="${shoulder_mass}">
         <origin xyz="0.0 0.0 0.0" rpy="0 0 0" />
       </xacro:cylinder_inertial>
@@ -207,5 +207,5 @@
         </geometry>
       </collision>
-      <xacro:cylinder_inertial radius="0.6" length="0.12" mass="${wrist_1_mass}">
+      <xacro:cylinder_inertial radius="0.06" length="0.12" mass="${wrist_1_mass}">
         <origin xyz="0.0 0.0 0.0" rpy="0 0 0" />
       </xacro:cylinder_inertial>
@@ -238,5 +238,5 @@
         </geometry>
       </collision>
-      <xacro:cylinder_inertial radius="0.6" length="0.12" mass="${wrist_2_mass}">
+      <xacro:cylinder_inertial radius="0.06" length="0.12" mass="${wrist_2_mass}">
         <origin xyz="0.0 0.0 0.0" rpy="0 0 0" />
       </xacro:cylinder_inertial>
@@ -269,5 +269,5 @@
         </geometry>
       </collision>
-      <xacro:cylinder_inertial radius="0.6" length="0.12" mass="${wrist_3_mass}">
+      <xacro:cylinder_inertial radius="0.04" length="0.04" mass="${wrist_3_mass}">
         <origin xyz="0.0 0.0 0.0" rpy="0 0 0" />
       </xacro:cylinder_inertial>

Commit message: Limit joint limits (solves planning problems)
This commit restricts the joints to the actually reachable angles.
Without this commit, planning between the following joint angles times
out with a "plan not found" error, even though there is a valid IK
solution for them:

   joint_group_positions{-2.811, 0.336, -0.666, -1.459, 1.306, 1.778};
   joint_group_positions = {-2.938, 3.007, -0.999, -0.685, -1.334, -1.242};

The reason is that it's impossible for the ur5_shoulder_lift_joint to go
from 0.336 to 3.007 without colliding with the robot structure, even though
both joint angles are technically within the joint angles of the robot.
Similarly, the ur5_elbow_joint can never reach values outside of [-pi,
pi] without self-collision. This makes the planning space discontinuous.

After this commit, the planning for the joint targets above now fails
immediately instead of timing out, because the joint angles are outside
the joint limits. Also, IK will now never return an unreachable set of
joint angles.

File: mobipick_description/urdf/ur5/ur5.urdf.xacro (robot description, xacro)
@@ -114,9 +114,12 @@
       <origin xyz="0.0 ${shoulder_offset} 0.0" rpy="0.0 ${pi / 2.0} 0.0" />
       <axis xyz="0 1 0" />
-      <xacro:unless value="${joint_limited}">
-        <limit lower="${-2.0 * pi}" upper="${2.0 * pi}" effort="150.0" velocity="3.15"/>
-      </xacro:unless>
-      <xacro:if value="${joint_limited}">
-        <limit lower="${-pi}" upper="${pi}" effort="150.0" velocity="3.15"/>
+      <!-- Reachable joint angles are limited by the robot structure to these
+           values. It's important to restrict the joint angles, otherwise the
+           planning space is discontinuous. -->
+      <xacro:unless value="${joint_limited}">
+        <limit lower="${-pi - 0.82}" upper="0.82" effort="150.0" velocity="3.15"/>
+      </xacro:unless>
+      <xacro:if value="${joint_limited}">
+        <limit lower="${-pi - 0.82}" upper="0.82" effort="150.0" velocity="3.15"/>
       </xacro:if>
       <dynamics damping="0.0" friction="0.0"/>
@@ -146,5 +149,8 @@
       <axis xyz="0 1 0" />
       <xacro:unless value="${joint_limited}">
-        <limit lower="${-2.0 * pi}" upper="${2.0 * pi}" effort="150.0" velocity="3.15"/>
+        <!-- This joint has to be limited to the reachable angles even in the
+             non-joint-limited version, otherwise the planning space is
+             discontinuous. -->
+        <limit lower="${-pi}" upper="${pi}" effort="150.0" velocity="3.15"/>
       </xacro:unless>
       <xacro:if value="${joint_limited}">
