Commit message: Fix typo: measurment -> measurement

File: mobipick_description/urdf/robotiq_ft_300/robotiq_ft_300.urdf.xacro (robot description, xacro)
@@ -33,5 +33,5 @@
         </link>
         <!-- virtual measurement frame -->
-        <joint name="${prefix}measurment_joint" type="fixed" >
+        <joint name="${prefix}measurement_joint" type="fixed" >
             <origin xyz="0 0 0.01625" rpy="0 0 0" />
             <parent link="${prefix}fts_robotside" />

File: mobipick_description/urdf/robotiq_ft_300/robotiq_fts150.urdf.xacro (robot description, xacro)
@@ -30,5 +30,5 @@
         </link>
         <!-- virtual measurement frame -->
-        <joint name="${prefix}measurment_joint" type="fixed" >
+        <joint name="${prefix}measurement_joint" type="fixed" >
             <origin xyz="0 0 0.01625" rpy="0 0 0" />
             <parent link="${prefix}fts_robotside" />

Commit message: ft_sensor: Fix whitespace

File: mobipick_description/urdf/robotiq_ft_300/robotiq_ft_300.urdf.xacro (robot description, xacro)
@@ -1,49 +1,49 @@
 <?xml version="1.0"?>
 <robot xmlns:xacro="http://ros.org/wiki/xacro" name="robotiq_ft_300">
-    <xacro:macro name="robotiq_ft_300" params="parent prefix *origin">
-        <!-- mount the fts to the robot -->
-        <joint name="${prefix}fts_fix" type="fixed" >
-            <!--In most cases origin would be flange adapter plate: <origin xyz="0 0 0.009" rpy="0 0 0"/> /-->
-            <xacro:insert_block name="origin" />
-            <parent link="${parent}" />
-            <child link="${prefix}fts_robotside" />
-        </joint>
-        <link name="${prefix}fts_robotside">
-            <inertial>
-                <origin xyz="0 0 0.01875" rpy="0 0 0"/>
-                <mass value="0.3"/>
-                <!-- <inertia ixx="0.000140625" ixy="0" ixz="0" iyy="0.000140625" iyz="0" izz="0.000246094" /> /-->
-		<inertia ixx="0.000262" ixy="0" ixz="1" iyy="0.000265" iyz="1" izz="0.000219" />
-            </inertial>
-            <visual>
-                <origin xyz="0 0 0" rpy="0 0 0" />
-                <geometry>
-                    <mesh filename="package://mobipick_description/meshes/robotiq_ft_300/visual/robotiq_ft_300.stl"/>
-                </geometry>
-		<material name="">
-		  <color rgba="0.25 0.25 0.25 1" />
-		</material>
-            </visual>
-            <collision>
-                <origin xyz="0 0 0" rpy="0 0 0" />
-                <geometry>
-                    <mesh filename="package://mobipick_description/meshes/robotiq_ft_300/collision/robotiq_ft_300.stl"/>
-                </geometry>
-            </collision>
-        </link>
-        <!-- virtual measurement frame -->
-        <joint name="${prefix}measurement_joint" type="fixed" >
-            <origin xyz="0 0 0.01625" rpy="0 0 0" />
-            <parent link="${prefix}fts_robotside" />
-            <child link="${prefix}robotiq_force_torque_frame_id" />
-        </joint>
-        <link name="${prefix}robotiq_force_torque_frame_id"/>
-        <!-- toolside frame -->
-        <joint name="${prefix}toolside_joint" type="fixed" >
-            <origin xyz="0 0 0.0375" rpy="0 0 0" />
-            <parent link="${prefix}fts_robotside" />
-            <child link="${prefix}fts_toolside" />
-        </joint>
-        <link name="${prefix}fts_toolside"/>
-    </xacro:macro>
+  <xacro:macro name="robotiq_ft_300" params="parent prefix *origin">
+    <!-- mount the fts to the robot -->
+    <joint name="${prefix}fts_fix" type="fixed" >
+      <!--In most cases origin would be flange adapter plate: <origin xyz="0 0 0.009" rpy="0 0 0"/> /-->
+      <xacro:insert_block name="origin" />
+      <parent link="${parent}" />
+      <child link="${prefix}fts_robotside" />
+    </joint>
+    <link name="${prefix}fts_robotside">
+      <inertial>
+        <origin xyz="0 0 0.01875" rpy="0 0 0"/>
+        <mass value="0.3"/>
+        <!-- <inertia ixx="0.000140625" ixy="0" ixz="0" iyy="0.000140625" iyz="0" izz="0.000246094" /> /-->
+        <inertia ixx="0.000262" ixy="0" ixz="1" iyy="0.000265" iyz="1" izz="0.000219" />
+      </inertial>
+      <visual>
+        <origin xyz="0 0 0" rpy="0 0 0" />
+        <geometry>
+          <mesh filename="package://mobipick_description/meshes/robotiq_ft_300/visual/robotiq_ft_300.stl"/>
+        </geometry>
+        <material name="">
+          <color rgba="0.25 0.25 0.25 1" />
+        </material>
+      </visual>
+      <collision>
+        <origin xyz="0 0 0" rpy="0 0 0" />
+        <geometry>
+          <mesh filename="package://mobipick_description/meshes/robotiq_ft_300/collision/robotiq_ft_300.stl"/>
+        </geometry>
+      </collision>
+    </link>
+    <!-- virtual measurement frame -->
+    <joint name="${prefix}measurement_joint" type="fixed" >
+      <origin xyz="0 0 0.01625" rpy="0 0 0" />
+      <parent link="${prefix}fts_robotside" />
+      <child link="${prefix}robotiq_force_torque_frame_id" />
+    </joint>
+    <link name="${prefix}robotiq_force_torque_frame_id"/>
+    <!-- toolside frame -->
+    <joint name="${prefix}toolside_joint" type="fixed" >
+      <origin xyz="0 0 0.0375" rpy="0 0 0" />
+      <parent link="${prefix}fts_robotside" />
+      <child link="${prefix}fts_toolside" />
+    </joint>
+    <link name="${prefix}fts_toolside"/>
+  </xacro:macro>
 </robot>

Commit message: ft_sensor: Add gazebo color

File: mobipick_description/urdf/robotiq_ft_300/robotiq_ft_300.urdf.xacro (robot description, xacro)
@@ -32,4 +32,7 @@
       </collision>
     </link>
+    <gazebo reference="${prefix}fts_robotside">
+      <material>Gazebo/FlatBlack</material>
+    </gazebo>
     <!-- virtual measurement frame -->
     <joint name="${prefix}measurement_joint" type="fixed" >

Commit message: URDF: Rotate FT sensor to match real cable

File: mobipick_description/urdf/robotiq_ft_300/robotiq_ft_300.urdf.xacro (robot description, xacro)
@@ -17,5 +17,5 @@
       </inertial>
       <visual>
-        <origin xyz="0 0 0" rpy="0 0 0" />
+        <origin xyz="0 0 0" rpy="0 0 ${pi/2}" />
         <geometry>
           <mesh filename="package://mobipick_description/meshes/robotiq_ft_300/visual/robotiq_ft_300.stl"/>
@@ -26,5 +26,5 @@
       </visual>
       <collision>
-        <origin xyz="0 0 0" rpy="0 0 0" />
+        <origin xyz="0 0 0" rpy="0 0 ${pi/2}" />
         <geometry>
           <mesh filename="package://mobipick_description/meshes/robotiq_ft_300/collision/robotiq_ft_300.stl"/>
