Commit message: Use ${xtion_cam_py}

File: mobipick_description/urdf/sensors/dual_xtions.urdf.xacro (robot description, xacro)
@@ -25,5 +25,5 @@
       <parent link="dual_xtion_mount_link" />
       <child link="dual_xtion_bottom_link" />
-      <origin xyz="0.045 0.069 0.032" rpy="0 -0.262 0" />
+      <origin xyz="0.045 ${xtion_cam_py} 0.032" rpy="0 -0.262 0" />
     </joint>
     <sensor_xtion camera_name="dual_xtion_bottom" />
@@ -31,5 +31,5 @@
       <parent link="dual_xtion_mount_link" />
       <child link="dual_xtion_top_link" />
-      <origin xyz="0.045 0.069 -0.032" rpy="0 0.262 0" />
+      <origin xyz="0.045 ${xtion_cam_py} -0.032" rpy="0 0.262 0" />
     </joint>
     <sensor_xtion camera_name="dual_xtion_top" />

Commit message: dual_xtions: Switch top + bottom xtion

File: mobipick_description/urdf/sensors/dual_xtions.urdf.xacro (robot description, xacro)
@@ -25,5 +25,5 @@
       <parent link="dual_xtion_mount_link" />
       <child link="dual_xtion_bottom_link" />
-      <origin xyz="0.045 ${xtion_cam_py} 0.032" rpy="0 -0.262 0" />
+      <origin xyz="0.045 ${xtion_cam_py} -0.032" rpy="0 0.262 0" />
     </joint>
     <sensor_xtion camera_name="dual_xtion_bottom" />
@@ -31,5 +31,5 @@
       <parent link="dual_xtion_mount_link" />
       <child link="dual_xtion_top_link" />
-      <origin xyz="0.045 ${xtion_cam_py} -0.032" rpy="0 0.262 0" />
+      <origin xyz="0.045 ${xtion_cam_py} 0.032" rpy="0 -0.262 0" />
     </joint>
     <sensor_xtion camera_name="dual_xtion_top" />

Commit message: dual_xtions: Add color, collision and inertial

File: mobipick_description/urdf/sensors/dual_xtions.urdf.xacro (robot description, xacro)
@@ -2,7 +2,4 @@
   <xacro:include filename="$(find mobipick_description)/urdf/common_properties.urdf.xacro" />
   <xacro:property name="dual_xtion_mount_mass" value="0.060" />
-  <xacro:property name="dual_xtion_mount_x" value="0.02" />   <!-- TODO HENDRIK -->
-  <xacro:property name="dual_xtion_mount_y" value="0.02" />   <!-- TODO HENDRIK -->
-  <xacro:property name="dual_xtion_mount_z" value="0.10" />   <!-- TODO HENDRIK -->
   <xacro:property name="xtion_mass" value="0.170" />
   <!-- distance between center of camera and camera_link -->
@@ -43,5 +40,22 @@
           <mesh scale="0.001 0.001 0.001" filename="package://mobipick_description/meshes/sensors/peotrac_mount.stl" />
         </geometry>
+        <xacro:insert_block name="material_black" />
       </visual>
+      <collision>
+        <origin xyz="0 0 0" rpy="0 0 0" />
+        <geometry>
+          <mesh scale="0.001 0.001 0.001" filename="package://mobipick_description/meshes/sensors/peotrac_mount.stl" />
+        </geometry>
+      </collision>
+      <inertial>
+        <mass value="${dual_xtion_mount_mass}" />
+        <origin xyz="0.0 0.015565191 0.014843559" rpy="0 0 0" />
+        <inertia ixx="${dual_xtion_mount_mass * 0.00054183681}"
+                 ixy="${dual_xtion_mount_mass * -0.0000000014037452}"
+                 ixz="${dual_xtion_mount_mass * -0.0000000034183191}"
+                 iyy="${dual_xtion_mount_mass * 0.00081506484}"
+                 iyz="${dual_xtion_mount_mass * 0.00012522968}"
+                 izz="${dual_xtion_mount_mass * 0.0008327177}" />
+      </inertial>
     </link>
     <gazebo reference="dual_xtion_${side}_mount_link">
