Commit message: URDF: Update Astra pose, add mesh

File: mobipick_description/urdf/sensors/gripper_cam.urdf.xacro (robot description, xacro)
@@ -4,9 +4,9 @@
   <xacro:property name="astra_s_mass" value="0.300" />
   <!-- distance between center of camera and camera_link -->
-  <xacro:property name="astra_cam_py" value="0.057"/>
+  <xacro:property name="astra_cam_py" value="0.0485"/>
   <xacro:macro name="gripper_cam" params="">
     <sensor_mount />
     <joint name="gripper_cam_joint" type="fixed">
-      <origin xyz="0.01 0.10 ${-astra_cam_py}" rpy="${-pi/2} 0.0 ${-30 * (pi / 180)}" />
+      <origin xyz="-0.032 0.033 -0.065" rpy="${pi/2} ${pi/2} ${-pi/2}" />
       <parent link="sensor_mount_link"/>
       <child link="gripper_cam_link"/>
@@ -46,13 +46,7 @@
     <link name="${camera_name}_link">
       <visual>
-        <!--
-          <origin xyz="-0.01 -0.068 0" rpy="${-pi/2} -${pi} ${-pi/2}"/>
-          <geometry>
-            <mesh filename="package://turtlebot_description/meshes/sensors/astra.dae"/>
-          </geometry>
-        -->
-        <origin xyz="${-0.0325 / 2} ${-astra_cam_py} 0.0" />
+        <origin xyz="0 0 0" />
         <geometry>
-          <box size="0.0325 0.12 0.0375" />
+          <mesh filename="package://mobipick_description/meshes/sensors/astra_mini.stl"/>
         </geometry>
         <xacro:insert_block name="material_black" />

Commit message: Rename gripper_cam -> gripper_astra

File: mobipick_description/urdf/sensors/gripper_cam.urdf.xacro (robot description, xacro)
@@ -7,10 +7,10 @@
   <xacro:macro name="gripper_cam" params="">
     <sensor_mount />
-    <joint name="gripper_cam_joint" type="fixed">
+    <joint name="gripper_astra_joint" type="fixed">
       <origin xyz="-0.032 0.033 -0.065" rpy="${pi/2} ${pi/2} ${-pi/2}" />
       <parent link="sensor_mount_link"/>
-      <child link="gripper_cam_link"/>
+      <child link="gripper_astra_link"/>
     </joint>
-    <sensor_astra_mini_s camera_name="gripper_cam" />
+    <sensor_astra_mini_s camera_name="gripper_astra" />
   </xacro:macro>
   <xacro:macro name="sensor_mount">

Commit message: Update mesh + URDF to new sensor_mount

File: mobipick_description/urdf/sensors/gripper_cam.urdf.xacro (robot description, xacro)
@@ -2,4 +2,6 @@
   <xacro:include filename="$(find mobipick_description)/urdf/common_properties.urdf.xacro" />
   <xacro:property name="sensor_mount_mass" value="0.060" />
+  <xacro:property name="sensor_mount_bracket_mass" value="0.040" />
+  <xacro:property name="sensor_mount_pico_holder_mass" value="0.020" />
   <xacro:property name="astra_s_mass" value="0.300" />
   <!-- distance between center of camera and camera_link -->
@@ -29,14 +31,76 @@
       <inertial>
         <mass value="${sensor_mount_mass}" />
-        <origin xyz="0.012318905 0.040711384 -0.005891052" rpy="0 0 0" />
-        <inertia ixx="${sensor_mount_mass * 0.0017886943}"
-          ixy="${sensor_mount_mass * 0.0000058410139}"
-          ixz="${sensor_mount_mass * 0.00000052824433}"
-          iyy="${sensor_mount_mass * 0.00077641599}"
-          iyz="${sensor_mount_mass * -0.00037632235}"
-          izz="${sensor_mount_mass * 0.0011250528}" />
+        <origin xyz="-0.006815249 0.054455677 -0.011470736" rpy="0 0 0" />
+        <inertia ixx="${sensor_mount_mass * 0.0018998439}"
+          ixy="${sensor_mount_mass * 0.0000011290362}"
+          ixz="${sensor_mount_mass * -0.000004403006}"
+          iyy="${sensor_mount_mass * 0.0013046557}"
+          iyz="${sensor_mount_mass * 0.00004099457}"
+          izz="${sensor_mount_mass * 0.00062646503}" />
       </inertial>
     </link>
     <gazebo reference="sensor_mount_link">
+      <material>Gazebo/Grey</material>
+    </gazebo>
+    <joint name="sensor_mount_bracket_joint" type="fixed">
+      <origin xyz="0 0 0" rpy="0 0 0" />
+      <parent link="sensor_mount_link"/>
+      <child link="sensor_mount_bracket_link" />
+    </joint>
+    <link name="sensor_mount_bracket_link">
+      <visual>
+        <geometry>
+          <mesh filename="package://mobipick_description/meshes/sensors/sensor_mount_bracket.stl" scale="0.001 0.001 0.001" />
+        </geometry>
+        <xacro:insert_block name="material_almost_white" />
+      </visual>
+      <collision>
+        <geometry>
+          <mesh filename="package://mobipick_description/meshes/sensors/sensor_mount_bracket.stl" scale="0.001 0.001 0.001" />
+        </geometry>
+      </collision>
+      <inertial>
+        <mass value="${sensor_mount_bracket_mass}" />
+        <origin xyz="-0.006750000 -0.030390745 0.000000062" rpy="0 0 0" />
+        <inertia ixx="${sensor_mount_bracket_mass * 0.0010335255}"
+          ixy="${sensor_mount_bracket_mass * 0.00000001092523}"
+          ixz="${sensor_mount_bracket_mass * -0.00000012318317}"
+          iyy="${sensor_mount_bracket_mass * 0.00087473292}"
+          iyz="${sensor_mount_bracket_mass * -0.000000049903018}"
+          izz="${sensor_mount_bracket_mass * 0.00019156915}" />
+      </inertial>
+    </link>
+    <gazebo reference="sensor_mount_bracket_link">
+      <material>Gazebo/Grey</material>
+    </gazebo>
+    <joint name="sensor_mount_pico_holder_joint" type="fixed">
+      <origin xyz="0 0 0" rpy="0 0 0" />
+      <parent link="sensor_mount_link"/>
+      <child link="sensor_mount_pico_holder_link" />
+    </joint>
+    <link name="sensor_mount_pico_holder_link">
+      <visual>
+        <geometry>
+          <mesh filename="package://mobipick_description/meshes/sensors/sensor_mount_pico_holder.stl" scale="0.001 0.001 0.001" />
+        </geometry>
+        <xacro:insert_block name="material_almost_white" />
+      </visual>
+      <collision>
+        <geometry>
+          <mesh filename="package://mobipick_description/meshes/sensors/sensor_mount_pico_holder.stl" scale="0.001 0.001 0.001" />
+        </geometry>
+      </collision>
+      <inertial>
+        <mass value="${sensor_mount_pico_holder_mass}" />
+        <origin xyz="0.001609901 0.102978844 0.008159077" rpy="0 0 0" />
+        <inertia ixx="${sensor_mount_pico_holder_mass * 0.00024619688}"
+          ixy="${sensor_mount_pico_holder_mass * 0.000027175325}"
+          ixz="${sensor_mount_pico_holder_mass * 0.000000014504396}"
+          iyy="${sensor_mount_pico_holder_mass * 0.00023794332}"
+          iyz="${sensor_mount_pico_holder_mass * -0.0000000015705397}"
+          izz="${sensor_mount_pico_holder_mass * 0.000071808769}" />
+      </inertial>
+    </link>
+    <gazebo reference="sensor_mount_pico_holder_link">
       <material>Gazebo/Grey</material>
     </gazebo>

Commit message: URDF: Add pico flexx

File: mobipick_description/urdf/sensors/gripper_cam.urdf.xacro (robot description, xacro)
@@ -5,4 +5,5 @@
   <xacro:property name="sensor_mount_pico_holder_mass" value="0.020" />
   <xacro:property name="astra_s_mass" value="0.300" />
+  <xacro:property name="pico_flexx_mass" value="0.008" />
   <!-- distance between center of camera and camera_link -->
   <xacro:property name="astra_cam_py" value="0.0485"/>
@@ -15,4 +16,10 @@
     </joint>
     <sensor_astra_mini_s camera_name="gripper_astra" />
+    <joint name="gripper_pico_flexx_joint" type="fixed">
+      <origin xyz="0.011 0.106 0.008" rpy="${-pi/2} 0.0 -0.458" />
+      <parent link="sensor_mount_link"/>
+      <child link="gripper_pico_flexx_link"/>
+    </joint>
+    <sensor_pico_flexx camera_name="gripper_pico_flexx" />
   </xacro:macro>
   <xacro:macro name="sensor_mount">
@@ -106,5 +113,7 @@
     </gazebo>
   </xacro:macro>
-  <!-- Orbbec Astra Mini S -->
+  <!-- ##################################################################### -->
+  <!-- ######################## Orbbec Astra Mini S ######################## -->
+  <!-- ##################################################################### -->
   <xacro:macro name="sensor_astra_mini_s" params="camera_name">
     <link name="${camera_name}_link">
@@ -182,5 +191,4 @@
           <depthImageCameraInfoTopicName>depth_registered/camera_info</depthImageCameraInfoTopicName>
           <frameName>${camera_name}_depth_optical_frame</frameName>
-          <baseline>0.1</baseline>
           <distortion_k1>0.0</distortion_k1>
           <distortion_k2>0.0</distortion_k2>
@@ -189,7 +197,86 @@
           <distortion_t2>0.0</distortion_t2>
           <pointCloudCutoff>0.35</pointCloudCutoff>  <!-- measured on real camera (same as data sheet) -->
+          <pointCloudCutoffMax>3.50</pointCloudCutoffMax>
         </plugin>
       </sensor>
     </gazebo>
   </xacro:macro>
+  <!-- ######################################################################### -->
+  <!-- ######################## PMD CamBoard pico flexx ######################## -->
+  <!-- ######################################################################### -->
+  <xacro:macro name="sensor_pico_flexx" params="camera_name">
+    <link name="${camera_name}_link">
+      <visual>
+        <origin xyz="0 0 0" />
+        <geometry>
+          <mesh filename="package://mobipick_description/meshes/sensors/pico_flexx.dae"/>
+        </geometry>
+        <xacro:insert_block name="material_black" />
+      </visual>
+      <collision>
+        <origin xyz="${0.0072 / 2} 0.0 0.0" />
+        <geometry>
+          <box size="0.0072 0.068 0.017" />
+        </geometry>
+      </collision>
+      <xacro:box_inertial mass="${pico_flexx_mass}" x="0.0072" y="0.068" z="0.017">
+        <origin xyz="${0.0072 / 2} 0.0 0.0" />
+      </xacro:box_inertial>
+    </link>
+    <gazebo reference="${camera_name}_link">
+      <material>Gazebo/FlatBlack</material>
+    </gazebo>
+    <joint name="${camera_name}_depth_joint" type="fixed">
+      <origin xyz="0.0072 0.0081 0.0" rpy="0 0 0" />
+      <parent link="${camera_name}_link"/>
+      <child link="${camera_name}_frame" />
+    </joint>
+    <link name="${camera_name}_frame"/>
+    <joint name="${camera_name}_optical_joint" type="fixed">
+      <origin xyz="0 0 0" rpy="${-pi/2} 0 ${-pi/2}" />
+      <parent link="${camera_name}_frame" />
+      <child link="${camera_name}_optical_frame" />
+    </joint>
+    <link name="${camera_name}_optical_frame"/>
+    <sim_pico_flexx/>
+  </xacro:macro>
+  <xacro:macro name="sim_pico_flexx">
+    <gazebo reference="${camera_name}_frame">
+      <sensor type="depth" name="${camera_name}">
+        <always_on>true</always_on>
+        <update_rate>1.0</update_rate>
+        <camera>
+          <horizontal_fov>${60.0 * pi/180.0}</horizontal_fov>
+          <image>
+            <!-- <format>B8G8R8</format> -->
+            <format>L8</format>
+            <width>224</width>
+            <height>171</height>
+          </image>
+          <clip>
+            <near>0.10</near>
+            <far>4.0</far>
+          </clip>
+        </camera>
+        <plugin name="kinect_${camera_name}_controller" filename="libgazebo_ros_openni_kinect.so">
+          <cameraName>${camera_name}</cameraName>
+          <alwaysOn>true</alwaysOn>
+          <updateRate>1.0</updateRate>
+          <imageTopicName>image_mono8</imageTopicName>
+          <depthImageTopicName>image_depth</depthImageTopicName>
+          <pointCloudTopicName>points</pointCloudTopicName>
+          <cameraInfoTopicName>camera_info</cameraInfoTopicName>
+          <depthImageCameraInfoTopicName>depth/camera_info</depthImageCameraInfoTopicName>
+          <frameName>${camera_name}_optical_frame</frameName>
+          <distortion_k1>0.0</distortion_k1>
+          <distortion_k2>0.0</distortion_k2>
+          <distortion_k3>0.0</distortion_k3>
+          <distortion_t1>0.0</distortion_t1>
+          <distortion_t2>0.0</distortion_t2>
+          <pointCloudCutoff>0.10</pointCloudCutoff>
+          <pointCloudCutoffMax>4.0</pointCloudCutoffMax>
+        </plugin>
+      </sensor>
+    </gazebo>
+  </xacro:macro>
 </robot>

Commit message: URDF: Shift pico_holder origin to rotation center
This is only a refactoring (the resulting TF doesn't change much). Shifting the rotation center makes it easier to adjust the angle of the pico flexx.

File: mobipick_description/urdf/sensors/gripper_cam.urdf.xacro (robot description, xacro)
@@ -17,6 +17,6 @@
     <sensor_astra_mini_s camera_name="gripper_astra" />
     <joint name="gripper_pico_flexx_joint" type="fixed">
-      <origin xyz="0.011 0.106 0.008" rpy="${-pi/2} 0.0 -0.458" />
-      <parent link="sensor_mount_link"/>
+      <origin xyz="0.01545 0.0001 0.008" rpy="${-pi/2} 0.0 -0.03650298564336946" />
+      <parent link="sensor_mount_pico_holder_link"/>
       <child link="gripper_pico_flexx_link"/>
     </joint>
@@ -82,5 +82,5 @@
     </gazebo>
     <joint name="sensor_mount_pico_holder_joint" type="fixed">
-      <origin xyz="0 0 0" rpy="0 0 0" />
+      <origin xyz="-0.00325 0.11187 0" rpy="0 0 ${-24.15 / 180.0 * pi}" /> <!-- angle can be adjusted from -15 to -50 degrees (corresponds to downward angle of the pico flexx) -->
       <parent link="sensor_mount_link"/>
       <child link="sensor_mount_pico_holder_link" />

Commit message: URDF: Calibrate pico flexx angle

File: mobipick_description/urdf/sensors/gripper_cam.urdf.xacro (robot description, xacro)
@@ -82,5 +82,5 @@
     </gazebo>
     <joint name="sensor_mount_pico_holder_joint" type="fixed">
-      <origin xyz="-0.00325 0.11187 0" rpy="0 0 ${-24.15 / 180.0 * pi}" /> <!-- angle can be adjusted from -15 to -50 degrees (corresponds to downward angle of the pico flexx) -->
+      <origin xyz="-0.00325 0.11187 0" rpy="0 0 ${-33.5 / 180.0 * pi}" /> <!-- angle can be adjusted from -15 to -50 degrees (corresponds to downward angle of the pico flexx) -->
       <parent link="sensor_mount_link"/>
       <child link="sensor_mount_pico_holder_link" />

Commit message: URDF: Extrinsic calibration for mobipick-hb
This makes things a bit better, but not much. Also it seems to be wrong
that the distance between the cameras is -0.031 (should be -0.025), and
all other values are close to 0.

File: mobipick_description/urdf/sensors/gripper_cam.urdf.xacro (robot description, xacro)
@@ -157,6 +157,6 @@
     <link name="${camera_name}_depth_frame"/>
     <joint name="${camera_name}_depth_optical_joint" type="fixed">
-      <origin xyz="0 0 0" rpy="${-pi/2} 0 ${-pi/2}" />
-      <parent link="${camera_name}_depth_frame" />
+      <origin xyz="-0.0314828066046 -0.000433828244333 0.00121080854987" rpy="0.01174712568115136 0.010416276323763485 -0.0028859908965827175" />   <!-- calibrated 2018-06-07 on mobipick-hbi (16112110432) -->
+      <parent link="${camera_name}_rgb_optical_frame" />
       <child link="${camera_name}_depth_optical_frame" />
     </joint>

Commit message: URDF: Fix typo

File: mobipick_description/urdf/sensors/gripper_cam.urdf.xacro (robot description, xacro)
@@ -157,5 +157,5 @@
     <link name="${camera_name}_depth_frame"/>
     <joint name="${camera_name}_depth_optical_joint" type="fixed">
-      <origin xyz="-0.0314828066046 -0.000433828244333 0.00121080854987" rpy="0.01174712568115136 0.010416276323763485 -0.0028859908965827175" />   <!-- calibrated 2018-06-07 on mobipick-hbi (16112110432) -->
+      <origin xyz="-0.0314828066046 -0.000433828244333 0.00121080854987" rpy="0.01174712568115136 0.010416276323763485 -0.0028859908965827175" />   <!-- calibrated 2018-06-07 on mobipick-hb (16112110432) -->
       <parent link="${camera_name}_rgb_optical_frame" />
       <child link="${camera_name}_depth_optical_frame" />

Commit message: Improve Astra calibration (depth_ir_offset_x)

File: mobipick_description/urdf/sensors/gripper_cam.urdf.xacro (robot description, xacro)
@@ -157,5 +157,5 @@
     <link name="${camera_name}_depth_frame"/>
     <joint name="${camera_name}_depth_optical_joint" type="fixed">
-      <origin xyz="-0.0314828066046 -0.000433828244333 0.00121080854987" rpy="0.01174712568115136 0.010416276323763485 -0.0028859908965827175" />   <!-- calibrated 2018-06-07 on mobipick-hb (16112110432) -->
+      <origin xyz="-0.025 0 0" rpy="0 0 0" />   <!-- calibration not necessary, depth_ir_offset used instead -->
       <parent link="${camera_name}_rgb_optical_frame" />
       <child link="${camera_name}_depth_optical_frame" />

Commit message: 1cm padding on gripper_astra_cam for  moveit collision checking

File: mobipick_description/urdf/sensors/gripper_cam.urdf.xacro (robot description, xacro)
@@ -128,5 +128,5 @@
         <origin xyz="${-0.0325 / 2} ${-astra_cam_py} 0.0" />
         <geometry>
-          <box size="0.0325 0.12 0.0375" />
+          <box size="0.0525 0.14 0.0575" /> <!-- padded 0.01 for moveit collision checking-->
         </geometry>
       </collision>

Commit message: Add logical camera

File: mobipick_description/urdf/sensors/gripper_cam.urdf.xacro (robot description, xacro)
@@ -150,4 +150,28 @@
     </joint>
     <link name="${prefix}${camera_name}_rgb_optical_frame"/>
+    <joint name="${prefix}${camera_name}_rgb_logical_joint" type="fixed">
+      <origin xyz="0 0 0" rpy="0 0 0" />
+      <parent link="${prefix}${camera_name}_rgb_frame" />
+      <child link="${prefix}${camera_name}_rgb_logical_frame" />
+    </joint>
+    <link name="${prefix}${camera_name}_rgb_logical_frame"/>
+    <gazebo reference="${prefix}${camera_name}_rgb_logical_frame">
+      <sensor name="logical_camera" type="logical_camera">
+        <logical_camera>
+          <near>0.05</near>
+          <far>3.50</far>
+          <horizontal_fov>${60.0 * pi/180.0}</horizontal_fov>
+          <aspect_ratio>${640.0/480.0}</aspect_ratio>
+        </logical_camera>
+        <visualize>false</visualize>
+        <always_on>true</always_on>
+        <update_rate>10</update_rate>
+        <plugin name="logical_camera_plugin" filename="liblogical_camera_plugin.so">
+          <cameraName>${prefix}${camera_name}</cameraName>
+          <imageTopicName>rgb/logical_image</imageTopicName>
+          <frameName>${prefix}${camera_name}_rgb_logical_frame</frameName>
+        </plugin>
+      </sensor>
+    </gazebo>
     <joint name="${prefix}${camera_name}_depth_joint" type="fixed">
       <origin xyz="0 -0.02 0" rpy="0 0 0" />
