Commit message: tune physics parameters for relay, fix bounding box, make it coincide with visual model, fix inertia tensor

File: mobipick_gazebo/urdf/relay.urdf.xacro (robot description, xacro)
@@ -1,22 +1,21 @@
 <robot  xmlns:xacro="http://ros.org/wiki/xacro" name="relay_model">
   <xacro:include filename="$(find mobipick_description)/urdf/common_properties.urdf.xacro" />
-  <xacro:property name="mass" value="0.500" />
+  <xacro:property name="mass" value="0.1" />
+  <xacro:property name="bb_width" value="0.106" />
+  <xacro:property name="bb_length" value="0.046" />
+  <xacro:property name="bb_height" value="0.056" />
+  <xacro:macro name="box_inertia" params="m x y z">
+    <inertia   ixx="${m*(y*y+z*z)/12}" ixy = "0" ixz = "0"
+               iyy="${m*(x*x+z*z)/12}" iyz = "0"
+               izz="${m*(x*x+z*z)/12}" />
+  </xacro:macro>
   <link name="relay">
-    <!-- <xacro:cylinder_inertial radius="${radius}" length="${height}" mass="${mass}">
-      <origin xyz="0 0 ${height/2}" rpy="0 0 0" />
-    </xacro:cylinder_inertial> -->
     <inertial>
-      <origin xyz="-0.03071469 0.02435085 0.02356763" rpy="0 0 0" />
+      <origin xyz="0 0 0" rpy="0 0 1.57" />
       <mass value="${mass}" />
-      <inertia
-        ixx="${mass * 0.003988511412844956}"
-        ixy="${mass * 0.0004112614213275305}"
-        ixz="${mass * 0.00003166287680811595}"
-        iyy="${mass * 0.0016270423052260282}"
-        iyz="${mass * 0.0000807201704454}"
-        izz="${mass * 0.00534355593909}" />
+      <xacro:box_inertia m="${mass}" x="${bb_width}" y="${bb_length}" z="${bb_height}" />
     </inertial>
     <visual>
-      <origin xyz="0 0 0" rpy="0 0 0" />
+      <origin xyz="-0.0025 -0.0445 -0.022" rpy="0 0 0" />
       <geometry>
         <mesh filename="package://mobipick_gazebo/meshes/relay.stl" scale="0.1 0.1 0.1" />
@@ -26,5 +25,5 @@
       <origin xyz="0 0 0" rpy="0 0 0" />
       <geometry>
-        <mesh filename="package://mobipick_gazebo/meshes/relay.stl" scale="0.1 0.1 0.1" />
+        <box size="${bb_height} ${bb_width} ${bb_length}" />
       </geometry>
     </collision>

Commit message: Replace relay mesh with final textured version
This rotates the mesh by 90 degrees, so grasp poses will have to be
re-teached.

File: mobipick_gazebo/urdf/relay.urdf.xacro (robot description, xacro)
@@ -2,7 +2,7 @@
   <xacro:include filename="$(find mobipick_description)/urdf/common_properties.urdf.xacro" />
   <xacro:property name="mass" value="0.1" />
-  <xacro:property name="bb_width" value="0.106" />
-  <xacro:property name="bb_length" value="0.046" />
-  <xacro:property name="bb_height" value="0.056" />
+  <xacro:property name="bb_size_x" value="0.0575" />
+  <xacro:property name="bb_size_y" value="0.0451" />
+  <xacro:property name="bb_size_z" value="0.104364" />
   <xacro:macro name="box_inertia" params="m x y z">
     <inertia   ixx="${m*(y*y+z*z)/12}" ixy = "0" ixz = "0"
@@ -12,10 +12,10 @@
   <link name="relay">
     <inertial>
-      <origin xyz="0 0 0" rpy="0 0 1.57" />
+      <origin xyz="0 0 0" rpy="0 0 0" />
       <mass value="${mass}" />
-      <xacro:box_inertia m="${mass}" x="${bb_width}" y="${bb_length}" z="${bb_height}" />
+      <xacro:box_inertia m="${mass}" x="${bb_size_x}" y="${bb_size_y}" z="${bb_size_z}" />
     </inertial>
     <visual>
-      <origin xyz="0 -0.015 0" rpy="-1.5708 0 0" />
+      <origin xyz="0 0 0" rpy="0 0 0" />
       <geometry>
         <mesh filename="package://mobipick_gazebo/meshes/relay.dae" scale="1 1 1" />
@@ -25,5 +25,5 @@
       <origin xyz="0 0 0" rpy="0 0 0" />
       <geometry>
-        <box size="${bb_height} ${bb_width} ${bb_length}" />
+        <box size="${bb_size_x} ${bb_size_y} ${bb_size_z}" />
       </geometry>
     </collision>
