Commit message: gazebo: Fix tall_table.urdf.xacro

File: mobipick_gazebo/urdf/tall_table.urdf.xacro (robot description, xacro)
@@ -1,14 +1,13 @@
 <?xml version="1.0"?>
-<robot name="table">
-  <property name="table_height" value="1.0" />
-  <property name="table_width" value="1.0" />
-  <property name="table_depth" value="2.0" />
-  <property name="leg_radius" value="0.02" />
-  <property name="table_x" value="0.0" />
-  <property name="table_y" value="0.0" />
-  <property name="table_z" value="0.0" />
-  <property name="table_top_thickness" value="0.05"/>
-  <property name="M_PI" value="3.1415926535897931" />
-  <!-- tabletop height is .55+.01+.025=.585 -->
+<robot xmlns:xacro="http://ros.org/wiki/xacro" name="table">
+  <xacro:property name="table_height" value="1.0" />
+  <xacro:property name="table_width" value="1.0" />
+  <xacro:property name="table_depth" value="2.0" />
+  <xacro:property name="leg_radius" value="0.02" />
+  <xacro:property name="table_x" value="0.0" />
+  <xacro:property name="table_y" value="0.0" />
+  <xacro:property name="table_z" value="0.0" />
+  <xacro:property name="table_top_thickness" value="0.05"/>
+  <xacro:property name="M_PI" value="3.1415926535897931" />
   <link name="table_top_link">
     <inertial>

Commit message: gazebo: Adjust table dimensions to actual demo table

File: mobipick_gazebo/urdf/tall_table.urdf.xacro (robot description, xacro)
@@ -1,7 +1,7 @@
 <?xml version="1.0"?>
 <robot xmlns:xacro="http://ros.org/wiki/xacro" name="table">
-  <xacro:property name="table_height" value="1.0" />
-  <xacro:property name="table_width" value="1.0" />
-  <xacro:property name="table_depth" value="2.0" />
+  <xacro:property name="table_height" value="0.94" />
+  <xacro:property name="table_width" value="0.70" />
+  <xacro:property name="table_depth" value="0.70" />
   <xacro:property name="leg_radius" value="0.02" />
   <xacro:property name="table_x" value="0.0" />

Commit message: adapted environment for easier detection of power drill

File: mobipick_gazebo/urdf/tall_table.urdf.xacro (robot description, xacro)
@@ -32,5 +32,5 @@
   </link>
   <gazebo reference="table_top_link">
-    <material>Gazebo/Wood</material>
+    <!--<material>Gazebo/Wood</material>-->
     <mu1>1.0</mu1>
     <mu2>1.0</mu2>

Commit message: Adapt height of table to the ones from Berghoffstraße

File: mobipick_gazebo/urdf/tall_table.urdf.xacro (robot description, xacro)
@@ -1,5 +1,5 @@
 <?xml version="1.0"?>
 <robot xmlns:xacro="http://ros.org/wiki/xacro" name="table">
-  <xacro:property name="table_height" value="0.94" />
+  <xacro:property name="table_height" value="0.73" />
   <xacro:property name="table_width" value="0.70" />
   <xacro:property name="table_depth" value="0.70" />

Commit message: adapted table high

File: mobipick_gazebo/urdf/tall_table.urdf.xacro (robot description, xacro)
@@ -1,5 +1,5 @@
 <?xml version="1.0"?>
 <robot xmlns:xacro="http://ros.org/wiki/xacro" name="table">
-  <xacro:property name="table_height" value="0.73" />
+  <xacro:property name="table_height" value="0.78" />
   <xacro:property name="table_width" value="0.70" />
   <xacro:property name="table_depth" value="0.70" />

Commit message: Gazebo: Adjust table dimensions to actual table
This stops the robot trying to press the power drill into the table
during placing.

File: mobipick_gazebo/urdf/tall_table.urdf.xacro (robot description, xacro)
@@ -1,7 +1,7 @@
 <?xml version="1.0"?>
 <robot xmlns:xacro="http://ros.org/wiki/xacro" name="table">
-  <xacro:property name="table_height" value="0.78" />
-  <xacro:property name="table_width" value="0.70" />
-  <xacro:property name="table_depth" value="0.70" />
+  <xacro:property name="table_height" value="0.72" />
+  <xacro:property name="table_width" value="0.80" />
+  <xacro:property name="table_depth" value="0.80" />
   <xacro:property name="leg_radius" value="0.02" />
   <xacro:property name="table_x" value="0.0" />

Commit message: Split out table xacro macro
This makes the table width, height etc. configurable

File: mobipick_gazebo/urdf/tall_table.urdf.xacro (robot description, xacro)
@@ -1,160 +1,5 @@
 <?xml version="1.0"?>
 <robot xmlns:xacro="http://ros.org/wiki/xacro" name="table">
-  <xacro:property name="table_height" value="0.72" />
-  <xacro:property name="table_width" value="0.80" />
-  <xacro:property name="table_depth" value="0.80" />
-  <xacro:property name="leg_radius" value="0.02" />
-  <xacro:property name="table_x" value="0.0" />
-  <xacro:property name="table_y" value="0.0" />
-  <xacro:property name="table_z" value="0.0" />
-  <xacro:property name="table_top_thickness" value="0.05"/>
-  <xacro:property name="M_PI" value="3.1415926535897931" />
-  <link name="table_top_link">
-    <inertial>
-      <mass value="1.0" />
-      <origin xyz="${table_x} ${table_y} ${table_z + table_height - table_top_thickness/2}" />
-      <inertia ixx="1" ixy="0"  ixz="0"
-               iyy="1" iyz="0"
-               izz="1" />
-    </inertial>
-    <visual>
-      <origin xyz="${table_x} ${table_y} ${table_z + table_height - table_top_thickness/2}" />
-      <geometry>
-        <box size="${table_width} ${table_depth} ${table_top_thickness}" />
-      </geometry>
-    </visual>
-    <collision>
-      <origin xyz="${table_x} ${table_y} ${table_z + table_height - table_top_thickness/2}" />
-      <geometry>
-        <box size="${table_width} ${table_depth} ${table_top_thickness}" />
-      </geometry>
-    </collision>
-  </link>
-  <gazebo reference="table_top_link">
-    <!--<material>Gazebo/Wood</material>-->
-    <mu1>1.0</mu1>
-    <mu2>1.0</mu2>
-    <kp>1000000.0</kp>
-    <kd>1.0</kd>
-  </gazebo>
-  <joint name="leg1_joint" type="fixed" >
-    <parent link="table_top_link" />
-    <origin xyz="${table_x + table_width/2} ${table_y + table_depth/2} ${table_z + table_height}" rpy="0 0 0" />
-    <child link="leg1_link" />
-  </joint>
-  <link name="leg1_link">
-    <inertial>
-      <mass value="1.0" />
-      <origin xyz="0 0 ${-table_height/2}" />
-      <inertia ixx="0.1" ixy="0"  ixz="0"
-               iyy="0.1" iyz="0"
-               izz="0.01" />
-    </inertial>
-    <visual>
-      <origin xyz="0.0 0.0 ${-table_height/2}" rpy="0 0 0" />
-      <geometry>
-        <cylinder radius="${leg_radius}" length="${table_height}" />
-      </geometry>
-    </visual>
-    <collision>
-      <origin xyz="0.0 0.0 ${-table_height/2}" rpy="0.0 0.0 0.0" />
-      <geometry>
-        <cylinder radius="${leg_radius}" length="${table_height}" />
-      </geometry>
-    </collision>
-  </link>
-  <gazebo reference="leg1_link">
-    <material>Gazebo/Red</material>
-  </gazebo>
-  <joint name="leg2_joint" type="fixed" >
-    <parent link="table_top_link" />
-    <origin xyz="${table_x - table_width/2} ${table_y + table_depth/2} ${table_z + table_height}" rpy="0 0 0" />
-    <child link="leg2_link" />
-  </joint>
-  <link name="leg2_link">
-    <inertial>
-      <mass value="1.0" />
-      <origin xyz="0 0 ${-table_height/2}" />
-      <inertia ixx="0.1" ixy="0"  ixz="0"
-               iyy="0.1" iyz="0"
-               izz="0.01" />
-    </inertial>
-    <visual>
-      <origin xyz="0.0 0.0 ${-table_height/2}" rpy="0 0 0" />
-      <geometry>
-        <cylinder radius="${leg_radius}" length="${table_height}" />
-      </geometry>
-    </visual>
-    <collision>
-      <origin xyz="0.0 0.0 ${-table_height/2}" rpy="0.0 0.0 0.0" />
-      <geometry>
-        <cylinder radius="${leg_radius}" length="${table_height}" />
-      </geometry>
-    </collision>
-  </link>
-  <gazebo reference="leg2_link">
-    <material>Gazebo/Red</material>
-  </gazebo>
-  <joint name="leg3_joint" type="fixed" >
-    <parent link="table_top_link" />
-    <origin xyz="${table_x + table_width/2} ${table_y - table_depth/2} ${table_z + table_height}" rpy="0 0 0" />
-    <child link="leg3_link" />
-  </joint>
-  <link name="leg3_link">
-    <inertial>
-      <mass value="1.0" />
-      <origin xyz="0 0 ${-table_height/2}" />
-      <inertia ixx="0.1" ixy="0"  ixz="0"
-               iyy="0.1" iyz="0"
-               izz="0.01" />
-    </inertial>
-    <visual>
-      <origin xyz="0.0 0.0 ${-table_height/2}" rpy="0 0 0" />
-      <geometry>
-        <cylinder radius="${leg_radius}" length="${table_height}" />
-      </geometry>
-    </visual>
-    <collision>
-      <origin xyz="0.0 0.0 ${-table_height/2}" rpy="0.0 0.0 0.0" />
-      <geometry>
-        <cylinder radius="${leg_radius}" length="${table_height}" />
-      </geometry>
-    </collision>
-  </link>
-  <gazebo reference="leg3_link">
-    <material>Gazebo/Red</material>
-  </gazebo>
-  <joint name="leg4_joint" type="fixed" >
-    <parent link="table_top_link" />
-    <origin xyz="${table_x - table_width/2} ${table_y - table_depth/2} ${table_z + table_height}" rpy="0 0 0" />
-    <child link="leg4_link" />
-  </joint>
-  <link name="leg4_link">
-    <inertial>
-      <mass value="1.0" />
-      <origin xyz="0 0 ${-table_height/2}" />
-      <inertia ixx="0.1" ixy="0"  ixz="0"
-               iyy="0.1" iyz="0"
-               izz="0.01" />
-    </inertial>
-    <visual>
-      <origin xyz="0.0 0.0 ${-table_height/2}" rpy="0 0 0" />
-      <geometry>
-        <cylinder radius="${leg_radius}" length="${table_height}" />
-      </geometry>
-    </visual>
-    <collision>
-      <origin xyz="0.0 0.0 ${-table_height/2}" rpy="0.0 0.0 0.0" />
-      <geometry>
-        <cylinder radius="${leg_radius}" length="${table_height}" />
-      </geometry>
-    </collision>
-  </link>
-  <gazebo reference="leg4_link">
-    <material>Gazebo/Red</material>
-  </gazebo>
-  <gazebo>
-    <static>true</static>
-    <canonicalBody>table_top_link</canonicalBody>
-  </gazebo>
+  <xacro:include filename="$(find mobipick_gazebo)/urdf/include/table.urdf.xacro" />
+  <xacro:table height="0.72" width="0.80" depth="0.80" leg_radius="0.02" table_top_thickness="0.05" x="0.0" y="0.0" z="0.0" />
 </robot>
