Commit message: tune physics parameters for multimeter, fix bounding box, make it coincide with visual model

File: mobipick_gazebo/urdf/multimeter.urdf.xacro (robot description, xacro)
@@ -1,22 +1,21 @@
 <robot  xmlns:xacro="http://ros.org/wiki/xacro" name="multimeter_model">
   <xacro:include filename="$(find mobipick_description)/urdf/common_properties.urdf.xacro" />
-  <xacro:property name="mass" value="0.500" />
+  <xacro:property name="mass" value="0.1" />
+  <xacro:property name="bb_width" value="0.042" />
+  <xacro:property name="bb_length" value="0.086" />
+  <xacro:property name="bb_height" value="0.177" />
+  <xacro:macro name="box_inertia" params="m x y z">
+    <inertia   ixx="${m*(y*y+z*z)/12}" ixy = "0" ixz = "0"
+               iyy="${m*(x*x+z*z)/12}" iyz = "0"
+               izz="${m*(x*x+z*z)/12}" />
+  </xacro:macro>
   <link name="multimeter">
-    <!-- <xacro:cylinder_inertial radius="${radius}" length="${height}" mass="${mass}">
-      <origin xyz="0 0 ${height/2}" rpy="0 0 0" />
-    </xacro:cylinder_inertial> -->
     <inertial>
-      <origin xyz="-0.03071469 0.02435085 0.02356763" rpy="0 0 0" />
+      <origin xyz="0 0 0" rpy="0 0 0" />
       <mass value="${mass}" />
-      <inertia
-        ixx="${mass * 0.003988511412844956}"
-        ixy="${mass * 0.0004112614213275305}"
-        ixz="${mass * 0.00003166287680811595}"
-        iyy="${mass * 0.0016270423052260282}"
-        iyz="${mass * 0.0000807201704454}"
-        izz="${mass * 0.00534355593909}" />
+      <xacro:box_inertia m="${mass}" x="${bb_width}" y="${bb_length}" z="${bb_height}" />
     </inertial>
     <visual>
-      <origin xyz="0 0 0" rpy="0 0 0" />
+      <origin xyz="-0.075 -0.089 -0.154" rpy="0 0 0" />
       <geometry>
         <mesh filename="package://mobipick_gazebo/meshes/multimeter.stl" scale="0.001 0.001 0.001" />
@@ -26,5 +25,5 @@
       <origin xyz="0 0 0" rpy="0 0 0" />
       <geometry>
-        <mesh filename="package://mobipick_gazebo/meshes/multimeter.stl" scale="0.001 0.001 0.001" />
+        <box size="${bb_height} ${bb_width} ${bb_length}"/>
       </geometry>
     </collision>

Commit message: add texture to multimeter

File: mobipick_gazebo/urdf/multimeter.urdf.xacro (robot description, xacro)
@@ -17,7 +17,7 @@
     </inertial>
     <visual>
-      <origin xyz="-0.075 -0.089 -0.154" rpy="0 0 0" />
+      <origin xyz="0 0 0" rpy="-1.5708 0 0" />
       <geometry>
-        <mesh filename="package://mobipick_gazebo/meshes/multimeter.stl" scale="0.001 0.001 0.001" />
+        <mesh filename="package://mobipick_gazebo/meshes/multimeter.dae" scale="1 1 1" />
       </geometry>
     </visual>

Commit message: Fix multimeter + screwdriver inertias

File: mobipick_gazebo/urdf/multimeter.urdf.xacro (robot description, xacro)
@@ -2,7 +2,7 @@
   <xacro:include filename="$(find mobipick_description)/urdf/common_properties.urdf.xacro" />
   <xacro:property name="mass" value="0.1" />
-  <xacro:property name="bb_width" value="0.042" />
-  <xacro:property name="bb_length" value="0.086" />
-  <xacro:property name="bb_height" value="0.177" />
+  <xacro:property name="bb_size_x" value="0.179500" />
+  <xacro:property name="bb_size_y" value="0.087488" />
+  <xacro:property name="bb_size_z" value="0.042064" />
   <xacro:macro name="box_inertia" params="m x y z">
     <inertia   ixx="${m*(y*y+z*z)/12}" ixy = "0" ixz = "0"
@@ -14,8 +14,8 @@
       <origin xyz="0 0 0" rpy="0 0 0" />
       <mass value="${mass}" />
-      <xacro:box_inertia m="${mass}" x="${bb_height}" y="${bb_length}" z="${bb_width}" />
+      <xacro:box_inertia m="${mass}" x="${bb_size_x}" y="${bb_size_y}" z="${bb_size_z}" />
     </inertial>
     <visual>
-      <origin xyz="0 0 0" rpy="-1.5708 0 0" />
+      <origin xyz="0 0 0" rpy="0 0 0" />
       <geometry>
         <mesh filename="package://mobipick_gazebo/meshes/multimeter.dae" scale="1 1 1" />
@@ -25,5 +25,5 @@
       <origin xyz="0 0 0" rpy="0 0 0" />
       <geometry>
-        <box size="${bb_height} ${bb_width} ${bb_length}"/>
+        <box size="${bb_size_x} ${bb_size_y} ${bb_size_z}" />
       </geometry>
     </collision>

File: mobipick_gazebo/urdf/screwdriver.urdf.xacro (robot description, xacro)
@@ -2,7 +2,7 @@
   <xacro:include filename="$(find mobipick_description)/urdf/common_properties.urdf.xacro" />
   <xacro:property name="mass" value="0.1" />
-  <xacro:property name="bb_width" value="0.036" />
-  <xacro:property name="bb_length" value="0.036" />
-  <xacro:property name="bb_height" value="0.24" />
+  <xacro:property name="bb_size_x" value="0.245" />
+  <xacro:property name="bb_size_y" value="0.034418" />
+  <xacro:property name="bb_size_z" value="0.034418" />
   <xacro:macro name="box_inertia" params="m x y z">
     <inertia   ixx="${m*(y*y+z*z)/12}" ixy = "0" ixz = "0"
@@ -12,10 +12,10 @@
   <link name="screwdriver">
     <inertial>
-      <origin xyz="0 0 0" rpy="0 0 1.57" />
+      <origin xyz="0 0 0" rpy="0 0 0" />
       <mass value="${mass}" />
-      <xacro:box_inertia m="${mass}" x="${bb_width}" y="${bb_length}" z="${bb_height}" />
+      <xacro:box_inertia m="${mass}" x="${bb_size_x}" y="${bb_size_y}" z="${bb_size_z}" />
     </inertial>
     <visual>
-        <origin xyz="0 0 0" rpy="-1.5708 0 0" />
+      <origin xyz="0 0 0" rpy="0 0 0" />
       <geometry>
         <mesh filename="package://mobipick_gazebo/meshes/screwdriver.dae" scale="1 1 1" />
@@ -25,5 +25,5 @@
       <origin xyz="0 0 0" rpy="0 0 0" />
       <geometry>
-        <box size="${bb_height} ${bb_width} ${bb_length}" />
+        <box size="${bb_size_x} ${bb_size_y} ${bb_size_z}" />
       </geometry>
     </collision>

Commit message: Add collision meshes for InCoRAP objects

File: mobipick_gazebo/urdf/multimeter.urdf.xacro (robot description, xacro)
@@ -25,5 +25,6 @@
       <origin xyz="0 0 0" rpy="0 0 0" />
       <geometry>
-        <box size="${bb_size_x} ${bb_size_y} ${bb_size_z}" />
+        <!-- <box size="${bb_size_x} ${bb_size_y} ${bb_size_z}" /> -->
+        <mesh filename="package://mobipick_gazebo/meshes/collision//multimeter.stl" />
       </geometry>
     </collision>

File: mobipick_gazebo/urdf/relay.urdf.xacro (robot description, xacro)
@@ -25,5 +25,6 @@
       <origin xyz="0 0 0" rpy="0 0 0" />
       <geometry>
-        <box size="${bb_size_x} ${bb_size_y} ${bb_size_z}" />
+        <!-- <box size="${bb_size_x} ${bb_size_y} ${bb_size_z}" /> -->
+        <mesh filename="package://mobipick_gazebo/meshes/collision/relay.stl" />
       </geometry>
     </collision>

File: mobipick_gazebo/urdf/screwdriver.urdf.xacro (robot description, xacro)
@@ -25,5 +25,6 @@
       <origin xyz="0 0 0" rpy="0 0 0" />
       <geometry>
-        <box size="${bb_size_x} ${bb_size_y} ${bb_size_z}" />
+        <!-- <box size="${bb_size_x} ${bb_size_y} ${bb_size_z}" /> -->
+        <mesh filename="package://mobipick_gazebo/meshes/collision/screwdriver.stl" />
       </geometry>
     </collision>

Commit message: gazebo: Change object mass to true measured values

File: mobipick_gazebo/urdf/multimeter.urdf.xacro (robot description, xacro)
@@ -1,5 +1,5 @@
 <robot  xmlns:xacro="http://ros.org/wiki/xacro" name="multimeter_model">
   <xacro:include filename="$(find mobipick_description)/urdf/common_properties.urdf.xacro" />
-  <xacro:property name="mass" value="0.1" />
+  <xacro:property name="mass" value="0.346" />
   <xacro:property name="bb_size_x" value="0.179500" />
   <xacro:property name="bb_size_y" value="0.087488" />

File: mobipick_gazebo/urdf/powerdrill.urdf.xacro (robot description, xacro)
@@ -1,5 +1,5 @@
 <robot  xmlns:xacro="http://ros.org/wiki/xacro" name="powerdrill_model">
   <xacro:include filename="$(find mobipick_description)/urdf/common_properties.urdf.xacro" />
-  <xacro:property name="mass" value="0.500" />
+  <xacro:property name="mass" value="1.284" />
   <link name="powerdrill">
     <!-- <xacro:cylinder_inertial radius="${radius}" length="${height}" mass="${mass}">

File: mobipick_gazebo/urdf/powerdrill_with_grip.urdf.xacro (robot description, xacro)
@@ -1,5 +1,5 @@
 <robot  xmlns:xacro="http://ros.org/wiki/xacro" name="powerdrill_with_grip_model">
   <xacro:include filename="$(find mobipick_description)/urdf/common_properties.urdf.xacro" />
-  <xacro:property name="mass" value="0.500" />
+  <xacro:property name="mass" value="1.284" />
   <link name="powerdrill_with_grip">
     <!-- <xacro:cylinder_inertial radius="${radius}" length="${height}" mass="${mass}">

File: mobipick_gazebo/urdf/relay.urdf.xacro (robot description, xacro)
@@ -1,5 +1,5 @@
 <robot  xmlns:xacro="http://ros.org/wiki/xacro" name="relay_model">
   <xacro:include filename="$(find mobipick_description)/urdf/common_properties.urdf.xacro" />
-  <xacro:property name="mass" value="0.1" />
+  <xacro:property name="mass" value="0.256" />
   <xacro:property name="bb_size_x" value="0.0575" />
   <xacro:property name="bb_size_y" value="0.0451" />

File: mobipick_gazebo/urdf/screwdriver.urdf.xacro (robot description, xacro)
@@ -1,5 +1,5 @@
 <robot  xmlns:xacro="http://ros.org/wiki/xacro" name="screwdriver_model">
   <xacro:include filename="$(find mobipick_description)/urdf/common_properties.urdf.xacro" />
-  <xacro:property name="mass" value="0.1" />
+  <xacro:property name="mass" value="0.118" />
   <xacro:property name="bb_size_x" value="0.245" />
   <xacro:property name="bb_size_y" value="0.034418" />
