Commit message: Remove roll rotation from powerdrill_with_grip
The roll=pi rotation in the URDF mean that the Gazebo pose and the mesh
pose were different. The object poses estimated by DOPE are based on the
mesh pose without any additional rotation. So in order to return the
same poses as DOPE on the real robot, the gazebo_object_publisher had to
apply another roll=pi rotation to the Gazebo pose. The logical_camera
plugin does not do this, so it returned incorrect poses.

This commit solves that problem by removing the roll=pi rotation from
the URDF, thereby making any special handling unnecessary.

File: mobipick_gazebo/urdf/powerdrill_with_grip.urdf.xacro (robot description, xacro)
@@ -18,5 +18,5 @@
     </inertial>
     <visual>
-      <origin xyz="0 0 0" rpy="${pi} 0 0" />
+      <origin xyz="0 0 0" rpy="0 0 0" />
       <geometry>
         <mesh filename="package://mobipick_gazebo/meshes/powerdrill_with_grip.dae" />
@@ -24,5 +24,5 @@
     </visual>
     <collision>
-      <origin xyz="0 0 0" rpy="${pi} 0 0" />
+      <origin xyz="0 0 0" rpy="0 0 0" />
       <geometry>
         <mesh filename="package://mobipick_gazebo/meshes/powerdrill_with_grip.dae" />

Commit message: powerdrill_with_grip URDF: Update inertia tensor
This intertia tensor was re-computed using Meshlab:

* Remeshing, Simplification and Reconstruction -> Create solid wireframe
  (to fix "mesh is not watertight" during computation of geometric
  measures)
* Scale by factor s=100
* compute geometric meshes
* divide resulting inertia tensor by (s^2 * volume)

File: mobipick_gazebo/urdf/powerdrill_with_grip.urdf.xacro (robot description, xacro)
@@ -3,17 +3,14 @@
   <xacro:property name="mass" value="1.284" />
   <link name="powerdrill_with_grip">
-    <!-- <xacro:cylinder_inertial radius="${radius}" length="${height}" mass="${mass}">
-      <origin xyz="0 0 ${height/2}" rpy="0 0 0" />
-    </xacro:cylinder_inertial> -->
     <inertial>
-      <origin xyz="0.01524081 -0.01376334 0.00190586" rpy="0 0 0" />
+      <origin xyz="0.01572397 0.00627010 -0.00088096" rpy="0 0 0" />
       <mass value="${mass}" />
       <inertia
-        ixx="${mass * 0.003988511412844956}"
-        ixy="${mass * -0.0004112614213275305}"
-        ixz="${mass * -0.00003166287680811595}"
-        iyy="${mass * 0.0016270423052260282}"
-        iyz="${mass * 0.0000807201704454}"
-        izz="${mass * 0.00534355593909}" />
+        ixx="${mass * 0.006644088398958405}"
+        ixy="${mass * -0.00021896180608560679}"
+        ixz="${mass * -4.562260404751529e-06}"
+        iyy="${mass * 0.002253199387886466}"
+        iyz="${mass * -3.265842622139487e-05}"
+        izz="${mass * 0.007951044267639611}" />
     </inertial>
     <visual>
