Commit message: Rename powerdrill -> power_drill

File: mobipick_gazebo/urdf/power_drill.urdf.xacro (robot description, xacro)
@@ -1,6 +1,6 @@
-<robot  xmlns:xacro="http://ros.org/wiki/xacro" name="powerdrill_model">
+<robot  xmlns:xacro="http://ros.org/wiki/xacro" name="power_drill_model">
   <xacro:include filename="$(find mobipick_description)/urdf/common_properties.urdf.xacro" />
   <xacro:property name="mass" value="1.284" />
-  <link name="powerdrill">
+  <link name="power_drill">
     <!-- <xacro:cylinder_inertial radius="${radius}" length="${height}" mass="${mass}">
       <origin xyz="0 0 ${height/2}" rpy="0 0 0" />
@@ -20,5 +20,5 @@
       <origin xyz="0 0 0" rpy="0 0 0" />
       <geometry>
-        <mesh filename="package://mobipick_gazebo/meshes/powerdrill.dae" />
+        <mesh filename="package://mobipick_gazebo/meshes/power_drill.dae" />
       </geometry>
     </visual>
@@ -26,5 +26,5 @@
       <origin xyz="0 0 0" rpy="0 0 0" />
       <geometry>
-        <mesh filename="package://mobipick_gazebo/meshes/powerdrill.dae" />
+        <mesh filename="package://mobipick_gazebo/meshes/power_drill.dae" />
       </geometry>
     </collision>

File: mobipick_gazebo/urdf/power_drill_with_grip.urdf.xacro (robot description, xacro)
@@ -1,6 +1,6 @@
-<robot  xmlns:xacro="http://ros.org/wiki/xacro" name="powerdrill_with_grip_model">
+<robot  xmlns:xacro="http://ros.org/wiki/xacro" name="power_drill_with_grip_model">
   <xacro:include filename="$(find mobipick_description)/urdf/common_properties.urdf.xacro" />
   <xacro:property name="mass" value="1.284" />
-  <link name="powerdrill_with_grip">
+  <link name="power_drill_with_grip">
     <inertial>
       <origin xyz="0.01572397 0.00627010 -0.00088096" rpy="0 0 0" />
@@ -17,5 +17,5 @@
       <origin xyz="0 0 0" rpy="0 0 0" />
       <geometry>
-        <mesh filename="package://mobipick_gazebo/meshes/powerdrill_with_grip.dae" />
+        <mesh filename="package://mobipick_gazebo/meshes/power_drill_with_grip.dae" />
       </geometry>
     </visual>
@@ -23,5 +23,5 @@
       <origin xyz="0 0 0" rpy="0 0 0" />
       <geometry>
-        <mesh filename="package://mobipick_gazebo/meshes/powerdrill_with_grip.dae" />
+        <mesh filename="package://mobipick_gazebo/meshes/power_drill_with_grip.dae" />
       </geometry>
     </collision>
