Commit message: Add collision mesh for klt

File: mobipick_gazebo/urdf/klt.urdf.xacro (robot description, xacro)
@@ -23,5 +23,5 @@
       <origin xyz="0 0 0" rpy="0 0 0" />
       <geometry>
-        <mesh filename="package://mobipick_gazebo/meshes/klt3147.dae" />
+        <mesh filename="package://mobipick_gazebo/meshes/collision/klt3147.stl" />
       </geometry>
     </collision>

Commit message: Rename mesh: klt3147 -> klt
This is for consistency with the other objects. Also, grasplan's
grasp_visualizer doesn't work if the object name is different from the
mesh filename.

File: mobipick_gazebo/urdf/klt.urdf.xacro (robot description, xacro)
@@ -17,5 +17,5 @@
       <origin xyz="0 0 0" rpy="0 0 0" />
       <geometry>
-        <mesh filename="package://mobipick_gazebo/meshes/klt3147.dae" />
+        <mesh filename="package://mobipick_gazebo/meshes/klt.dae" />
       </geometry>
     </visual>
@@ -23,5 +23,5 @@
       <origin xyz="0 0 0" rpy="0 0 0" />
       <geometry>
-        <mesh filename="package://mobipick_gazebo/meshes/collision/klt3147.stl" />
+        <mesh filename="package://mobipick_gazebo/meshes/collision/klt.stl" />
       </geometry>
     </collision>

Commit message: mobipick_gazebo: Use meshes from pbr_objects

File: mobipick_gazebo/urdf/klt.urdf.xacro (robot description, xacro)
@@ -17,5 +17,5 @@
       <origin xyz="0 0 0" rpy="0 0 0" />
       <geometry>
-        <mesh filename="package://mobipick_gazebo/meshes/klt.dae" />
+        <mesh filename="package://pbr_objects/meshes/klt/klt3147.obj" />
       </geometry>
     </visual>

File: mobipick_gazebo/urdf/multimeter.urdf.xacro (robot description, xacro)
@@ -19,5 +19,5 @@
       <origin xyz="0 0 0" rpy="0 0 0" />
       <geometry>
-        <mesh filename="package://mobipick_gazebo/meshes/multimeter.dae" scale="1 1 1" />
+        <mesh filename="package://pbr_objects/meshes/multimeter/multimeter.obj" scale="1 1 1" />
       </geometry>
     </visual>

File: mobipick_gazebo/urdf/power_drill_with_grip.urdf.xacro (robot description, xacro)
@@ -17,5 +17,5 @@
       <origin xyz="0 0 0" rpy="0 0 0" />
       <geometry>
-        <mesh filename="package://mobipick_gazebo/meshes/power_drill_with_grip.dae" />
+        <mesh filename="package://pbr_objects/meshes/power_drill_with_grip/power_drill_with_grip.obj" />
       </geometry>
     </visual>
@@ -23,5 +23,5 @@
       <origin xyz="0 0 0" rpy="0 0 0" />
       <geometry>
-        <mesh filename="package://mobipick_gazebo/meshes/power_drill_with_grip.dae" />
+        <mesh filename="package://pbr_objects/meshes/power_drill_with_grip/power_drill_with_grip.stl" />
       </geometry>
     </collision>

File: mobipick_gazebo/urdf/relay.urdf.xacro (robot description, xacro)
@@ -19,5 +19,5 @@
       <origin xyz="0 0 0" rpy="0 0 0" />
       <geometry>
-        <mesh filename="package://mobipick_gazebo/meshes/relay.dae" scale="1 1 1" />
+        <mesh filename="package://pbr_objects/meshes/relay/relay.obj" scale="1 1 1" />
       </geometry>
     </visual>

File: mobipick_gazebo/urdf/screwdriver.urdf.xacro (robot description, xacro)
@@ -19,5 +19,5 @@
       <origin xyz="0 0 0" rpy="0 0 0" />
       <geometry>
-        <mesh filename="package://mobipick_gazebo/meshes/screwdriver.dae" scale="1 1 1" />
+        <mesh filename="package://pbr_objects/meshes/screwdriver/screwdriver.obj" scale="1 1 1" />
       </geometry>
     </visual>

Commit message: Move simplified collision meshes to pbr_objects

File: mobipick_gazebo/urdf/klt.urdf.xacro (robot description, xacro)
@@ -23,5 +23,5 @@
       <origin xyz="0 0 0" rpy="0 0 0" />
       <geometry>
-        <mesh filename="package://mobipick_gazebo/meshes/collision/klt.stl" />
+        <mesh filename="package://pbr_objects/meshes/klt/klt_simplified.stl" />
       </geometry>
     </collision>-->

File: mobipick_gazebo/urdf/multimeter.urdf.xacro (robot description, xacro)
@@ -26,5 +26,5 @@
       <geometry>
          <box size="${bb_size_x} ${bb_size_y} ${bb_size_z}" />
-        <!--<mesh filename="package://mobipick_gazebo/meshes/collision//multimeter.stl" />-->
+        <!--<mesh filename="package://pbr_objects/meshes/multimeter//multimeter_simplified.stl" />-->
       </geometry>
     </collision>

File: mobipick_gazebo/urdf/power_drill_with_grip.urdf.xacro (robot description, xacro)
@@ -23,5 +23,5 @@
       <origin xyz="0 0 0" rpy="0 0 0" />
       <geometry>
-        <mesh filename="package://pbr_objects/meshes/power_drill_with_grip/power_drill_with_grip.stl" />
+        <mesh filename="package://pbr_objects/meshes/power_drill_with_grip/power_drill_with_grip_simplified.stl" />
       </geometry>
     </collision>

File: mobipick_gazebo/urdf/relay.urdf.xacro (robot description, xacro)
@@ -26,5 +26,5 @@
       <geometry>
          <box size="${bb_size_x} ${bb_size_y} ${bb_size_z}" />
-        <!--<mesh filename="package://mobipick_gazebo/meshes/collision/relay.stl" />-->
+        <!--<mesh filename="package://pbr_objects/meshes/relay/relay_simplified.stl" />-->
       </geometry>
     </collision>

File: mobipick_gazebo/urdf/screwdriver.urdf.xacro (robot description, xacro)
@@ -26,5 +26,5 @@
       <geometry>
         <box size="${bb_size_x} ${bb_size_y} ${bb_size_z}" />
-        <!-- mesh filename="package://mobipick_gazebo/meshes/collision/screwdriver.stl" / -->
+        <!-- mesh filename="package://pbr_objects/meshes/screwdriver/screwdriver_simplified.stl" / -->
       </geometry>
     </collision>
