Commit message: Adapted grasp poses for YCB objects, changed collision of soup can to cylinder

File: mobipick_gazebo/urdf/tomato_soup_can.urdf.xacro (robot description, xacro)
@@ -2,11 +2,11 @@
   <xacro:include filename="$(find mobipick_description)/urdf/common_properties.urdf.xacro" />
   <xacro:property name="mass" value="0.01" /><!-- TODO Measure mass -->
-  <xacro:property name="bb_size_x" value="0.06766" />
-  <xacro:property name="bb_size_y" value="0.10186" />
-  <xacro:property name="bb_size_z" value="0.06771" />
-  <xacro:macro name="box_inertia" params="m x y z">
-    <inertia   ixx="${m*(y*y+z*z)/12}" ixy = "0" ixz = "0"
-               iyy="${m*(x*x+z*z)/12}" iyz = "0"
-               izz="${m*(x*x+y*y)/12}" />
+  <xacro:property name="radius" value="0.034" />
+  <xacro:property name="height" value="0.10186" />
+  <xacro:macro name="cylinder_inertia" params="m r h">
+    <inertia  ixx="${m*(3*r*r+h*h)/12}" ixy = "0" ixz = "0"
+              iyy="${m*(3*r*r+h*h)/12}" iyz = "0"
+              izz="${m*r*r/2}"
+     />
   </xacro:macro>
   <link name="tomato_soup_can">
@@ -14,5 +14,5 @@
       <origin xyz="0 0 0" rpy="0 0 0" />
       <mass value="${mass}" />
-      <xacro:box_inertia m="${mass}" x="${bb_size_x}" y="${bb_size_y}" z="${bb_size_z}" />
+      <xacro:cylinder_inertia m="${mass}" r="${radius}" h="${height}" />
     </inertial>
     <visual>
@@ -23,7 +23,7 @@
     </visual>
     <collision>
-      <origin xyz="0 0 0" rpy="0 0 0" />
+      <origin xyz="0 0 0" rpy="1.57 0 0" />
       <geometry>
-         <box size="${bb_size_x} ${bb_size_y} ${bb_size_z}" />
+         <cylinder radius="${radius}" length="${height}" />
         <!--<mesh filename="package://pbr_objects/meshes/005_tomato_soup_can/005_tomato_soup_can.stl" />-->
       </geometry>
