Commit message: gazebo: Add barriers to tables

File: mobipick_gazebo/urdf/conf_room_table.urdf.xacro (robot description, xacro)
@@ -1,5 +1,41 @@
 <?xml version="1.0"?>
 <robot xmlns:xacro="http://ros.org/wiki/xacro" name="table">
+  <xacro:property name="width"               value="1.40" />
+  <xacro:property name="depth"               value="0.70" />
+  <xacro:property name="height"              value="0.72" />
+  <xacro:property name="leg_radius"          value="0.02" />
+  <xacro:property name="table_top_thickness" value="0.05" />
+  <xacro:property name="x"                   value="0.0" />
+  <xacro:property name="y"                   value="0.0" />
+  <xacro:property name="z"                   value="0.0" />
+  <xacro:property name="barrier_width"       value="${width + 2*leg_radius}" />
+  <xacro:property name="barrier_depth"       value="0.01" />
+  <xacro:property name="barrier_height"      value="0.30" />
   <xacro:include filename="$(find mobipick_gazebo)/urdf/include/table.urdf.xacro" />
-  <xacro:table height="0.72" width="1.40" depth="0.70" leg_radius="0.02" table_top_thickness="0.05" x="0.0" y="0.0" z="0.0" />
+  <xacro:table height="${height}" width="${width}" depth="${depth}" leg_radius="${leg_radius}" table_top_thickness="${table_top_thickness}" x="${x}" y="${y}" z="${z}" />
+  <joint name="barrier_joint" type="fixed" >
+    <parent link="table_top_link" />
+    <origin xyz="${x} ${y + depth/2 + leg_radius + barrier_depth/2} ${z + barrier_height/2}" rpy="0 0 0" />
+    <child link="barrier_link" />
+  </joint>
+  <link name="barrier_link">
+    <xacro:box_inertial x="${barrier_width}" y="${barrier_depth}" z="${barrier_height}" mass="10">
+      <origin xyz="0 0 0" />
+    </xacro:box_inertial>
+    <visual>
+      <origin xyz="0 0 0" />
+      <geometry>
+        <box size="${barrier_width} ${barrier_depth} ${barrier_height}" />
+      </geometry>
+    </visual>
+    <collision>
+      <origin xyz="0 0 0" />
+      <geometry>
+        <box size="${barrier_width} ${barrier_depth} ${barrier_height}" />
+      </geometry>
+    </collision>
+  </link>
+  <gazebo reference="barrier_link">
+    <material>Gazebo/Wood</material>
+  </gazebo>
 </robot>

Commit message: update tables demo gazebo environment to reflect current situation, now we have 3 tables placed on the corner

File: mobipick_gazebo/urdf/conf_room_table.urdf.xacro (robot description, xacro)
@@ -11,14 +11,14 @@
   <xacro:property name="barrier_width"       value="${width + 2*leg_radius}" />
   <xacro:property name="barrier_depth"       value="0.01" />
-  <xacro:property name="barrier_height"      value="0.30" />
+  <xacro:property name="barrier_height"      value="0.05" />
   <xacro:include filename="$(find mobipick_gazebo)/urdf/include/table.urdf.xacro" />
   <xacro:table height="${height}" width="${width}" depth="${depth}" leg_radius="${leg_radius}" table_top_thickness="${table_top_thickness}" x="${x}" y="${y}" z="${z}" />
   <joint name="barrier_joint" type="fixed" >
     <parent link="table_top_link" />
-    <origin xyz="${x} ${y + depth/2 + leg_radius + barrier_depth/2} ${z + barrier_height/2}" rpy="0 0 0" />
+    <origin xyz="${x} ${y + depth/2 + leg_radius + barrier_depth/2} 0.19" rpy="0 0 0" />
     <child link="barrier_link" />
   </joint>
   <link name="barrier_link">
-    <xacro:box_inertial x="${barrier_width}" y="${barrier_depth}" z="${barrier_height}" mass="10">
+    <xacro:box_inertial x="${barrier_width}" y="${barrier_depth}" z="${barrier_height}" mass="0.2">
       <origin xyz="0 0 0" />
     </xacro:box_inertial>
@@ -37,5 +37,5 @@
   </link>
   <gazebo reference="barrier_link">
-    <material>Gazebo/Wood</material>
+    <material>Gazebo/Black</material>
   </gazebo>
 </robot>

File: mobipick_gazebo/urdf/include/table.urdf.xacro (robot description, xacro)
@@ -50,5 +50,5 @@
     </link>
     <gazebo reference="leg1_link">
-      <material>Gazebo/Red</material>
+      <material>Gazebo/Grey</material>
     </gazebo>
     <joint name="leg2_joint" type="fixed" >
@@ -75,5 +75,5 @@
     </link>
     <gazebo reference="leg2_link">
-      <material>Gazebo/Red</material>
+      <material>Gazebo/Grey</material>
     </gazebo>
     <joint name="leg3_joint" type="fixed" >
@@ -100,5 +100,5 @@
     </link>
     <gazebo reference="leg3_link">
-      <material>Gazebo/Red</material>
+      <material>Gazebo/Grey</material>
     </gazebo>
     <joint name="leg4_joint" type="fixed" >
@@ -125,5 +125,5 @@
     </link>
     <gazebo reference="leg4_link">
-      <material>Gazebo/Red</material>
+      <material>Gazebo/Grey</material>
     </gazebo>
     <gazebo>

Commit message: gazebo tables_demo: Adjust to real environment
* shift tables to match the virtual_walls map from the real MiR
* move and rotate power drill so it is reachable by the robot for the
  pick_and_place demo
* shift barriers towards center of the table, like on the real tables

File: mobipick_gazebo/urdf/conf_room_table.urdf.xacro (robot description, xacro)
@@ -12,9 +12,12 @@
   <xacro:property name="barrier_depth"       value="0.01" />
   <xacro:property name="barrier_height"      value="0.05" />
+  <xacro:property name="barrier_x"           value="${x}" />
+  <xacro:property name="barrier_y"           value="${y + 0.10}" />
+  <xacro:property name="barrier_z"           value="${z + 0.19}" />
   <xacro:include filename="$(find mobipick_gazebo)/urdf/include/table.urdf.xacro" />
   <xacro:table height="${height}" width="${width}" depth="${depth}" leg_radius="${leg_radius}" table_top_thickness="${table_top_thickness}" x="${x}" y="${y}" z="${z}" />
   <joint name="barrier_joint" type="fixed" >
     <parent link="table_top_link" />
-    <origin xyz="${x} ${y + depth/2 + leg_radius + barrier_depth/2} 0.19" rpy="0 0 0" />
+    <origin xyz="${barrier_x} ${barrier_y} ${barrier_z}" rpy="0 0 0" />
     <child link="barrier_link" />
   </joint>

Commit message: gazebo tables_demo: Move table legs to match our tables

File: mobipick_gazebo/urdf/conf_room_table.urdf.xacro (robot description, xacro)
@@ -4,17 +4,18 @@
   <xacro:property name="depth"               value="0.70" />
   <xacro:property name="height"              value="0.72" />
-  <xacro:property name="leg_radius"          value="0.02" />
+  <xacro:property name="leg_radius"          value="0.015" />
+  <xacro:property name="leg_offet"           value="0.275" />
   <xacro:property name="table_top_thickness" value="0.05" />
   <xacro:property name="x"                   value="0.0" />
   <xacro:property name="y"                   value="0.0" />
   <xacro:property name="z"                   value="0.0" />
-  <xacro:property name="barrier_width"       value="${width + 2*leg_radius}" />
+  <xacro:property name="barrier_width"       value="${width}" />
   <xacro:property name="barrier_depth"       value="0.01" />
-  <xacro:property name="barrier_height"      value="0.05" />
+  <xacro:property name="barrier_height"      value="0.14" />
   <xacro:property name="barrier_x"           value="${x}" />
-  <xacro:property name="barrier_y"           value="${y + 0.10}" />
+  <xacro:property name="barrier_y"           value="${y + depth/2 + leg_radius - leg_offet + barrier_depth/2}" />
   <xacro:property name="barrier_z"           value="${z + 0.19}" />
   <xacro:include filename="$(find mobipick_gazebo)/urdf/include/table.urdf.xacro" />
-  <xacro:table height="${height}" width="${width}" depth="${depth}" leg_radius="${leg_radius}" table_top_thickness="${table_top_thickness}" x="${x}" y="${y}" z="${z}" />
+  <xacro:table height="${height}" width="${width}" depth="${depth}" leg_radius="${leg_radius}" leg_offet="${leg_offet}" table_top_thickness="${table_top_thickness}" x="${x}" y="${y}" z="${z}" />
   <joint name="barrier_joint" type="fixed" >
     <parent link="table_top_link" />

File: mobipick_gazebo/urdf/include/table.urdf.xacro (robot description, xacro)
@@ -2,5 +2,5 @@
 <robot xmlns:xacro="http://ros.org/wiki/xacro">
   <xacro:include filename="$(find mobipick_description)/urdf/common_properties.urdf.xacro" />
-  <xacro:macro name="table" params="height:=0.72 width:=0.80 depth:=0.80 leg_radius:=0.02 table_top_thickness:=0.05 x:=0.0 y:=0.0 z:=0.0">
+  <xacro:macro name="table" params="height:=0.72 width:=0.80 depth:=0.80 leg_radius:=0.02 leg_offet:=0.0 table_top_thickness:=0.05 x:=0.0 y:=0.0 z:=0.0">
     <link name="table_top_link">
       <xacro:box_inertial x="${width}" y="${depth}" z="${table_top_thickness}" mass="10">
@@ -29,5 +29,5 @@
     <joint name="leg1_joint" type="fixed" >
       <parent link="table_top_link" />
-      <origin xyz="${x + width/2} ${y + depth/2} ${z + height}" rpy="0 0 0" />
+      <origin xyz="${x + width/2} ${y + depth/2 - leg_offet} ${z + height}" rpy="0 0 0" />
       <child link="leg1_link" />
     </joint>
@@ -54,5 +54,5 @@
     <joint name="leg2_joint" type="fixed" >
       <parent link="table_top_link" />
-      <origin xyz="${x - width/2} ${y + depth/2} ${z + height}" rpy="0 0 0" />
+      <origin xyz="${x - width/2} ${y + depth/2 - leg_offet} ${z + height}" rpy="0 0 0" />
       <child link="leg2_link" />
     </joint>
@@ -79,5 +79,5 @@
     <joint name="leg3_joint" type="fixed" >
       <parent link="table_top_link" />
-      <origin xyz="${x + width/2} ${y - depth/2} ${z + height}" rpy="0 0 0" />
+      <origin xyz="${x + width/2} ${y - depth/2 + leg_offet} ${z + height}" rpy="0 0 0" />
       <child link="leg3_link" />
     </joint>
@@ -104,5 +104,5 @@
     <joint name="leg4_joint" type="fixed" >
       <parent link="table_top_link" />
-      <origin xyz="${x - width/2} ${y - depth/2} ${z + height}" rpy="0 0 0" />
+      <origin xyz="${x - width/2} ${y - depth/2 + leg_offet} ${z + height}" rpy="0 0 0" />
       <child link="leg4_link" />
     </joint>

Commit message: made conf_room_table.urdf parameters configureable

File: mobipick_gazebo/urdf/conf_room_table.urdf.xacro (robot description, xacro)
@@ -1,21 +1,30 @@
 <?xml version="1.0"?>
 <robot xmlns:xacro="http://ros.org/wiki/xacro" name="table">
-  <xacro:property name="width"               value="1.40" />
-  <xacro:property name="depth"               value="0.70" />
-  <xacro:property name="height"              value="0.72" />
-  <xacro:property name="leg_radius"          value="0.015" />
-  <xacro:property name="leg_offet"           value="0.275" />
-  <xacro:property name="table_top_thickness" value="0.05" />
-  <xacro:property name="x"                   value="0.0" />
-  <xacro:property name="y"                   value="0.0" />
-  <xacro:property name="z"                   value="0.0" />
+  <xacro:arg name="width"               default="1.40" />
+  <xacro:arg name="depth"               default="0.70" />
+  <xacro:arg name="height"              default="0.72" />
+  <xacro:arg name="leg_radius"          default="0.015" />
+  <xacro:arg name="leg_offset"           default="0.275" />
+  <xacro:arg name="table_top_thickness" default="0.05" />
+  <xacro:arg name="x"                   default="0.0" />
+  <xacro:arg name="y"                   default="0.0" />
+  <xacro:arg name="z"                   default="0.0" />
+  <xacro:property name="width"               value="$(arg width)" />
+  <xacro:property name="depth"               value="$(arg depth)" />
+  <xacro:property name="height"              value="$(arg height)" />
+  <xacro:property name="leg_radius"          value="$(arg leg_radius)" />
+  <xacro:property name="leg_offset"           value="$(arg leg_offset)" />
+  <xacro:property name="table_top_thickness" value="$(arg table_top_thickness)" />
+  <xacro:property name="x"                   value="$(arg x)" />
+  <xacro:property name="y"                   value="$(arg y)" />
+  <xacro:property name="z"                   value="$(arg z)" />
   <xacro:property name="barrier_width"       value="${width}" />
   <xacro:property name="barrier_depth"       value="0.01" />
   <xacro:property name="barrier_height"      value="0.14" />
   <xacro:property name="barrier_x"           value="${x}" />
-  <xacro:property name="barrier_y"           value="${y + depth/2 + leg_radius - leg_offet + barrier_depth/2}" />
+  <xacro:property name="barrier_y"           value="${y + depth/2 + leg_radius - leg_offset + barrier_depth/2}" />
   <xacro:property name="barrier_z"           value="${z + 0.19}" />
   <xacro:include filename="$(find mobipick_gazebo)/urdf/include/table.urdf.xacro" />
-  <xacro:table height="${height}" width="${width}" depth="${depth}" leg_radius="${leg_radius}" leg_offet="${leg_offet}" table_top_thickness="${table_top_thickness}" x="${x}" y="${y}" z="${z}" />
+  <xacro:table height="${height}" width="${width}" depth="${depth}" leg_radius="${leg_radius}" leg_offset="${leg_offset}" table_top_thickness="${table_top_thickness}" x="${x}" y="${y}" z="${z}" />
   <joint name="barrier_joint" type="fixed" >
     <parent link="table_top_link" />

Commit message: cic_tables gazebo: Remove table laser scan barriers
These were removed in reality, so this commit updates the Gazebo
simulation accordingly. Turns out they are not needed; localization
works fine without them (on the real robot).

File: mobipick_gazebo/urdf/conf_room_table.urdf.xacro (robot description, xacro)
@@ -10,4 +10,5 @@
   <xacro:arg name="y"                   default="0.0" />
   <xacro:arg name="z"                   default="0.0" />
+  <xacro:arg name="with_barrier"        default="true" />
   <xacro:property name="width"               value="$(arg width)" />
   <xacro:property name="depth"               value="$(arg depth)" />
@@ -19,4 +20,5 @@
   <xacro:property name="y"                   value="$(arg y)" />
   <xacro:property name="z"                   value="$(arg z)" />
+  <xacro:property name="with_barrier"        value="$(arg with_barrier)" />
   <xacro:property name="barrier_width"       value="${width}" />
   <xacro:property name="barrier_depth"       value="0.01" />
@@ -27,28 +29,30 @@
   <xacro:include filename="$(find mobipick_gazebo)/urdf/include/table.urdf.xacro" />
   <xacro:table height="${height}" width="${width}" depth="${depth}" leg_radius="${leg_radius}" leg_offset="${leg_offset}" table_top_thickness="${table_top_thickness}" x="${x}" y="${y}" z="${z}" />
-  <joint name="barrier_joint" type="fixed" >
-    <parent link="table_top_link" />
-    <origin xyz="${barrier_x} ${barrier_y} ${barrier_z}" rpy="0 0 0" />
-    <child link="barrier_link" />
-  </joint>
-  <link name="barrier_link">
-    <xacro:box_inertial x="${barrier_width}" y="${barrier_depth}" z="${barrier_height}" mass="0.2">
-      <origin xyz="0 0 0" />
-    </xacro:box_inertial>
-    <visual>
-      <origin xyz="0 0 0" />
-      <geometry>
-        <box size="${barrier_width} ${barrier_depth} ${barrier_height}" />
-      </geometry>
-    </visual>
-    <collision>
-      <origin xyz="0 0 0" />
-      <geometry>
-        <box size="${barrier_width} ${barrier_depth} ${barrier_height}" />
-      </geometry>
-    </collision>
-  </link>
-  <gazebo reference="barrier_link">
-    <material>Gazebo/Black</material>
-  </gazebo>
+  <xacro:if value="${with_barrier}">
+    <joint name="barrier_joint" type="fixed" >
+      <parent link="table_top_link" />
+      <origin xyz="${barrier_x} ${barrier_y} ${barrier_z}" rpy="0 0 0" />
+      <child link="barrier_link" />
+    </joint>
+    <link name="barrier_link">
+      <xacro:box_inertial x="${barrier_width}" y="${barrier_depth}" z="${barrier_height}" mass="0.2">
+        <origin xyz="0 0 0" />
+      </xacro:box_inertial>
+      <visual>
+        <origin xyz="0 0 0" />
+        <geometry>
+          <box size="${barrier_width} ${barrier_depth} ${barrier_height}" />
+        </geometry>
+      </visual>
+      <collision>
+        <origin xyz="0 0 0" />
+        <geometry>
+          <box size="${barrier_width} ${barrier_depth} ${barrier_height}" />
+        </geometry>
+      </collision>
+    </link>
+    <gazebo reference="barrier_link">
+      <material>Gazebo/Black</material>
+    </gazebo>
+  </xacro:if>
 </robot>
