Commit message: Use includes for static objects, add more

File: mobipick_gazebo/urdf/static/static_multimeter.urdf.xacro (robot description, xacro)
@@ -1,32 +1,4 @@
 <robot  xmlns:xacro="http://ros.org/wiki/xacro" name="multimeter_model">
-  <xacro:include filename="$(find mobipick_description)/urdf/common_properties.urdf.xacro" />
-  <xacro:property name="mass" value="0.1" />
-  <xacro:property name="bb_width" value="0.042" />
-  <xacro:property name="bb_length" value="0.086" />
-  <xacro:property name="bb_height" value="0.177" />
-  <xacro:macro name="box_inertia" params="m x y z">
-    <inertia   ixx="${m*(y*y+z*z)/12}" ixy = "0" ixz = "0"
-               iyy="${m*(x*x+z*z)/12}" iyz = "0"
-               izz="${m*(x*x+y*y)/12}" />
-  </xacro:macro>
-  <link name="multimeter">
-    <inertial>
-      <origin xyz="0 0 0" rpy="0 0 0" />
-      <mass value="${mass}" />
-      <xacro:box_inertia m="${mass}" x="${bb_height}" y="${bb_length}" z="${bb_width}" />
-    </inertial>
-    <visual>
-      <origin xyz="0 0 0" rpy="-1.5708 0 0" />
-      <geometry>
-        <mesh filename="package://mobipick_gazebo/meshes/multimeter.dae" scale="1 1 1" />
-      </geometry>
-    </visual>
-    <collision>
-      <origin xyz="0 0 0" rpy="0 0 0" />
-      <geometry>
-        <box size="${bb_height} ${bb_width} ${bb_length}"/>
-      </geometry>
-    </collision>
-  </link>
+  <xacro:include filename="$(find mobipick_gazebo)/urdf/multimeter.urdf.xacro" />
   <gazebo>
     <static>true</static>

File: mobipick_gazebo/urdf/static/static_relay.urdf.xacro (robot description, xacro)
@@ -1,32 +1,4 @@
 <robot  xmlns:xacro="http://ros.org/wiki/xacro" name="relay_model">
-  <xacro:include filename="$(find mobipick_description)/urdf/common_properties.urdf.xacro" />
-  <xacro:property name="mass" value="0.1" />
-  <xacro:property name="bb_width" value="0.106" />
-  <xacro:property name="bb_length" value="0.046" />
-  <xacro:property name="bb_height" value="0.056" />
-  <xacro:macro name="box_inertia" params="m x y z">
-    <inertia   ixx="${m*(y*y+z*z)/12}" ixy = "0" ixz = "0"
-               iyy="${m*(x*x+z*z)/12}" iyz = "0"
-               izz="${m*(x*x+y*y)/12}" />
-  </xacro:macro>
-  <link name="relay">
-    <inertial>
-      <origin xyz="0 0 0" rpy="0 0 1.57" />
-      <mass value="${mass}" />
-      <xacro:box_inertia m="${mass}" x="${bb_width}" y="${bb_length}" z="${bb_height}" />
-    </inertial>
-    <visual>
-      <origin xyz="0 -0.015 0" rpy="-1.5708 0 0" />
-      <geometry>
-        <mesh filename="package://mobipick_gazebo/meshes/relay.dae" scale="1 1 1" />
-      </geometry>
-    </visual>
-    <collision>
-      <origin xyz="0 0 0" rpy="0 0 0" />
-      <geometry>
-        <box size="${bb_height} ${bb_width} ${bb_length}" />
-      </geometry>
-    </collision>
-  </link>
+  <xacro:include filename="$(find mobipick_gazebo)/urdf/relay.urdf.xacro" />
   <gazebo>
     <static>true</static>

File: mobipick_gazebo/urdf/static/static_screwdriver.urdf.xacro (robot description, xacro)
@@ -1,32 +1,4 @@
 <robot  xmlns:xacro="http://ros.org/wiki/xacro" name="screwdriver_model">
-  <xacro:include filename="$(find mobipick_description)/urdf/common_properties.urdf.xacro" />
-  <xacro:property name="mass" value="0.1" />
-  <xacro:property name="bb_width" value="0.036" />
-  <xacro:property name="bb_length" value="0.036" />
-  <xacro:property name="bb_height" value="0.24" />
-  <xacro:macro name="box_inertia" params="m x y z">
-    <inertia   ixx="${m*(y*y+z*z)/12}" ixy = "0" ixz = "0"
-               iyy="${m*(x*x+z*z)/12}" iyz = "0"
-               izz="${m*(x*x+y*y)/12}" />
-  </xacro:macro>
-  <link name="screwdriver">
-    <inertial>
-      <origin xyz="0 0 0" rpy="0 0 1.57" />
-      <mass value="${mass}" />
-      <xacro:box_inertia m="${mass}" x="${bb_width}" y="${bb_length}" z="${bb_height}" />
-    </inertial>
-    <visual>
-        <origin xyz="0 0 0" rpy="-1.5708 0 0" />
-      <geometry>
-        <mesh filename="package://mobipick_gazebo/meshes/screwdriver.dae" scale="1 1 1" />
-      </geometry>
-    </visual>
-    <collision>
-      <origin xyz="0 0 0" rpy="0 0 0" />
-      <geometry>
-        <box size="${bb_height} ${bb_width} ${bb_length}" />
-      </geometry>
-    </collision>
-  </link>
+  <xacro:include filename="$(find mobipick_gazebo)/urdf/screwdriver.urdf.xacro" />
   <gazebo>
     <static>true</static>
