Commit message: table.urdf: Fix inertials
This doesn't really matter at the moment, because we set "static" to
"true". Better to fix it anyway.

File: mobipick_gazebo/urdf/include/table.urdf.xacro (robot description, xacro)
@@ -1,13 +1,10 @@
 <?xml version="1.0"?>
 <robot xmlns:xacro="http://ros.org/wiki/xacro">
+  <xacro:include filename="$(find mobipick_description)/urdf/common_properties.urdf.xacro" />
   <xacro:macro name="table" params="height:=0.72 width:=0.80 depth:=0.80 leg_radius:=0.02 table_top_thickness:=0.05 x:=0.0 y:=0.0 z:=0.0">
     <link name="table_top_link">
-      <inertial>
-        <mass value="1.0" />
+      <xacro:box_inertial x="${width}" y="${depth}" z="${table_top_thickness}" mass="10">
         <origin xyz="${x} ${y} ${z + height - table_top_thickness/2}" />
-        <inertia ixx="1" ixy="0"  ixz="0"
-                 iyy="1" iyz="0"
-                 izz="1" />
-      </inertial>
+      </xacro:box_inertial>
       <visual>
         <origin xyz="${x} ${y} ${z + height - table_top_thickness/2}" />
@@ -36,11 +33,7 @@
     </joint>
     <link name="leg1_link">
-      <inertial>
-        <mass value="1.0" />
+      <xacro:cylinder_inertial radius="${leg_radius}" length="${height}" mass="2.0">
         <origin xyz="0 0 ${-height/2}" />
-        <inertia ixx="0.1" ixy="0"  ixz="0"
-                 iyy="0.1" iyz="0"
-                 izz="0.01" />
-      </inertial>
+      </xacro:cylinder_inertial>
       <visual>
         <origin xyz="0.0 0.0 ${-height/2}" rpy="0 0 0" />
@@ -65,11 +58,7 @@
     </joint>
     <link name="leg2_link">
-      <inertial>
-        <mass value="1.0" />
+      <xacro:cylinder_inertial radius="${leg_radius}" length="${height}" mass="2.0">
         <origin xyz="0 0 ${-height/2}" />
-        <inertia ixx="0.1" ixy="0"  ixz="0"
-                 iyy="0.1" iyz="0"
-                 izz="0.01" />
-      </inertial>
+      </xacro:cylinder_inertial>
       <visual>
         <origin xyz="0.0 0.0 ${-height/2}" rpy="0 0 0" />
@@ -94,11 +83,7 @@
     </joint>
     <link name="leg3_link">
-      <inertial>
-        <mass value="1.0" />
+      <xacro:cylinder_inertial radius="${leg_radius}" length="${height}" mass="2.0">
         <origin xyz="0 0 ${-height/2}" />
-        <inertia ixx="0.1" ixy="0"  ixz="0"
-                 iyy="0.1" iyz="0"
-                 izz="0.01" />
-      </inertial>
+      </xacro:cylinder_inertial>
       <visual>
         <origin xyz="0.0 0.0 ${-height/2}" rpy="0 0 0" />
@@ -123,11 +108,7 @@
     </joint>
     <link name="leg4_link">
-      <inertial>
-        <mass value="1.0" />
+      <xacro:cylinder_inertial radius="${leg_radius}" length="${height}" mass="2.0">
         <origin xyz="0 0 ${-height/2}" />
-        <inertia ixx="0.1" ixy="0"  ixz="0"
-                 iyy="0.1" iyz="0"
-                 izz="0.01" />
-      </inertial>
+      </xacro:cylinder_inertial>
       <visual>
         <origin xyz="0.0 0.0 ${-height/2}" rpy="0 0 0" />
@@ -148,5 +129,4 @@
     <gazebo>
       <static>true</static>
-      <canonicalBody>table_top_link</canonicalBody>
     </gazebo>
   </xacro:macro>

Commit message: fixed typo in table leg_offset parameter

File: mobipick_gazebo/urdf/include/table.urdf.xacro (robot description, xacro)
@@ -2,5 +2,5 @@
 <robot xmlns:xacro="http://ros.org/wiki/xacro">
   <xacro:include filename="$(find mobipick_description)/urdf/common_properties.urdf.xacro" />
-  <xacro:macro name="table" params="height:=0.72 width:=0.80 depth:=0.80 leg_radius:=0.02 leg_offet:=0.0 table_top_thickness:=0.05 x:=0.0 y:=0.0 z:=0.0">
+  <xacro:macro name="table" params="height:=0.72 width:=0.80 depth:=0.80 leg_radius:=0.02 leg_offset:=0.0 table_top_thickness:=0.05 x:=0.0 y:=0.0 z:=0.0">
     <link name="table_top_link">
       <xacro:box_inertial x="${width}" y="${depth}" z="${table_top_thickness}" mass="10">
@@ -29,5 +29,5 @@
     <joint name="leg1_joint" type="fixed" >
       <parent link="table_top_link" />
-      <origin xyz="${x + width/2} ${y + depth/2 - leg_offet} ${z + height}" rpy="0 0 0" />
+      <origin xyz="${x + width/2} ${y + depth/2 - leg_offset} ${z + height}" rpy="0 0 0" />
       <child link="leg1_link" />
     </joint>
@@ -54,5 +54,5 @@
     <joint name="leg2_joint" type="fixed" >
       <parent link="table_top_link" />
-      <origin xyz="${x - width/2} ${y + depth/2 - leg_offet} ${z + height}" rpy="0 0 0" />
+      <origin xyz="${x - width/2} ${y + depth/2 - leg_offset} ${z + height}" rpy="0 0 0" />
       <child link="leg2_link" />
     </joint>
@@ -79,5 +79,5 @@
     <joint name="leg3_joint" type="fixed" >
       <parent link="table_top_link" />
-      <origin xyz="${x + width/2} ${y - depth/2 + leg_offet} ${z + height}" rpy="0 0 0" />
+      <origin xyz="${x + width/2} ${y - depth/2 + leg_offset} ${z + height}" rpy="0 0 0" />
       <child link="leg3_link" />
     </joint>
@@ -104,5 +104,5 @@
     <joint name="leg4_joint" type="fixed" >
       <parent link="table_top_link" />
-      <origin xyz="${x - width/2} ${y - depth/2 + leg_offet} ${z + height}" rpy="0 0 0" />
+      <origin xyz="${x - width/2} ${y - depth/2 + leg_offset} ${z + height}" rpy="0 0 0" />
       <child link="leg4_link" />
     </joint>
