Commit message: URDF: Adjust cable guide wrist clamp to real robot

File: mobipick_description/urdf/cable_guide/cable_guide.urdf.xacro (robot description, xacro)
@@ -12,5 +12,5 @@
   <xacro:property name="clamp_mass" value="0.50" />
   <xacro:property name="wrist_clamp_mass" value="0.200" />
-  <xacro:property name="wrist_clamp_yaw" value="0.2" />
+  <xacro:property name="wrist_clamp_yaw" value="0.36" />
   <xacro:property name="terminal_element_x_length" value="0.044" />
   <xacro:property name="terminal_element_y_length" value="0.045" />
@@ -210,5 +210,5 @@
     </link>
     <joint name="${prefix}cable_guide_wrist_3_tube_joint" type="fixed">
-      <origin xyz="0 0 ${-(0.05 / 2)}" rpy="0 0 0" />
+      <origin xyz="0 0 ${-(0.08 / 2)}" rpy="0 0 0" />
       <parent link="${prefix}cable_guide_terminal_element_link" />
       <child link="${prefix}cable_guide_wrist_3_tube_link" />
@@ -217,15 +217,15 @@
       <visual>
         <geometry>
-          <cylinder radius="${tube_radius}" length="0.05"/>
-        </geometry>
-        <xacro:insert_block name="material_black" />
-      </visual>
-      <collision>
-        <origin xyz="0 0 0" rpy="0 0 0" />
-        <geometry>
-          <cylinder radius="${tube_radius}" length="0.05"/>
-        </geometry>
-      </collision>
-      <xacro:cylinder_inertial radius="${tube_radius}" length="0.05" mass="${tube_mass}">
+          <cylinder radius="${tube_radius}" length="0.08"/>
+        </geometry>
+        <xacro:insert_block name="material_black" />
+      </visual>
+      <collision>
+        <origin xyz="0 0 0" rpy="0 0 0" />
+        <geometry>
+          <cylinder radius="${tube_radius}" length="0.08"/>
+        </geometry>
+      </collision>
+      <xacro:cylinder_inertial radius="${tube_radius}" length="0.08" mass="${tube_mass}">
         <origin xyz="0.0 0.0 0.0" rpy="0 0 0" />
       </xacro:cylinder_inertial>

Commit message: do not use cable_guide_wrist_3 for the hb-robot and forward robot/robot_version everywhere correctly

File: mobipick_description/urdf/cable_guide/cable_guide.urdf.xacro (robot description, xacro)
@@ -2,4 +2,7 @@
 <robot xmlns:xacro="http://ros.org/wiki/xacro">
   <xacro:include filename="$(find mobipick_description)/urdf/common_properties.urdf.xacro" />
+  <!-- cable guide on Wrist 3 is optional-->
+  <xacro:arg name="cable_guide_wrist_3" default="true" />
+  <xacro:property name="cable_guide_wrist_3" value="$(arg cable_guide_wrist_3)" />
   <!-- constants coped from ur_description: -->
   <xacro:property name="shoulder_offset" value="0.136" />
@@ -159,79 +162,81 @@
     </gazebo>
     <!-- wrist_3 -->
-    <joint name="${prefix}cable_guide_wrist_clamp_joint" type="fixed">
-      <origin xyz="0 0 -0.03" rpy="0 0 ${wrist_clamp_yaw}" />
-      <parent link="${prefix}ur5_wrist_3_link" />
-      <child link="${prefix}cable_guide_wrist_clamp_link" />
-    </joint>
-    <link name="${prefix}cable_guide_wrist_clamp_link">
-      <visual>
-        <geometry>
-          <mesh filename="package://mobipick_description/meshes/cable_guide/visual/wrist_clamp_TR_918_012.dae" />
-        </geometry>
-        <xacro:insert_block name="material_black" />
-      </visual>
-      <collision>
-        <geometry>
-          <mesh filename="package://mobipick_description/meshes/cable_guide/collision/wrist_clamp_TR_918_012.stl" />
-        </geometry>
-      </collision>
-      <inertial>
-        <mass value="${wrist_clamp_mass}" />
-        <origin xyz="0.0 0.05549427 -0.0" rpy="0 0 0" />
-        <inertia ixx="${wrist_clamp_mass *  0.0042434960684663275}"
-                 ixy="${wrist_clamp_mass * -2.2400373470288125e-06}"
-                 ixz="${wrist_clamp_mass *  4.4523467998712435e-08}"
-                 iyy="${wrist_clamp_mass *  0.0005344100748342659}"
-                 iyz="${wrist_clamp_mass * -5.1403149429916256e-08}"
-                 izz="${wrist_clamp_mass *  0.004767239872136627}" />
-      </inertial>
-    </link>
-    <joint name="${prefix}cable_guide_terminal_element_joint" type="fixed">
-      <origin xyz="-0.029 0.142 0.007" rpy="0 0 0" />
-      <parent link="${prefix}cable_guide_wrist_clamp_link" />
-      <child link="${prefix}cable_guide_terminal_element_link" />
-    </joint>
-    <link name="${prefix}cable_guide_terminal_element_link">
-      <visual>
-        <geometry>
-          <mesh filename="package://mobipick_description/meshes/cable_guide/visual/terminal_element_TL_30_01_Z1.dae" />
-        </geometry>
-        <xacro:insert_block name="material_black" />
-      </visual>
-      <collision>
-        <origin xyz="0 0 0" rpy="0 0 0" />
-        <geometry>
-          <box size="${terminal_element_x_length} ${terminal_element_y_length} ${terminal_element_z_length} " />
-        </geometry>
-      </collision>
-      <xacro:box_inertial x="${terminal_element_x_length}" y="${terminal_element_y_length}" z="${terminal_element_z_length}" mass="${terminal_element_mass}">
-        <origin xyz="0.0 0.0 0.0" rpy="0 0 0" />
-      </xacro:box_inertial>
-    </link>
-    <joint name="${prefix}cable_guide_wrist_3_tube_joint" type="fixed">
-      <origin xyz="0 0 ${-(0.08 / 2)}" rpy="0 0 0" />
-      <parent link="${prefix}cable_guide_terminal_element_link" />
-      <child link="${prefix}cable_guide_wrist_3_tube_link" />
-    </joint>
-    <link name="${prefix}cable_guide_wrist_3_tube_link">
-      <visual>
-        <geometry>
-          <cylinder radius="${tube_radius}" length="0.08"/>
-        </geometry>
-        <xacro:insert_block name="material_black" />
-      </visual>
-      <collision>
-        <origin xyz="0 0 0" rpy="0 0 0" />
-        <geometry>
-          <cylinder radius="${tube_radius}" length="0.08"/>
-        </geometry>
-      </collision>
-      <xacro:cylinder_inertial radius="${tube_radius}" length="0.08" mass="${tube_mass}">
-        <origin xyz="0.0 0.0 0.0" rpy="0 0 0" />
-      </xacro:cylinder_inertial>
-    </link>
-    <gazebo reference="${prefix}cable_guide_wrist_3_tube_link">
-      <material>Gazebo/FlatBlack</material>
-    </gazebo>
+    <xacro:if value="${cable_guide_wrist_3}">
+      <joint name="${prefix}cable_guide_wrist_clamp_joint" type="fixed">
+        <origin xyz="0 0 -0.03" rpy="0 0 ${wrist_clamp_yaw}" />
+        <parent link="${prefix}ur5_wrist_3_link" />
+        <child link="${prefix}cable_guide_wrist_clamp_link" />
+      </joint>
+      <link name="${prefix}cable_guide_wrist_clamp_link">
+        <visual>
+          <geometry>
+            <mesh filename="package://mobipick_description/meshes/cable_guide/visual/wrist_clamp_TR_918_012.dae" />
+          </geometry>
+          <xacro:insert_block name="material_black" />
+        </visual>
+        <collision>
+          <geometry>
+            <mesh filename="package://mobipick_description/meshes/cable_guide/collision/wrist_clamp_TR_918_012.stl" />
+          </geometry>
+        </collision>
+        <inertial>
+          <mass value="${wrist_clamp_mass}" />
+          <origin xyz="0.0 0.05549427 -0.0" rpy="0 0 0" />
+          <inertia ixx="${wrist_clamp_mass *  0.0042434960684663275}"
+                  ixy="${wrist_clamp_mass * -2.2400373470288125e-06}"
+                  ixz="${wrist_clamp_mass *  4.4523467998712435e-08}"
+                  iyy="${wrist_clamp_mass *  0.0005344100748342659}"
+                  iyz="${wrist_clamp_mass * -5.1403149429916256e-08}"
+                  izz="${wrist_clamp_mass *  0.004767239872136627}" />
+        </inertial>
+      </link>
+      <joint name="${prefix}cable_guide_terminal_element_joint" type="fixed">
+        <origin xyz="-0.029 0.142 0.007" rpy="0 0 0" />
+        <parent link="${prefix}cable_guide_wrist_clamp_link" />
+        <child link="${prefix}cable_guide_terminal_element_link" />
+      </joint>
+      <link name="${prefix}cable_guide_terminal_element_link">
+        <visual>
+          <geometry>
+            <mesh filename="package://mobipick_description/meshes/cable_guide/visual/terminal_element_TL_30_01_Z1.dae" />
+          </geometry>
+          <xacro:insert_block name="material_black" />
+        </visual>
+        <collision>
+          <origin xyz="0 0 0" rpy="0 0 0" />
+          <geometry>
+            <box size="${terminal_element_x_length} ${terminal_element_y_length} ${terminal_element_z_length} " />
+          </geometry>
+        </collision>
+        <xacro:box_inertial x="${terminal_element_x_length}" y="${terminal_element_y_length}" z="${terminal_element_z_length}" mass="${terminal_element_mass}">
+          <origin xyz="0.0 0.0 0.0" rpy="0 0 0" />
+        </xacro:box_inertial>
+      </link>
+      <joint name="${prefix}cable_guide_wrist_3_tube_joint" type="fixed">
+        <origin xyz="0 0 ${-(0.08 / 2)}" rpy="0 0 0" />
+        <parent link="${prefix}cable_guide_terminal_element_link" />
+        <child link="${prefix}cable_guide_wrist_3_tube_link" />
+      </joint>
+      <link name="${prefix}cable_guide_wrist_3_tube_link">
+        <visual>
+          <geometry>
+            <cylinder radius="${tube_radius}" length="0.08"/>
+          </geometry>
+          <xacro:insert_block name="material_black" />
+        </visual>
+        <collision>
+          <origin xyz="0 0 0" rpy="0 0 0" />
+          <geometry>
+            <cylinder radius="${tube_radius}" length="0.08"/>
+          </geometry>
+        </collision>
+        <xacro:cylinder_inertial radius="${tube_radius}" length="0.08" mass="${tube_mass}">
+          <origin xyz="0.0 0.0 0.0" rpy="0 0 0" />
+        </xacro:cylinder_inertial>
+      </link>
+      <gazebo reference="${prefix}cable_guide_wrist_3_tube_link">
+        <material>Gazebo/FlatBlack</material>
+      </gazebo>
+    </xacro:if>
   </xacro:macro>
 </robot>

File: mobipick_description/urdf/mobipick/mobipick_v1_model.urdf.xacro (robot description, xacro)
@@ -15,4 +15,6 @@
   <xacro:arg name="joint_limits_parameters_file" default="$(find mobipick_description)/config/joint_limits.yaml"/>  <!-- path the to the yaml with the ur5 joint limits. -->
   <xacro:arg name="kinematics_config" default="$(find mobipick_description)/config/ur5_calibration.yaml"/>  <!-- path the to the yaml with the arms calibration parameters. -->
+  <!-- mobipick-hb does not have a cable guide at the wrist, allowing it to take pictures facing up -->
+  <xacro:arg name="cable_guide_wrist_3" default="${str(robot == 'mobipick-os')}" />
   <!-- ############# MIR100 BASE ############## -->
   <xacro:include filename="$(find mir_description)/urdf/include/mir_100_v1.urdf.xacro" />

File: mobipick_moveit_config/config/mobipick.srdf.xacro (robot description, xacro)
@@ -15,4 +15,9 @@
         <xacro:property name="tf_prefix" value="${tf_prefix_}/"/>
     </xacro:unless>
+    <xacro:arg name="robot_version" default="os" />      <!-- can be "mobipick-hb" or "mobipick-os" -->
+    <xacro:property name="robot_version" value="$(arg robot_version)" />  <!-- necessary because args cannot be accessed inside ${} expressions -->
+    <!-- mobipick-hb does not have a cable guide at the wrist, allowing it to take pictures facing up -->
+    <xacro:arg name="cable_guide_wrist_3" default="${str(robot_version == 'os')}" />
+    <xacro:property name="cable_guide_wrist_3" value="$(arg cable_guide_wrist_3)" />
     <!--GROUPS: Representation of a set of joints and links. This can be useful for specifying DOF to plan for, defining arms, end effectors, etc-->
     <!--LINKS: When a link is specified, the parent joint of that link (if it exists) is automatically included-->
@@ -177,5 +182,7 @@
     <disable_collisions link1="${tf_prefix}back_laser_link" link2="${tf_prefix}cable_guide_terminal_element_link" reason="Never"/>
     <disable_collisions link1="${tf_prefix}back_laser_link" link2="${tf_prefix}cable_guide_upper_arm_tube_link" reason="Never"/>
+    <xacro:if value="${cable_guide_wrist_3}">
     <disable_collisions link1="${tf_prefix}back_laser_link" link2="${tf_prefix}cable_guide_wrist_3_tube_link" reason="Never"/>
+    </xacro:if>
     <disable_collisions link1="${tf_prefix}back_laser_link" link2="${tf_prefix}cable_guide_wrist_clamp_link" reason="Never"/>
     <disable_collisions link1="${tf_prefix}back_laser_link" link2="${tf_prefix}eef_forward_cam_link" reason="Never"/>
@@ -232,5 +239,7 @@
     <disable_collisions link1="${tf_prefix}base_link" link2="${tf_prefix}cable_guide_terminal_element_link" reason="User"/>
     <disable_collisions link1="${tf_prefix}base_link" link2="${tf_prefix}cable_guide_upper_arm_tube_link" reason="Never"/>
+    <xacro:if value="${cable_guide_wrist_3}">
     <disable_collisions link1="${tf_prefix}base_link" link2="${tf_prefix}cable_guide_wrist_3_tube_link" reason="User"/>
+    </xacro:if>
     <disable_collisions link1="${tf_prefix}base_link" link2="${tf_prefix}cable_guide_wrist_clamp_link" reason="User"/>
     <disable_collisions link1="${tf_prefix}base_link" link2="${tf_prefix}eef_forward_cam_link" reason="User"/>
@@ -286,5 +295,7 @@
     <disable_collisions link1="${tf_prefix}bl_caster_rotation_link" link2="${tf_prefix}cable_guide_terminal_element_link" reason="Never"/>
     <disable_collisions link1="${tf_prefix}bl_caster_rotation_link" link2="${tf_prefix}cable_guide_upper_arm_tube_link" reason="Never"/>
+    <xacro:if value="${cable_guide_wrist_3}">
     <disable_collisions link1="${tf_prefix}bl_caster_rotation_link" link2="${tf_prefix}cable_guide_wrist_3_tube_link" reason="Never"/>
+    </xacro:if>
     <disable_collisions link1="${tf_prefix}bl_caster_rotation_link" link2="${tf_prefix}cable_guide_wrist_clamp_link" reason="Never"/>
     <disable_collisions link1="${tf_prefix}bl_caster_rotation_link" link2="${tf_prefix}eef_forward_cam_link" reason="Never"/>
@@ -339,5 +350,7 @@
     <disable_collisions link1="${tf_prefix}bl_caster_wheel_link" link2="${tf_prefix}cable_guide_terminal_element_link" reason="Never"/>
     <disable_collisions link1="${tf_prefix}bl_caster_wheel_link" link2="${tf_prefix}cable_guide_upper_arm_tube_link" reason="Never"/>
+    <xacro:if value="${cable_guide_wrist_3}">
     <disable_collisions link1="${tf_prefix}bl_caster_wheel_link" link2="${tf_prefix}cable_guide_wrist_3_tube_link" reason="Never"/>
+    </xacro:if>
     <disable_collisions link1="${tf_prefix}bl_caster_wheel_link" link2="${tf_prefix}cable_guide_wrist_clamp_link" reason="Never"/>
     <disable_collisions link1="${tf_prefix}bl_caster_wheel_link" link2="${tf_prefix}eef_forward_cam_link" reason="Never"/>
@@ -391,5 +404,7 @@
     <disable_collisions link1="${tf_prefix}br_caster_rotation_link" link2="${tf_prefix}cable_guide_terminal_element_link" reason="Never"/>
     <disable_collisions link1="${tf_prefix}br_caster_rotation_link" link2="${tf_prefix}cable_guide_upper_arm_tube_link" reason="Never"/>
+    <xacro:if value="${cable_guide_wrist_3}">
     <disable_collisions link1="${tf_prefix}br_caster_rotation_link" link2="${tf_prefix}cable_guide_wrist_3_tube_link" reason="Never"/>
+    </xacro:if>
     <disable_collisions link1="${tf_prefix}br_caster_rotation_link" link2="${tf_prefix}cable_guide_wrist_clamp_link" reason="Never"/>
     <disable_collisions link1="${tf_prefix}br_caster_rotation_link" link2="${tf_prefix}eef_forward_cam_link" reason="Never"/>
@@ -442,5 +457,7 @@
     <disable_collisions link1="${tf_prefix}br_caster_wheel_link" link2="${tf_prefix}cable_guide_terminal_element_link" reason="Never"/>
     <disable_collisions link1="${tf_prefix}br_caster_wheel_link" link2="${tf_prefix}cable_guide_upper_arm_tube_link" reason="Never"/>
+    <xacro:if value="${cable_guide_wrist_3}">
     <disable_collisions link1="${tf_prefix}br_caster_wheel_link" link2="${tf_prefix}cable_guide_wrist_3_tube_link" reason="Never"/>
+    </xacro:if>
     <disable_collisions link1="${tf_prefix}br_caster_wheel_link" link2="${tf_prefix}cable_guide_wrist_clamp_link" reason="Never"/>
     <disable_collisions link1="${tf_prefix}br_caster_wheel_link" link2="${tf_prefix}eef_forward_cam_link" reason="Never"/>
@@ -522,5 +539,7 @@
     <disable_collisions link1="${tf_prefix}cable_guide_clamp2_link" link2="${tf_prefix}cable_guide_terminal_element_link" reason="Never"/>
     <disable_collisions link1="${tf_prefix}cable_guide_clamp2_link" link2="${tf_prefix}cable_guide_upper_arm_tube_link" reason="Default"/>
+    <xacro:if value="${cable_guide_wrist_3}">
     <disable_collisions link1="${tf_prefix}cable_guide_clamp2_link" link2="${tf_prefix}cable_guide_wrist_3_tube_link" reason="Never"/>
+    </xacro:if>
     <disable_collisions link1="${tf_prefix}cable_guide_clamp2_link" link2="${tf_prefix}cable_guide_wrist_clamp_link" reason="Never"/>
     <disable_collisions link1="${tf_prefix}cable_guide_clamp2_link" link2="${tf_prefix}eef_forward_cam_link" reason="Never"/>
@@ -564,5 +583,7 @@
     <disable_collisions link1="${tf_prefix}cable_guide_clamp3_link" link2="${tf_prefix}cable_guide_terminal_element_link" reason="Never"/>
     <disable_collisions link1="${tf_prefix}cable_guide_clamp3_link" link2="${tf_prefix}cable_guide_upper_arm_tube_link" reason="Never"/>
+    <xacro:if value="${cable_guide_wrist_3}">
     <disable_collisions link1="${tf_prefix}cable_guide_clamp3_link" link2="${tf_prefix}cable_guide_wrist_3_tube_link" reason="Never"/>
+    </xacro:if>
     <disable_collisions link1="${tf_prefix}cable_guide_clamp3_link" link2="${tf_prefix}cable_guide_wrist_clamp_link" reason="Never"/>
     <disable_collisions link1="${tf_prefix}cable_guide_clamp3_link" link2="${tf_prefix}eef_forward_cam_link" reason="Never"/>
@@ -636,5 +657,7 @@
     <disable_collisions link1="${tf_prefix}cable_guide_forearm_tube_link" link2="${tf_prefix}ur5_wrist_1_link" reason="Never"/>
     <disable_collisions link1="${tf_prefix}cable_guide_forearm_tube_link" link2="${tf_prefix}ur5_wrist_2_link" reason="Never"/>
+    <xacro:if value="${cable_guide_wrist_3}">
     <disable_collisions link1="${tf_prefix}cable_guide_terminal_element_link" link2="${tf_prefix}cable_guide_wrist_3_tube_link" reason="Adjacent"/>
+    </xacro:if>
     <disable_collisions link1="${tf_prefix}cable_guide_terminal_element_link" link2="${tf_prefix}cable_guide_wrist_clamp_link" reason="Adjacent"/>
     <disable_collisions link1="${tf_prefix}cable_guide_terminal_element_link" link2="${tf_prefix}eef_forward_cam_link" reason="Never"/>
@@ -693,4 +716,5 @@
     <disable_collisions link1="${tf_prefix}cable_guide_upper_arm_tube_link" link2="${tf_prefix}ur5_wrist_2_link" reason="Never"/>
     <disable_collisions link1="${tf_prefix}cable_guide_upper_arm_tube_link" link2="${tf_prefix}ur5_wrist_3_link" reason="Never"/>
+    <xacro:if value="${cable_guide_wrist_3}">
     <disable_collisions link1="${tf_prefix}cable_guide_wrist_3_tube_link" link2="${tf_prefix}cable_guide_wrist_clamp_link" reason="Never"/>
     <disable_collisions link1="${tf_prefix}cable_guide_wrist_3_tube_link" link2="${tf_prefix}eef_forward_cam_link" reason="Never"/>
@@ -724,4 +748,5 @@
     <disable_collisions link1="${tf_prefix}cable_guide_wrist_3_tube_link" link2="${tf_prefix}ur5_wrist_2_link" reason="Never"/>
     <disable_collisions link1="${tf_prefix}cable_guide_wrist_3_tube_link" link2="${tf_prefix}ur5_wrist_3_link" reason="Never"/>
+    </xacro:if>
     <disable_collisions link1="${tf_prefix}cable_guide_wrist_clamp_link" link2="${tf_prefix}eef_forward_cam_link" reason="Never"/>
     <disable_collisions link1="${tf_prefix}cable_guide_wrist_clamp_link" link2="${tf_prefix}eef_main_cam_link" reason="Default"/>
