Commit message: Big rename

File: mobipick_description/urdf/structure/mobipick_structure.urdf.xacro (robot description, xacro)
@@ -3,5 +3,5 @@
   <xacro:property name="pi" value="3.14159265" />
   <xacro:macro name="structure" params="prefix height">
-    <link name="${prefix}StructPartDown">
+    <link name="${prefix}part_down">
       <inertial>
         <origin xyz="0 0 0.3278534031" rpy="${1.5 * pi} ${0.5 * pi} ${0.5 * pi}" />
@@ -18,5 +18,5 @@
         <origin xyz="0 0 0" rpy="0 0 0" />
         <geometry>
-          <mesh filename="package://mobipick_description/meshes/structure/visual/PartDown.stl" />
+          <mesh filename="package://mobipick_description/meshes/structure/visual/part_down.stl" />
         </geometry>
         <material name="">
@@ -27,9 +27,9 @@
         <origin xyz="0 0 0" rpy="0 0 0" />
         <geometry>
-          <mesh filename="package://mobipick_description/meshes/structure/collision/PartDown.stl" />
+          <mesh filename="package://mobipick_description/meshes/structure/collision/part_down.stl" />
         </geometry>
       </collision>
     </link>
-    <link name="${prefix}StructPartUp">
+    <link name="${prefix}part_up">
       <inertial>
         <origin xyz="0 0 0.3535849057" rpy="${1.5 * pi} ${0.5 * pi} ${0.5 * pi}" />
@@ -46,5 +46,5 @@
         <origin xyz="0 0 0" rpy="0 0 0" />
         <geometry>
-          <mesh filename="package://mobipick_description/meshes/structure/visual/PartUp.stl" />
+          <mesh filename="package://mobipick_description/meshes/structure/visual/part_up.stl" />
         </geometry>
         <material name="">
@@ -55,9 +55,9 @@
         <origin xyz="0 0 0" rpy="0 0 0" />
         <geometry>
-          <mesh filename="package://mobipick_description/meshes/structure/collision/PartUp.stl" />
+          <mesh filename="package://mobipick_description/meshes/structure/collision/part_up.stl" />
         </geometry>
       </collision>
     </link>
-    <link name="${prefix}StructTischaufbau">
+    <link name="${prefix}pedestal">
       <inertial>
         <origin xyz="0 0 0.1532210441" rpy="${0.5 * pi} ${0.5 * pi} 0" />
@@ -74,5 +74,5 @@
         <origin xyz="0 0 0" rpy="0 0 0" />
         <geometry>
-          <mesh filename="package://mobipick_description/meshes/structure/visual/Tischaufbau.stl" />
+          <mesh filename="package://mobipick_description/meshes/structure/visual/pedestal.stl" />
         </geometry>
         <material name="">
@@ -83,13 +83,13 @@
         <origin xyz="0 0 0" rpy="0 0 0" />
         <geometry>
-          <mesh filename="package://mobipick_description/meshes/structure/collision/Tischaufbau.stl" />
+          <mesh filename="package://mobipick_description/meshes/structure/collision/pedestal.stl" />
         </geometry>
       </collision>
     </link>
-    <link name="${prefix}StructBaseSupport"/>
+    <link name="${prefix}pedestal_surface"/>
     <!-- <joint name="${prefix}structure_vertical_joint" type="prismatic">
       <origin xyz="0 0 ${0.04}" rpy="0 0 0" />
-      <parent link="${prefix}StructPartDown" />
-      <child link="${prefix}StructPartUp" />
+      <parent link="${prefix}part_down" />
+      <child link="${prefix}part_up" />
       <axis xyz="0 0 1" />
       <limit effort="1000.0" lower="0.01" upper="0.25" velocity="0.01"/>
@@ -97,18 +97,18 @@
     <joint name="${prefix}structure_vertical_joint" type="fixed">
       <origin xyz="0 0 ${0.04 + height}" rpy="0 0 0" />
-      <parent link="${prefix}StructPartDown" />
-      <child link="${prefix}StructPartUp" />
+      <parent link="${prefix}part_down" />
+      <child link="${prefix}part_up" />
       <axis xyz="0 0 1" />
     </joint>
     <joint name="${prefix}Tischaufbau_joint" type="fixed">
       <origin xyz="0 0 0.44" rpy="0 0 0" />
-      <parent link="${prefix}StructPartUp" />
-      <child link="${prefix}StructTischaufbau" />
+      <parent link="${prefix}part_up" />
+      <child link="${prefix}pedestal" />
       <axis xyz="0 0 1" />
     </joint>
     <joint name="${prefix}Tischaufbau_base_joint" type="fixed">
       <origin xyz="0 0 0.25" rpy="0 0 0" />
-      <parent link="${prefix}StructTischaufbau" />
-      <child link="${prefix}StructBaseSupport" />
+      <parent link="${prefix}pedestal" />
+      <child link="${prefix}pedestal_surface" />
       <axis xyz="0 0 1" />
     </joint>

File: mobipick_description/urdf/structure/mobipick_structure_model.urdf.xacro (robot description, xacro)
@@ -8,5 +8,5 @@
   <joint name="world_joint" type="fixed">
     <parent link="world" />
-    <child link="StructPartDown" />
+    <child link="part_down" />
     <origin xyz="0.0 0.0 0.0" rpy="0.0 0.0 0.0" />
   </joint>

Commit message: urdf: Move structure meshes to v1/

File: mobipick_description/urdf/structure/mobipick_structure.urdf.xacro (robot description, xacro)
@@ -18,5 +18,5 @@
         <origin xyz="0 0 0" rpy="0 0 0" />
         <geometry>
-          <mesh filename="package://mobipick_description/meshes/structure/visual/part_down.stl" />
+          <mesh filename="package://mobipick_description/meshes/structure/visual/v1/part_down.stl" />
         </geometry>
         <xacro:insert_block name="material_aluminum" />
@@ -25,5 +25,5 @@
         <origin xyz="0 0 0" rpy="0 0 0" />
         <geometry>
-          <mesh filename="package://mobipick_description/meshes/structure/collision/part_down.stl" />
+          <mesh filename="package://mobipick_description/meshes/structure/collision/v1/part_down.stl" />
         </geometry>
       </collision>
@@ -47,5 +47,5 @@
         <origin xyz="0 0 0" rpy="0 0 0" />
         <geometry>
-          <mesh filename="package://mobipick_description/meshes/structure/visual/part_up.stl" />
+          <mesh filename="package://mobipick_description/meshes/structure/visual/v1/part_up.stl" />
         </geometry>
         <xacro:insert_block name="material_aluminum" />
@@ -54,5 +54,5 @@
         <origin xyz="0 0 0" rpy="0 0 0" />
         <geometry>
-          <mesh filename="package://mobipick_description/meshes/structure/collision/part_up.stl" />
+          <mesh filename="package://mobipick_description/meshes/structure/collision/v1/part_up.stl" />
         </geometry>
       </collision>
@@ -76,5 +76,5 @@
         <origin xyz="0 0 0" rpy="0 0 0" />
         <geometry>
-          <mesh filename="package://mobipick_description/meshes/structure/visual/pedestal.stl" />
+          <mesh filename="package://mobipick_description/meshes/structure/visual/v1/pedestal.stl" />
         </geometry>
         <xacro:insert_block name="material_aluminum" />
@@ -83,5 +83,5 @@
         <origin xyz="0 0 0" rpy="0 0 0" />
         <geometry>
-          <mesh filename="package://mobipick_description/meshes/structure/collision/pedestal.stl" />
+          <mesh filename="package://mobipick_description/meshes/structure/collision/v1/pedestal.stl" />
         </geometry>
       </collision>

Commit message: urdf: Remove spurious axis defs for fixed joints

File: mobipick_description/urdf/structure/mobipick_structure.urdf.xacro (robot description, xacro)
@@ -106,5 +106,4 @@
       <parent link="${prefix}part_down" />
       <child link="${prefix}part_up" />
-      <axis xyz="0 0 1" />
     </joint>
     <joint name="${prefix}Tischaufbau_joint" type="fixed">
@@ -112,5 +111,4 @@
       <parent link="${prefix}part_up" />
       <child link="${prefix}pedestal" />
-      <axis xyz="0 0 1" />
     </joint>
     <xacro:if value="${variant == 'v1'}">
@@ -124,5 +122,4 @@
       <parent link="${prefix}pedestal" />
       <child link="${prefix}pedestal_surface" />
-      <axis xyz="0 0 1" />
     </joint>
   </xacro:macro>

Commit message: urdf: Add mobipick covers

File: mobipick_description/urdf/structure/mobipick_structure.urdf.xacro (robot description, xacro)
@@ -2,4 +2,9 @@
 <robot xmlns:xacro="http://ros.org/wiki/xacro">
   <xacro:include filename="$(find mobipick_description)/urdf/common_properties.urdf.xacro" />
+  <xacro:property name="structure_length" value="0.740" />   <!-- x -->
+  <xacro:property name="structure_width"  value="0.530" />   <!-- y -->
+  <xacro:property name="structure_height" value="0.538" />   <!-- z -->
+  <xacro:property name="cover_thickness"  value="0.004" />
+  <xacro:property name="cover_height"     value="0.528" />
   <!-- variant can be one of:
        - v1: The original Mobipick in Bremen, built for the Hybr-iT project
@@ -123,4 +128,144 @@
       <child link="${prefix}pedestal_surface" />
     </joint>
+    <xacro:if value="${variant == 'v2'}">
+      <!-- cover_front -->
+      <joint name="${prefix}cover_front_joint" type="fixed">
+        <origin xyz="${structure_length / 2 + cover_thickness / 2} 0 ${structure_height - cover_height / 2}" rpy="0 0 0" />
+        <parent link="${prefix}part_down" />
+        <child link="${prefix}cover_front_link" />
+      </joint>
+      <link name="${prefix}cover_front_link">
+        <xacro:box_inertial mass="1.648" x="${cover_thickness}" y="${structure_width + 2 * cover_thickness}" z="${cover_height}">
+          <origin xyz="0 0 0" />
+        </xacro:box_inertial>
+        <visual>
+          <origin xyz="0 0 0" rpy="0 0 0" />
+          <geometry>
+            <mesh filename="package://mobipick_description/meshes/structure/visual/v2/cover_short_side.dae" />
+          </geometry>
+        </visual>
+        <collision>
+          <origin xyz="0 0 0" rpy="0 0 0" />
+          <geometry>
+            <mesh filename="package://mobipick_description/meshes/structure/visual/v2/cover_short_side.dae" />
+          </geometry>
+        </collision>
+      </link>
+      <!-- cover_back -->
+      <joint name="${prefix}cover_back_joint" type="fixed">
+        <origin xyz="${-(structure_length / 2 + cover_thickness / 2)} 0 ${structure_height - cover_height / 2}" rpy="0 0 ${pi}" />
+        <parent link="${prefix}part_down" />
+        <child link="${prefix}cover_back_link" />
+      </joint>
+      <link name="${prefix}cover_back_link">
+        <xacro:box_inertial mass="1.648" x="${cover_thickness}" y="${structure_width + 2 * cover_thickness}" z="${cover_height}">
+          <origin xyz="0 0 0" />
+        </xacro:box_inertial>
+        <visual>
+          <origin xyz="0 0 0" rpy="0 0 0" />
+          <geometry>
+            <mesh filename="package://mobipick_description/meshes/structure/visual/v2/cover_short_side.dae" />
+          </geometry>
+        </visual>
+        <collision>
+          <origin xyz="0 0 0" rpy="0 0 0" />
+          <geometry>
+            <mesh filename="package://mobipick_description/meshes/structure/visual/v2/cover_short_side.dae" />
+          </geometry>
+        </collision>
+      </link>
+      <!-- cover_left -->
+      <joint name="${prefix}cover_left_joint" type="fixed">
+        <origin xyz="0 ${structure_width / 2 + cover_thickness / 2} ${structure_height - cover_height / 2}" rpy="0 0 ${pi / 2}" />
+        <parent link="${prefix}part_down" />
+        <child link="${prefix}cover_left_link" />
+      </joint>
+      <link name="${prefix}cover_left_link">
+        <xacro:box_inertial mass="2.266" x="${cover_thickness}" y="${structure_length}" z="${cover_height}">
+          <origin xyz="0 0 0" />
+        </xacro:box_inertial>
+        <visual>
+          <origin xyz="0 0 0" rpy="0 0 0" />
+          <geometry>
+            <mesh filename="package://mobipick_description/meshes/structure/visual/v2/cover_long_side.dae" />
+          </geometry>
+        </visual>
+        <collision>
+          <origin xyz="0 0 0" rpy="0 0 0" />
+          <geometry>
+            <mesh filename="package://mobipick_description/meshes/structure/visual/v2/cover_long_side.dae" />
+          </geometry>
+        </collision>
+      </link>
+      <!-- cover_right -->
+      <joint name="${prefix}cover_right_joint" type="fixed">
+        <origin xyz="0 ${-(structure_width / 2 + cover_thickness / 2)} ${structure_height - cover_height / 2}" rpy="0 0 ${-pi / 2}" />
+        <parent link="${prefix}part_down" />
+        <child link="${prefix}cover_right_link" />
+      </joint>
+      <link name="${prefix}cover_right_link">
+        <xacro:box_inertial mass="2.266" x="${cover_thickness}" y="${structure_length}" z="${cover_height}">
+          <origin xyz="0 0 0" />
+        </xacro:box_inertial>
+        <visual>
+          <origin xyz="0 0 0" rpy="0 0 0" />
+          <geometry>
+            <mesh filename="package://mobipick_description/meshes/structure/visual/v2/cover_long_side.dae" />
+          </geometry>
+        </visual>
+        <collision>
+          <origin xyz="0 0 0" rpy="0 0 0" />
+          <geometry>
+            <mesh filename="package://mobipick_description/meshes/structure/visual/v2/cover_long_side.dae" />
+          </geometry>
+        </collision>
+      </link>
+      <!-- cover_top_front -->
+      <joint name="${prefix}cover_top_front_joint" type="fixed">
+        <origin xyz="${structure_length / 4} 0 ${structure_height + cover_thickness / 2}" rpy="0 0 ${pi}" />
+        <parent link="${prefix}part_down" />
+        <child link="${prefix}cover_top_front_link" />
+      </joint>
+      <link name="${prefix}cover_top_front_link">
+        <xacro:box_inertial mass="0.946" x="${cover_thickness}" y="${structure_length}" z="${cover_height}">
+          <origin xyz="0 0 0" />
+        </xacro:box_inertial>
+        <visual>
+          <origin xyz="0 0 0" rpy="0 0 0" />
+          <geometry>
+            <mesh filename="package://mobipick_description/meshes/structure/visual/v2/cover_top.dae" />
+          </geometry>
+        </visual>
+        <collision>
+          <origin xyz="0 0 0" rpy="0 0 0" />
+          <geometry>
+            <mesh filename="package://mobipick_description/meshes/structure/visual/v2/cover_top.dae" />
+          </geometry>
+        </collision>
+      </link>
+      <!-- cover_top_back -->
+      <joint name="${prefix}cover_top_back_joint" type="fixed">
+        <origin xyz="${-structure_length / 4} 0 ${structure_height + cover_thickness / 2}" rpy="0 0 0" />
+        <parent link="${prefix}part_down" />
+        <child link="${prefix}cover_top_back_link" />
+      </joint>
+      <link name="${prefix}cover_top_back_link">
+        <xacro:box_inertial mass="0.946" x="${cover_thickness}" y="${structure_length}" z="${cover_height}">
+          <origin xyz="0 0 0" />
+        </xacro:box_inertial>
+        <visual>
+          <origin xyz="0 0 0" rpy="0 0 0" />
+          <geometry>
+            <mesh filename="package://mobipick_description/meshes/structure/visual/v2/cover_top.dae" />
+          </geometry>
+        </visual>
+        <collision>
+          <origin xyz="0 0 0" rpy="0 0 0" />
+          <geometry>
+            <mesh filename="package://mobipick_description/meshes/structure/visual/v2/cover_top.dae" />
+          </geometry>
+        </collision>
+      </link>
+    </xacro:if>
   </xacro:macro>
 </robot>
