Commit message: urdf: Add mobipick covers

File: mobipick_moveit_config/config/mobipick.srdf.xacro (robot description, xacro)
@@ -170,4 +170,10 @@
     <disable_collisions link1="${tf_prefix}back_laser_link" link2="${tf_prefix}sensor_mount_link" reason="Never" />
     <disable_collisions link1="${tf_prefix}back_laser_link" link2="${tf_prefix}sensor_mount_pico_holder_link" reason="Never" />
+    <disable_collisions link1="${tf_prefix}back_laser_link" link2="${tf_prefix}structure_cover_back_link" reason="Never" />
+    <disable_collisions link1="${tf_prefix}back_laser_link" link2="${tf_prefix}structure_cover_front_link" reason="Never" />
+    <disable_collisions link1="${tf_prefix}back_laser_link" link2="${tf_prefix}structure_cover_left_link" reason="Never" />
+    <disable_collisions link1="${tf_prefix}back_laser_link" link2="${tf_prefix}structure_cover_right_link" reason="Never" />
+    <disable_collisions link1="${tf_prefix}back_laser_link" link2="${tf_prefix}structure_cover_top_back_link" reason="Never" />
+    <disable_collisions link1="${tf_prefix}back_laser_link" link2="${tf_prefix}structure_cover_top_front_link" reason="Never" />
     <disable_collisions link1="${tf_prefix}back_laser_link" link2="${tf_prefix}structure_part_down" reason="Never" />
     <disable_collisions link1="${tf_prefix}back_laser_link" link2="${tf_prefix}structure_part_up" reason="Never" />
@@ -195,4 +201,10 @@
     <disable_collisions link1="${tf_prefix}base_link" link2="${tf_prefix}right_wheel_link" reason="Adjacent" />
     <disable_collisions link1="${tf_prefix}base_link" link2="${tf_prefix}sensor_mount_bracket_link" reason="Never" />
+    <disable_collisions link1="${tf_prefix}base_link" link2="${tf_prefix}structure_cover_back_link" reason="Never" />
+    <disable_collisions link1="${tf_prefix}base_link" link2="${tf_prefix}structure_cover_front_link" reason="Never" />
+    <disable_collisions link1="${tf_prefix}base_link" link2="${tf_prefix}structure_cover_left_link" reason="Never" />
+    <disable_collisions link1="${tf_prefix}base_link" link2="${tf_prefix}structure_cover_right_link" reason="Never" />
+    <disable_collisions link1="${tf_prefix}base_link" link2="${tf_prefix}structure_cover_top_back_link" reason="Never" />
+    <disable_collisions link1="${tf_prefix}base_link" link2="${tf_prefix}structure_cover_top_front_link" reason="Never" />
     <disable_collisions link1="${tf_prefix}base_link" link2="${tf_prefix}structure_part_down" reason="Adjacent" />
     <disable_collisions link1="${tf_prefix}base_link" link2="${tf_prefix}structure_part_up" reason="Never" />
@@ -234,4 +246,10 @@
     <disable_collisions link1="${tf_prefix}bl_caster_rotation_link" link2="${tf_prefix}sensor_mount_link" reason="Never" />
     <disable_collisions link1="${tf_prefix}bl_caster_rotation_link" link2="${tf_prefix}sensor_mount_pico_holder_link" reason="Never" />
+    <disable_collisions link1="${tf_prefix}bl_caster_rotation_link" link2="${tf_prefix}structure_cover_back_link" reason="Never" />
+    <disable_collisions link1="${tf_prefix}bl_caster_rotation_link" link2="${tf_prefix}structure_cover_front_link" reason="Never" />
+    <disable_collisions link1="${tf_prefix}bl_caster_rotation_link" link2="${tf_prefix}structure_cover_left_link" reason="Never" />
+    <disable_collisions link1="${tf_prefix}bl_caster_rotation_link" link2="${tf_prefix}structure_cover_right_link" reason="Never" />
+    <disable_collisions link1="${tf_prefix}bl_caster_rotation_link" link2="${tf_prefix}structure_cover_top_back_link" reason="Never" />
+    <disable_collisions link1="${tf_prefix}bl_caster_rotation_link" link2="${tf_prefix}structure_cover_top_front_link" reason="Never" />
     <disable_collisions link1="${tf_prefix}bl_caster_rotation_link" link2="${tf_prefix}structure_part_down" reason="Never" />
     <disable_collisions link1="${tf_prefix}bl_caster_rotation_link" link2="${tf_prefix}structure_part_up" reason="Never" />
@@ -272,4 +290,10 @@
     <disable_collisions link1="${tf_prefix}bl_caster_wheel_link" link2="${tf_prefix}sensor_mount_link" reason="Never" />
     <disable_collisions link1="${tf_prefix}bl_caster_wheel_link" link2="${tf_prefix}sensor_mount_pico_holder_link" reason="Never" />
+    <disable_collisions link1="${tf_prefix}bl_caster_wheel_link" link2="${tf_prefix}structure_cover_back_link" reason="Never" />
+    <disable_collisions link1="${tf_prefix}bl_caster_wheel_link" link2="${tf_prefix}structure_cover_front_link" reason="Never" />
+    <disable_collisions link1="${tf_prefix}bl_caster_wheel_link" link2="${tf_prefix}structure_cover_left_link" reason="Never" />
+    <disable_collisions link1="${tf_prefix}bl_caster_wheel_link" link2="${tf_prefix}structure_cover_right_link" reason="Never" />
+    <disable_collisions link1="${tf_prefix}bl_caster_wheel_link" link2="${tf_prefix}structure_cover_top_back_link" reason="Never" />
+    <disable_collisions link1="${tf_prefix}bl_caster_wheel_link" link2="${tf_prefix}structure_cover_top_front_link" reason="Never" />
     <disable_collisions link1="${tf_prefix}bl_caster_wheel_link" link2="${tf_prefix}structure_part_down" reason="Never" />
     <disable_collisions link1="${tf_prefix}bl_caster_wheel_link" link2="${tf_prefix}structure_part_up" reason="Never" />
@@ -309,4 +333,10 @@
     <disable_collisions link1="${tf_prefix}br_caster_rotation_link" link2="${tf_prefix}sensor_mount_link" reason="Never" />
     <disable_collisions link1="${tf_prefix}br_caster_rotation_link" link2="${tf_prefix}sensor_mount_pico_holder_link" reason="Never" />
+    <disable_collisions link1="${tf_prefix}br_caster_rotation_link" link2="${tf_prefix}structure_cover_back_link" reason="Never" />
+    <disable_collisions link1="${tf_prefix}br_caster_rotation_link" link2="${tf_prefix}structure_cover_front_link" reason="Never" />
+    <disable_collisions link1="${tf_prefix}br_caster_rotation_link" link2="${tf_prefix}structure_cover_left_link" reason="Never" />
+    <disable_collisions link1="${tf_prefix}br_caster_rotation_link" link2="${tf_prefix}structure_cover_right_link" reason="Never" />
+    <disable_collisions link1="${tf_prefix}br_caster_rotation_link" link2="${tf_prefix}structure_cover_top_back_link" reason="Never" />
+    <disable_collisions link1="${tf_prefix}br_caster_rotation_link" link2="${tf_prefix}structure_cover_top_front_link" reason="Never" />
     <disable_collisions link1="${tf_prefix}br_caster_rotation_link" link2="${tf_prefix}structure_part_down" reason="Never" />
     <disable_collisions link1="${tf_prefix}br_caster_rotation_link" link2="${tf_prefix}structure_part_up" reason="Never" />
@@ -345,4 +375,10 @@
     <disable_collisions link1="${tf_prefix}br_caster_wheel_link" link2="${tf_prefix}sensor_mount_link" reason="Never" />
     <disable_collisions link1="${tf_prefix}br_caster_wheel_link" link2="${tf_prefix}sensor_mount_pico_holder_link" reason="Never" />
+    <disable_collisions link1="${tf_prefix}br_caster_wheel_link" link2="${tf_prefix}structure_cover_back_link" reason="Never" />
+    <disable_collisions link1="${tf_prefix}br_caster_wheel_link" link2="${tf_prefix}structure_cover_front_link" reason="Never" />
+    <disable_collisions link1="${tf_prefix}br_caster_wheel_link" link2="${tf_prefix}structure_cover_left_link" reason="Never" />
+    <disable_collisions link1="${tf_prefix}br_caster_wheel_link" link2="${tf_prefix}structure_cover_right_link" reason="Never" />
+    <disable_collisions link1="${tf_prefix}br_caster_wheel_link" link2="${tf_prefix}structure_cover_top_back_link" reason="Never" />
+    <disable_collisions link1="${tf_prefix}br_caster_wheel_link" link2="${tf_prefix}structure_cover_top_front_link" reason="Never" />
     <disable_collisions link1="${tf_prefix}br_caster_wheel_link" link2="${tf_prefix}structure_part_down" reason="Never" />
     <disable_collisions link1="${tf_prefix}br_caster_wheel_link" link2="${tf_prefix}structure_part_up" reason="Never" />
@@ -380,4 +416,10 @@
     <disable_collisions link1="${tf_prefix}fl_caster_rotation_link" link2="${tf_prefix}sensor_mount_link" reason="Never" />
     <disable_collisions link1="${tf_prefix}fl_caster_rotation_link" link2="${tf_prefix}sensor_mount_pico_holder_link" reason="Never" />
+    <disable_collisions link1="${tf_prefix}fl_caster_rotation_link" link2="${tf_prefix}structure_cover_back_link" reason="Never" />
+    <disable_collisions link1="${tf_prefix}fl_caster_rotation_link" link2="${tf_prefix}structure_cover_front_link" reason="Never" />
+    <disable_collisions link1="${tf_prefix}fl_caster_rotation_link" link2="${tf_prefix}structure_cover_left_link" reason="Never" />
+    <disable_collisions link1="${tf_prefix}fl_caster_rotation_link" link2="${tf_prefix}structure_cover_right_link" reason="Never" />
+    <disable_collisions link1="${tf_prefix}fl_caster_rotation_link" link2="${tf_prefix}structure_cover_top_back_link" reason="Never" />
+    <disable_collisions link1="${tf_prefix}fl_caster_rotation_link" link2="${tf_prefix}structure_cover_top_front_link" reason="Never" />
     <disable_collisions link1="${tf_prefix}fl_caster_rotation_link" link2="${tf_prefix}structure_part_down" reason="Never" />
     <disable_collisions link1="${tf_prefix}fl_caster_rotation_link" link2="${tf_prefix}structure_part_up" reason="Never" />
@@ -414,4 +456,10 @@
     <disable_collisions link1="${tf_prefix}fl_caster_wheel_link" link2="${tf_prefix}sensor_mount_link" reason="Never" />
     <disable_collisions link1="${tf_prefix}fl_caster_wheel_link" link2="${tf_prefix}sensor_mount_pico_holder_link" reason="Never" />
+    <disable_collisions link1="${tf_prefix}fl_caster_wheel_link" link2="${tf_prefix}structure_cover_back_link" reason="Never" />
+    <disable_collisions link1="${tf_prefix}fl_caster_wheel_link" link2="${tf_prefix}structure_cover_front_link" reason="Never" />
+    <disable_collisions link1="${tf_prefix}fl_caster_wheel_link" link2="${tf_prefix}structure_cover_left_link" reason="Never" />
+    <disable_collisions link1="${tf_prefix}fl_caster_wheel_link" link2="${tf_prefix}structure_cover_right_link" reason="Never" />
+    <disable_collisions link1="${tf_prefix}fl_caster_wheel_link" link2="${tf_prefix}structure_cover_top_back_link" reason="Never" />
+    <disable_collisions link1="${tf_prefix}fl_caster_wheel_link" link2="${tf_prefix}structure_cover_top_front_link" reason="Never" />
     <disable_collisions link1="${tf_prefix}fl_caster_wheel_link" link2="${tf_prefix}structure_part_down" reason="Never" />
     <disable_collisions link1="${tf_prefix}fl_caster_wheel_link" link2="${tf_prefix}structure_part_up" reason="Never" />
@@ -447,4 +495,10 @@
     <disable_collisions link1="${tf_prefix}fr_caster_rotation_link" link2="${tf_prefix}sensor_mount_link" reason="Never" />
     <disable_collisions link1="${tf_prefix}fr_caster_rotation_link" link2="${tf_prefix}sensor_mount_pico_holder_link" reason="Never" />
+    <disable_collisions link1="${tf_prefix}fr_caster_rotation_link" link2="${tf_prefix}structure_cover_back_link" reason="Never" />
+    <disable_collisions link1="${tf_prefix}fr_caster_rotation_link" link2="${tf_prefix}structure_cover_front_link" reason="Never" />
+    <disable_collisions link1="${tf_prefix}fr_caster_rotation_link" link2="${tf_prefix}structure_cover_left_link" reason="Never" />
+    <disable_collisions link1="${tf_prefix}fr_caster_rotation_link" link2="${tf_prefix}structure_cover_right_link" reason="Never" />
+    <disable_collisions link1="${tf_prefix}fr_caster_rotation_link" link2="${tf_prefix}structure_cover_top_back_link" reason="Never" />
+    <disable_collisions link1="${tf_prefix}fr_caster_rotation_link" link2="${tf_prefix}structure_cover_top_front_link" reason="Never" />
     <disable_collisions link1="${tf_prefix}fr_caster_rotation_link" link2="${tf_prefix}structure_part_down" reason="Never" />
     <disable_collisions link1="${tf_prefix}fr_caster_rotation_link" link2="${tf_prefix}structure_part_up" reason="Never" />
@@ -479,4 +533,10 @@
     <disable_collisions link1="${tf_prefix}fr_caster_wheel_link" link2="${tf_prefix}sensor_mount_link" reason="Never" />
     <disable_collisions link1="${tf_prefix}fr_caster_wheel_link" link2="${tf_prefix}sensor_mount_pico_holder_link" reason="Never" />
+    <disable_collisions link1="${tf_prefix}fr_caster_wheel_link" link2="${tf_prefix}structure_cover_back_link" reason="Never" />
+    <disable_collisions link1="${tf_prefix}fr_caster_wheel_link" link2="${tf_prefix}structure_cover_front_link" reason="Never" />
+    <disable_collisions link1="${tf_prefix}fr_caster_wheel_link" link2="${tf_prefix}structure_cover_left_link" reason="Never" />
+    <disable_collisions link1="${tf_prefix}fr_caster_wheel_link" link2="${tf_prefix}structure_cover_right_link" reason="Never" />
+    <disable_collisions link1="${tf_prefix}fr_caster_wheel_link" link2="${tf_prefix}structure_cover_top_back_link" reason="Never" />
+    <disable_collisions link1="${tf_prefix}fr_caster_wheel_link" link2="${tf_prefix}structure_cover_top_front_link" reason="Never" />
     <disable_collisions link1="${tf_prefix}fr_caster_wheel_link" link2="${tf_prefix}structure_part_down" reason="Never" />
     <disable_collisions link1="${tf_prefix}fr_caster_wheel_link" link2="${tf_prefix}structure_part_up" reason="Never" />
@@ -510,4 +570,10 @@
     <disable_collisions link1="${tf_prefix}front_laser_link" link2="${tf_prefix}sensor_mount_link" reason="Never" />
     <disable_collisions link1="${tf_prefix}front_laser_link" link2="${tf_prefix}sensor_mount_pico_holder_link" reason="Never" />
+    <disable_collisions link1="${tf_prefix}front_laser_link" link2="${tf_prefix}structure_cover_back_link" reason="Never" />
+    <disable_collisions link1="${tf_prefix}front_laser_link" link2="${tf_prefix}structure_cover_front_link" reason="Never" />
+    <disable_collisions link1="${tf_prefix}front_laser_link" link2="${tf_prefix}structure_cover_left_link" reason="Never" />
+    <disable_collisions link1="${tf_prefix}front_laser_link" link2="${tf_prefix}structure_cover_right_link" reason="Never" />
+    <disable_collisions link1="${tf_prefix}front_laser_link" link2="${tf_prefix}structure_cover_top_back_link" reason="Never" />
+    <disable_collisions link1="${tf_prefix}front_laser_link" link2="${tf_prefix}structure_cover_top_front_link" reason="Never" />
     <disable_collisions link1="${tf_prefix}front_laser_link" link2="${tf_prefix}structure_part_down" reason="Never" />
     <disable_collisions link1="${tf_prefix}front_laser_link" link2="${tf_prefix}structure_part_up" reason="Never" />
@@ -765,4 +831,10 @@
     <disable_collisions link1="${tf_prefix}left_wheel_link" link2="${tf_prefix}sensor_mount_link" reason="Never" />
     <disable_collisions link1="${tf_prefix}left_wheel_link" link2="${tf_prefix}sensor_mount_pico_holder_link" reason="Never" />
+    <disable_collisions link1="${tf_prefix}left_wheel_link" link2="${tf_prefix}structure_cover_back_link" reason="Never" />
+    <disable_collisions link1="${tf_prefix}left_wheel_link" link2="${tf_prefix}structure_cover_front_link" reason="Never" />
+    <disable_collisions link1="${tf_prefix}left_wheel_link" link2="${tf_prefix}structure_cover_left_link" reason="Never" />
+    <disable_collisions link1="${tf_prefix}left_wheel_link" link2="${tf_prefix}structure_cover_right_link" reason="Never" />
+    <disable_collisions link1="${tf_prefix}left_wheel_link" link2="${tf_prefix}structure_cover_top_back_link" reason="Never" />
+    <disable_collisions link1="${tf_prefix}left_wheel_link" link2="${tf_prefix}structure_cover_top_front_link" reason="Never" />
     <disable_collisions link1="${tf_prefix}left_wheel_link" link2="${tf_prefix}structure_part_down" reason="Never" />
     <disable_collisions link1="${tf_prefix}left_wheel_link" link2="${tf_prefix}structure_part_up" reason="Never" />
@@ -779,4 +851,10 @@
     <disable_collisions link1="${tf_prefix}right_wheel_link" link2="${tf_prefix}sensor_mount_link" reason="Never" />
     <disable_collisions link1="${tf_prefix}right_wheel_link" link2="${tf_prefix}sensor_mount_pico_holder_link" reason="Never" />
+    <disable_collisions link1="${tf_prefix}right_wheel_link" link2="${tf_prefix}structure_cover_back_link" reason="Never" />
+    <disable_collisions link1="${tf_prefix}right_wheel_link" link2="${tf_prefix}structure_cover_front_link" reason="Never" />
+    <disable_collisions link1="${tf_prefix}right_wheel_link" link2="${tf_prefix}structure_cover_left_link" reason="Never" />
+    <disable_collisions link1="${tf_prefix}right_wheel_link" link2="${tf_prefix}structure_cover_right_link" reason="Never" />
+    <disable_collisions link1="${tf_prefix}right_wheel_link" link2="${tf_prefix}structure_cover_top_back_link" reason="Never" />
+    <disable_collisions link1="${tf_prefix}right_wheel_link" link2="${tf_prefix}structure_cover_top_front_link" reason="Never" />
     <disable_collisions link1="${tf_prefix}right_wheel_link" link2="${tf_prefix}structure_part_down" reason="Never" />
     <disable_collisions link1="${tf_prefix}right_wheel_link" link2="${tf_prefix}structure_part_up" reason="Never" />
@@ -805,4 +883,49 @@
     <disable_collisions link1="${tf_prefix}sensor_mount_pico_holder_link" link2="${tf_prefix}ur5_wrist_2_link" reason="Never" />
     <disable_collisions link1="${tf_prefix}sensor_mount_pico_holder_link" link2="${tf_prefix}ur5_wrist_3_link" reason="Never" />
+    <disable_collisions link1="${tf_prefix}structure_cover_back_link" link2="${tf_prefix}structure_cover_front_link" reason="Never" />
+    <disable_collisions link1="${tf_prefix}structure_cover_back_link" link2="${tf_prefix}structure_cover_left_link" reason="Never" />
+    <disable_collisions link1="${tf_prefix}structure_cover_back_link" link2="${tf_prefix}structure_cover_right_link" reason="Never" />
+    <disable_collisions link1="${tf_prefix}structure_cover_back_link" link2="${tf_prefix}structure_cover_top_back_link" reason="Never" />
+    <disable_collisions link1="${tf_prefix}structure_cover_back_link" link2="${tf_prefix}structure_cover_top_front_link" reason="Never" />
+    <disable_collisions link1="${tf_prefix}structure_cover_back_link" link2="${tf_prefix}structure_part_down" reason="Adjacent" />
+    <disable_collisions link1="${tf_prefix}structure_cover_back_link" link2="${tf_prefix}structure_part_up" reason="Never" />
+    <disable_collisions link1="${tf_prefix}structure_cover_back_link" link2="${tf_prefix}structure_pedestal" reason="Never" />
+    <disable_collisions link1="${tf_prefix}structure_cover_back_link" link2="${tf_prefix}ur5_base_link" reason="Never" />
+    <disable_collisions link1="${tf_prefix}structure_cover_back_link" link2="${tf_prefix}ur5_shoulder_link" reason="Never" />
+    <disable_collisions link1="${tf_prefix}structure_cover_front_link" link2="${tf_prefix}structure_cover_left_link" reason="Never" />
+    <disable_collisions link1="${tf_prefix}structure_cover_front_link" link2="${tf_prefix}structure_cover_right_link" reason="Never" />
+    <disable_collisions link1="${tf_prefix}structure_cover_front_link" link2="${tf_prefix}structure_cover_top_back_link" reason="Never" />
+    <disable_collisions link1="${tf_prefix}structure_cover_front_link" link2="${tf_prefix}structure_cover_top_front_link" reason="Never" />
+    <disable_collisions link1="${tf_prefix}structure_cover_front_link" link2="${tf_prefix}structure_part_down" reason="Adjacent" />
+    <disable_collisions link1="${tf_prefix}structure_cover_front_link" link2="${tf_prefix}structure_part_up" reason="Never" />
+    <disable_collisions link1="${tf_prefix}structure_cover_front_link" link2="${tf_prefix}structure_pedestal" reason="Never" />
+    <disable_collisions link1="${tf_prefix}structure_cover_front_link" link2="${tf_prefix}ur5_base_link" reason="Never" />
+    <disable_collisions link1="${tf_prefix}structure_cover_front_link" link2="${tf_prefix}ur5_shoulder_link" reason="Never" />
+    <disable_collisions link1="${tf_prefix}structure_cover_left_link" link2="${tf_prefix}structure_cover_right_link" reason="Never" />
+    <disable_collisions link1="${tf_prefix}structure_cover_left_link" link2="${tf_prefix}structure_cover_top_back_link" reason="Never" />
+    <disable_collisions link1="${tf_prefix}structure_cover_left_link" link2="${tf_prefix}structure_cover_top_front_link" reason="Never" />
+    <disable_collisions link1="${tf_prefix}structure_cover_left_link" link2="${tf_prefix}structure_part_down" reason="Adjacent" />
+    <disable_collisions link1="${tf_prefix}structure_cover_left_link" link2="${tf_prefix}structure_part_up" reason="Never" />
+    <disable_collisions link1="${tf_prefix}structure_cover_left_link" link2="${tf_prefix}structure_pedestal" reason="Never" />
+    <disable_collisions link1="${tf_prefix}structure_cover_left_link" link2="${tf_prefix}ur5_base_link" reason="Never" />
+    <disable_collisions link1="${tf_prefix}structure_cover_left_link" link2="${tf_prefix}ur5_shoulder_link" reason="Never" />
+    <disable_collisions link1="${tf_prefix}structure_cover_right_link" link2="${tf_prefix}structure_cover_top_back_link" reason="Never" />
+    <disable_collisions link1="${tf_prefix}structure_cover_right_link" link2="${tf_prefix}structure_cover_top_front_link" reason="Never" />
+    <disable_collisions link1="${tf_prefix}structure_cover_right_link" link2="${tf_prefix}structure_part_down" reason="Adjacent" />
+    <disable_collisions link1="${tf_prefix}structure_cover_right_link" link2="${tf_prefix}structure_part_up" reason="Never" />
+    <disable_collisions link1="${tf_prefix}structure_cover_right_link" link2="${tf_prefix}structure_pedestal" reason="Never" />
+    <disable_collisions link1="${tf_prefix}structure_cover_right_link" link2="${tf_prefix}ur5_base_link" reason="Never" />
+    <disable_collisions link1="${tf_prefix}structure_cover_right_link" link2="${tf_prefix}ur5_shoulder_link" reason="Never" />
+    <disable_collisions link1="${tf_prefix}structure_cover_top_back_link" link2="${tf_prefix}structure_cover_top_front_link" reason="Default" />
+    <disable_collisions link1="${tf_prefix}structure_cover_top_back_link" link2="${tf_prefix}structure_part_down" reason="Adjacent" />
+    <disable_collisions link1="${tf_prefix}structure_cover_top_back_link" link2="${tf_prefix}structure_part_up" reason="Default" />
+    <disable_collisions link1="${tf_prefix}structure_cover_top_back_link" link2="${tf_prefix}structure_pedestal" reason="Never" />
+    <disable_collisions link1="${tf_prefix}structure_cover_top_back_link" link2="${tf_prefix}ur5_base_link" reason="Never" />
+    <disable_collisions link1="${tf_prefix}structure_cover_top_back_link" link2="${tf_prefix}ur5_shoulder_link" reason="Never" />
+    <disable_collisions link1="${tf_prefix}structure_cover_top_front_link" link2="${tf_prefix}structure_part_down" reason="Adjacent" />
+    <disable_collisions link1="${tf_prefix}structure_cover_top_front_link" link2="${tf_prefix}structure_part_up" reason="Default" />
+    <disable_collisions link1="${tf_prefix}structure_cover_top_front_link" link2="${tf_prefix}structure_pedestal" reason="Never" />
+    <disable_collisions link1="${tf_prefix}structure_cover_top_front_link" link2="${tf_prefix}ur5_base_link" reason="Never" />
+    <disable_collisions link1="${tf_prefix}structure_cover_top_front_link" link2="${tf_prefix}ur5_shoulder_link" reason="Never" />
     <disable_collisions link1="${tf_prefix}structure_part_down" link2="${tf_prefix}structure_part_up" reason="Adjacent" />
     <disable_collisions link1="${tf_prefix}structure_part_down" link2="${tf_prefix}structure_pedestal" reason="Never" />
