Commit message: remove cable_guide_wrist_3 as option and split into hb and os version

File: mobipick_moveit_config/config/mobipick_hb.srdf.xacro (robot description, xacro)
@@ -5,4 +5,5 @@
 -->
 <robot xmlns:xacro="http://ros.org/wiki/xacro" name="mobipick">
+    <!-- This version of Mobipick does not have a cable guide at the wrist, allowing it to take pictures facing up -->
     <!-- Use the arg tf_prefix to set the tf_prefix property. Use a dummy tf_prefix_ property to avoid a leading / if
          the prefix is not set, without using eval (which is not supported on indigo). -->
@@ -15,9 +16,4 @@
         <xacro:property name="tf_prefix" value="${tf_prefix_}/"/>
     </xacro:unless>
-    <xacro:arg name="robot_version" default="os" />      <!-- can be "mobipick-hb" or "mobipick-os" -->
-    <xacro:property name="robot_version" value="$(arg robot_version)" />  <!-- necessary because args cannot be accessed inside ${} expressions -->
-    <!-- mobipick-hb does not have a cable guide at the wrist, allowing it to take pictures facing up -->
-    <xacro:arg name="cable_guide_wrist_3" default="${str(robot_version == 'os')}" />
-    <xacro:property name="cable_guide_wrist_3" value="$(arg cable_guide_wrist_3)" />
     <!--GROUPS: Representation of a set of joints and links. This can be useful for specifying DOF to plan for, defining arms, end effectors, etc-->
     <!--LINKS: When a link is specified, the parent joint of that link (if it exists) is automatically included-->
@@ -182,7 +178,4 @@
     <disable_collisions link1="${tf_prefix}back_laser_link" link2="${tf_prefix}cable_guide_terminal_element_link" reason="Never"/>
     <disable_collisions link1="${tf_prefix}back_laser_link" link2="${tf_prefix}cable_guide_upper_arm_tube_link" reason="Never"/>
-    <xacro:if value="${cable_guide_wrist_3}">
-    <disable_collisions link1="${tf_prefix}back_laser_link" link2="${tf_prefix}cable_guide_wrist_3_tube_link" reason="Never"/>
-    </xacro:if>
     <disable_collisions link1="${tf_prefix}back_laser_link" link2="${tf_prefix}cable_guide_wrist_clamp_link" reason="Never"/>
     <disable_collisions link1="${tf_prefix}back_laser_link" link2="${tf_prefix}eef_forward_cam_link" reason="Never"/>
@@ -239,7 +232,4 @@
     <disable_collisions link1="${tf_prefix}base_link" link2="${tf_prefix}cable_guide_terminal_element_link" reason="User"/>
     <disable_collisions link1="${tf_prefix}base_link" link2="${tf_prefix}cable_guide_upper_arm_tube_link" reason="Never"/>
-    <xacro:if value="${cable_guide_wrist_3}">
-    <disable_collisions link1="${tf_prefix}base_link" link2="${tf_prefix}cable_guide_wrist_3_tube_link" reason="User"/>
-    </xacro:if>
     <disable_collisions link1="${tf_prefix}base_link" link2="${tf_prefix}cable_guide_wrist_clamp_link" reason="User"/>
     <disable_collisions link1="${tf_prefix}base_link" link2="${tf_prefix}eef_forward_cam_link" reason="User"/>
@@ -295,7 +285,4 @@
     <disable_collisions link1="${tf_prefix}bl_caster_rotation_link" link2="${tf_prefix}cable_guide_terminal_element_link" reason="Never"/>
     <disable_collisions link1="${tf_prefix}bl_caster_rotation_link" link2="${tf_prefix}cable_guide_upper_arm_tube_link" reason="Never"/>
-    <xacro:if value="${cable_guide_wrist_3}">
-    <disable_collisions link1="${tf_prefix}bl_caster_rotation_link" link2="${tf_prefix}cable_guide_wrist_3_tube_link" reason="Never"/>
-    </xacro:if>
     <disable_collisions link1="${tf_prefix}bl_caster_rotation_link" link2="${tf_prefix}cable_guide_wrist_clamp_link" reason="Never"/>
     <disable_collisions link1="${tf_prefix}bl_caster_rotation_link" link2="${tf_prefix}eef_forward_cam_link" reason="Never"/>
@@ -350,7 +337,4 @@
     <disable_collisions link1="${tf_prefix}bl_caster_wheel_link" link2="${tf_prefix}cable_guide_terminal_element_link" reason="Never"/>
     <disable_collisions link1="${tf_prefix}bl_caster_wheel_link" link2="${tf_prefix}cable_guide_upper_arm_tube_link" reason="Never"/>
-    <xacro:if value="${cable_guide_wrist_3}">
-    <disable_collisions link1="${tf_prefix}bl_caster_wheel_link" link2="${tf_prefix}cable_guide_wrist_3_tube_link" reason="Never"/>
-    </xacro:if>
     <disable_collisions link1="${tf_prefix}bl_caster_wheel_link" link2="${tf_prefix}cable_guide_wrist_clamp_link" reason="Never"/>
     <disable_collisions link1="${tf_prefix}bl_caster_wheel_link" link2="${tf_prefix}eef_forward_cam_link" reason="Never"/>
@@ -404,7 +388,4 @@
     <disable_collisions link1="${tf_prefix}br_caster_rotation_link" link2="${tf_prefix}cable_guide_terminal_element_link" reason="Never"/>
     <disable_collisions link1="${tf_prefix}br_caster_rotation_link" link2="${tf_prefix}cable_guide_upper_arm_tube_link" reason="Never"/>
-    <xacro:if value="${cable_guide_wrist_3}">
-    <disable_collisions link1="${tf_prefix}br_caster_rotation_link" link2="${tf_prefix}cable_guide_wrist_3_tube_link" reason="Never"/>
-    </xacro:if>
     <disable_collisions link1="${tf_prefix}br_caster_rotation_link" link2="${tf_prefix}cable_guide_wrist_clamp_link" reason="Never"/>
     <disable_collisions link1="${tf_prefix}br_caster_rotation_link" link2="${tf_prefix}eef_forward_cam_link" reason="Never"/>
@@ -457,7 +438,4 @@
     <disable_collisions link1="${tf_prefix}br_caster_wheel_link" link2="${tf_prefix}cable_guide_terminal_element_link" reason="Never"/>
     <disable_collisions link1="${tf_prefix}br_caster_wheel_link" link2="${tf_prefix}cable_guide_upper_arm_tube_link" reason="Never"/>
-    <xacro:if value="${cable_guide_wrist_3}">
-    <disable_collisions link1="${tf_prefix}br_caster_wheel_link" link2="${tf_prefix}cable_guide_wrist_3_tube_link" reason="Never"/>
-    </xacro:if>
     <disable_collisions link1="${tf_prefix}br_caster_wheel_link" link2="${tf_prefix}cable_guide_wrist_clamp_link" reason="Never"/>
     <disable_collisions link1="${tf_prefix}br_caster_wheel_link" link2="${tf_prefix}eef_forward_cam_link" reason="Never"/>
@@ -539,7 +517,4 @@
     <disable_collisions link1="${tf_prefix}cable_guide_clamp2_link" link2="${tf_prefix}cable_guide_terminal_element_link" reason="Never"/>
     <disable_collisions link1="${tf_prefix}cable_guide_clamp2_link" link2="${tf_prefix}cable_guide_upper_arm_tube_link" reason="Default"/>
-    <xacro:if value="${cable_guide_wrist_3}">
-    <disable_collisions link1="${tf_prefix}cable_guide_clamp2_link" link2="${tf_prefix}cable_guide_wrist_3_tube_link" reason="Never"/>
-    </xacro:if>
     <disable_collisions link1="${tf_prefix}cable_guide_clamp2_link" link2="${tf_prefix}cable_guide_wrist_clamp_link" reason="Never"/>
     <disable_collisions link1="${tf_prefix}cable_guide_clamp2_link" link2="${tf_prefix}eef_forward_cam_link" reason="Never"/>
@@ -583,7 +558,4 @@
     <disable_collisions link1="${tf_prefix}cable_guide_clamp3_link" link2="${tf_prefix}cable_guide_terminal_element_link" reason="Never"/>
     <disable_collisions link1="${tf_prefix}cable_guide_clamp3_link" link2="${tf_prefix}cable_guide_upper_arm_tube_link" reason="Never"/>
-    <xacro:if value="${cable_guide_wrist_3}">
-    <disable_collisions link1="${tf_prefix}cable_guide_clamp3_link" link2="${tf_prefix}cable_guide_wrist_3_tube_link" reason="Never"/>
-    </xacro:if>
     <disable_collisions link1="${tf_prefix}cable_guide_clamp3_link" link2="${tf_prefix}cable_guide_wrist_clamp_link" reason="Never"/>
     <disable_collisions link1="${tf_prefix}cable_guide_clamp3_link" link2="${tf_prefix}eef_forward_cam_link" reason="Never"/>
@@ -657,7 +629,4 @@
     <disable_collisions link1="${tf_prefix}cable_guide_forearm_tube_link" link2="${tf_prefix}ur5_wrist_1_link" reason="Never"/>
     <disable_collisions link1="${tf_prefix}cable_guide_forearm_tube_link" link2="${tf_prefix}ur5_wrist_2_link" reason="Never"/>
-    <xacro:if value="${cable_guide_wrist_3}">
-    <disable_collisions link1="${tf_prefix}cable_guide_terminal_element_link" link2="${tf_prefix}cable_guide_wrist_3_tube_link" reason="Adjacent"/>
-    </xacro:if>
     <disable_collisions link1="${tf_prefix}cable_guide_terminal_element_link" link2="${tf_prefix}cable_guide_wrist_clamp_link" reason="Adjacent"/>
     <disable_collisions link1="${tf_prefix}cable_guide_terminal_element_link" link2="${tf_prefix}eef_forward_cam_link" reason="Never"/>
@@ -716,37 +685,4 @@
     <disable_collisions link1="${tf_prefix}cable_guide_upper_arm_tube_link" link2="${tf_prefix}ur5_wrist_2_link" reason="Never"/>
     <disable_collisions link1="${tf_prefix}cable_guide_upper_arm_tube_link" link2="${tf_prefix}ur5_wrist_3_link" reason="Never"/>
-    <xacro:if value="${cable_guide_wrist_3}">
-    <disable_collisions link1="${tf_prefix}cable_guide_wrist_3_tube_link" link2="${tf_prefix}cable_guide_wrist_clamp_link" reason="Never"/>
-    <disable_collisions link1="${tf_prefix}cable_guide_wrist_3_tube_link" link2="${tf_prefix}eef_forward_cam_link" reason="Never"/>
-    <disable_collisions link1="${tf_prefix}cable_guide_wrist_3_tube_link" link2="${tf_prefix}eef_main_cam_link" reason="Never"/>
-    <disable_collisions link1="${tf_prefix}cable_guide_wrist_3_tube_link" link2="${tf_prefix}fl_caster_rotation_link" reason="Never"/>
-    <disable_collisions link1="${tf_prefix}cable_guide_wrist_3_tube_link" link2="${tf_prefix}fl_caster_wheel_link" reason="Never"/>
-    <disable_collisions link1="${tf_prefix}cable_guide_wrist_3_tube_link" link2="${tf_prefix}fr_caster_rotation_link" reason="Never"/>
-    <disable_collisions link1="${tf_prefix}cable_guide_wrist_3_tube_link" link2="${tf_prefix}fr_caster_wheel_link" reason="Never"/>
-    <disable_collisions link1="${tf_prefix}cable_guide_wrist_3_tube_link" link2="${tf_prefix}front_laser_link" reason="Never"/>
-    <disable_collisions link1="${tf_prefix}cable_guide_wrist_3_tube_link" link2="${tf_prefix}ft300_mounting_plate" reason="Never"/>
-    <disable_collisions link1="${tf_prefix}cable_guide_wrist_3_tube_link" link2="${tf_prefix}ft300_sensor" reason="Never"/>
-    <disable_collisions link1="${tf_prefix}cable_guide_wrist_3_tube_link" link2="${tf_prefix}gripper_coupling_link" reason="Never"/>
-    <disable_collisions link1="${tf_prefix}cable_guide_wrist_3_tube_link" link2="${tf_prefix}gripper_left_inner_finger" reason="Never"/>
-    <disable_collisions link1="${tf_prefix}cable_guide_wrist_3_tube_link" link2="${tf_prefix}gripper_left_inner_knuckle" reason="Never"/>
-    <disable_collisions link1="${tf_prefix}cable_guide_wrist_3_tube_link" link2="${tf_prefix}gripper_left_outer_finger" reason="Never"/>
-    <disable_collisions link1="${tf_prefix}cable_guide_wrist_3_tube_link" link2="${tf_prefix}gripper_left_outer_knuckle" reason="Never"/>
-    <disable_collisions link1="${tf_prefix}cable_guide_wrist_3_tube_link" link2="${tf_prefix}gripper_left_robotiq_fingertip_65mm" reason="Never"/>
-    <disable_collisions link1="${tf_prefix}cable_guide_wrist_3_tube_link" link2="${tf_prefix}gripper_right_inner_finger" reason="Never"/>
-    <disable_collisions link1="${tf_prefix}cable_guide_wrist_3_tube_link" link2="${tf_prefix}gripper_right_inner_knuckle" reason="Never"/>
-    <disable_collisions link1="${tf_prefix}cable_guide_wrist_3_tube_link" link2="${tf_prefix}gripper_right_outer_finger" reason="Never"/>
-    <disable_collisions link1="${tf_prefix}cable_guide_wrist_3_tube_link" link2="${tf_prefix}gripper_right_outer_knuckle" reason="Never"/>
-    <disable_collisions link1="${tf_prefix}cable_guide_wrist_3_tube_link" link2="${tf_prefix}gripper_right_robotiq_fingertip_65mm" reason="Never"/>
-    <disable_collisions link1="${tf_prefix}cable_guide_wrist_3_tube_link" link2="${tf_prefix}gripper_robotiq_arg2f_base_link" reason="Never"/>
-    <disable_collisions link1="${tf_prefix}cable_guide_wrist_3_tube_link" link2="${tf_prefix}left_wheel_link" reason="Never"/>
-    <disable_collisions link1="${tf_prefix}cable_guide_wrist_3_tube_link" link2="${tf_prefix}right_wheel_link" reason="Never"/>
-    <disable_collisions link1="${tf_prefix}cable_guide_wrist_3_tube_link" link2="${tf_prefix}sensor_mount_bracket_link" reason="Never"/>
-    <disable_collisions link1="${tf_prefix}cable_guide_wrist_3_tube_link" link2="${tf_prefix}sensor_mount_link" reason="Never"/>
-    <disable_collisions link1="${tf_prefix}cable_guide_wrist_3_tube_link" link2="${tf_prefix}sensor_mount_pico_holder_link" reason="Never"/>
-    <disable_collisions link1="${tf_prefix}cable_guide_wrist_3_tube_link" link2="${tf_prefix}structure_part_down" reason="User"/>
-    <disable_collisions link1="${tf_prefix}cable_guide_wrist_3_tube_link" link2="${tf_prefix}structure_part_up" reason="User"/>
-    <disable_collisions link1="${tf_prefix}cable_guide_wrist_3_tube_link" link2="${tf_prefix}ur5_wrist_2_link" reason="Never"/>
-    <disable_collisions link1="${tf_prefix}cable_guide_wrist_3_tube_link" link2="${tf_prefix}ur5_wrist_3_link" reason="Never"/>
-    </xacro:if>
     <disable_collisions link1="${tf_prefix}cable_guide_wrist_clamp_link" link2="${tf_prefix}eef_forward_cam_link" reason="Never"/>
     <disable_collisions link1="${tf_prefix}cable_guide_wrist_clamp_link" link2="${tf_prefix}eef_main_cam_link" reason="Default"/>
