Commit message: Re-run moveit_setup_assistant
Version of moveit_setup_assistant: 1.1.4

* Fixes slow execution (move to observation pose, move to transport pose, move to handover pose) because default_velocity_scaling_factor and default_acceleration_scaling_factor were moved to a different namespace
* Fixes warning: "MoveGroup launched without ~default_planning_pipeline..."

File: mobipick_moveit_config/config/mobipick.srdf.xacro (robot description, xacro)
@@ -1,3 +1,3 @@
-<?xml version="1.0" ?>
+<?xml version="1.0" encoding="UTF-8"?>
 <!--This does not replace URDF, and is not an extension of URDF.
     This is a format for representing semantic information about the robot structure.
@@ -7,11 +7,11 @@
     <!-- Use the arg tf_prefix to set the tf_prefix property. Use a dummy tf_prefix_ property to avoid a leading / if
          the prefix is not set, without using eval (which is not supported on indigo). -->
-    <xacro:arg name="tf_prefix" default="" />
-    <xacro:property name="tf_prefix_" value="$(arg tf_prefix)" />
+    <xacro:arg name="tf_prefix" default=""/>
+    <xacro:property name="tf_prefix_" value="$(arg tf_prefix)"/>
     <xacro:if value="${tf_prefix_ == ''}">
-        <xacro:property name="tf_prefix" value="" />
+        <xacro:property name="tf_prefix" value=""/>
     </xacro:if>
     <xacro:unless value="${tf_prefix_ == ''}">
-        <xacro:property name="tf_prefix" value="${tf_prefix_}/" />
+        <xacro:property name="tf_prefix" value="${tf_prefix_}/"/>
     </xacro:unless>
     <!--GROUPS: Representation of a set of joints and links. This can be useful for specifying DOF to plan for, defining arms, end effectors, etc-->
@@ -21,1271 +21,1277 @@
     <!--SUBGROUPS: Groups can also be formed by referencing to already defined group names-->
     <group name="arm">
-        <chain base_link="${tf_prefix}ur5_base_link" tip_link="${tf_prefix}gripper_tcp" />
+        <chain base_link="${tf_prefix}ur5_base_link" tip_link="${tf_prefix}gripper_tcp"/>
     </group>
     <group name="gripper">
-        <link name="${tf_prefix}gripper_robotiq_arg2f_base_link" />
-        <link name="${tf_prefix}gripper_left_outer_knuckle" />
-        <link name="${tf_prefix}gripper_left_outer_finger" />
-        <link name="${tf_prefix}gripper_left_inner_finger" />
-        <link name="${tf_prefix}gripper_left_robotiq_fingertip_65mm" />
-        <link name="${tf_prefix}gripper_left_inner_knuckle" />
-        <link name="${tf_prefix}gripper_right_inner_knuckle" />
-        <link name="${tf_prefix}gripper_right_outer_knuckle" />
-        <link name="${tf_prefix}gripper_right_outer_finger" />
-        <link name="${tf_prefix}gripper_right_inner_finger" />
-        <link name="${tf_prefix}gripper_right_robotiq_fingertip_65mm" />
-        <!-- <joint name="${tf_prefix}gripper_finger_joint" /> -->
+        <link name="${tf_prefix}gripper_robotiq_arg2f_base_link"/>
+        <link name="${tf_prefix}gripper_left_outer_knuckle"/>
+        <link name="${tf_prefix}gripper_left_outer_finger"/>
+        <link name="${tf_prefix}gripper_left_inner_finger"/>
+        <link name="${tf_prefix}gripper_left_robotiq_fingertip_65mm"/>
+        <link name="${tf_prefix}gripper_left_inner_knuckle"/>
+        <link name="${tf_prefix}gripper_right_inner_knuckle"/>
+        <link name="${tf_prefix}gripper_right_outer_knuckle"/>
+        <link name="${tf_prefix}gripper_right_outer_finger"/>
+        <link name="${tf_prefix}gripper_right_inner_finger"/>
+        <link name="${tf_prefix}gripper_right_robotiq_fingertip_65mm"/>
+        <!-- <joint name="${tf_prefix}gripper_finger_joint"/> -->
     </group>
     <!--GROUP STATES: Purpose: Define a named state for a particular group, in terms of joint values. This is useful to define states like 'folded arms'-->
     <group_state name="home" group="arm">
-        <joint name="${tf_prefix}ur5_shoulder_pan_joint" value="0.00" />
-        <joint name="${tf_prefix}ur5_shoulder_lift_joint" value="-2.60" />
-        <joint name="${tf_prefix}ur5_elbow_joint" value="2.43" />
-        <joint name="${tf_prefix}ur5_wrist_1_joint" value="-2.05" />
-        <joint name="${tf_prefix}ur5_wrist_2_joint" value="-1.57" />
-        <joint name="${tf_prefix}ur5_wrist_3_joint" value="3.14" />
+        <joint name="${tf_prefix}ur5_shoulder_pan_joint" value="0.00"/>
+        <joint name="${tf_prefix}ur5_shoulder_lift_joint" value="-2.60"/>
+        <joint name="${tf_prefix}ur5_elbow_joint" value="2.43"/>
+        <joint name="${tf_prefix}ur5_wrist_1_joint" value="-2.05"/>
+        <joint name="${tf_prefix}ur5_wrist_2_joint" value="-1.57"/>
+        <joint name="${tf_prefix}ur5_wrist_3_joint" value="3.14"/>
     </group_state>
     <!-- observation poses for a 100 cm high table directly adjacent to the robot -->
     <group_state name="observe100cm_front" group="arm">
-        <joint name="${tf_prefix}ur5_shoulder_pan_joint" value="0.00" />
-        <joint name="${tf_prefix}ur5_shoulder_lift_joint" value="-2.30" />
-        <joint name="${tf_prefix}ur5_elbow_joint" value="2.44" />
-        <joint name="${tf_prefix}ur5_wrist_1_joint" value="-0.95" />
-        <joint name="${tf_prefix}ur5_wrist_2_joint" value="1.57" />
-        <joint name="${tf_prefix}ur5_wrist_3_joint" value="4.71" />
+        <joint name="${tf_prefix}ur5_shoulder_pan_joint" value="0.00"/>
+        <joint name="${tf_prefix}ur5_shoulder_lift_joint" value="-2.30"/>
+        <joint name="${tf_prefix}ur5_elbow_joint" value="2.44"/>
+        <joint name="${tf_prefix}ur5_wrist_1_joint" value="-0.95"/>
+        <joint name="${tf_prefix}ur5_wrist_2_joint" value="1.57"/>
+        <joint name="${tf_prefix}ur5_wrist_3_joint" value="4.71"/>
     </group_state>
     <group_state name="observe100cm_left" group="arm">
-        <joint name="${tf_prefix}ur5_shoulder_pan_joint" value="1.57" />
-        <joint name="${tf_prefix}ur5_shoulder_lift_joint" value="-2.30" />
-        <joint name="${tf_prefix}ur5_elbow_joint" value="2.44" />
-        <joint name="${tf_prefix}ur5_wrist_1_joint" value="-0.95" />
-        <joint name="${tf_prefix}ur5_wrist_2_joint" value="1.57" />
-        <joint name="${tf_prefix}ur5_wrist_3_joint" value="4.71" />
+        <joint name="${tf_prefix}ur5_shoulder_pan_joint" value="1.57"/>
+        <joint name="${tf_prefix}ur5_shoulder_lift_joint" value="-2.30"/>
+        <joint name="${tf_prefix}ur5_elbow_joint" value="2.44"/>
+        <joint name="${tf_prefix}ur5_wrist_1_joint" value="-0.95"/>
+        <joint name="${tf_prefix}ur5_wrist_2_joint" value="1.57"/>
+        <joint name="${tf_prefix}ur5_wrist_3_joint" value="4.71"/>
     </group_state>
     <group_state name="observe100cm_right" group="arm">
-        <joint name="${tf_prefix}ur5_shoulder_pan_joint" value="-1.57" />
-        <joint name="${tf_prefix}ur5_shoulder_lift_joint" value="-2.30" />
-        <joint name="${tf_prefix}ur5_elbow_joint" value="2.44" />
-        <joint name="${tf_prefix}ur5_wrist_1_joint" value="-0.95" />
-        <joint name="${tf_prefix}ur5_wrist_2_joint" value="1.57" />
-        <joint name="${tf_prefix}ur5_wrist_3_joint" value="4.71" />
+        <joint name="${tf_prefix}ur5_shoulder_pan_joint" value="-1.57"/>
+        <joint name="${tf_prefix}ur5_shoulder_lift_joint" value="-2.30"/>
+        <joint name="${tf_prefix}ur5_elbow_joint" value="2.44"/>
+        <joint name="${tf_prefix}ur5_wrist_1_joint" value="-0.95"/>
+        <joint name="${tf_prefix}ur5_wrist_2_joint" value="1.57"/>
+        <joint name="${tf_prefix}ur5_wrist_3_joint" value="4.71"/>
     </group_state>
     <group_state name="observe100cm_back" group="arm">
-        <joint name="${tf_prefix}ur5_shoulder_pan_joint" value="3.14" />
-        <joint name="${tf_prefix}ur5_shoulder_lift_joint" value="-2.30" />
-        <joint name="${tf_prefix}ur5_elbow_joint" value="2.44" />
-        <joint name="${tf_prefix}ur5_wrist_1_joint" value="-0.95" />
-        <joint name="${tf_prefix}ur5_wrist_2_joint" value="1.57" />
-        <joint name="${tf_prefix}ur5_wrist_3_joint" value="4.71" />
+        <joint name="${tf_prefix}ur5_shoulder_pan_joint" value="3.14"/>
+        <joint name="${tf_prefix}ur5_shoulder_lift_joint" value="-2.30"/>
+        <joint name="${tf_prefix}ur5_elbow_joint" value="2.44"/>
+        <joint name="${tf_prefix}ur5_wrist_1_joint" value="-0.95"/>
+        <joint name="${tf_prefix}ur5_wrist_2_joint" value="1.57"/>
+        <joint name="${tf_prefix}ur5_wrist_3_joint" value="4.71"/>
     </group_state>
     <group_state name="transport" group="arm">
-        <joint name="${tf_prefix}ur5_shoulder_pan_joint" value="-0.897" />
-        <joint name="${tf_prefix}ur5_shoulder_lift_joint" value="-1.88" />
-        <joint name="${tf_prefix}ur5_elbow_joint" value="2.14" />
-        <joint name="${tf_prefix}ur5_wrist_1_joint" value="-1.83" />
-        <joint name="${tf_prefix}ur5_wrist_2_joint" value="-1.58" />
-        <joint name="${tf_prefix}ur5_wrist_3_joint" value="3.81" />
+        <joint name="${tf_prefix}ur5_shoulder_pan_joint" value="-0.897"/>
+        <joint name="${tf_prefix}ur5_shoulder_lift_joint" value="-1.88"/>
+        <joint name="${tf_prefix}ur5_elbow_joint" value="2.14"/>
+        <joint name="${tf_prefix}ur5_wrist_1_joint" value="-1.83"/>
+        <joint name="${tf_prefix}ur5_wrist_2_joint" value="-1.58"/>
+        <joint name="${tf_prefix}ur5_wrist_3_joint" value="3.81"/>
     </group_state>
     <group_state name="place_1" group="arm">
-        <joint name="${tf_prefix}ur5_shoulder_pan_joint" value="-1.72" />
-        <joint name="${tf_prefix}ur5_shoulder_lift_joint" value="-1.836" />
-        <joint name="${tf_prefix}ur5_elbow_joint" value="1.76" />
-        <joint name="${tf_prefix}ur5_wrist_1_joint" value="-1.52" />
-        <joint name="${tf_prefix}ur5_wrist_2_joint" value="-1.57" />
-        <joint name="${tf_prefix}ur5_wrist_3_joint" value="2.89" />
+        <joint name="${tf_prefix}ur5_shoulder_pan_joint" value="-1.72"/>
+        <joint name="${tf_prefix}ur5_shoulder_lift_joint" value="-1.836"/>
+        <joint name="${tf_prefix}ur5_elbow_joint" value="1.76"/>
+        <joint name="${tf_prefix}ur5_wrist_1_joint" value="-1.52"/>
+        <joint name="${tf_prefix}ur5_wrist_2_joint" value="-1.57"/>
+        <joint name="${tf_prefix}ur5_wrist_3_joint" value="2.89"/>
     </group_state>
     <group_state name="above" group="arm">
-        <joint name="${tf_prefix}ur5_shoulder_pan_joint" value="-1.72" />
-        <joint name="${tf_prefix}ur5_shoulder_lift_joint" value="-0.79" />
-        <joint name="${tf_prefix}ur5_elbow_joint" value="0.71" />
-        <joint name="${tf_prefix}ur5_wrist_1_joint" value="-1.52" />
-        <joint name="${tf_prefix}ur5_wrist_2_joint" value="-1.57" />
-        <joint name="${tf_prefix}ur5_wrist_3_joint" value="1.1" />
+        <joint name="${tf_prefix}ur5_shoulder_pan_joint" value="-1.72"/>
+        <joint name="${tf_prefix}ur5_shoulder_lift_joint" value="-0.79"/>
+        <joint name="${tf_prefix}ur5_elbow_joint" value="0.71"/>
+        <joint name="${tf_prefix}ur5_wrist_1_joint" value="-1.52"/>
+        <joint name="${tf_prefix}ur5_wrist_2_joint" value="-1.57"/>
+        <joint name="${tf_prefix}ur5_wrist_3_joint" value="1.1"/>
     </group_state>
     <group_state name="tucked" group="arm">
-        <joint name="${tf_prefix}ur5_shoulder_pan_joint" value="0.0" />
-        <joint name="${tf_prefix}ur5_shoulder_lift_joint" value="-2.37" />
-        <joint name="${tf_prefix}ur5_elbow_joint" value="2.37" />
-        <joint name="${tf_prefix}ur5_wrist_1_joint" value="-1.15" />
-        <joint name="${tf_prefix}ur5_wrist_2_joint" value="1.57" />
-        <joint name="${tf_prefix}ur5_wrist_3_joint" value="4.71" />
+        <joint name="${tf_prefix}ur5_shoulder_pan_joint" value="0.0"/>
+        <joint name="${tf_prefix}ur5_shoulder_lift_joint" value="-2.37"/>
+        <joint name="${tf_prefix}ur5_elbow_joint" value="2.37"/>
+        <joint name="${tf_prefix}ur5_wrist_1_joint" value="-1.15"/>
+        <joint name="${tf_prefix}ur5_wrist_2_joint" value="1.57"/>
+        <joint name="${tf_prefix}ur5_wrist_3_joint" value="4.71"/>
     </group_state>
     <group_state name="open" group="gripper">
-        <joint name="${tf_prefix}gripper_finger_joint" value="0" />
+        <joint name="${tf_prefix}gripper_finger_joint" value="0"/>
     </group_state>
     <group_state name="closed" group="gripper">
-        <joint name="${tf_prefix}gripper_finger_joint" value="0.755" />
+        <joint name="${tf_prefix}gripper_finger_joint" value="0.755"/>
     </group_state>
     <!--END EFFECTOR: Purpose: Represent information about an end effector.-->
-    <end_effector name="end_effector" parent_link="${tf_prefix}gripper_tcp" group="gripper" />
+    <end_effector name="end_effector" parent_link="${tf_prefix}gripper_tcp" group="gripper"/>
     <!--VIRTUAL JOINT: Purpose: this element defines a virtual joint between a robot link and an external frame of reference (considered fixed with respect to the robot)-->
-    <virtual_joint name="${tf_prefix}virtual_joint" type="floating" parent_frame="${tf_prefix}odom_comb" child_link="${tf_prefix}base_footprint" />
+    <virtual_joint name="${tf_prefix}virtual_joint" type="floating" parent_frame="${tf_prefix}odom_comb" child_link="${tf_prefix}base_footprint"/>
     <!--PASSIVE JOINT: Purpose: this element is used to mark joints that are not actuated-->
-    <passive_joint name="${tf_prefix}virtual_joint" />
-    <passive_joint name="${tf_prefix}bl_caster_rotation_joint" />
-    <passive_joint name="${tf_prefix}bl_caster_wheel_joint" />
-    <passive_joint name="${tf_prefix}br_caster_rotation_joint" />
-    <passive_joint name="${tf_prefix}br_caster_wheel_joint" />
-    <passive_joint name="${tf_prefix}fl_caster_rotation_joint" />
-    <passive_joint name="${tf_prefix}fl_caster_wheel_joint" />
-    <passive_joint name="${tf_prefix}fr_caster_rotation_joint" />
-    <passive_joint name="${tf_prefix}fr_caster_wheel_joint" />
+    <passive_joint name="${tf_prefix}virtual_joint"/>
+    <passive_joint name="${tf_prefix}bl_caster_rotation_joint"/>
+    <passive_joint name="${tf_prefix}bl_caster_wheel_joint"/>
+    <passive_joint name="${tf_prefix}br_caster_rotation_joint"/>
+    <passive_joint name="${tf_prefix}br_caster_wheel_joint"/>
+    <passive_joint name="${tf_prefix}fl_caster_rotation_joint"/>
+    <passive_joint name="${tf_prefix}fl_caster_wheel_joint"/>
+    <passive_joint name="${tf_prefix}fr_caster_rotation_joint"/>
+    <passive_joint name="${tf_prefix}fr_caster_wheel_joint"/>
     <!--DISABLE COLLISIONS: By default it is assumed that any link of the robot could potentially come into collision with any other link in the robot. This tag disables collision checking between a specified pair of links. -->
-    <disable_collisions link1="${tf_prefix}back_laser_link" link2="${tf_prefix}base_link" reason="Adjacent" />
-    <disable_collisions link1="${tf_prefix}back_laser_link" link2="${tf_prefix}bl_caster_rotation_link" reason="Never" />
-    <disable_collisions link1="${tf_prefix}back_laser_link" link2="${tf_prefix}bl_caster_wheel_link" reason="Never" />
-    <disable_collisions link1="${tf_prefix}back_laser_link" link2="${tf_prefix}br_caster_rotation_link" reason="Never" />
-    <disable_collisions link1="${tf_prefix}back_laser_link" link2="${tf_prefix}br_caster_wheel_link" reason="Never" />
-    <disable_collisions link1="${tf_prefix}back_laser_link" link2="${tf_prefix}cable_guide_clamp1_link" reason="Never" />
-    <disable_collisions link1="${tf_prefix}back_laser_link" link2="${tf_prefix}cable_guide_clamp2_link" reason="Never" />
-    <disable_collisions link1="${tf_prefix}back_laser_link" link2="${tf_prefix}cable_guide_clamp3_link" reason="Never" />
-    <disable_collisions link1="${tf_prefix}back_laser_link" link2="${tf_prefix}cable_guide_clamp4_link" reason="Never" />
-    <disable_collisions link1="${tf_prefix}back_laser_link" link2="${tf_prefix}cable_guide_forearm_tube_link" reason="Never" />
-    <disable_collisions link1="${tf_prefix}back_laser_link" link2="${tf_prefix}cable_guide_terminal_element_link" reason="Never" />
-    <disable_collisions link1="${tf_prefix}back_laser_link" link2="${tf_prefix}cable_guide_upper_arm_tube_link" reason="Never" />
-    <disable_collisions link1="${tf_prefix}back_laser_link" link2="${tf_prefix}cable_guide_wrist_3_tube_link" reason="Never" />
-    <disable_collisions link1="${tf_prefix}back_laser_link" link2="${tf_prefix}cable_guide_wrist_clamp_link" reason="Never" />
-    <disable_collisions link1="${tf_prefix}back_laser_link" link2="${tf_prefix}fl_caster_rotation_link" reason="Never" />
-    <disable_collisions link1="${tf_prefix}back_laser_link" link2="${tf_prefix}fl_caster_wheel_link" reason="Never" />
-    <disable_collisions link1="${tf_prefix}back_laser_link" link2="${tf_prefix}fr_caster_rotation_link" reason="Never" />
-    <disable_collisions link1="${tf_prefix}back_laser_link" link2="${tf_prefix}fr_caster_wheel_link" reason="Never" />
-    <disable_collisions link1="${tf_prefix}back_laser_link" link2="${tf_prefix}front_laser_link" reason="Never" />
-    <disable_collisions link1="${tf_prefix}back_laser_link" link2="${tf_prefix}fts_robotside" reason="Never" />
-    <disable_collisions link1="${tf_prefix}back_laser_link" link2="${tf_prefix}gripper_astra_link" reason="Never" />
-    <disable_collisions link1="${tf_prefix}back_laser_link" link2="${tf_prefix}gripper_coupling_link" reason="Never" />
-    <disable_collisions link1="${tf_prefix}back_laser_link" link2="${tf_prefix}gripper_left_inner_finger" reason="User" />
-    <disable_collisions link1="${tf_prefix}back_laser_link" link2="${tf_prefix}gripper_left_inner_knuckle" reason="User" />
-    <disable_collisions link1="${tf_prefix}back_laser_link" link2="${tf_prefix}gripper_left_outer_finger" reason="User" />
-    <disable_collisions link1="${tf_prefix}back_laser_link" link2="${tf_prefix}gripper_left_outer_knuckle" reason="Never" />
-    <disable_collisions link1="${tf_prefix}back_laser_link" link2="${tf_prefix}gripper_left_robotiq_fingertip_65mm" reason="User" />
-    <disable_collisions link1="${tf_prefix}back_laser_link" link2="${tf_prefix}gripper_pico_flexx_link" reason="Never" />
-    <disable_collisions link1="${tf_prefix}back_laser_link" link2="${tf_prefix}gripper_right_inner_finger" reason="Never" />
-    <disable_collisions link1="${tf_prefix}back_laser_link" link2="${tf_prefix}gripper_right_inner_knuckle" reason="User" />
-    <disable_collisions link1="${tf_prefix}back_laser_link" link2="${tf_prefix}gripper_right_outer_finger" reason="Never" />
-    <disable_collisions link1="${tf_prefix}back_laser_link" link2="${tf_prefix}gripper_right_outer_knuckle" reason="Never" />
-    <disable_collisions link1="${tf_prefix}back_laser_link" link2="${tf_prefix}gripper_right_robotiq_fingertip_65mm" reason="Never" />
-    <disable_collisions link1="${tf_prefix}back_laser_link" link2="${tf_prefix}gripper_robotiq_arg2f_base_link" reason="Never" />
-    <disable_collisions link1="${tf_prefix}back_laser_link" link2="${tf_prefix}left_wheel_link" reason="Never" />
-    <disable_collisions link1="${tf_prefix}back_laser_link" link2="${tf_prefix}right_wheel_link" reason="Never" />
-    <disable_collisions link1="${tf_prefix}back_laser_link" link2="${tf_prefix}sensor_mount_bracket_link" reason="Never" />
-    <disable_collisions link1="${tf_prefix}back_laser_link" link2="${tf_prefix}sensor_mount_link" reason="Never" />
-    <disable_collisions link1="${tf_prefix}back_laser_link" link2="${tf_prefix}sensor_mount_pico_holder_link" reason="Never" />
-    <disable_collisions link1="${tf_prefix}back_laser_link" link2="${tf_prefix}structure_cover_back_link" reason="Never" />
-    <disable_collisions link1="${tf_prefix}back_laser_link" link2="${tf_prefix}structure_cover_front_link" reason="Never" />
-    <disable_collisions link1="${tf_prefix}back_laser_link" link2="${tf_prefix}structure_cover_left_link" reason="Never" />
-    <disable_collisions link1="${tf_prefix}back_laser_link" link2="${tf_prefix}structure_cover_right_link" reason="Never" />
-    <disable_collisions link1="${tf_prefix}back_laser_link" link2="${tf_prefix}structure_cover_top_back_link" reason="Never" />
-    <disable_collisions link1="${tf_prefix}back_laser_link" link2="${tf_prefix}structure_cover_top_front_link" reason="Never" />
-    <disable_collisions link1="${tf_prefix}back_laser_link" link2="${tf_prefix}structure_part_down" reason="Never" />
-    <disable_collisions link1="${tf_prefix}back_laser_link" link2="${tf_prefix}structure_part_up" reason="Never" />
-    <disable_collisions link1="${tf_prefix}back_laser_link" link2="${tf_prefix}structure_pedestal" reason="Never" />
-    <disable_collisions link1="${tf_prefix}back_laser_link" link2="${tf_prefix}ur5_base_link" reason="Never" />
-    <disable_collisions link1="${tf_prefix}back_laser_link" link2="${tf_prefix}ur5_forearm_link" reason="Never" />
-    <disable_collisions link1="${tf_prefix}back_laser_link" link2="${tf_prefix}ur5_shoulder_link" reason="Never" />
-    <disable_collisions link1="${tf_prefix}back_laser_link" link2="${tf_prefix}ur5_upper_arm_link" reason="Never" />
-    <disable_collisions link1="${tf_prefix}back_laser_link" link2="${tf_prefix}ur5_wrist_1_link" reason="Never" />
-    <disable_collisions link1="${tf_prefix}back_laser_link" link2="${tf_prefix}ur5_wrist_2_link" reason="Never" />
-    <disable_collisions link1="${tf_prefix}back_laser_link" link2="${tf_prefix}ur5_wrist_3_link" reason="Never" />
-    <disable_collisions link1="${tf_prefix}base_link" link2="${tf_prefix}bl_caster_rotation_link" reason="Adjacent" />
-    <disable_collisions link1="${tf_prefix}base_link" link2="${tf_prefix}bl_caster_wheel_link" reason="Never" />
-    <disable_collisions link1="${tf_prefix}base_link" link2="${tf_prefix}br_caster_rotation_link" reason="Adjacent" />
-    <disable_collisions link1="${tf_prefix}base_link" link2="${tf_prefix}br_caster_wheel_link" reason="Never" />
-    <disable_collisions link1="${tf_prefix}base_link" link2="${tf_prefix}cable_guide_clamp1_link" reason="Never" />
-    <disable_collisions link1="${tf_prefix}base_link" link2="${tf_prefix}cable_guide_clamp2_link" reason="Never" />
-    <disable_collisions link1="${tf_prefix}base_link" link2="${tf_prefix}cable_guide_clamp3_link" reason="Never" />
-    <disable_collisions link1="${tf_prefix}base_link" link2="${tf_prefix}cable_guide_clamp4_link" reason="Never" />
-    <disable_collisions link1="${tf_prefix}base_link" link2="${tf_prefix}cable_guide_forearm_tube_link" reason="Never" />
-    <disable_collisions link1="${tf_prefix}base_link" link2="${tf_prefix}cable_guide_terminal_element_link" reason="User" />
-    <disable_collisions link1="${tf_prefix}base_link" link2="${tf_prefix}cable_guide_upper_arm_tube_link" reason="Never" />
-    <disable_collisions link1="${tf_prefix}base_link" link2="${tf_prefix}cable_guide_wrist_3_tube_link" reason="User" />
-    <disable_collisions link1="${tf_prefix}base_link" link2="${tf_prefix}cable_guide_wrist_clamp_link" reason="User" />
-    <disable_collisions link1="${tf_prefix}base_link" link2="${tf_prefix}fl_caster_rotation_link" reason="Adjacent" />
-    <disable_collisions link1="${tf_prefix}base_link" link2="${tf_prefix}fl_caster_wheel_link" reason="Never" />
-    <disable_collisions link1="${tf_prefix}base_link" link2="${tf_prefix}fr_caster_rotation_link" reason="Adjacent" />
-    <disable_collisions link1="${tf_prefix}base_link" link2="${tf_prefix}fr_caster_wheel_link" reason="Never" />
-    <disable_collisions link1="${tf_prefix}base_link" link2="${tf_prefix}front_laser_link" reason="Adjacent" />
-    <disable_collisions link1="${tf_prefix}base_link" link2="${tf_prefix}fts_robotside" reason="Never" />
-    <disable_collisions link1="${tf_prefix}base_link" link2="${tf_prefix}gripper_astra_link" reason="User" />
-    <disable_collisions link1="${tf_prefix}base_link" link2="${tf_prefix}gripper_coupling_link" reason="Never" />
-    <disable_collisions link1="${tf_prefix}base_link" link2="${tf_prefix}gripper_left_inner_finger" reason="User" />
-    <disable_collisions link1="${tf_prefix}base_link" link2="${tf_prefix}gripper_left_inner_knuckle" reason="User" />
-    <disable_collisions link1="${tf_prefix}base_link" link2="${tf_prefix}gripper_left_outer_finger" reason="User" />
-    <disable_collisions link1="${tf_prefix}base_link" link2="${tf_prefix}gripper_left_outer_knuckle" reason="User" />
-    <disable_collisions link1="${tf_prefix}base_link" link2="${tf_prefix}gripper_left_robotiq_fingertip_65mm" reason="User" />
-    <disable_collisions link1="${tf_prefix}base_link" link2="${tf_prefix}gripper_pico_flexx_link" reason="User" />
-    <disable_collisions link1="${tf_prefix}base_link" link2="${tf_prefix}gripper_right_inner_finger" reason="User" />
-    <disable_collisions link1="${tf_prefix}base_link" link2="${tf_prefix}gripper_right_inner_knuckle" reason="User" />
-    <disable_collisions link1="${tf_prefix}base_link" link2="${tf_prefix}gripper_right_outer_finger" reason="User" />
-    <disable_collisions link1="${tf_prefix}base_link" link2="${tf_prefix}gripper_right_outer_knuckle" reason="User" />
-    <disable_collisions link1="${tf_prefix}base_link" link2="${tf_prefix}gripper_right_robotiq_fingertip_65mm" reason="User" />
-    <disable_collisions link1="${tf_prefix}base_link" link2="${tf_prefix}gripper_robotiq_arg2f_base_link" reason="User" />
-    <disable_collisions link1="${tf_prefix}base_link" link2="${tf_prefix}left_wheel_link" reason="Adjacent" />
-    <disable_collisions link1="${tf_prefix}base_link" link2="${tf_prefix}right_wheel_link" reason="Adjacent" />
-    <disable_collisions link1="${tf_prefix}base_link" link2="${tf_prefix}sensor_mount_bracket_link" reason="Never" />
-    <disable_collisions link1="${tf_prefix}base_link" link2="${tf_prefix}sensor_mount_link" reason="User" />
-    <disable_collisions link1="${tf_prefix}base_link" link2="${tf_prefix}sensor_mount_pico_holder_link" reason="User" />
-    <disable_collisions link1="${tf_prefix}base_link" link2="${tf_prefix}structure_cover_back_link" reason="Never" />
-    <disable_collisions link1="${tf_prefix}base_link" link2="${tf_prefix}structure_cover_front_link" reason="Never" />
-    <disable_collisions link1="${tf_prefix}base_link" link2="${tf_prefix}structure_cover_left_link" reason="Never" />
-    <disable_collisions link1="${tf_prefix}base_link" link2="${tf_prefix}structure_cover_right_link" reason="Never" />
-    <disable_collisions link1="${tf_prefix}base_link" link2="${tf_prefix}structure_cover_top_back_link" reason="Never" />
-    <disable_collisions link1="${tf_prefix}base_link" link2="${tf_prefix}structure_cover_top_front_link" reason="Never" />
-    <disable_collisions link1="${tf_prefix}base_link" link2="${tf_prefix}structure_part_down" reason="Adjacent" />
-    <disable_collisions link1="${tf_prefix}base_link" link2="${tf_prefix}structure_part_up" reason="Never" />
-    <disable_collisions link1="${tf_prefix}base_link" link2="${tf_prefix}structure_pedestal" reason="Never" />
-    <disable_collisions link1="${tf_prefix}base_link" link2="${tf_prefix}ur5_base_link" reason="Never" />
-    <disable_collisions link1="${tf_prefix}base_link" link2="${tf_prefix}ur5_forearm_link" reason="Never" />
-    <disable_collisions link1="${tf_prefix}base_link" link2="${tf_prefix}ur5_shoulder_link" reason="Never" />
-    <disable_collisions link1="${tf_prefix}base_link" link2="${tf_prefix}ur5_upper_arm_link" reason="Never" />
-    <disable_collisions link1="${tf_prefix}base_link" link2="${tf_prefix}ur5_wrist_1_link" reason="Never" />
-    <disable_collisions link1="${tf_prefix}base_link" link2="${tf_prefix}ur5_wrist_2_link" reason="Never" />
-    <disable_collisions link1="${tf_prefix}base_link" link2="${tf_prefix}ur5_wrist_3_link" reason="Never" />
-    <disable_collisions link1="${tf_prefix}bl_caster_rotation_link" link2="${tf_prefix}bl_caster_wheel_link" reason="Adjacent" />
-    <disable_collisions link1="${tf_prefix}bl_caster_rotation_link" link2="${tf_prefix}br_caster_rotation_link" reason="Never" />
-    <disable_collisions link1="${tf_prefix}bl_caster_rotation_link" link2="${tf_prefix}br_caster_wheel_link" reason="Never" />
-    <disable_collisions link1="${tf_prefix}bl_caster_rotation_link" link2="${tf_prefix}cable_guide_clamp1_link" reason="Never" />
-    <disable_collisions link1="${tf_prefix}bl_caster_rotation_link" link2="${tf_prefix}cable_guide_clamp2_link" reason="Never" />
-    <disable_collisions link1="${tf_prefix}bl_caster_rotation_link" link2="${tf_prefix}cable_guide_clamp3_link" reason="Never" />
-    <disable_collisions link1="${tf_prefix}bl_caster_rotation_link" link2="${tf_prefix}cable_guide_clamp4_link" reason="Never" />
-    <disable_collisions link1="${tf_prefix}bl_caster_rotation_link" link2="${tf_prefix}cable_guide_forearm_tube_link" reason="Never" />
-    <disable_collisions link1="${tf_prefix}bl_caster_rotation_link" link2="${tf_prefix}cable_guide_terminal_element_link" reason="Never" />
-    <disable_collisions link1="${tf_prefix}bl_caster_rotation_link" link2="${tf_prefix}cable_guide_upper_arm_tube_link" reason="Never" />
-    <disable_collisions link1="${tf_prefix}bl_caster_rotation_link" link2="${tf_prefix}cable_guide_wrist_3_tube_link" reason="Never" />
-    <disable_collisions link1="${tf_prefix}bl_caster_rotation_link" link2="${tf_prefix}cable_guide_wrist_clamp_link" reason="Never" />
-    <disable_collisions link1="${tf_prefix}bl_caster_rotation_link" link2="${tf_prefix}fl_caster_rotation_link" reason="Never" />
-    <disable_collisions link1="${tf_prefix}bl_caster_rotation_link" link2="${tf_prefix}fl_caster_wheel_link" reason="Never" />
-    <disable_collisions link1="${tf_prefix}bl_caster_rotation_link" link2="${tf_prefix}fr_caster_rotation_link" reason="Never" />
-    <disable_collisions link1="${tf_prefix}bl_caster_rotation_link" link2="${tf_prefix}fr_caster_wheel_link" reason="Never" />
-    <disable_collisions link1="${tf_prefix}bl_caster_rotation_link" link2="${tf_prefix}front_laser_link" reason="Never" />
-    <disable_collisions link1="${tf_prefix}bl_caster_rotation_link" link2="${tf_prefix}fts_robotside" reason="Never" />
-    <disable_collisions link1="${tf_prefix}bl_caster_rotation_link" link2="${tf_prefix}gripper_astra_link" reason="Never" />
-    <disable_collisions link1="${tf_prefix}bl_caster_rotation_link" link2="${tf_prefix}gripper_coupling_link" reason="Never" />
-    <disable_collisions link1="${tf_prefix}bl_caster_rotation_link" link2="${tf_prefix}gripper_left_inner_finger" reason="Never" />
-    <disable_collisions link1="${tf_prefix}bl_caster_rotation_link" link2="${tf_prefix}gripper_left_inner_knuckle" reason="Never" />
-    <disable_collisions link1="${tf_prefix}bl_caster_rotation_link" link2="${tf_prefix}gripper_left_outer_finger" reason="Never" />
-    <disable_collisions link1="${tf_prefix}bl_caster_rotation_link" link2="${tf_prefix}gripper_left_outer_knuckle" reason="Never" />
-    <disable_collisions link1="${tf_prefix}bl_caster_rotation_link" link2="${tf_prefix}gripper_left_robotiq_fingertip_65mm" reason="Never" />
-    <disable_collisions link1="${tf_prefix}bl_caster_rotation_link" link2="${tf_prefix}gripper_pico_flexx_link" reason="Never" />
-    <disable_collisions link1="${tf_prefix}bl_caster_rotation_link" link2="${tf_prefix}gripper_right_inner_finger" reason="Never" />
-    <disable_collisions link1="${tf_prefix}bl_caster_rotation_link" link2="${tf_prefix}gripper_right_inner_knuckle" reason="Never" />
-    <disable_collisions link1="${tf_prefix}bl_caster_rotation_link" link2="${tf_prefix}gripper_right_outer_finger" reason="Never" />
-    <disable_collisions link1="${tf_prefix}bl_caster_rotation_link" link2="${tf_prefix}gripper_right_outer_knuckle" reason="Never" />
-    <disable_collisions link1="${tf_prefix}bl_caster_rotation_link" link2="${tf_prefix}gripper_right_robotiq_fingertip_65mm" reason="Never" />
-    <disable_collisions link1="${tf_prefix}bl_caster_rotation_link" link2="${tf_prefix}gripper_robotiq_arg2f_base_link" reason="Never" />
-    <disable_collisions link1="${tf_prefix}bl_caster_rotation_link" link2="${tf_prefix}left_wheel_link" reason="Never" />
-    <disable_collisions link1="${tf_prefix}bl_caster_rotation_link" link2="${tf_prefix}right_wheel_link" reason="Never" />
-    <disable_collisions link1="${tf_prefix}bl_caster_rotation_link" link2="${tf_prefix}sensor_mount_bracket_link" reason="Never" />
-    <disable_collisions link1="${tf_prefix}bl_caster_rotation_link" link2="${tf_prefix}sensor_mount_link" reason="Never" />
-    <disable_collisions link1="${tf_prefix}bl_caster_rotation_link" link2="${tf_prefix}sensor_mount_pico_holder_link" reason="Never" />
-    <disable_collisions link1="${tf_prefix}bl_caster_rotation_link" link2="${tf_prefix}structure_cover_back_link" reason="Never" />
-    <disable_collisions link1="${tf_prefix}bl_caster_rotation_link" link2="${tf_prefix}structure_cover_front_link" reason="Never" />
-    <disable_collisions link1="${tf_prefix}bl_caster_rotation_link" link2="${tf_prefix}structure_cover_left_link" reason="Never" />
-    <disable_collisions link1="${tf_prefix}bl_caster_rotation_link" link2="${tf_prefix}structure_cover_right_link" reason="Never" />
-    <disable_collisions link1="${tf_prefix}bl_caster_rotation_link" link2="${tf_prefix}structure_cover_top_back_link" reason="Never" />
-    <disable_collisions link1="${tf_prefix}bl_caster_rotation_link" link2="${tf_prefix}structure_cover_top_front_link" reason="Never" />
-    <disable_collisions link1="${tf_prefix}bl_caster_rotation_link" link2="${tf_prefix}structure_part_down" reason="Never" />
-    <disable_collisions link1="${tf_prefix}bl_caster_rotation_link" link2="${tf_prefix}structure_part_up" reason="Never" />
-    <disable_collisions link1="${tf_prefix}bl_caster_rotation_link" link2="${tf_prefix}structure_pedestal" reason="Never" />
-    <disable_collisions link1="${tf_prefix}bl_caster_rotation_link" link2="${tf_prefix}ur5_base_link" reason="Never" />
-    <disable_collisions link1="${tf_prefix}bl_caster_rotation_link" link2="${tf_prefix}ur5_forearm_link" reason="Never" />
-    <disable_collisions link1="${tf_prefix}bl_caster_rotation_link" link2="${tf_prefix}ur5_shoulder_link" reason="Never" />
-    <disable_collisions link1="${tf_prefix}bl_caster_rotation_link" link2="${tf_prefix}ur5_upper_arm_link" reason="Never" />
-    <disable_collisions link1="${tf_prefix}bl_caster_rotation_link" link2="${tf_prefix}ur5_wrist_1_link" reason="Never" />
-    <disable_collisions link1="${tf_prefix}bl_caster_rotation_link" link2="${tf_prefix}ur5_wrist_2_link" reason="Never" />
-    <disable_collisions link1="${tf_prefix}bl_caster_rotation_link" link2="${tf_prefix}ur5_wrist_3_link" reason="Never" />
-    <disable_collisions link1="${tf_prefix}bl_caster_wheel_link" link2="${tf_prefix}br_caster_rotation_link" reason="Never" />
-    <disable_collisions link1="${tf_prefix}bl_caster_wheel_link" link2="${tf_prefix}br_caster_wheel_link" reason="Never" />
-    <disable_collisions link1="${tf_prefix}bl_caster_wheel_link" link2="${tf_prefix}cable_guide_clamp1_link" reason="Never" />
-    <disable_collisions link1="${tf_prefix}bl_caster_wheel_link" link2="${tf_prefix}cable_guide_clamp2_link" reason="Never" />
-    <disable_collisions link1="${tf_prefix}bl_caster_wheel_link" link2="${tf_prefix}cable_guide_clamp3_link" reason="Never" />
-    <disable_collisions link1="${tf_prefix}bl_caster_wheel_link" link2="${tf_prefix}cable_guide_clamp4_link" reason="Never" />
-    <disable_collisions link1="${tf_prefix}bl_caster_wheel_link" link2="${tf_prefix}cable_guide_forearm_tube_link" reason="Never" />
-    <disable_collisions link1="${tf_prefix}bl_caster_wheel_link" link2="${tf_prefix}cable_guide_terminal_element_link" reason="Never" />
-    <disable_collisions link1="${tf_prefix}bl_caster_wheel_link" link2="${tf_prefix}cable_guide_upper_arm_tube_link" reason="Never" />
-    <disable_collisions link1="${tf_prefix}bl_caster_wheel_link" link2="${tf_prefix}cable_guide_wrist_3_tube_link" reason="Never" />
-    <disable_collisions link1="${tf_prefix}bl_caster_wheel_link" link2="${tf_prefix}cable_guide_wrist_clamp_link" reason="Never" />
-    <disable_collisions link1="${tf_prefix}bl_caster_wheel_link" link2="${tf_prefix}fl_caster_rotation_link" reason="Never" />
-    <disable_collisions link1="${tf_prefix}bl_caster_wheel_link" link2="${tf_prefix}fl_caster_wheel_link" reason="Never" />
-    <disable_collisions link1="${tf_prefix}bl_caster_wheel_link" link2="${tf_prefix}fr_caster_rotation_link" reason="Never" />
-    <disable_collisions link1="${tf_prefix}bl_caster_wheel_link" link2="${tf_prefix}fr_caster_wheel_link" reason="Never" />
-    <disable_collisions link1="${tf_prefix}bl_caster_wheel_link" link2="${tf_prefix}front_laser_link" reason="Never" />
-    <disable_collisions link1="${tf_prefix}bl_caster_wheel_link" link2="${tf_prefix}fts_robotside" reason="Never" />
-    <disable_collisions link1="${tf_prefix}bl_caster_wheel_link" link2="${tf_prefix}gripper_astra_link" reason="Never" />
-    <disable_collisions link1="${tf_prefix}bl_caster_wheel_link" link2="${tf_prefix}gripper_coupling_link" reason="Never" />
-    <disable_collisions link1="${tf_prefix}bl_caster_wheel_link" link2="${tf_prefix}gripper_left_inner_finger" reason="Never" />
-    <disable_collisions link1="${tf_prefix}bl_caster_wheel_link" link2="${tf_prefix}gripper_left_inner_knuckle" reason="Never" />
-    <disable_collisions link1="${tf_prefix}bl_caster_wheel_link" link2="${tf_prefix}gripper_left_outer_finger" reason="Never" />
-    <disable_collisions link1="${tf_prefix}bl_caster_wheel_link" link2="${tf_prefix}gripper_left_outer_knuckle" reason="Never" />
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