Commit message: srdf: Add ready_for_packing pose
... copied from pose_teacher.

File: mobipick_moveit_config/config/mobipick.srdf.xacro (robot description, xacro)
@@ -110,4 +110,12 @@
         <joint name="${tf_prefix}ur5_wrist_2_joint" value="1.57"/>
         <joint name="${tf_prefix}ur5_wrist_3_joint" value="4.71"/>
+    </group_state>
+    <group_state name="ready_for_packing" group="arm">
+        <joint name="${tf_prefix}ur5_shoulder_pan_joint" value="0.0"/>
+        <joint name="${tf_prefix}ur5_shoulder_lift_joint" value="-2.68"/>
+        <joint name="${tf_prefix}ur5_elbow_joint" value="2.80"/>
+        <joint name="${tf_prefix}ur5_wrist_1_joint" value="-1.84"/>
+        <joint name="${tf_prefix}ur5_wrist_2_joint" value="-1.57"/>
+        <joint name="${tf_prefix}ur5_wrist_3_joint" value="3.14"/>
     </group_state>
     <!-- NOTE: Using MoveIt to plan gripper opening/closing trajectories does not work (see README). -->

Commit message: srdf: Move "above" group state to be lower
This is used for "placing" (until we have a proper place action) in the
tables demo. Moving it lower prevents the objects from dropping too far
if we forget to catch them.

File: mobipick_moveit_config/config/mobipick.srdf.xacro (robot description, xacro)
@@ -96,10 +96,10 @@
     </group_state>
     <group_state name="above" group="arm">
-        <joint name="${tf_prefix}ur5_shoulder_pan_joint" value="-1.72"/>
-        <joint name="${tf_prefix}ur5_shoulder_lift_joint" value="-0.79"/>
-        <joint name="${tf_prefix}ur5_elbow_joint" value="0.71"/>
-        <joint name="${tf_prefix}ur5_wrist_1_joint" value="-1.52"/>
+        <joint name="${tf_prefix}ur5_shoulder_pan_joint" value="-1.57"/>
+        <joint name="${tf_prefix}ur5_shoulder_lift_joint" value="-0.42"/>
+        <joint name="${tf_prefix}ur5_elbow_joint" value="0.74"/>
+        <joint name="${tf_prefix}ur5_wrist_1_joint" value="-1.94"/>
         <joint name="${tf_prefix}ur5_wrist_2_joint" value="-1.57"/>
-        <joint name="${tf_prefix}ur5_wrist_3_joint" value="1.1"/>
+        <joint name="${tf_prefix}ur5_wrist_3_joint" value="1.57"/>
     </group_state>
     <group_state name="tucked" group="arm">

Commit message: SRDF: Add untangle_cable_guide right group states

File: mobipick_moveit_config/config/mobipick.srdf.xacro (robot description, xacro)
@@ -118,4 +118,20 @@
         <joint name="${tf_prefix}ur5_wrist_2_joint" value="-1.57"/>
         <joint name="${tf_prefix}ur5_wrist_3_joint" value="3.14"/>
+    </group_state>
+    <group_state name="untangle_cable_guide_1_right" group="arm">
+        <joint name="${tf_prefix}ur5_shoulder_pan_joint" value="-1.57"/>
+        <joint name="${tf_prefix}ur5_shoulder_lift_joint" value="-2.30"/>
+        <joint name="${tf_prefix}ur5_elbow_joint" value="2.44"/>
+        <joint name="${tf_prefix}ur5_wrist_1_joint" value="-2.59"/>
+        <joint name="${tf_prefix}ur5_wrist_2_joint" value="-1.57"/>
+        <joint name="${tf_prefix}ur5_wrist_3_joint" value="3.88"/>
+    </group_state>
+    <group_state name="untangle_cable_guide_2_right" group="arm">
+        <joint name="${tf_prefix}ur5_shoulder_pan_joint" value="-1.57"/>
+        <joint name="${tf_prefix}ur5_shoulder_lift_joint" value="-2.30"/>
+        <joint name="${tf_prefix}ur5_elbow_joint" value="2.44"/>
+        <joint name="${tf_prefix}ur5_wrist_1_joint" value="-2.59"/>
+        <joint name="${tf_prefix}ur5_wrist_2_joint" value="-1.58"/>
+        <joint name="${tf_prefix}ur5_wrist_3_joint" value="3.10"/>
     </group_state>
     <!-- NOTE: Using MoveIt to plan gripper opening/closing trajectories does not work (see README). -->

Commit message: SRDF: Add handover group state

File: mobipick_moveit_config/config/mobipick.srdf.xacro (robot description, xacro)
@@ -134,4 +134,12 @@
         <joint name="${tf_prefix}ur5_wrist_2_joint" value="-1.58"/>
         <joint name="${tf_prefix}ur5_wrist_3_joint" value="3.10"/>
+    </group_state>
+    <group_state name="handover" group="arm">
+        <joint name="${tf_prefix}ur5_shoulder_pan_joint" value="-0.8814045223823461"/>
+        <joint name="${tf_prefix}ur5_shoulder_lift_joint" value="-0.9537410855135158"/>
+        <joint name="${tf_prefix}ur5_elbow_joint" value="1.3274989660102516"/>
+        <joint name="${tf_prefix}ur5_wrist_1_joint" value="-0.3573771398701102"/>
+        <joint name="${tf_prefix}ur5_wrist_2_joint" value="0.685091341557877"/>
+        <joint name="${tf_prefix}ur5_wrist_3_joint" value="1.548322337092717"/>
     </group_state>
     <!-- NOTE: Using MoveIt to plan gripper opening/closing trajectories does not work (see README). -->

Commit message: added smart_factory nav poses and arm configurations

File: mobipick_moveit_config/config/mobipick.srdf.xacro (robot description, xacro)
@@ -71,4 +71,12 @@
         <joint name="${tf_prefix}ur5_wrist_3_joint" value="4.71"/>
     </group_state>
+    <group_state name="observe_workstation_right" group="arm">
+        <joint name="${tf_prefix}ur5_shoulder_pan_joint" value="-1.761"/>
+        <joint name="${tf_prefix}ur5_shoulder_lift_joint" value="-2.301"/>
+        <joint name="${tf_prefix}ur5_elbow_joint" value="2.44"/>
+        <joint name="${tf_prefix}ur5_wrist_1_joint" value="-0.95"/>
+        <joint name="${tf_prefix}ur5_wrist_2_joint" value="1.57"/>
+        <joint name="${tf_prefix}ur5_wrist_3_joint" value="4.71"/>
+    </group_state>
     <group_state name="observe100cm_back" group="arm">
         <joint name="${tf_prefix}ur5_shoulder_pan_joint" value="3.14"/>
@@ -136,10 +144,18 @@
     </group_state>
     <group_state name="handover" group="arm">
-        <joint name="${tf_prefix}ur5_shoulder_pan_joint" value="-0.8814045223823461"/>
-        <joint name="${tf_prefix}ur5_shoulder_lift_joint" value="-0.9537410855135158"/>
-        <joint name="${tf_prefix}ur5_elbow_joint" value="1.3274989660102516"/>
-        <joint name="${tf_prefix}ur5_wrist_1_joint" value="-0.3573771398701102"/>
-        <joint name="${tf_prefix}ur5_wrist_2_joint" value="0.685091341557877"/>
-        <joint name="${tf_prefix}ur5_wrist_3_joint" value="1.548322337092717"/>
+        <joint name="${tf_prefix}ur5_shoulder_pan_joint" value="-0.88"/>
+        <joint name="${tf_prefix}ur5_shoulder_lift_joint" value="-0.95"/>
+        <joint name="${tf_prefix}ur5_elbow_joint" value="1.327"/>
+        <joint name="${tf_prefix}ur5_wrist_1_joint" value="-0.357"/>
+        <joint name="${tf_prefix}ur5_wrist_2_joint" value="0.685"/>
+        <joint name="${tf_prefix}ur5_wrist_3_joint" value="1.548"/>
+    </group_state>
+    <group_state name="handover_truck_assembly" group="arm">
+        <joint name="${tf_prefix}ur5_shoulder_pan_joint" value="-2.071"/>
+        <joint name="${tf_prefix}ur5_shoulder_lift_joint" value="-1.286"/>
+        <joint name="${tf_prefix}ur5_elbow_joint" value="1.809"/>
+        <joint name="${tf_prefix}ur5_wrist_1_joint" value="-0.193"/>
+        <joint name="${tf_prefix}ur5_wrist_2_joint" value="0.007"/>
+        <joint name="${tf_prefix}ur5_wrist_3_joint" value="1.214"/>
     </group_state>
     <!-- NOTE: Using MoveIt to plan gripper opening/closing trajectories does not work (see README). -->

Commit message: change handover pose to ease the navigation workstation pose

File: mobipick_moveit_config/config/mobipick.srdf.xacro (robot description, xacro)
@@ -144,5 +144,5 @@
     </group_state>
     <group_state name="handover" group="arm">
-        <joint name="${tf_prefix}ur5_shoulder_pan_joint" value="-0.88"/>
+        <joint name="${tf_prefix}ur5_shoulder_pan_joint" value="-1.465"/>
         <joint name="${tf_prefix}ur5_shoulder_lift_joint" value="-0.95"/>
         <joint name="${tf_prefix}ur5_elbow_joint" value="1.327"/>
